Commit message: updated description

File: mini_pupper_description/urdf/_d435.urdf.xacro (robot description, xacro)
@@ -8,6 +8,6 @@
 <robot name="sensor_d435" xmlns:xacro="http://ros.org/wiki/xacro">
   <!-- Includes -->
-  <xacro:include filename="$(find realsense2_description)/urdf/_materials.urdf.xacro" />
-  <xacro:include filename="$(find realsense2_description)/urdf/_usb_plug.urdf.xacro" />
+  <xacro:include filename="$(find mini_pupper_description)/urdf/_materials.urdf.xacro" />
+  <xacro:include filename="$(find mini_pupper_description)/urdf/_usb_plug.urdf.xacro" />
   <xacro:macro name="sensor_d435" params="parent *origin name:=camera use_nominal_extrinsics:=true add_plug:=false use_mesh:=true">
     <xacro:property name="M_PI" value="3.1415926535897931" />
@@ -53,5 +53,5 @@
           <origin xyz="${d435_zero_depth_to_glass + d435_glass_to_front} ${-d435_cam_depth_py} 0" rpy="${M_PI/2} 0 ${M_PI/2}"/>
           <geometry>
-            <mesh filename="package://realsense2_description/meshes/d435.dae" />
+            <mesh filename="package://mini_pupper_description/meshes/d435.dae" />
           </geometry>
         </xacro:if>

File: mini_pupper_description/urdf/mini_pupper_description.urdf (robot description, URDF)
Before this commit: robot mini_pupper_description, 38 links, 37 joints
Links:
- link camera_link: geometry collision box size=0.02505 0.09 0.025; visual mesh filename=package://mini_pupper_description/meshes/d435.dae
