Commit message: Fix lidar frame_id

File: mini_pupper_description/urdf/mini_pupper_description.urdf.xacro (robot description, xacro)
@@ -151,4 +151,18 @@
     <child
       link="lidar" />
+    <axis
+      xyz="0 0 0" />
+  </joint>
+  <link name="lidar_link" />
+  <joint
+    name="lidar_link_joint"
+    type="fixed">
+    <origin
+      xyz="0 0 0"
+      rpy="0 0 0" />
+    <parent
+      link="lidar" />
+    <child
+      link="lidar_link" />
     <axis
       xyz="0 0 0" />

Commit message: Update bringup launch file and URDF to support real Mini Pupper (#45)
Co-authored-by: 0nhc <thefoxfoxfox@outlook.com>

File: mini_pupper_description/urdf/mini_pupper_description.urdf.xacro (robot description, xacro)
@@ -106,5 +106,5 @@
       <origin
         xyz="1.56706411611127E-05 -5.16565672073303E-13 -0.0191835739440227"
-        rpy="0 0 0" />
+        rpy="0 0 -1.57" />
       <mass
         value="0.0001" />
@@ -120,5 +120,5 @@
       <origin
         xyz="0 0 0"
-        rpy="0 0 0" />
+        rpy="0 0 -1.57" />
       <geometry>
         <mesh
@@ -134,5 +134,5 @@
       <origin
         xyz="0 0 0"
-        rpy="0 0 0" />
+        rpy="0 0 -1.57" />
       <geometry>
         <mesh
@@ -146,9 +146,23 @@
     <origin
       xyz="-0.070475 0.0001 0.08"
-      rpy="0 0 0" />
+      rpy="0 0 1.57" />
     <parent
       link="base_link" />
     <child
       link="lidar" />
+    <axis
+      xyz="0 0 0" />
+  </joint>
+  <link name="lidar_link" />
+  <joint
+    name="lidar_link_joint"
+    type="fixed">
+    <origin
+      xyz="0 0 0"
+      rpy="0 0 0" />
+    <parent
+      link="lidar" />
+    <child
+      link="lidar_link" />
     <axis
       xyz="0 0 0" />

Commit message: fix lidar link inconsistent issue

File: mini_pupper_description/urdf/mini_pupper_description.urdf.xacro (robot description, xacro)
@@ -102,5 +102,5 @@
   </joint>
   <link
-    name="lidar">
+    name="lidar_link">
     <inertial>
       <origin
@@ -149,18 +149,4 @@
     <parent
       link="base_link" />
-    <child
-      link="lidar" />
-    <axis
-      xyz="0 0 0" />
-  </joint>
-  <link name="lidar_link" />
-  <joint
-    name="lidar_link_joint"
-    type="fixed">
-    <origin
-      xyz="0 0 0"
-      rpy="0 0 0" />
-    <parent
-      link="lidar" />
     <child
       link="lidar_link" />
@@ -1740,9 +1726,8 @@
     <material>Gazebo/FlatBlack</material>
   </gazebo>
-  <gazebo reference="lidar">
+  <gazebo reference="lidar_link">
     <material>Gazebo/FlatBlack</material>
     <sensor type="ray" name="lidar">
       <always_on>true</always_on>
-      <visualize>false</visualize>
       <update_rate>30</update_rate>
       <pose>0 0 0 0 0 0</pose>
