Commit message: add gazebo supporting in description file

File: mini_pupper_description/urdf/mini_pupper_description.urdf (robot description, URDF)
Before this commit: robot mini_pupper_description, 17 links, 16 joints
Links:
- link base_link: mass 0.190607936684523 -> 0.2
- link lb1: mass 0.0267711576459679 -> 0.025
- link lb2: mass 0.00429044082420202 -> 0.025
- link lb3: mass 0.000584099405055381 -> 0.025
- link lbfoot: mass 0.00125666639937702 -> 0.025
- link lf1: mass 0.0265603147825122 -> 0.025
- link lf2: mass 0.00429044082169227 -> 0.025
- link lf3: mass 0.000584099405055383 -> 0.025
- link lffoot: mass 0.00125666639937702 -> 0.025
- link rb1: mass 0.0269414287477286 -> 0.025
- link rb2: mass 0.00426203115074646 -> 0.025
- link rb3: mass 0.000584099405055381 -> 0.025
- link rbfoot: mass 0.00125666639937702 -> 0.025
- link rf1: mass 0.02656031490036 -> 0.025
- link rf2: mass 0.0042620311539195 -> 0.025
- link rf3: mass 0.000584099405055381 -> 0.025
- link rffoot: mass 0.00125666639937702 -> 0.025
Joints:
- joint base_lb1: limit lower=-3.14 upper=3.14 effort=0 velocity=0 -> lower=-3.14 upper=3.14 effort=2 velocity=1
- joint base_lf1: limit lower=-3.14 upper=3.14 effort=0 velocity=0 -> lower=-3.14 upper=3.14 effort=2 velocity=1
- joint base_rb1: limit lower=-3.14 upper=3.14 effort=0 velocity=0 -> lower=-3.14 upper=3.14 effort=2 velocity=1
- joint base_rf1: limit lower=-3.14 upper=3.14 effort=0 velocity=0 -> lower=-3.14 upper=3.14 effort=2 velocity=1
- joint lb1_lb2: limit lower=-3.14 upper=3.14 effort=0 velocity=0 -> lower=-3.14 upper=3.14 effort=2 velocity=1
- joint lb2_lb3: limit lower=-3.14 upper=3.14 effort=0 velocity=0 -> lower=-3.14 upper=3.14 effort=2 velocity=1
- joint lf1_lf2: limit lower=-3.14 upper=3.14 effort=0 velocity=0 -> lower=-3.14 upper=3.14 effort=2 velocity=1
- joint lf2_lf3: limit lower=-3.14 upper=3.14 effort=0 velocity=0 -> lower=-3.14 upper=3.14 effort=2 velocity=1
- joint rb1_rb2: limit lower=-3.14 upper=3.14 effort=0 velocity=0 -> lower=-3.14 upper=3.14 effort=2 velocity=1
- joint rb2_rb3: limit lower=-3.14 upper=3.14 effort=0 velocity=0 -> lower=-3.14 upper=3.14 effort=2 velocity=1
- joint rf1_rf2: limit lower=-3.14 upper=3.14 effort=0 velocity=0 -> lower=-3.14 upper=3.14 effort=2 velocity=1
- joint rf2_rf3: limit lower=-3.14 upper=3.14 effort=0 velocity=0 -> lower=-3.14 upper=3.14 effort=2 velocity=1

Commit message: added gazebo plugins and changed robotmodel

File: mini_pupper_description/urdf/mini_pupper_description.urdf (robot description, URDF)
Before this commit: robot mini_pupper_description, 17 links, 16 joints
Links:
- added link imu_link, mass 0.001
- added link lidar, mass 0.05; collision mesh filename=package://mini_pupper_description/meshes/lidar.STL; visual mesh filename=package://mini_pupper_description/meshes/lidar.STL
- added link lpb1, mass 0.025; collision mesh filename=package://mini_pupper_description/meshes/lpb1.STL; visual mesh filename=package://mini_pupper_description/meshes/lpb1.STL
- added link lpb2, mass 0.025; collision mesh filename=package://mini_pupper_description/meshes/lpb2.STL; visual mesh filename=package://mini_pupper_description/meshes/lpb2.STL
- added link lpf1, mass 0.025; collision mesh filename=package://mini_pupper_description/meshes/lpf1.STL; visual mesh filename=package://mini_pupper_description/meshes/lpf1.STL
- added link lpf2, mass 0.025; collision mesh filename=package://mini_pupper_description/meshes/lpf2.STL; visual mesh filename=package://mini_pupper_description/meshes/lpf2.STL
- added link rpb1, mass 0.025; collision mesh filename=package://mini_pupper_description/meshes/rpb1.STL; visual mesh filename=package://mini_pupper_description/meshes/rpb1.STL
- added link rpb2, mass 0.025; collision mesh filename=package://mini_pupper_description/meshes/rpb2.STL; visual mesh filename=package://mini_pupper_description/meshes/rpb2.STL
- added link rpf1, mass 0.025; collision mesh filename=package://mini_pupper_description/meshes/rpf1.STL; visual mesh filename=package://mini_pupper_description/meshes/rpf1.STL
- added link rpf2, mass 0.025; collision mesh filename=package://mini_pupper_description/meshes/rpf2.STL; visual mesh filename=package://mini_pupper_description/meshes/rpf2.STL
- added link yellow_plate, mass 0.1; collision mesh filename=package://mini_pupper_description/meshes/yellow_plate.STL; visual mesh filename=package://mini_pupper_description/meshes/yellow_plate.STL
Joints:
- removed joint lb3_lbfoot
- removed joint lf3_lffoot
- removed joint rb3_rbfoot
- removed joint rf3_rffoot
- added joint base_lidar: type fixed, parent base_link, child lidar, origin xyz=-0.0521000000000001 0 0.0784999999999999 rpy=0 0 0, axis 0 0 0
- added joint base_yellowplate: type fixed, parent base_link, child yellow_plate, origin xyz=0.0556975724826061 -0.000166914683579864 0.0700000000000001 rpy=0 0 0, axis 0 0 0
- added joint imu_joint: type fixed, parent base_link, child imu_link
- added joint lb1_plate: type fixed, parent lb1, child lpb1, origin xyz=0.0107599999999999 0.0307 0.013 rpy=0 0 0, axis 0 0 0
- added joint lb2_plate: type fixed, parent lb2, child lpb2, origin xyz=0 0.0100000000000007 -0.0500000000000001 rpy=0 0 0, axis 0 0 0
- added joint lb3_foot: type fixed, parent lb3, child lbfoot, origin xyz=0 0 -0.056 rpy=0 0 0, axis 0 0 0
- added joint lf1_plate: type fixed, parent lf1, child lpf1, origin xyz=0.0107600000007337 0.0306999999992666 0.0130000000001585 rpy=0 0 0, axis 0 0 0
- added joint lf2_plate: type fixed, parent lf2, child lpf2, origin xyz=0 0.00999999999998141 -0.0500000000003035 rpy=0 0 0, axis 0 0 0
- added joint lf3_foot: type fixed, parent lf3, child lffoot, origin xyz=0 -4.9999999999939E-05 -0.056 rpy=0 0 0, axis 0 0 0
- added joint rb1_plate: type fixed, parent rb1, child rpb1, origin xyz=0.0107578315199995 -0.0307000000000005 0.0129999999999966 rpy=0 0 0, axis 0 0 0
- added joint rb2_plate: type fixed, parent rb2, child rpb2, origin xyz=0 -0.0099999999999994 -0.0500000000000005 rpy=0 0 0, axis 0 0 0
- added joint rb3_foot: type fixed, parent rb3, child rbfoot, origin xyz=0 0 -0.056 rpy=0 0 0, axis 0 0 0
- added joint rf1_plate: type fixed, parent rf1, child rpf1, origin xyz=0.0107599999999999 -0.0306999999999999 0.013 rpy=0 0 0, axis 0 0 0
- added joint rf2_plate: type fixed, parent rf2, child rpf2, origin xyz=0 -0.00999999999999994 -0.0499999999999996 rpy=0 0 0, axis 0 0 0
- added joint rf3_foot: type fixed, parent rf3, child rffoot, origin xyz=0 0 -0.056 rpy=0 0 0, axis 0 0 0
- joint base_lb1: limit lower=-3.14 upper=3.14 effort=2 velocity=1 -> lower=-3.14 upper=3.14 effort=2 velocity=1.5
- joint base_lf1: limit lower=-3.14 upper=3.14 effort=2 velocity=1 -> lower=-3.14 upper=3.14 effort=2 velocity=1.5
- joint base_rb1: limit lower=-3.14 upper=3.14 effort=2 velocity=1 -> lower=-3.14 upper=3.14 effort=2 velocity=1.5
- joint base_rf1: limit lower=-3.14 upper=3.14 effort=2 velocity=1 -> lower=-3.14 upper=3.14 effort=2 velocity=1.5
- joint lb1_lb2: limit lower=-3.14 upper=3.14 effort=2 velocity=1 -> lower=-3.14 upper=3.14 effort=2 velocity=1.5
- joint lb2_lb3: limit lower=-3.14 upper=3.14 effort=2 velocity=1 -> lower=-3.14 upper=3.14 effort=2 velocity=1.5
- joint lf1_lf2: limit lower=-3.14 upper=3.14 effort=2 velocity=1 -> lower=-3.14 upper=3.14 effort=2 velocity=1.5
- joint lf2_lf3: limit lower=-3.14 upper=3.14 effort=2 velocity=1 -> lower=-3.14 upper=3.14 effort=2 velocity=1.5
- joint rb1_rb2: limit lower=-3.14 upper=3.14 effort=2 velocity=1 -> lower=-3.14 upper=3.14 effort=2 velocity=1.5
- joint rb2_rb3: limit lower=-3.14 upper=3.14 effort=2 velocity=1 -> lower=-3.14 upper=3.14 effort=2 velocity=1.5
- joint rf1_rf2: limit lower=-3.14 upper=3.14 effort=2 velocity=1 -> lower=-3.14 upper=3.14 effort=2 velocity=1.5
- joint rf2_rf3: limit lower=-3.14 upper=3.14 effort=2 velocity=1 -> lower=-3.14 upper=3.14 effort=2 velocity=1.5

Commit message: Update mini_pupper_description.urdf

File: mini_pupper_description/urdf/mini_pupper_description.urdf (robot description, URDF)
Before this commit: robot mini_pupper_description, 28 links, 27 joints
Links:
- added link camera_bottom_screw_frame
- added link camera_color_frame
- added link camera_color_optical_frame
- added link camera_depth_frame
- added link camera_depth_optical_frame
- added link camera_infra1_frame
- added link camera_infra1_optical_frame
- added link camera_infra2_frame
- added link camera_infra2_optical_frame
- added link camera_link, mass 0.072; collision box size=0.02505 0.09 0.025; visual mesh filename=package://realsense2_description/meshes/d435.dae
- link base_link: mass 0.2 -> 0.7
- link lb1: mass 0.025 -> 0.25
- link lb2: mass 0.025 -> 0.125
- link lb3: mass 0.025 -> 0.0625
- link lbfoot: mass 0.025 -> 0.0625
- link lf1: mass 0.025 -> 0.25
- link lf2: mass 0.025 -> 0.125
- link lf3: mass 0.025 -> 0.0625
- link lffoot: mass 0.025 -> 0.0625
- link lidar: mass 0.05 -> 0.270
- link lpb1: mass 0.025 -> 0.005
- link lpb2: mass 0.025 -> 0.005
- link lpf1: mass 0.025 -> 0.005
- link lpf2: mass 0.025 -> 0.005
- link rb1: mass 0.025 -> 0.25
- link rb2: mass 0.025 -> 0.125
- link rb3: mass 0.025 -> 0.0625
- link rbfoot: mass 0.025 -> 0.0625
- link rf1: mass 0.025 -> 0.25
- link rf2: mass 0.025 -> 0.125
- link rf3: mass 0.025 -> 0.0625
- link rffoot: mass 0.025 -> 0.0625
- link rpb1: mass 0.025 -> 0.005
- link rpb2: mass 0.025 -> 0.005
- link rpf1: mass 0.025 -> 0.005
- link rpf2: mass 0.025 -> 0.005
- link yellow_plate: mass 0.1 -> 0.3
Joints:
- added joint camera_color_joint: type fixed, parent camera_link, child camera_color_frame, origin xyz=0 0.015 0 rpy=0 0 0
- added joint camera_color_optical_joint: type fixed, parent camera_color_frame, child camera_color_optical_frame, origin xyz=0 0 0 rpy=-1.5707963267948966 0 -1.5707963267948966
- added joint camera_depth_joint: type fixed, parent camera_link, child camera_depth_frame, origin xyz=0 0 0 rpy=0 0 0
- added joint camera_depth_optical_joint: type fixed, parent camera_depth_frame, child camera_depth_optical_frame, origin xyz=0 0 0 rpy=-1.5707963267948966 0 -1.5707963267948966
- added joint camera_infra1_joint: type fixed, parent camera_link, child camera_infra1_frame, origin xyz=0 0.0 0 rpy=0 0 0
- added joint camera_infra1_optical_joint: type fixed, parent camera_infra1_frame, child camera_infra1_optical_frame, origin xyz=0 0 0 rpy=-1.5707963267948966 0 -1.5707963267948966
- added joint camera_infra2_joint: type fixed, parent camera_link, child camera_infra2_frame, origin xyz=0 -0.05 0 rpy=0 0 0
- added joint camera_infra2_optical_joint: type fixed, parent camera_infra2_frame, child camera_infra2_optical_frame, origin xyz=0 0 0 rpy=-1.5707963267948966 0 -1.5707963267948966
- added joint camera_joint: type fixed, parent base_link, child camera_bottom_screw_frame, origin xyz=0.08 0.0 0.07 rpy=0 0 0
- added joint camera_link_joint: type fixed, parent camera_bottom_screw_frame, child camera_link, origin xyz=0.010600000000000002 0.0175 0.0125 rpy=0 0 0
- joint base_lb1: limit lower=-3.14 upper=3.14 effort=2 velocity=1.5 -> lower=-3.14 upper=3.14 effort=5 velocity=1.5
- joint base_lf1: limit lower=-3.14 upper=3.14 effort=2 velocity=1.5 -> lower=-3.14 upper=3.14 effort=5 velocity=1.5
- joint base_rb1: limit lower=-3.14 upper=3.14 effort=2 velocity=1.5 -> lower=-3.14 upper=3.14 effort=5 velocity=1.5
- joint base_rf1: limit lower=-3.14 upper=3.14 effort=2 velocity=1.5 -> lower=-3.14 upper=3.14 effort=5 velocity=1.5
- joint lb1_lb2: limit lower=-3.14 upper=3.14 effort=2 velocity=1.5 -> lower=-3.14 upper=3.14 effort=5 velocity=1.5
- joint lb2_lb3: limit lower=-3.14 upper=3.14 effort=2 velocity=1.5 -> lower=-3.14 upper=3.14 effort=5 velocity=1.5
- joint lf1_lf2: limit lower=-3.14 upper=3.14 effort=2 velocity=1.5 -> lower=-3.14 upper=3.14 effort=5 velocity=1.5
- joint lf2_lf3: limit lower=-3.14 upper=3.14 effort=2 velocity=1.5 -> lower=-3.14 upper=3.14 effort=5 velocity=1.5
- joint rb1_rb2: limit lower=-3.14 upper=3.14 effort=2 velocity=1.5 -> lower=-3.14 upper=3.14 effort=5 velocity=1.5
- joint rb2_rb3: limit lower=-3.14 upper=3.14 effort=2 velocity=1.5 -> lower=-3.14 upper=3.14 effort=5 velocity=1.5
- joint rf1_rf2: limit lower=-3.14 upper=3.14 effort=2 velocity=1.5 -> lower=-3.14 upper=3.14 effort=5 velocity=1.5
- joint rf2_rf3: limit lower=-3.14 upper=3.14 effort=2 velocity=1.5 -> lower=-3.14 upper=3.14 effort=5 velocity=1.5

Commit message: update urdf

File: mini_pupper_description/urdf/mini_pupper_description.urdf (robot description, URDF)
Before this commit: robot mini_pupper_description, 38 links, 37 joints
Links:
- link lidar: mass 0.270 -> 0.27
Joints:
- joint base_lidar: origin xyz=-0.0521000000000001 0 0.0784999999999999 rpy=0 0 0 -> xyz=-0.070475 0.0001 0.08 rpy=0 0 0

File: mini_pupper_description/urdf/mini_pupper_description.urdf.xacro (robot description, xacro)
@@ -103,15 +103,15 @@
     <inertial>
       <origin
-        xyz="-6.93889390390723E-18 2.26160114015493E-18 -0.0182071701877274"
-        rpy="0 0 0" />
-      <mass
-        value="0.270" />
-      <inertia
-        ixx="8.26918371378652E-06"
-        ixy="-1.02105106862017E-21"
-        ixz="-8.80189643038176E-22"
-        iyy="8.26918371378652E-06"
-        iyz="3.14750181540702E-22"
-        izz="9.10852801583898E-06" />
+        xyz="1.56706411611127E-05 -5.16565672073303E-13 -0.0191835739440227"
+        rpy="0 0 0" />
+      <mass
+        value="0.27" />
+      <inertia
+        ixx="8.74731426973985E-06"
+        ixy="-6.66781590704156E-08"
+        ixz="1.89196685410159E-11"
+        iyy="8.70097486591694E-06"
+        iyz="-1.13397577799603E-17"
+        izz="9.98821295317784E-06" />
     </inertial>
     <visual>
@@ -143,5 +143,5 @@
     type="fixed">
     <origin
-      xyz="-0.0521000000000001 0 0.0784999999999999"
+      xyz="-0.070475 0.0001 0.08"
       rpy="0 0 0" />
     <parent

Commit message: update

File: mini_pupper_description/urdf/mini_pupper_description.urdf (robot description, URDF)
Before this commit: robot mini-pupper, 39 links, 38 joints
Links:
- link base_inertia: mass 0.2 -> 0.190607936684523

Commit message: add mini_pupper_control and update README

File: mini_pupper_description/urdf/mini_pupper_description.urdf (robot description, URDF)
Before this commit: robot mini-pupper, 39 links, 38 joints
Links:
- link base_inertia: mass 0.190607936684523 -> 0.2

File: mini_pupper_description/urdf/mini_pupper_description.urdf.xacro (robot description, xacro)
@@ -1779,5 +1779,5 @@
   <gazebo>
     <plugin filename="libgazebo_ros2_control.so" name="gazebo_ros2_control">
-      <parameters>$(find mini_pupper_gazebo)/config/ros_control/ros_control.yaml</parameters>
+      <parameters>$(find mini_pupper_control)/config/ros_control/ros_control.yaml</parameters>
     </plugin>
   </gazebo>

Commit message: Fix urdf

File: mini_pupper_description/urdf/mini_pupper_description.urdf (robot description, URDF)
Before this commit: robot mini-pupper, 39 links, 38 joints
Joints:
- joint base_lidar: origin xyz=-0.070475 0.0001 0.08 rpy=0 0 0 -> xyz=-0.070475 0.0001 0.08 rpy=0 0 1.57

File: mini_pupper_description/urdf/mini_pupper_description.urdf.xacro (robot description, xacro)
@@ -106,5 +106,5 @@
       <origin
         xyz="1.56706411611127E-05 -5.16565672073303E-13 -0.0191835739440227"
-        rpy="0 0 0" />
+        rpy="0 0 -1.57" />
       <mass
         value="0.0001" />
@@ -120,5 +120,5 @@
       <origin
         xyz="0 0 0"
-        rpy="0 0 0" />
+        rpy="0 0 -1.57" />
       <geometry>
         <mesh
@@ -134,5 +134,5 @@
       <origin
         xyz="0 0 0"
-        rpy="0 0 0" />
+        rpy="0 0 -1.57" />
       <geometry>
         <mesh
@@ -146,5 +146,5 @@
     <origin
       xyz="-0.070475 0.0001 0.08"
-      rpy="0 0 0" />
+      rpy="0 0 1.57" />
     <parent
       link="base_link" />
