Commit message: add: mini pupper 2 urdf working in rviz

File: mini_pupper_description/urdf/mini_pupper_description.urdf (robot description, URDF)
Before this commit: robot mini-pupper, 39 links, 38 joints
Links:
- removed link camera_bottom_screw_frame
- removed link camera_color_frame
- removed link camera_color_optical_frame
- removed link camera_depth_frame
- removed link camera_depth_optical_frame
- removed link camera_infra1_frame
- removed link camera_infra1_optical_frame
- removed link camera_infra2_frame
- removed link camera_infra2_optical_frame
- removed link camera_link
- removed link lidar
- removed link lpb1
- removed link lpb2
- removed link lpf1
- removed link lpf2
- removed link rpb1
- removed link rpb2
- removed link rpf1
- removed link rpf2
- removed link yellow_plate
- added link Board_PCB, mass 0.014261552601793053; collision mesh filename=package://mini_pupper_description/meshes/Board_PCB.stl scale=1 1 1; visual mesh filename=package://mini_pupper_description/meshes/Board_PCB.stl scale=1 1 1
- added link Board_connectors_1, mass 0.004688613655947816; collision mesh filename=package://mini_pupper_description/meshes/Board_connectors_1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 scale=1 1 1; visual mesh filename=package://mini_pupper_description/meshes/Board_connectors_1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 scale=1 1 1
- added link Board_connectors_2, mass 0.0019746031301169403; collision mesh filename=package://mini_pupper_description/meshes/Board_connectors_2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 scale=1 1 1; visual mesh filename=package://mini_pupper_description/meshes/Board_connectors_2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 scale=1 1 1
- added link Body_front, mass 0.00785515871148119; collision mesh filename=package://mini_pupper_description/meshes/Body_front.stl scale=1 1 1; visual mesh filename=package://mini_pupper_description/meshes/Body_front.stl scale=1 1 1
- added link Shell_Hip_Left_1, mass 0.002573897544461238; collision mesh filename=package://mini_pupper_description/meshes/Shell_Hip_Left_1.s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 scale=1 1 1; visual mesh filename=package://mini_pupper_description/meshes/Shell_Hip_Left_1.s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 scale=1 1 1
- added link Shell_Hip_Left_2, mass 0.002573897544461238; collision mesh filename=package://mini_pupper_description/meshes/Shell_Hip_Left_2.s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 scale=1 1 1; visual mesh filename=package://mini_pupper_description/meshes/Shell_Hip_Left_2.s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 scale=1 1 1
- added link Shell_Hip_Right_1, mass 0.002396251664132183; collision mesh filename=package://mini_pupper_description/meshes/Shell_Hip_Right_1.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 scale=1 1 1; visual mesh filename=package://mini_pupper_description/meshes/Shell_Hip_Right_1.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 scale=1 1 1
- added link Shell_Hip_Right_2, mass 0.002396251664132183; collision mesh filename=package://mini_pupper_description/meshes/Shell_Hip_Right_2.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 scale=1 1 1; visual mesh filename=package://mini_pupper_description/meshes/Shell_Hip_Right_2.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 scale=1 1 1
- added link Shell_Leg_Upper_LeftSide_1, mass 0.00223142111318912; collision mesh filename=package://mini_pupper_description/meshes/Shell_Leg_Upper_Le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 scale=1 1 1; visual mesh filename=package://mini_pupper_description/meshes/Shell_Leg_Upper_Le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 scale=1 1 1
- added link Shell_Leg_Upper_LeftSide_2, mass 0.00223142111318912; collision mesh filename=package://mini_pupper_description/meshes/Shell_Leg_Upper_Le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 scale=1 1 1; visual mesh filename=package://mini_pupper_description/meshes/Shell_Leg_Upper_Le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 scale=1 1 1
- added link Shell_Leg_Upper_RightSide_1, mass 0.0022016115622538724; collision mesh filename=package://mini_pupper_description/meshes/Shell_Leg_Upper_Ri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 scale=1 1 1; visual mesh filename=package://mini_pupper_description/meshes/Shell_Leg_Upper_Ri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 scale=1 1 1
- added link Shell_Leg_Upper_RightSide_2, mass 0.0022016115622538724; collision mesh filename=package://mini_pupper_description/meshes/Shell_Leg_Upper_Ri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 scale=1 1 1; visual mesh filename=package://mini_pupper_description/meshes/Shell_Leg_Upper_Ri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 scale=1 1 1
- added link Shell_Side, mass 0.0051928835390001775; collision mesh filename=package://mini_pupper_description/meshes/Shell_Side.stl scale=1 1 1; visual mesh filename=package://mini_pupper_description/meshes/Shell_Side.stl scale=1 1 1
- link base_inertia: mass 0.2 -> 0.09818420433466489
- link base_link: geometry collision mesh filename=package://mini_pupper_description/meshes/base_link.stl scale=1 1 1; visual mesh filename=package://mini_pupper_description/meshes/base_link.stl scale=1 1 1
- link lb1: mass 0.00025 -> 0.020769030189864354; geometry collision mesh filename=package://mini_pupper_description/meshes/lb1.stl scale=1 1 1; visual mesh filename=package://mini_pupper_description/meshes/lb1.stl scale=1 1 1
- link lb2: mass 0.00125 -> 0.0019057729925095609; geometry collision mesh filename=package://mini_pupper_description/meshes/lb2.stl scale=1 1 1; visual mesh filename=package://mini_pupper_description/meshes/lb2.stl scale=1 1 1
- link lb3: mass 0.000625 -> 0.001144346207072784; geometry collision mesh filename=package://mini_pupper_description/meshes/lb3.stl scale=1 1 1; visual mesh filename=package://mini_pupper_description/meshes/lb3.stl scale=1 1 1
- link lbfoot: mass 0.000625 -> 0.0014053107976262874; geometry collision mesh filename=package://mini_pupper_description/meshes/lbfoot.stl scale=1 1 1; visual mesh filename=package://mini_pupper_description/meshes/lbfoot.stl scale=1 1 1
- link lf1: mass 0.0025 -> 0.020769030109708524; geometry collision mesh filename=package://mini_pupper_description/meshes/lf1.stl scale=1 1 1; visual mesh filename=package://mini_pupper_description/meshes/lf1.stl scale=1 1 1
- link lf2: mass 0.00125 -> 0.0019057729925096327; geometry collision mesh filename=package://mini_pupper_description/meshes/lf2.stl scale=1 1 1; visual mesh filename=package://mini_pupper_description/meshes/lf2.stl scale=1 1 1
- link lf3: mass 0.000625 -> 0.0011438144457690698; geometry collision mesh filename=package://mini_pupper_description/meshes/lf3.stl scale=1 1 1; visual mesh filename=package://mini_pupper_description/meshes/lf3.stl scale=1 1 1
- link lffoot: mass 0.000625 -> 0.0014053107976262874; geometry collision mesh filename=package://mini_pupper_description/meshes/lffoot.stl scale=1 1 1; visual mesh filename=package://mini_pupper_description/meshes/lffoot.stl scale=1 1 1
- link rb1: mass 0.0025 -> 0.020769549324363486; geometry collision mesh filename=package://mini_pupper_description/meshes/rb1.stl scale=1 1 1; visual mesh filename=package://mini_pupper_description/meshes/rb1.stl scale=1 1 1
- link rb2: mass 0.00125 -> 0.0019057729926311429; geometry collision mesh filename=package://mini_pupper_description/meshes/rb2.stl scale=1 1 1; visual mesh filename=package://mini_pupper_description/meshes/rb2.stl scale=1 1 1
- link rb3: mass 0.000625 -> 0.0011440535724654094; geometry collision mesh filename=package://mini_pupper_description/meshes/rb3.stl scale=1 1 1; visual mesh filename=package://mini_pupper_description/meshes/rb3.stl scale=1 1 1
- link rbfoot: mass 0.000625 -> 0.0014053107976262874; geometry collision mesh filename=package://mini_pupper_description/meshes/rbfoot.stl scale=1 1 1; visual mesh filename=package://mini_pupper_description/meshes/rbfoot.stl scale=1 1 1
- link rf1: mass 0.0025 -> 0.020769549324466178; geometry collision mesh filename=package://mini_pupper_description/meshes/rf1.stl scale=1 1 1; visual mesh filename=package://mini_pupper_description/meshes/rf1.stl scale=1 1 1
- link rf2: mass 0.00125 -> 0.0019057729924780605; geometry collision mesh filename=package://mini_pupper_description/meshes/rf2.stl scale=1 1 1; visual mesh filename=package://mini_pupper_description/meshes/rf2.stl scale=1 1 1
- link rf3: mass 0.000625 -> 0.001143490701517533; geometry collision mesh filename=package://mini_pupper_description/meshes/rf3.stl scale=1 1 1; visual mesh filename=package://mini_pupper_description/meshes/rf3.stl scale=1 1 1
- link rffoot: mass 0.000625 -> 0.0014053107976262874; geometry collision mesh filename=package://mini_pupper_description/meshes/rffoot.stl scale=1 1 1; visual mesh filename=package://mini_pupper_description/meshes/rffoot.stl scale=1 1 1
Joints:
- removed joint base_lidar
- removed joint base_yellowplate
- removed joint camera_color_joint
- removed joint camera_color_optical_joint
- removed joint camera_depth_joint
- removed joint camera_depth_optical_joint
- removed joint camera_infra1_joint
- removed joint camera_infra1_optical_joint
- removed joint camera_infra2_joint
- removed joint camera_infra2_optical_joint
- removed joint camera_joint
- removed joint camera_link_joint
- removed joint lb1_plate
- removed joint lb2_plate
- removed joint lf1_plate
- removed joint lf2_plate
- removed joint rb1_plate
- removed joint rb2_plate
- removed joint rf1_plate
- removed joint rf2_plate
- added joint base_board: type fixed, parent base_link, child Board_PCB, origin xyz=-0.087701 -0.023255 0.026457 rpy=0 0 0
- added joint base_cn1: type fixed, parent Board_PCB, child Board_connectors_1, origin xyz=0.149035 0.023472 0.0 rpy=0 0 0
- added joint base_cn2: type fixed, parent Board_PCB, child Board_connectors_2, origin xyz=0.042355 0.0235 0.0 rpy=0 0 0
- added joint base_front: type fixed, parent base_link, child Body_front, origin xyz=0.089299 0.000245 -0.015543 rpy=0 0 0
- added joint base_sides: type fixed, parent base_link, child Shell_Side, origin xyz=-0.002701 -0.029755 -0.016293 rpy=0 0 0
- added joint lb1_hip: type fixed, parent lb1, child Shell_Hip_Left_2, origin xyz=-0.006266 0.0145 0.013 rpy=0 0 0
- added joint lb2_shell: type fixed, parent lb2, child Shell_Leg_Upper_LeftSide_2, origin xyz=0.0 0.003 -0.019 rpy=0 0 0
- added joint lf1_hip: type fixed, parent lf1, child Shell_Hip_Left_1, origin xyz=0.034266 0.0145 0.013 rpy=0 0 0
- added joint lf2_shell: type fixed, parent lf2, child Shell_Leg_Upper_LeftSide_1, origin xyz=-3e-06 0.003 -0.019 rpy=0 0 0
- added joint rb2_hip: type fixed, parent rb1, child Shell_Hip_Right_2, origin xyz=-0.006266 -0.014493 0.013007 rpy=0 0 0
- added joint rb2_shell: type fixed, parent rb2, child Shell_Leg_Upper_RightSide_2, origin xyz=0.0 -0.003011 -0.018998 rpy=0 0 0
- added joint rf1_hip: type fixed, parent rf1, child Shell_Hip_Right_1, origin xyz=0.034266 -0.0145 0.013 rpy=0 0 0
- added joint rf2_shell: type fixed, parent rf2, child Shell_Leg_Upper_RightSide_1, origin xyz=0.0 -0.003 -0.019 rpy=0 0 0
- joint base_lb1: axis 1 0 0 -> 1.0 0.0 0.0; limit lower=-3.14 upper=3.14 effort=50 velocity=15 -> lower=-3.141593 upper=3.141593 effort=5 velocity=1.5; origin xyz=-0.05886 0.0235 0.0171 rpy=0 0 0 -> xyz=-0.042701 0.023745 5.7e-05 rpy=0 0 0
- joint base_lf1: axis 1 0 0 -> 1.0 0.0 0.0; limit lower=-3.14 upper=3.14 effort=50 velocity=15 -> lower=-3.141593 upper=3.141593 effort=5 velocity=1.5; origin xyz=0.06014 0.0235 0.0171 rpy=0 0 0 -> xyz=0.037299 0.023745 5.7e-05 rpy=0 0 0
- joint base_rb1: axis 1 0 0 -> 1.0 0.0 0.0; limit lower=-3.14 upper=3.14 effort=50 velocity=15 -> lower=-3.141593 upper=3.141593 effort=5 velocity=1.5; origin xyz=-0.05886 -0.0235 0.0171 rpy=0 0 0 -> xyz=-0.042701 -0.023255 5.7e-05 rpy=0 0 0
- joint base_rf1: axis 1 0 0 -> 1.0 0.0 0.0; limit lower=-3.14 upper=3.14 effort=50 velocity=15 -> lower=-3.141593 upper=3.141593 effort=5 velocity=1.5; origin xyz=0.06014 -0.0235 0.0171 rpy=0 0 0 -> xyz=0.037299 -0.023255 5.7e-05 rpy=0 0 0
- joint lb1_lb2: axis 0 1 0 -> 0.0 1.0 -0.0; limit lower=-3.14 upper=3.14 effort=50 velocity=15 -> lower=-3.141593 upper=3.141593 effort=5 velocity=1.5; origin xyz=-4E-05 0.0197 0 rpy=0 0 0 -> xyz=-0.025666 0.0177 0.0 rpy=0 0 0
- joint lb2_lb3: axis 0 1 0 -> 0.0 1.0 -0.0; limit lower=-3.14 upper=3.14 effort=50 velocity=15 -> lower=-3.141593 upper=3.141593 effort=5 velocity=1.5; origin xyz=0 0.00475 -0.05 rpy=0 0 0 -> xyz=0.0 0.003 -0.05 rpy=0 0 0
- joint lb3_foot: axis 0 0 0 -> (none); origin xyz=0 0 -0.056 rpy=0 0 0 -> xyz=0.004524 0.00375 -0.059571 rpy=0 0 0
- joint lf1_lf2: axis 0 1 0 -> 0.0 1.0 -0.0; limit lower=-3.14 upper=3.14 effort=50 velocity=15 -> lower=-3.141593 upper=3.141593 effort=5 velocity=1.5; origin xyz=-4E-05 0.0197 0 rpy=0 0 0 -> xyz=0.014866 0.0177 0.0 rpy=0 0 0
- joint lf2_lf3: axis 0 1 0 -> 0.0 1.0 -0.0; limit lower=-3.14 upper=3.14 effort=50 velocity=15 -> lower=-3.141593 upper=3.141593 effort=5 velocity=1.5; origin xyz=0 0.00475 -0.05 rpy=0 0 0 -> xyz=-6e-06 0.003 -0.05 rpy=0 0 0
- joint lf3_foot: axis 0 0 0 -> (none); origin xyz=0 -4.9999999999939E-05 -0.056 rpy=0 0 0 -> xyz=0.00453 0.00375 -0.05957 rpy=0 0 0
- joint rb1_rb2: axis 0 1 0 -> 0.0 1.0 0.0; limit lower=-3.14 upper=3.14 effort=50 velocity=15 -> lower=-3.141593 upper=3.141593 effort=5 velocity=1.5; origin xyz=-4E-05 -0.0197 0 rpy=0 0 0 -> xyz=-0.025666 -0.0177 9e-06 rpy=0 0 0
- joint rb2_rb3: axis 0 1 0 -> 0.0 1.0 0.0; limit lower=-3.14 upper=3.14 effort=50 velocity=15 -> lower=-3.141593 upper=3.141593 effort=5 velocity=1.5; origin xyz=0 -0.00475 -0.05 rpy=0 0 0 -> xyz=0.0 -0.003028 -0.049998 rpy=0 0 0
- joint rb3_foot: axis 0 0 0 -> (none); origin xyz=0 0 -0.056 rpy=0 0 0 -> xyz=0.004524 -0.003782 -0.059568 rpy=0 0 0
- joint rf1_rf2: axis 0 1 0 -> 0.0 1.0 0.0; limit lower=-3.14 upper=3.14 effort=50 velocity=15 -> lower=-3.141593 upper=3.141593 effort=5 velocity=1.5; origin xyz=-4E-05 -0.0197 0 rpy=0 0 0 -> xyz=0.014866 -0.0177 0.0 rpy=0 0 0
- joint rf2_rf3: axis 0 1 0 -> 0.0 1.0 0.0; limit lower=-3.14 upper=3.14 effort=50 velocity=15 -> lower=-3.141593 upper=3.141593 effort=5 velocity=1.5; origin xyz=0 -0.00475 -0.05 rpy=0 0 0 -> xyz=0.0 -0.003 -0.05 rpy=0 0 0
- joint rf3_foot: axis 0 0 0 -> (none); origin xyz=0 0 -0.056 rpy=0 0 0 -> xyz=0.004524 -0.00375 -0.059571 rpy=0 0 0
