Commit message: add: mini pupper 2 urdf working in rviz

File: mini_pupper_description/urdf/mini_pupper_description.urdf.xacro (robot description, xacro)
@@ -1,27 +1,18 @@
-<?xml version="1.0"?>
-<robot name="mini-pupper" xmlns:xacro="http://ros.org/wiki/xacro">
-  <xacro:include filename="$(find mini_pupper_description)/urdf/_d435.urdf.xacro" />
+<?xml version="1.0" ?>
+<robot name="mini_pupper" xmlns:xacro="http://www.ros.org/wiki/xacro">
+  <xacro:include filename="$(find mini_pupper_description)/urdf/materials.xacro" />
+  <!-- <xacro:include filename="$(find mini_pupper_description)/urdf/mini_pupper_description.trans" /> -->
   <link name="base_link">
     <visual>
-      <origin
-        xyz="0 0 0"
-        rpy="0 0 0" />
-      <geometry>
-        <mesh
-          filename="file://$(find mini_pupper_description)/meshes/base_link.STL" />
-      </geometry>
-      <material
-        name="">
-        <color
-          rgba="0.2 0.2 0.2 1" />
-      </material>
-    </visual>
-    <collision>
-      <origin
-        xyz="0 0 0"
-        rpy="0 0 0" />
-      <geometry>
-        <mesh
-          filename="file://$(find mini_pupper_description)/meshes/base_link.STL" />
+      <origin xyz="0 0 0" rpy="0 0 0"/>
+      <geometry>
+        <mesh filename="package://mini_pupper_description/meshes/base_link.stl" scale="1 1 1"/>
+      </geometry>
+      <material name="opaque252525"/>
+    </visual>
+    <collision>
+      <origin xyz="0 0 0" rpy="0 0 0"/>
+      <geometry>
+        <mesh filename="package://mini_pupper_description/meshes/base_link.stl" scale="1 1 1"/>
       </geometry>
     </collision>
@@ -29,1460 +20,762 @@
   <link name="base_inertia">
     <inertial>
-      <origin
-        xyz="0.00660426498064391 8.26976427410632E-06 0.0200623332889016"
-        rpy="0 0 0" />
-      <mass
-        value="0.07" />
-      <inertia
-        ixx="3.3463402501291E-05"
-        ixy="-2.80059099694232E-07"
-        ixz="1.59673474113324E-08"
-        iyy="9.73631866262367E-05"
-        iyz="2.90091309171363E-09"
-        izz="0.00010929561287651" />
-    </inertial>
+      <origin xyz="-0.008866664732250966 0.0006462612742260995 -0.007154314406453802" rpy="0 0 0"/>
+      <mass value="0.09818420433466489"/>
+      <inertia ixx="5.2e-05" iyy="0.000244" izz="0.000252" ixy="1e-06" iyz="1e-06" ixz="-1e-05"/>
+    </inertial>
+  </link>
+  <link name="lf1">
+    <inertial>
+      <origin xyz="0.020109281613098752 0.002331771723067172 0.0064994497731911665" rpy="0 0 0"/>
+      <mass value="0.020769030109708524"/>
+      <inertia ixx="2e-06" iyy="4e-06" izz="3e-06" ixy="-0.0" iyz="-0.0" ixz="-0.0"/>
+    </inertial>
+    <visual>
+      <origin xyz="-0.037299 -0.023745 -5.7e-05" rpy="0 0 0"/>
+      <geometry>
+        <mesh filename="package://mini_pupper_description/meshes/lf1.stl" scale="1 1 1"/>
+      </geometry>
+      <material name="opaque666666"/>
+    </visual>
+    <collision>
+      <origin xyz="-0.037299 -0.023745 -5.7e-05" rpy="0 0 0"/>
+      <geometry>
+        <mesh filename="package://mini_pupper_description/meshes/lf1.stl" scale="1 1 1"/>
+      </geometry>
+    </collision>
+  </link>
+  <link name="lf2">
+    <inertial>
+      <origin xyz="-2.5728896106275156e-06 0.0009860558893138652 -0.018261345499916863" rpy="0 0 0"/>
+      <mass value="0.0019057729925096327"/>
+      <inertia ixx="0.0" iyy="0.0" izz="0.0" ixy="0.0" iyz="0.0" ixz="-0.0"/>
+    </inertial>
+    <visual>
+      <origin xyz="-0.052165 -0.041445 -5.7e-05" rpy="0 0 0"/>
+      <geometry>
+        <mesh filename="package://mini_pupper_description/meshes/lf2.stl" scale="1 1 1"/>
+      </geometry>
+      <material name="opaque636363"/>
+    </visual>
+    <collision>
+      <origin xyz="-0.052165 -0.041445 -5.7e-05" rpy="0 0 0"/>
+      <geometry>
+        <mesh filename="package://mini_pupper_description/meshes/lf2.stl" scale="1 1 1"/>
+      </geometry>
+    </collision>
+  </link>
+  <link name="lf3">
+    <inertial>
+      <origin xyz="0.0007046107744873437 0.0034550275861905885 -0.016225601428628958" rpy="0 0 0"/>
+      <mass value="0.0011438144457690698"/>
+      <inertia ixx="1e-06" iyy="1e-06" izz="0.0" ixy="-0.0" iyz="0.0" ixz="0.0"/>
+    </inertial>
+    <visual>
+      <origin xyz="-0.052159 -0.044445 0.049943" rpy="0 0 0"/>
+      <geometry>
+        <mesh filename="package://mini_pupper_description/meshes/lf3.stl" scale="1 1 1"/>
+      </geometry>
+      <material name="opaque252525"/>
+    </visual>
+    <collision>
+      <origin xyz="-0.052159 -0.044445 0.049943" rpy="0 0 0"/>
+      <geometry>
+        <mesh filename="package://mini_pupper_description/meshes/lf3.stl" scale="1 1 1"/>
+      </geometry>
+    </collision>
+  </link>
+  <link name="rf1">
+      <inertial>
+      <origin xyz="0.020106742599110078 -0.00233237781568562 0.006497900858401761" rpy="0 0 0"/>
+      <mass value="0.020769549324466178"/>
+      <inertia ixx="2e-06" iyy="4e-06" izz="3e-06" ixy="0.0" iyz="-0.0" ixz="-0.0"/>
+    </inertial>
+    <visual>
+      <origin xyz="-0.037299 0.023255 -5.7e-05" rpy="0 0 0"/>
+      <geometry>
+        <mesh filename="package://mini_pupper_description/meshes/rf1.stl" scale="1 1 1"/>
+      </geometry>
+      <material name="opaque666666"/>
+    </visual>
+    <collision>
+      <origin xyz="-0.037299 0.023255 -5.7e-05" rpy="0 0 0"/>
+      <geometry>
+        <mesh filename="package://mini_pupper_description/meshes/rf1.stl" scale="1 1 1"/>
+      </geometry>
+    </collision>
+  </link>
+  <link name="rf2">
+    <inertial>
+      <origin xyz="-4.1025190424676117e-07 -0.0009866275794596438 -0.018261345629717353" rpy="0 0 0"/>
+      <mass value="0.0019057729924780605"/>
+      <inertia ixx="0.0" iyy="0.0" izz="0.0" ixy="-0.0" iyz="-0.0" ixz="-0.0"/>
+    </inertial>
+    <visual>
+      <origin xyz="-0.052165 0.040955 -5.7e-05" rpy="0 0 0"/>
+      <geometry>
+        <mesh filename="package://mini_pupper_description/meshes/rf2.stl" scale="1 1 1"/>
+      </geometry>
+      <material name="opaque636363"/>
+    </visual>
+    <collision>
+      <origin xyz="-0.052165 0.040955 -5.7e-05" rpy="0 0 0"/>
+      <geometry>
+        <mesh filename="package://mini_pupper_description/meshes/rf2.stl" scale="1 1 1"/>
+      </geometry>
+    </collision>
+  </link>
+  <link name="rf3">
+    <inertial>
+      <origin xyz="0.0007030898236521158 -0.003457422744677939 -0.016230262912113935" rpy="0 0 0"/>
+      <mass value="0.001143490701517533"/>
+      <inertia ixx="1e-06" iyy="1e-06" izz="0.0" ixy="0.0" iyz="-0.0" ixz="0.0"/>
+    </inertial>
+    <visual>
+      <origin xyz="-0.052165 0.043955 0.049943" rpy="0 0 0"/>
+      <geometry>
+        <mesh filename="package://mini_pupper_description/meshes/rf3.stl" scale="1 1 1"/>
+      </geometry>
+      <material name="opaque252525"/>
+    </visual>
+    <collision>
+      <origin xyz="-0.052165 0.043955 0.049943" rpy="0 0 0"/>
+      <geometry>
+        <mesh filename="package://mini_pupper_description/meshes/rf3.stl" scale="1 1 1"/>
+      </geometry>
+    </collision>
+  </link>
+  <link name="rb1">
+    <inertial>
+      <origin xyz="-0.020107177922528044 -0.0023288309787250286 0.006502376356642127" rpy="0 0 0"/>
+      <mass value="0.020769549324363486"/>
+      <inertia ixx="2e-06" iyy="4e-06" izz="3e-06" ixy="-0.0" iyz="-0.0" ixz="-0.0"/>
+    </inertial>
+    <visual>
+      <origin xyz="0.042701 0.023255 -5.7e-05" rpy="0 0 0"/>
+      <geometry>
+        <mesh filename="package://mini_pupper_description/meshes/rb1.stl" scale="1 1 1"/>
+      </geometry>
+      <material name="opaque666666"/>
+    </visual>
+    <collision>
+      <origin xyz="0.042701 0.023255 -5.7e-05" rpy="0 0 0"/>
+      <geometry>
+        <mesh filename="package://mini_pupper_description/meshes/rb1.stl" scale="1 1 1"/>
+      </geometry>
+    </collision>
+  </link>
+  <link name="rb2">
+    <inertial>
+      <origin xyz="-2.5070667000748337e-08 -0.000996585764066693 -0.018260149861185754" rpy="0 0 0"/>
+      <mass value="0.0019057729926311429"/>
+      <inertia ixx="0.0" iyy="0.0" izz="0.0" ixy="-0.0" iyz="-0.0" ixz="-0.0"/>
+    </inertial>
+    <visual>
+      <origin xyz="0.068367 0.040955 -6.6e-05" rpy="0 0 0"/>
+      <geometry>
+        <mesh filename="package://mini_pupper_description/meshes/rb2.stl" scale="1 1 1"/>
+      </geometry>
+      <material name="opaque636363"/>
+    </visual>
+    <collision>
+      <origin xyz="0.068367 0.040955 -6.6e-05" rpy="0 0 0"/>
+      <geometry>
+        <mesh filename="package://mini_pupper_description/meshes/rb2.stl" scale="1 1 1"/>
+      </geometry>
+    </collision>
+  </link>
+  <link name="rb3">
+    <inertial>
+      <origin xyz="0.0007031309185970697 -0.0034624258831375196 -0.016220094399306113" rpy="0 0 0"/>
+      <mass value="0.0011440535724654094"/>
+      <inertia ixx="1e-06" iyy="1e-06" izz="0.0" ixy="0.0" iyz="-0.0" ixz="0.0"/>
+    </inertial>
+    <visual>
+      <origin xyz="0.068367 0.043983 0.049932" rpy="0 0 0"/>
+      <geometry>
+        <mesh filename="package://mini_pupper_description/meshes/rb3.stl" scale="1 1 1"/>
+      </geometry>
+      <material name="opaque252525"/>
+    </visual>
+    <collision>
+      <origin xyz="0.068367 0.043983 0.049932" rpy="0 0 0"/>
+      <geometry>
+        <mesh filename="package://mini_pupper_description/meshes/rb3.stl" scale="1 1 1"/>
+      </geometry>
+    </collision>
+  </link>
+  <link name="lb1">
+    <inertial>
+      <origin xyz="-0.020109716415830967 0.0023317718989125207 0.006499556305653081" rpy="0 0 0"/>
+      <mass value="0.020769030189864354"/>
+      <inertia ixx="2e-06" iyy="4e-06" izz="3e-06" ixy="0.0" iyz="0.0" ixz="-0.0"/>
+    </inertial>
+    <visual>
+      <origin xyz="0.042701 -0.023745 -5.7e-05" rpy="0 0 0"/>
+      <geometry>
+        <mesh filename="package://mini_pupper_description/meshes/lb1.stl" scale="1 1 1"/>
+      </geometry>
+      <material name="opaque666666"/>
+    </visual>
+    <collision>
+      <origin xyz="0.042701 -0.023745 -5.7e-05" rpy="0 0 0"/>
+      <geometry>
+        <mesh filename="package://mini_pupper_description/meshes/lb1.stl" scale="1 1 1"/>
+      </geometry>
+    </collision>
+  </link>
+  <link name="lb2">
+    <inertial>
+      <origin xyz="-2.486178994620669e-08 0.0009860564153100007 -0.01826134562993383" rpy="0 0 0"/>
+      <mass value="0.0019057729925095609"/>
+      <inertia ixx="0.0" iyy="0.0" izz="0.0" ixy="0.0" iyz="0.0" ixz="-0.0"/>
+    </inertial>
+    <visual>
+      <origin xyz="0.068367 -0.041445 -5.7e-05" rpy="0 0 0"/>
+      <geometry>
+        <mesh filename="package://mini_pupper_description/meshes/lb2.stl" scale="1 1 1"/>
+      </geometry>
+      <material name="opaque636363"/>
+    </visual>
+    <collision>
+      <origin xyz="0.068367 -0.041445 -5.7e-05" rpy="0 0 0"/>
+      <geometry>
+        <mesh filename="package://mini_pupper_description/meshes/lb2.stl" scale="1 1 1"/>
+      </geometry>
+    </collision>
+  </link>
+  <link name="lb3">
+    <inertial>
+      <origin xyz="0.0007030123702261443 0.0034519487133846394 -0.016218113385159758" rpy="0 0 0"/>
+      <mass value="0.001144346207072784"/>
+      <inertia ixx="1e-06" iyy="1e-06" izz="0.0" ixy="-0.0" iyz="0.0" ixz="0.0"/>
+    </inertial>
+    <visual>
+      <origin xyz="0.068367 -0.044445 0.049943" rpy="0 0 0"/>
+      <geometry>
+        <mesh filename="package://mini_pupper_description/meshes/lb3.stl" scale="1 1 1"/>
+      </geometry>
+      <material name="opaque252525"/>
+    </visual>
+    <collision>
+      <origin xyz="0.068367 -0.044445 0.049943" rpy="0 0 0"/>
+      <geometry>
+        <mesh filename="package://mini_pupper_description/meshes/lb3.stl" scale="1 1 1"/>
+      </geometry>
+    </collision>
+  </link>
+  <link name="Body_front">
+    <inertial>
+      <origin xyz="-0.005538678480206852 -0.00020424196520824284 0.020222593513387798" rpy="0 0 0"/>
+      <mass value="0.00785515871148119"/>
+      <inertia ixx="5e-06" iyy="2e-06" izz="4e-06" ixy="-0.0" iyz="-0.0" ixz="-0.0"/>
+    </inertial>
+    <visual>
+      <origin xyz="-0.089299 -0.000245 0.015543" rpy="0 0 0"/>
+      <geometry>
+        <mesh filename="package://mini_pupper_description/meshes/Body_front.stl" scale="1 1 1"/>
+      </geometry>
+      <material name="opaque2552210"/>
+    </visual>
+    <collision>
+      <origin xyz="-0.089299 -0.000245 0.015543" rpy="0 0 0"/>
+      <geometry>
+        <mesh filename="package://mini_pupper_description/meshes/Body_front.stl" scale="1 1 1"/>
+      </geometry>
+    </collision>
+  </link>
+  <link name="Board_PCB">
+    <inertial>
+      <origin xyz="0.08946128454598752 0.025716073555853 -3.6415040620890043e-05" rpy="0 0 0"/>
+      <mass value="0.014261552601793053"/>
+      <inertia ixx="4e-06" iyy="3.5e-05" izz="3.9e-05" ixy="0.0" iyz="0.0" ixz="0.0"/>
+    </inertial>
+    <visual>
+      <origin xyz="0.087701 0.023255 -0.026457" rpy="0 0 0"/>
+      <geometry>
+        <mesh filename="package://mini_pupper_description/meshes/Board_PCB.stl" scale="1 1 1"/>
+      </geometry>
+      <material name="opaque646464"/>
+    </visual>
+    <collision>
+      <origin xyz="0.087701 0.023255 -0.026457" rpy="0 0 0"/>
+      <geometry>
+        <mesh filename="package://mini_pupper_description/meshes/Board_PCB.stl" scale="1 1 1"/>
+      </geometry>
+    </collision>
+  </link>
+  <link name="Board_connectors_1">
+    <inertial>
+      <origin xyz="-0.07276303117117414 -0.002323344081837563 -0.0010631239213060653" rpy="0 0 0"/>
+      <mass value="0.004688613655947816"/>
+      <inertia ixx="0.0" iyy="1.5e-05" izz="1.6e-05" ixy="-1e-06" iyz="0.0" ixz="0.0"/>
+    </inertial>
+    <visual>
+      <origin xyz="-0.061334 -0.000217 -0.026457" rpy="0 0 0"/>
+      <geometry>
+        <mesh filename="package://mini_pupper_description/meshes/Board_connectors_1.stl" scale="1 1 1"/>
+      </geometry>
+      <material name="opaque2491590"/>
+    </visual>
+    <collision>
+      <origin xyz="-0.061334 -0.000217 -0.026457" rpy="0 0 0"/>
+      <geometry>
+        <mesh filename="package://mini_pupper_description/meshes/Board_connectors_1.stl" scale="1 1 1"/>
+      </geometry>
+    </collision>
+  </link>
+  <link name="Board_connectors_2">
+    <inertial>
+      <origin xyz="0.008233541174180986 -0.002138369786547657 -0.00030110978110910874" rpy="0 0 0"/>
+      <mass value="0.0019746031301169403"/>
+      <inertia ixx="0.0" iyy="3e-06" izz="4e-06" ixy="-0.0" iyz="0.0" ixz="0.0"/>
+    </inertial>
+    <visual>
+      <origin xyz="0.045346 -0.000245 -0.026457" rpy="0 0 0"/>
+      <geometry>
+        <mesh filename="package://mini_pupper_description/meshes/Board_connectors_2.stl" scale="1 1 1"/>
+      </geometry>
+      <material name="opaque255255255"/>
+    </visual>
+    <collision>
+      <origin xyz="0.045346 -0.000245 -0.026457" rpy="0 0 0"/>
+      <geometry>
+        <mesh filename="package://mini_pupper_description/meshes/Board_connectors_2.stl" scale="1 1 1"/>
+      </geometry>
+    </collision>
+  </link>
+  <link name="rffoot">
+    <inertial>
+      <origin xyz="-0.0024634044240561814 -2.8557999392359035e-07 0.007801816226636768" rpy="0 0 0"/>
+      <mass value="0.0014053107976262874"/>
+      <inertia ixx="0.0" iyy="0.0" izz="0.0" ixy="0.0" iyz="-0.0" ixz="-0.0"/>
+    </inertial>
+    <visual>
+      <origin xyz="-0.056689 0.047705 0.109514" rpy="0 0 0"/>
+      <geometry>
+        <mesh filename="package://mini_pupper_description/meshes/rffoot.stl" scale="1 1 1"/>
+      </geometry>
+      <material name="opaque666666"/>
+    </visual>
+    <collision>
+      <origin xyz="-0.056689 0.047705 0.109514" rpy="0 0 0"/>
+      <geometry>
+        <mesh filename="package://mini_pupper_description/meshes/rffoot.stl" scale="1 1 1"/>
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