Commit message: restore mp1 files

File: mini_pupper_description/urdf/mini_pupper_description.urdf (robot description, URDF)
Before this commit: robot mini-pupper, 29 links, 28 joints
Links:
- removed link lidar_link
- added link camera_bottom_screw_frame
- added link camera_color_frame
- added link camera_color_optical_frame
- added link camera_depth_frame
- added link camera_depth_optical_frame
- added link camera_infra1_frame
- added link camera_infra1_optical_frame
- added link camera_infra2_frame
- added link camera_infra2_optical_frame
- added link camera_link, mass 0.0072; collision box size=0.02505 0.09 0.025; visual mesh filename=file://$(find mini_pupper_description)/meshes/d435.dae
- added link lidar, mass 0.0001; collision mesh filename=file://$(find mini_pupper_description)/meshes/lidar.STL; visual mesh filename=file://$(find mini_pupper_description)/meshes/lidar.STL
- link base_inertia: mass 0.07 -> 0.2
- link base_link: geometry collision mesh filename=file://$(find mini_pupper_description)/meshes/base_link.STL; visual mesh filename=file://$(find mini_pupper_description)/meshes/base_link.STL
- link lb1: mass 0.025 -> 0.00025; geometry collision mesh filename=file://$(find mini_pupper_description)/meshes/lb1.STL; visual mesh filename=file://$(find mini_pupper_description)/meshes/lb1.STL
- link lb2: mass 0.0125 -> 0.00125; geometry collision mesh filename=file://$(find mini_pupper_description)/meshes/lb2.STL; visual mesh filename=file://$(find mini_pupper_description)/meshes/lb2.STL
- link lb3: mass 0.00625 -> 0.000625; geometry collision mesh filename=file://$(find mini_pupper_description)/meshes/lb3.STL; visual mesh filename=file://$(find mini_pupper_description)/meshes/lb3.STL
- link lbfoot: mass 0.00625 -> 0.000625; geometry collision mesh filename=file://$(find mini_pupper_description)/meshes/lbfoot.STL; visual mesh filename=file://$(find mini_pupper_description)/meshes/lbfoot.STL
- link lf1: mass 0.025 -> 0.0025; geometry collision mesh filename=file://$(find mini_pupper_description)/meshes/lf1.STL; visual mesh filename=file://$(find mini_pupper_description)/meshes/lf1.STL
- link lf2: mass 0.0125 -> 0.00125; geometry collision mesh filename=file://$(find mini_pupper_description)/meshes/lf2.STL; visual mesh filename=file://$(find mini_pupper_description)/meshes/lf2.STL
- link lf3: mass 0.00625 -> 0.000625; geometry collision mesh filename=file://$(find mini_pupper_description)/meshes/lf3.STL; visual mesh filename=file://$(find mini_pupper_description)/meshes/lf3.STL
- link lffoot: mass 0.00625 -> 0.000625; geometry collision mesh filename=file://$(find mini_pupper_description)/meshes/lffoot.STL; visual mesh filename=file://$(find mini_pupper_description)/meshes/lffoot.STL
- link lpb1: geometry collision mesh filename=file://$(find mini_pupper_description)/meshes/lpb1.STL; visual mesh filename=file://$(find mini_pupper_description)/meshes/lpb1.STL
- link lpb2: geometry collision mesh filename=file://$(find mini_pupper_description)/meshes/lpb2.STL; visual mesh filename=file://$(find mini_pupper_description)/meshes/lpb2.STL
- link lpf1: geometry collision mesh filename=file://$(find mini_pupper_description)/meshes/lpf1.STL; visual mesh filename=file://$(find mini_pupper_description)/meshes/lpf1.STL
- link lpf2: geometry collision mesh filename=file://$(find mini_pupper_description)/meshes/lpf2.STL; visual mesh filename=file://$(find mini_pupper_description)/meshes/lpf2.STL
- link rb1: mass 0.025 -> 0.0025; geometry collision mesh filename=file://$(find mini_pupper_description)/meshes/rb1.STL; visual mesh filename=file://$(find mini_pupper_description)/meshes/rb1.STL
- link rb2: mass 0.0125 -> 0.00125; geometry collision mesh filename=file://$(find mini_pupper_description)/meshes/rb2.STL; visual mesh filename=file://$(find mini_pupper_description)/meshes/rb2.STL
- link rb3: mass 0.00625 -> 0.000625; geometry collision mesh filename=file://$(find mini_pupper_description)/meshes/rb3.STL; visual mesh filename=file://$(find mini_pupper_description)/meshes/rb3.STL
- link rbfoot: mass 0.00625 -> 0.000625; geometry collision mesh filename=file://$(find mini_pupper_description)/meshes/rbfoot.STL; visual mesh filename=file://$(find mini_pupper_description)/meshes/rbfoot.STL
- link rf1: mass 0.025 -> 0.0025; geometry collision mesh filename=file://$(find mini_pupper_description)/meshes/rf1.STL; visual mesh filename=file://$(find mini_pupper_description)/meshes/rf1.STL
- link rf2: mass 0.0125 -> 0.00125; geometry collision mesh filename=file://$(find mini_pupper_description)/meshes/rf2.STL; visual mesh filename=file://$(find mini_pupper_description)/meshes/rf2.STL
- link rf3: mass 0.00625 -> 0.000625; geometry collision mesh filename=file://$(find mini_pupper_description)/meshes/rf3.STL; visual mesh filename=file://$(find mini_pupper_description)/meshes/rf3.STL
- link rffoot: mass 0.00625 -> 0.000625; geometry collision mesh filename=file://$(find mini_pupper_description)/meshes/rffoot.STL; visual mesh filename=file://$(find mini_pupper_description)/meshes/rffoot.STL
- link rpb1: geometry collision mesh filename=file://$(find mini_pupper_description)/meshes/rpb1.STL; visual mesh filename=file://$(find mini_pupper_description)/meshes/rpb1.STL
- link rpb2: geometry collision mesh filename=file://$(find mini_pupper_description)/meshes/rpb2.STL; visual mesh filename=file://$(find mini_pupper_description)/meshes/rpb2.STL
- link rpf1: geometry collision mesh filename=file://$(find mini_pupper_description)/meshes/rpf1.STL; visual mesh filename=file://$(find mini_pupper_description)/meshes/rpf1.STL
- link rpf2: geometry collision mesh filename=file://$(find mini_pupper_description)/meshes/rpf2.STL; visual mesh filename=file://$(find mini_pupper_description)/meshes/rpf2.STL
- link yellow_plate: mass 0.03 -> 0.002; geometry collision mesh filename=file://$(find mini_pupper_description)/meshes/yellow_plate.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; visual mesh filename=file://$(find mini_pupper_description)/meshes/yellow_plate.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
Joints:
- added joint camera_color_joint: type fixed, parent camera_link, child camera_color_frame, origin xyz=0 0.015 0 rpy=0 0 0
- added joint camera_color_optical_joint: type fixed, parent camera_color_frame, child camera_color_optical_frame, origin xyz=0 0 0 rpy=-1.5707963267948966 0 -1.5707963267948966
- added joint camera_depth_joint: type fixed, parent camera_link, child camera_depth_frame, origin xyz=0 0 0 rpy=0 0 0
- added joint camera_depth_optical_joint: type fixed, parent camera_depth_frame, child camera_depth_optical_frame, origin xyz=0 0 0 rpy=-1.5707963267948966 0 -1.5707963267948966
- added joint camera_infra1_joint: type fixed, parent camera_link, child camera_infra1_frame, origin xyz=0 0.0 0 rpy=0 0 0
- added joint camera_infra1_optical_joint: type fixed, parent camera_infra1_frame, child camera_infra1_optical_frame, origin xyz=0 0 0 rpy=-1.5707963267948966 0 -1.5707963267948966
- added joint camera_infra2_joint: type fixed, parent camera_link, child camera_infra2_frame, origin xyz=0 -0.05 0 rpy=0 0 0
- added joint camera_infra2_optical_joint: type fixed, parent camera_infra2_frame, child camera_infra2_optical_frame, origin xyz=0 0 0 rpy=-1.5707963267948966 0 -1.5707963267948966
- added joint camera_joint: type fixed, parent base_link, child camera_bottom_screw_frame, origin xyz=0.08 0.0 0.07 rpy=0 0 0
- added joint camera_link_joint: type fixed, parent camera_bottom_screw_frame, child camera_link, origin xyz=0.010600000000000002 0.0175 0.0125 rpy=0 0 0
- joint base_lb1: limit lower=-3.14 upper=3.14 effort=5 velocity=1.5 -> lower=-3.14 upper=3.14 effort=50 velocity=15
- joint base_lf1: limit lower=-3.14 upper=3.14 effort=5 velocity=1.5 -> lower=-3.14 upper=3.14 effort=50 velocity=15
- joint base_lidar: child lidar_link -> lidar
- joint base_rb1: limit lower=-3.14 upper=3.14 effort=5 velocity=1.5 -> lower=-3.14 upper=3.14 effort=50 velocity=15
- joint base_rf1: limit lower=-3.14 upper=3.14 effort=5 velocity=1.5 -> lower=-3.14 upper=3.14 effort=50 velocity=15
- joint lb1_lb2: limit lower=-3.14 upper=3.14 effort=5 velocity=1.5 -> lower=-3.14 upper=3.14 effort=50 velocity=15
- joint lb2_lb3: limit lower=-3.14 upper=3.14 effort=5 velocity=1.5 -> lower=-3.14 upper=3.14 effort=50 velocity=15
- joint lf1_lf2: limit lower=-3.14 upper=3.14 effort=5 velocity=1.5 -> lower=-3.14 upper=3.14 effort=50 velocity=15
- joint lf2_lf3: limit lower=-3.14 upper=3.14 effort=5 velocity=1.5 -> lower=-3.14 upper=3.14 effort=50 velocity=15
- joint rb1_rb2: limit lower=-3.14 upper=3.14 effort=5 velocity=1.5 -> lower=-3.14 upper=3.14 effort=50 velocity=15
- joint rb2_rb3: limit lower=-3.14 upper=3.14 effort=5 velocity=1.5 -> lower=-3.14 upper=3.14 effort=50 velocity=15
- joint rf1_rf2: limit lower=-3.14 upper=3.14 effort=5 velocity=1.5 -> lower=-3.14 upper=3.14 effort=50 velocity=15
- joint rf2_rf3: limit lower=-3.14 upper=3.14 effort=5 velocity=1.5 -> lower=-3.14 upper=3.14 effort=50 velocity=15

Commit message: tidy and merge description files of two robot models

File: mini_pupper_description/urdf/mini_pupper_description.urdf (robot description, URDF)
Before this commit: robot mini-pupper, 39 links, 38 joints
Links:
- link camera_link: geometry collision box size=0.02505 0.09 0.025; visual mesh filename=file://$(find mini_pupper_description)/mini_pupper_meshes/m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
- link lb1: geometry collision mesh filename=file://$(find mini_pupper_description)/mini_pupper_meshes/m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; visual mesh filename=file://$(find mini_pupper_description)/mini_pupper_meshes/m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
- link lb2: geometry collision mesh filename=file://$(find mini_pupper_description)/mini_pupper_meshes/m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; visual mesh filename=file://$(find mini_pupper_description)/mini_pupper_meshes/m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
- link lb3: geometry collision mesh filename=file://$(find mini_pupper_description)/mini_pupper_meshes/m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; visual mesh filename=file://$(find mini_pupper_description)/mini_pupper_meshes/m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
- link lbfoot: geometry collision mesh filename=file://$(find mini_pupper_description)/mini_pupper_meshes/m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; visual mesh filename=file://$(find mini_pupper_description)/mini_pupper_meshes/m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
- link lf1: geometry collision mesh filename=file://$(find mini_pupper_description)/mini_pupper_meshes/m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; visual mesh filename=file://$(find mini_pupper_description)/mini_pupper_meshes/m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
- link lf2: geometry collision mesh filename=file://$(find mini_pupper_description)/mini_pupper_meshes/m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; visual mesh filename=file://$(find mini_pupper_description)/mini_pupper_meshes/m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
- link lf3: geometry collision mesh filename=file://$(find mini_pupper_description)/meshes/lf3.STL; visual mesh filename=file://$(find mini_pupper_description)/mini_pupper_meshes/m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
- link lffoot: geometry collision mesh filename=file://$(find mini_pupper_description)/mini_pupper_meshes/m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; visual mesh filename=file://$(find mini_pupper_description)/mini_pupper_meshes/m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
- link lidar: geometry collision mesh filename=file://$(find mini_pupper_description)/mini_pupper_meshes/m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; visual mesh filename=file://$(find mini_pupper_description)/mini_pupper_meshes/m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
- link lpb1: geometry collision mesh filename=file://$(find mini_pupper_description)/mini_pupper_meshes/m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; visual mesh filename=file://$(find mini_pupper_description)/mini_pupper_meshes/m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
- link lpb2: geometry collision mesh filename=file://$(find mini_pupper_description)/mini_pupper_meshes/m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; visual mesh filename=file://$(find mini_pupper_description)/mini_pupper_meshes/m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
- link lpf1: geometry collision mesh filename=file://$(find mini_pupper_description)/mini_pupper_meshes/m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; visual mesh filename=file://$(find mini_pupper_description)/mini_pupper_meshes/m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
- link lpf2: geometry collision mesh filename=file://$(find mini_pupper_description)/mini_pupper_meshes/m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; visual mesh filename=file://$(find mini_pupper_description)/mini_pupper_meshes/m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
- link rb1: geometry collision mesh filename=file://$(find mini_pupper_description)/mini_pupper_meshes/m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; visual mesh filename=file://$(find mini_pupper_description)/mini_pupper_meshes/m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
- link rb2: geometry collision mesh filename=file://$(find mini_pupper_description)/mini_pupper_meshes/m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; visual mesh filename=file://$(find mini_pupper_description)/mini_pupper_meshes/m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
- link rb3: geometry collision mesh filename=file://$(find mini_pupper_description)/mini_pupper_meshes/m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; visual mesh filename=file://$(find mini_pupper_description)/mini_pupper_meshes/m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
- link rbfoot: geometry collision mesh filename=file://$(find mini_pupper_description)/mini_pupper_meshes/m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; visual mesh filename=file://$(find mini_pupper_description)/mini_pupper_meshes/m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
- link rf1: geometry collision mesh filename=file://$(find mini_pupper_description)/mini_pupper_meshes/m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; visual mesh filename=file://$(find mini_pupper_description)/mini_pupper_meshes/m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
- link rf2: geometry collision mesh filename=file://$(find mini_pupper_description)/mini_pupper_meshes/m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; visual mesh filename=file://$(find mini_pupper_description)/mini_pupper_meshes/m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
- link rf3: geometry collision mesh filename=file://$(find mini_pupper_description)/mini_pupper_meshes/m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; visual mesh filename=file://$(find mini_pupper_description)/mini_pupper_meshes/m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
- link rffoot: geometry collision mesh filename=file://$(find mini_pupper_description)/mini_pupper_meshes/m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; visual mesh filename=file://$(find mini_pupper_description)/mini_pupper_meshes/m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
- link rpb1: geometry collision mesh filename=file://$(find mini_pupper_description)/mini_pupper_meshes/m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; visual mesh filename=file://$(find mini_pupper_description)/mini_pupper_meshes/m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
- link rpb2: geometry collision mesh filename=file://$(find mini_pupper_description)/mini_pupper_meshes/m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; visual mesh filename=file://$(find mini_pupper_description)/mini_pupper_meshes/m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
- link rpf1: geometry collision mesh filename=file://$(find mini_pupper_description)/mini_pupper_meshes/m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; visual mesh filename=file://$(find mini_pupper_description)/mini_pupper_meshes/m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
- link rpf2: geometry collision mesh filename=file://$(find mini_pupper_description)/mini_pupper_meshes/m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; visual mesh filename=file://$(find mini_pupper_description)/mini_pupper_meshes/m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

Commit message: fix urdf wrong path

File: mini_pupper_description/urdf/mini_pupper_description.urdf (robot description, URDF)
Before this commit: robot mini-pupper, 29 links, 28 joints
Links:
- link base_link: geometry collision mesh filename=package://mini_pupper_description/meshes/mini_pupper_base_l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; visual mesh filename=package://mini_pupper_description/meshes/mini_pupper_base_l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
- link lb1: geometry collision mesh filename=package://mini_pupper_description/meshes/mini_pupper_lb1.STL; visual mesh filename=package://mini_pupper_description/meshes/mini_pupper_lb1.STL
- link lb2: geometry collision mesh filename=package://mini_pupper_description/meshes/mini_pupper_lb2.STL; visual mesh filename=package://mini_pupper_description/meshes/mini_pupper_lb2.STL
- link lb3: geometry collision mesh filename=package://mini_pupper_description/meshes/mini_pupper_lb3.STL; visual mesh filename=package://mini_pupper_description/meshes/mini_pupper_lb3.STL
- link lbfoot: geometry collision mesh filename=package://mini_pupper_description/meshes/mini_pupper_lbfoot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; visual mesh filename=package://mini_pupper_description/meshes/mini_pupper_lbfoot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
- link lf1: geometry collision mesh filename=package://mini_pupper_description/meshes/mini_pupper_lf1.STL; visual mesh filename=package://mini_pupper_description/meshes/mini_pupper_lf1.STL
- link lf2: geometry collision mesh filename=package://mini_pupper_description/meshes/mini_pupper_lf2.STL; visual mesh filename=package://mini_pupper_description/meshes/mini_pupper_lf2.STL
- link lf3: geometry collision mesh filename=package://mini_pupper_description/meshes/mini_pupper_lf3.STL; visual mesh filename=package://mini_pupper_description/meshes/mini_pupper_lf3.STL
- link lffoot: geometry collision mesh filename=package://mini_pupper_description/meshes/mini_pupper_lffoot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; visual mesh filename=package://mini_pupper_description/meshes/mini_pupper_lffoot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
- link lidar_link: geometry collision mesh filename=package://mini_pupper_description/meshes/mini_pupper_lidar.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; visual mesh filename=package://mini_pupper_description/meshes/mini_pupper_lidar.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
- link lpb1: geometry collision mesh filename=package://mini_pupper_description/meshes/mini_pupper_lpb1.S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; visual mesh filename=package://mini_pupper_description/meshes/mini_pupper_lpb1.S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
- link lpb2: geometry collision mesh filename=package://mini_pupper_description/meshes/mini_pupper_lpb2.S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; visual mesh filename=package://mini_pupper_description/meshes/mini_pupper_lpb2.S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
- link lpf1: geometry collision mesh filename=package://mini_pupper_description/meshes/mini_pupper_lpf1.S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; visual mesh filename=package://mini_pupper_description/meshes/mini_pupper_lpf1.S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
- link lpf2: geometry collision mesh filename=package://mini_pupper_description/meshes/mini_pupper_lpf2.S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; visual mesh filename=package://mini_pupper_description/meshes/mini_pupper_lpf2.S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
- link rb1: geometry collision mesh filename=package://mini_pupper_description/meshes/mini_pupper_rb1.STL; visual mesh filename=package://mini_pupper_description/meshes/mini_pupper_rb1.STL
- link rb2: geometry collision mesh filename=package://mini_pupper_description/meshes/mini_pupper_rb2.STL; visual mesh filename=package://mini_pupper_description/meshes/mini_pupper_rb2.STL
- link rb3: geometry collision mesh filename=package://mini_pupper_description/meshes/mini_pupper_rb3.STL; visual mesh filename=package://mini_pupper_description/meshes/mini_pupper_rb3.STL
- link rbfoot: geometry collision mesh filename=package://mini_pupper_description/meshes/mini_pupper_rbfoot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; visual mesh filename=package://mini_pupper_description/meshes/mini_pupper_rbfoot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
- link rf1: geometry collision mesh filename=package://mini_pupper_description/meshes/mini_pupper_rf1.STL; visual mesh filename=package://mini_pupper_description/meshes/mini_pupper_rf1.STL
- link rf2: geometry collision mesh filename=package://mini_pupper_description/meshes/mini_pupper_rf2.STL; visual mesh filename=package://mini_pupper_description/meshes/mini_pupper_rf2.STL
- link rf3: geometry collision mesh filename=package://mini_pupper_description/meshes/mini_pupper_rf3.STL; visual mesh filename=package://mini_pupper_description/meshes/mini_pupper_rf3.STL
- link rffoot: geometry collision mesh filename=package://mini_pupper_description/meshes/mini_pupper_rffoot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; visual mesh filename=package://mini_pupper_description/meshes/mini_pupper_rffoot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
- link rpb1: geometry collision mesh filename=package://mini_pupper_description/meshes/mini_pupper_rpb1.S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; visual mesh filename=package://mini_pupper_description/meshes/mini_pupper_rpb1.S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
- link rpb2: geometry collision mesh filename=package://mini_pupper_description/meshes/mini_pupper_rpb2.S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; visual mesh filename=package://mini_pupper_description/meshes/mini_pupper_rpb2.S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
- link rpf1: geometry collision mesh filename=package://mini_pupper_description/meshes/mini_pupper_rpf1.S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; visual mesh filename=package://mini_pupper_description/meshes/mini_pupper_rpf1.S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
- link rpf2: geometry collision mesh filename=package://mini_pupper_description/meshes/mini_pupper_rpf2.S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; visual mesh filename=package://mini_pupper_description/meshes/mini_pupper_rpf2.S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
- link yellow_plate: geometry collision mesh filename=package://mini_pupper_description/meshes/mini_pupper_yellow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; visual mesh filename=package://mini_pupper_description/meshes/mini_pupper_yellow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
