Commit message: further tidy format and addition of removed dependent .urdf files

File: mini_pupper_description/urdf/mini_pupper_2_description.urdf (robot description, URDF)
Before this commit: robot mini_pupper_2, 33 links, 32 joints
Links:
- link Board_PCB: geometry collision mesh filename=package://mini_pupper_2_description/mini_pupper_2_meshes/mi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 scale=1 1 1; visual mesh filename=package://mini_pupper_2_description/mini_pupper_2_meshes/mi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 scale=1 1 1
- link Board_connectors_1: geometry collision mesh filename=package://mini_pupper_2_description/mini_pupper_2_meshes/mi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 scale=1 1 1; visual mesh filename=package://mini_pupper_2_description/mini_pupper_2_meshes/mi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 scale=1 1 1
- link Board_connectors_2: geometry collision mesh filename=package://mini_pupper_2_description/mini_pupper_2_meshes/mi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 scale=1 1 1; visual mesh filename=package://mini_pupper_2_description/mini_pupper_2_meshes/mi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 scale=1 1 1
- link Body_front: geometry collision mesh filename=package://mini_pupper_2_description/mini_pupper_2_meshes/mi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 scale=1 1 1; visual mesh filename=package://mini_pupper_2_description/mini_pupper_2_meshes/mi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 scale=1 1 1
- link Shell_Side: geometry collision mesh filename=package://mini_pupper_2_description/mini_pupper_2_meshes/mi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 scale=1 1 1; visual mesh filename=package://mini_pupper_2_description/mini_pupper_2_meshes/mi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 scale=1 1 1
- link base_link: geometry collision mesh filename=package://mini_pupper_2_description/mini_pupper_2_meshes/mi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 scale=1 1 1; visual mesh filename=package://mini_pupper_2_description/mini_pupper_2_meshes/mi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 scale=1 1 1
- link lb1: geometry collision mesh filename=package://mini_pupper_2_description/mini_pupper_2_meshes/mi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 scale=1 1 1; visual mesh filename=package://mini_pupper_2_description/mini_pupper_2_meshes/mi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 scale=1 1 1
- link lb2: geometry collision mesh filename=package://mini_pupper_2_description/mini_pupper_2_meshes/mi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 scale=1 1 1; visual mesh filename=package://mini_pupper_2_description/mini_pupper_2_meshes/mi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 scale=1 1 1
- link lb3: geometry collision mesh filename=package://mini_pupper_2_description/mini_pupper_2_meshes/mi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 scale=1 1 1; visual mesh filename=package://mini_pupper_2_description/mini_pupper_2_meshes/mi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 scale=1 1 1
- link lbfoot: geometry collision mesh filename=package://mini_pupper_2_description/mini_pupper_2_meshes/mi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 scale=1 1 1; visual mesh filename=package://mini_pupper_2_description/mini_pupper_2_meshes/mi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 scale=1 1 1
- link lf1: geometry collision mesh filename=package://mini_pupper_2_description/mini_pupper_2_meshes/mi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 scale=1 1 1; visual mesh filename=package://mini_pupper_2_description/mini_pupper_2_meshes/mi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 scale=1 1 1
- link lf2: geometry collision mesh filename=package://mini_pupper_2_description/mini_pupper_2_meshes/mi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 scale=1 1 1; visual mesh filename=package://mini_pupper_2_description/mini_pupper_2_meshes/mi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 scale=1 1 1
- link lf3: geometry collision mesh filename=package://mini_pupper_2_description/mini_pupper_2_meshes/mi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 scale=1 1 1; visual mesh filename=package://mini_pupper_2_description/mini_pupper_2_meshes/mi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 scale=1 1 1
- link lffoot: geometry collision mesh filename=package://mini_pupper_2_description/mini_pupper_2_meshes/mi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 scale=1 1 1; visual mesh filename=package://mini_pupper_2_description/mini_pupper_2_meshes/mi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 scale=1 1 1
- link lidar_link: geometry collision mesh filename=package://mini_pupper_2_description/mini_pupper_2_meshes/mi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; visual mesh filename=package://mini_pupper_2_description/mini_pupper_2_meshes/mi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
- link lpb1: geometry collision mesh filename=package://mini_pupper_2_description/mini_pupper_2_meshes/mi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 scale=1 1 1; visual mesh filename=package://mini_pupper_2_description/mini_pupper_2_meshes/mi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 scale=1 1 1
- link lpb2: geometry collision mesh filename=package://mini_pupper_2_description/mini_pupper_2_meshes/mi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 scale=1 1 1; visual mesh filename=package://mini_pupper_2_description/mini_pupper_2_meshes/mi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 scale=1 1 1
- link lpf1: geometry collision mesh filename=package://mini_pupper_2_description/mini_pupper_2_meshes/mi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 scale=1 1 1; visual mesh filename=package://mini_pupper_2_description/mini_pupper_2_meshes/mi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 scale=1 1 1
- link lpf2: geometry collision mesh filename=package://mini_pupper_2_description/mini_pupper_2_meshes/mi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 scale=1 1 1; visual mesh filename=package://mini_pupper_2_description/mini_pupper_2_meshes/mi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 scale=1 1 1
- link rb1: geometry collision mesh filename=package://mini_pupper_2_description/mini_pupper_2_meshes/mi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 scale=1 1 1; visual mesh filename=package://mini_pupper_2_description/mini_pupper_2_meshes/mi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 scale=1 1 1
- link rb2: geometry collision mesh filename=package://mini_pupper_2_description/mini_pupper_2_meshes/mi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 scale=1 1 1; visual mesh filename=package://mini_pupper_2_description/mini_pupper_2_meshes/mi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 scale=1 1 1
- link rb3: geometry collision mesh filename=package://mini_pupper_2_description/mini_pupper_2_meshes/mi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 scale=1 1 1; visual mesh filename=package://mini_pupper_2_description/mini_pupper_2_meshes/mi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 scale=1 1 1
- link rbfoot: geometry collision mesh filename=package://mini_pupper_2_description/mini_pupper_2_meshes/mi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 scale=1 1 1; visual mesh filename=package://mini_pupper_2_description/mini_pupper_2_meshes/mi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 scale=1 1 1
- link rf1: geometry collision mesh filename=package://mini_pupper_2_description/mini_pupper_2_meshes/mi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 scale=1 1 1; visual mesh filename=package://mini_pupper_2_description/mini_pupper_2_meshes/mi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 scale=1 1 1
- link rf2: geometry collision mesh filename=package://mini_pupper_2_description/mini_pupper_2_meshes/mi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 scale=1 1 1; visual mesh filename=package://mini_pupper_2_description/mini_pupper_2_meshes/mi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 scale=1 1 1
- link rf3: geometry collision mesh filename=package://mini_pupper_2_description/mini_pupper_2_meshes/mi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 scale=1 1 1; visual mesh filename=package://mini_pupper_2_description/mini_pupper_2_meshes/mi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 scale=1 1 1
- link rffoot: geometry collision mesh filename=package://mini_pupper_2_description/mini_pupper_2_meshes/mi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 scale=1 1 1; visual mesh filename=package://mini_pupper_2_description/mini_pupper_2_meshes/mi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 scale=1 1 1
- link rpb1: geometry collision mesh filename=package://mini_pupper_2_description/mini_pupper_2_meshes/mi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 scale=1 1 1; visual mesh filename=package://mini_pupper_2_description/mini_pupper_2_meshes/mi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 scale=1 1 1
- link rpb2: geometry collision mesh filename=package://mini_pupper_2_description/mini_pupper_2_meshes/mi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 scale=1 1 1; visual mesh filename=package://mini_pupper_2_description/mini_pupper_2_meshes/mi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 scale=1 1 1
- link rpf1: geometry collision mesh filename=package://mini_pupper_2_description/mini_pupper_2_meshes/mi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 scale=1 1 1; visual mesh filename=package://mini_pupper_2_description/mini_pupper_2_meshes/mi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 scale=1 1 1
- link rpf2: geometry collision mesh filename=package://mini_pupper_2_description/mini_pupper_2_meshes/mi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 scale=1 1 1; visual mesh filename=package://mini_pupper_2_description/mini_pupper_2_meshes/mi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 scale=1 1 1

Commit message: change paths in urdf files

File: mini_pupper_description/urdf/mini_pupper_2_description.urdf (robot description, URDF)
Before this commit: robot mini_pupper_2, 33 links, 32 joints
Links:
- link Board_PCB: geometry collision mesh filename=package://mini_pupper_description/mini_pupper_2_meshes/mini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 scale=1 1 1; visual mesh filename=package://mini_pupper_description/mini_pupper_2_meshes/mini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 scale=1 1 1
- link Board_connectors_1: geometry collision mesh filename=package://mini_pupper_description/mini_pupper_2_meshes/mini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 scale=1 1 1; visual mesh filename=package://mini_pupper_description/mini_pupper_2_meshes/mini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 scale=1 1 1
- link Board_connectors_2: geometry collision mesh filename=package://mini_pupper_description/mini_pupper_2_meshes/mini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 scale=1 1 1; visual mesh filename=package://mini_pupper_description/mini_pupper_2_meshes/mini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 scale=1 1 1
- link Body_front: geometry collision mesh filename=package://mini_pupper_description/mini_pupper_2_meshes/mini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 scale=1 1 1; visual mesh filename=package://mini_pupper_description/mini_pupper_2_meshes/mini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 scale=1 1 1
- link Shell_Side: geometry collision mesh filename=package://mini_pupper_description/mini_pupper_2_meshes/mini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 scale=1 1 1; visual mesh filename=package://mini_pupper_description/mini_pupper_2_meshes/mini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 scale=1 1 1
- link base_link: geometry collision mesh filename=package://mini_pupper_description/mini_pupper_2_meshes/mini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 scale=1 1 1; visual mesh filename=package://mini_pupper_description/mini_pupper_2_meshes/mini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 scale=1 1 1
- link lb1: geometry collision mesh filename=package://mini_pupper_description/mini_pupper_2_meshes/mini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 scale=1 1 1; visual mesh filename=package://mini_pupper_description/mini_pupper_2_meshes/mini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 scale=1 1 1
- link lb2: geometry collision mesh filename=package://mini_pupper_description/mini_pupper_2_meshes/mini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 scale=1 1 1; visual mesh filename=package://mini_pupper_description/mini_pupper_2_meshes/mini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 scale=1 1 1
- link lb3: geometry collision mesh filename=package://mini_pupper_description/mini_pupper_2_meshes/mini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 scale=1 1 1; visual mesh filename=package://mini_pupper_description/mini_pupper_2_meshes/mini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 scale=1 1 1
- link lbfoot: geometry collision mesh filename=package://mini_pupper_description/mini_pupper_2_meshes/mini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 scale=1 1 1; visual mesh filename=package://mini_pupper_description/mini_pupper_2_meshes/mini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 scale=1 1 1
- link lf1: geometry collision mesh filename=package://mini_pupper_description/mini_pupper_2_meshes/mini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 scale=1 1 1; visual mesh filename=package://mini_pupper_description/mini_pupper_2_meshes/mini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 scale=1 1 1
- link lf2: geometry collision mesh filename=package://mini_pupper_description/mini_pupper_2_meshes/mini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 scale=1 1 1; visual mesh filename=package://mini_pupper_description/mini_pupper_2_meshes/mini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 scale=1 1 1
- link lf3: geometry collision mesh filename=package://mini_pupper_description/mini_pupper_2_meshes/mini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 scale=1 1 1; visual mesh filename=package://mini_pupper_description/mini_pupper_2_meshes/mini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 scale=1 1 1
- link lffoot: geometry collision mesh filename=package://mini_pupper_description/mini_pupper_2_meshes/mini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 scale=1 1 1; visual mesh filename=package://mini_pupper_description/mini_pupper_2_meshes/mini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 scale=1 1 1
- link lidar_link: geometry collision mesh filename=package://mini_pupper_description/mini_pupper_2_meshes/mini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; visual mesh filename=package://mini_pupper_description/mini_pupper_2_meshes/mini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
- link lpb1: geometry collision mesh filename=package://mini_pupper_description/mini_pupper_2_meshes/mini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 scale=1 1 1; visual mesh filename=package://mini_pupper_description/mini_pupper_2_meshes/mini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 scale=1 1 1
- link lpb2: geometry collision mesh filename=package://mini_pupper_description/mini_pupper_2_meshes/mini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 scale=1 1 1; visual mesh filename=package://mini_pupper_description/mini_pupper_2_meshes/mini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 scale=1 1 1
- link lpf1: geometry collision mesh filename=package://mini_pupper_description/mini_pupper_2_meshes/mini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 scale=1 1 1; visual mesh filename=package://mini_pupper_description/mini_pupper_2_meshes/mini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 scale=1 1 1
- link lpf2: geometry collision mesh filename=package://mini_pupper_description/mini_pupper_2_meshes/mini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 scale=1 1 1; visual mesh filename=package://mini_pupper_description/mini_pupper_2_meshes/mini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 scale=1 1 1
- link rb1: geometry collision mesh filename=package://mini_pupper_description/mini_pupper_2_meshes/mini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 scale=1 1 1; visual mesh filename=package://mini_pupper_description/mini_pupper_2_meshes/mini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 scale=1 1 1
- link rb2: geometry collision mesh filename=package://mini_pupper_description/mini_pupper_2_meshes/mini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 scale=1 1 1; visual mesh filename=package://mini_pupper_description/mini_pupper_2_meshes/mini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 scale=1 1 1
- link rb3: geometry collision mesh filename=package://mini_pupper_description/mini_pupper_2_meshes/mini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 scale=1 1 1; visual mesh filename=package://mini_pupper_description/mini_pupper_2_meshes/mini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 scale=1 1 1
- link rbfoot: geometry collision mesh filename=package://mini_pupper_description/mini_pupper_2_meshes/mini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 scale=1 1 1; visual mesh filename=package://mini_pupper_description/mini_pupper_2_meshes/mini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 scale=1 1 1
- link rf1: geometry collision mesh filename=package://mini_pupper_description/mini_pupper_2_meshes/mini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 scale=1 1 1; visual mesh filename=package://mini_pupper_description/mini_pupper_2_meshes/mini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 scale=1 1 1
- link rf2: geometry collision mesh filename=package://mini_pupper_description/mini_pupper_2_meshes/mini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 scale=1 1 1; visual mesh filename=package://mini_pupper_description/mini_pupper_2_meshes/mini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 scale=1 1 1
- link rf3: geometry collision mesh filename=package://mini_pupper_description/mini_pupper_2_meshes/mini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 scale=1 1 1; visual mesh filename=package://mini_pupper_description/mini_pupper_2_meshes/mini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 scale=1 1 1
- link rffoot: geometry collision mesh filename=package://mini_pupper_description/mini_pupper_2_meshes/mini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 scale=1 1 1; visual mesh filename=package://mini_pupper_description/mini_pupper_2_meshes/mini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 scale=1 1 1
- link rpb1: geometry collision mesh filename=package://mini_pupper_description/mini_pupper_2_meshes/mini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 scale=1 1 1; visual mesh filename=package://mini_pupper_description/mini_pupper_2_meshes/mini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 scale=1 1 1
- link rpb2: geometry collision mesh filename=package://mini_pupper_description/mini_pupper_2_meshes/mini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 scale=1 1 1; visual mesh filename=package://mini_pupper_description/mini_pupper_2_meshes/mini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 scale=1 1 1
- link rpf1: geometry collision mesh filename=package://mini_pupper_description/mini_pupper_2_meshes/mini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 scale=1 1 1; visual mesh filename=package://mini_pupper_description/mini_pupper_2_meshes/mini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 scale=1 1 1
- link rpf2: geometry collision mesh filename=package://mini_pupper_description/mini_pupper_2_meshes/mini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 scale=1 1 1; visual mesh filename=package://mini_pupper_description/mini_pupper_2_meshes/mini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 scale=1 1 1

Commit message: adapt to urdf relative path

File: mini_pupper_description/urdf/mini_pupper_2_description.urdf (robot description, URDF)
Before this commit: robot mini_pupper_2, 33 links, 32 joints
Links:
- link Board_PCB: geometry collision mesh filename=package://mini_pupper_description/meshes/mini_pupper_2_Boar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 scale=1 1 1; visual mesh filename=package://mini_pupper_description/meshes/mini_pupper_2_Boar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 scale=1 1 1
- link Board_connectors_1: geometry collision mesh filename=package://mini_pupper_description/meshes/mini_pupper_2_Boar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 scale=1 1 1; visual mesh filename=package://mini_pupper_description/meshes/mini_pupper_2_Boar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 scale=1 1 1
- link Board_connectors_2: geometry collision mesh filename=package://mini_pupper_description/meshes/mini_pupper_2_Boar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 scale=1 1 1; visual mesh filename=package://mini_pupper_description/meshes/mini_pupper_2_Boar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 scale=1 1 1
- link Body_front: geometry collision mesh filename=package://mini_pupper_description/meshes/mini_pupper_2_Body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 scale=1 1 1; visual mesh filename=package://mini_pupper_description/meshes/mini_pupper_2_Body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 scale=1 1 1
- link Shell_Side: geometry collision mesh filename=package://mini_pupper_description/meshes/mini_pupper_2_Shel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 scale=1 1 1; visual mesh filename=package://mini_pupper_description/meshes/mini_pupper_2_Shel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 scale=1 1 1
- link base_link: geometry collision mesh filename=package://mini_pupper_description/meshes/mini_pupper_2_base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 scale=1 1 1; visual mesh filename=package://mini_pupper_description/meshes/mini_pupper_2_base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 scale=1 1 1
- link lb1: geometry collision mesh filename=package://mini_pupper_description/meshes/mini_pupper_2_lb1.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 scale=1 1 1; visual mesh filename=package://mini_pupper_description/meshes/mini_pupper_2_lb1.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 scale=1 1 1
- link lb2: geometry collision mesh filename=package://mini_pupper_description/meshes/mini_pupper_2_lb2.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 scale=1 1 1; visual mesh filename=package://mini_pupper_description/meshes/mini_pupper_2_lb2.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 scale=1 1 1
- link lb3: geometry collision mesh filename=package://mini_pupper_description/meshes/mini_pupper_2_lb3.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 scale=1 1 1; visual mesh filename=package://mini_pupper_description/meshes/mini_pupper_2_lb3.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 scale=1 1 1
- link lbfoot: geometry collision mesh filename=package://mini_pupper_description/meshes/mini_pupper_2_lbfo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 scale=1 1 1; visual mesh filename=package://mini_pupper_description/meshes/mini_pupper_2_lbfo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 scale=1 1 1
- link lf1: geometry collision mesh filename=package://mini_pupper_description/meshes/mini_pupper_2_lf1.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 scale=1 1 1; visual mesh filename=package://mini_pupper_description/meshes/mini_pupper_2_lf1.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 scale=1 1 1
- link lf2: geometry collision mesh filename=package://mini_pupper_description/meshes/mini_pupper_2_lf2.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 scale=1 1 1; visual mesh filename=package://mini_pupper_description/meshes/mini_pupper_2_lf2.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 scale=1 1 1
- link lf3: geometry collision mesh filename=package://mini_pupper_description/meshes/mini_pupper_2_lf3.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 scale=1 1 1; visual mesh filename=package://mini_pupper_description/meshes/mini_pupper_2_lf3.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 scale=1 1 1
- link lffoot: geometry collision mesh filename=package://mini_pupper_description/meshes/mini_pupper_2_lffo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 scale=1 1 1; visual mesh filename=package://mini_pupper_description/meshes/mini_pupper_2_lffo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 scale=1 1 1
- link lidar_link: geometry collision mesh filename=package://mini_pupper_description/meshes/mini_pupper_2_lida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; visual mesh filename=package://mini_pupper_description/meshes/mini_pupper_2_lida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
- link lpb1: geometry collision mesh filename=package://mini_pupper_description/meshes/mini_pupper_2_lpb1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 scale=1 1 1; visual mesh filename=package://mini_pupper_description/meshes/mini_pupper_2_lpb1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 scale=1 1 1
- link lpb2: geometry collision mesh filename=package://mini_pupper_description/meshes/mini_pupper_2_lpb2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 scale=1 1 1; visual mesh filename=package://mini_pupper_description/meshes/mini_pupper_2_lpb2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 scale=1 1 1
- link lpf1: geometry collision mesh filename=package://mini_pupper_description/meshes/mini_pupper_2_lpf1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 scale=1 1 1; visual mesh filename=package://mini_pupper_description/meshes/mini_pupper_2_lpf1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 scale=1 1 1
- link lpf2: geometry collision mesh filename=package://mini_pupper_description/meshes/mini_pupper_2_lpf2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 scale=1 1 1; visual mesh filename=package://mini_pupper_description/meshes/mini_pupper_2_lpf2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 scale=1 1 1
- link rb1: geometry collision mesh filename=package://mini_pupper_description/meshes/mini_pupper_2_rb1.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 scale=1 1 1; visual mesh filename=package://mini_pupper_description/meshes/mini_pupper_2_rb1.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 scale=1 1 1
- link rb2: geometry collision mesh filename=package://mini_pupper_description/meshes/mini_pupper_2_rb2.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 scale=1 1 1; visual mesh filename=package://mini_pupper_description/meshes/mini_pupper_2_rb2.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 scale=1 1 1
- link rb3: geometry collision mesh filename=package://mini_pupper_description/meshes/mini_pupper_2_rb3.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 scale=1 1 1; visual mesh filename=package://mini_pupper_description/meshes/mini_pupper_2_rb3.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 scale=1 1 1
- link rbfoot: geometry collision mesh filename=package://mini_pupper_description/meshes/mini_pupper_2_rbfo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 scale=1 1 1; visual mesh filename=package://mini_pupper_description/meshes/mini_pupper_2_rbfo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 scale=1 1 1
- link rf1: geometry collision mesh filename=package://mini_pupper_description/meshes/mini_pupper_2_rf1.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 scale=1 1 1; visual mesh filename=package://mini_pupper_description/meshes/mini_pupper_2_rf1.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 scale=1 1 1
- link rf2: geometry collision mesh filename=package://mini_pupper_description/meshes/mini_pupper_2_rf2.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 scale=1 1 1; visual mesh filename=package://mini_pupper_description/meshes/mini_pupper_2_rf2.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 scale=1 1 1
- link rf3: geometry collision mesh filename=package://mini_pupper_description/meshes/mini_pupper_2_rf3.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 scale=1 1 1; visual mesh filename=package://mini_pupper_description/meshes/mini_pupper_2_rf3.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 scale=1 1 1
- link rffoot: geometry collision mesh filename=package://mini_pupper_description/meshes/mini_pupper_2_rffo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 scale=1 1 1; visual mesh filename=package://mini_pupper_description/meshes/mini_pupper_2_rffo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 scale=1 1 1
- link rpb1: geometry collision mesh filename=package://mini_pupper_description/meshes/mini_pupper_2_rpb1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 scale=1 1 1; visual mesh filename=package://mini_pupper_description/meshes/mini_pupper_2_rpb1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 scale=1 1 1
- link rpb2: geometry collision mesh filename=package://mini_pupper_description/meshes/mini_pupper_2_rpb2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 scale=1 1 1; visual mesh filename=package://mini_pupper_description/meshes/mini_pupper_2_rpb2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 scale=1 1 1
- link rpf1: geometry collision mesh filename=package://mini_pupper_description/meshes/mini_pupper_2_rpf1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 scale=1 1 1; visual mesh filename=package://mini_pupper_description/meshes/mini_pupper_2_rpf1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 scale=1 1 1
- link rpf2: geometry collision mesh filename=package://mini_pupper_description/meshes/mini_pupper_2_rpf2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 scale=1 1 1; visual mesh filename=package://mini_pupper_description/meshes/mini_pupper_2_rpf2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 scale=1 1 1
