Commit message: add comment content

File: mini_pupper_description/urdf/mini_pupper_2_description.urdf (robot description, URDF)
Before this commit: robot mini_pupper_2, 33 links, 32 joints
Links:
- link Board_PCB: geometry collision mesh filename=package://mini_pupper_description/meshes/mini_pupper_2/mini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 scale=1 1 1; visual mesh filename=package://mini_pupper_description/meshes/mini_pupper_2/mini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 scale=1 1 1
- link Board_connectors_1: geometry collision mesh filename=package://mini_pupper_description/meshes/mini_pupper_2/mini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 scale=1 1 1; visual mesh filename=package://mini_pupper_description/meshes/mini_pupper_2/mini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 scale=1 1 1
- link Board_connectors_2: geometry collision mesh filename=package://mini_pupper_description/meshes/mini_pupper_2/mini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 scale=1 1 1; visual mesh filename=package://mini_pupper_description/meshes/mini_pupper_2/mini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 scale=1 1 1
- link Body_front: geometry collision mesh filename=package://mini_pupper_description/meshes/mini_pupper_2/mini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 scale=1 1 1; visual mesh filename=package://mini_pupper_description/meshes/mini_pupper_2/mini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 scale=1 1 1
- link Shell_Side: geometry collision mesh filename=package://mini_pupper_description/meshes/mini_pupper_2/mini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 scale=1 1 1; visual mesh filename=package://mini_pupper_description/meshes/mini_pupper_2/mini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 scale=1 1 1
- link base_link: geometry collision mesh filename=package://mini_pupper_description/meshes/mini_pupper_2/mini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 scale=1 1 1; visual mesh filename=package://mini_pupper_description/meshes/mini_pupper_2/mini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 scale=1 1 1
- link lb1: geometry collision mesh filename=package://mini_pupper_description/meshes/mini_pupper_2/mini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 scale=1 1 1; visual mesh filename=package://mini_pupper_description/meshes/mini_pupper_2/mini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 scale=1 1 1
- link lb2: geometry collision mesh filename=package://mini_pupper_description/meshes/mini_pupper_2/mini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 scale=1 1 1; visual mesh filename=package://mini_pupper_description/meshes/mini_pupper_2/mini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 scale=1 1 1
- link lb3: geometry collision mesh filename=package://mini_pupper_description/meshes/mini_pupper_2/mini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 scale=1 1 1; visual mesh filename=package://mini_pupper_description/meshes/mini_pupper_2/mini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 scale=1 1 1
- link lbfoot: geometry collision mesh filename=package://mini_pupper_description/meshes/mini_pupper_2/mini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 scale=1 1 1; visual mesh filename=package://mini_pupper_description/meshes/mini_pupper_2/mini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 scale=1 1 1
- link lf1: geometry collision mesh filename=package://mini_pupper_description/meshes/mini_pupper_2/mini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 scale=1 1 1; visual mesh filename=package://mini_pupper_description/meshes/mini_pupper_2/mini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 scale=1 1 1
- link lf2: geometry collision mesh filename=package://mini_pupper_description/meshes/mini_pupper_2/mini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 scale=1 1 1; visual mesh filename=package://mini_pupper_description/meshes/mini_pupper_2/mini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 scale=1 1 1
- link lf3: geometry collision mesh filename=package://mini_pupper_description/meshes/mini_pupper_2/mini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 scale=1 1 1; visual mesh filename=package://mini_pupper_description/meshes/mini_pupper_2/mini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 scale=1 1 1
- link lffoot: geometry collision mesh filename=package://mini_pupper_description/meshes/mini_pupper_2/mini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 scale=1 1 1; visual mesh filename=package://mini_pupper_description/meshes/mini_pupper_2/mini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 scale=1 1 1
- link lidar_link: geometry collision mesh filename=package://mini_pupper_description/meshes/mini_pupper_2/mini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; visual mesh filename=package://mini_pupper_description/meshes/mini_pupper_2/mini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
- link lpb1: geometry collision mesh filename=package://mini_pupper_description/meshes/mini_pupper_2/mini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 scale=1 1 1; visual mesh filename=package://mini_pupper_description/meshes/mini_pupper_2/mini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 scale=1 1 1
- link lpb2: geometry collision mesh filename=package://mini_pupper_description/meshes/mini_pupper_2/mini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 scale=1 1 1; visual mesh filename=package://mini_pupper_description/meshes/mini_pupper_2/mini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 scale=1 1 1
- link lpf1: geometry collision mesh filename=package://mini_pupper_description/meshes/mini_pupper_2/mini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 scale=1 1 1; visual mesh filename=package://mini_pupper_description/meshes/mini_pupper_2/mini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 scale=1 1 1
- link lpf2: geometry collision mesh filename=package://mini_pupper_description/meshes/mini_pupper_2/mini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 scale=1 1 1; visual mesh filename=package://mini_pupper_description/meshes/mini_pupper_2/mini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 scale=1 1 1
- link rb1: geometry collision mesh filename=package://mini_pupper_description/meshes/mini_pupper_2/mini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 scale=1 1 1; visual mesh filename=package://mini_pupper_description/meshes/mini_pupper_2/mini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 scale=1 1 1
- link rb2: geometry collision mesh filename=package://mini_pupper_description/meshes/mini_pupper_2/mini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 scale=1 1 1; visual mesh filename=package://mini_pupper_description/meshes/mini_pupper_2/mini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 scale=1 1 1
- link rb3: geometry collision mesh filename=package://mini_pupper_description/meshes/mini_pupper_2/mini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 scale=1 1 1; visual mesh filename=package://mini_pupper_description/meshes/mini_pupper_2/mini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 scale=1 1 1
- link rbfoot: geometry collision mesh filename=package://mini_pupper_description/meshes/mini_pupper_2/mini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 scale=1 1 1; visual mesh filename=package://mini_pupper_description/meshes/mini_pupper_2/mini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 scale=1 1 1
- link rf1: geometry collision mesh filename=package://mini_pupper_description/meshes/mini_pupper_2/mini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 scale=1 1 1; visual mesh filename=package://mini_pupper_description/meshes/mini_pupper_2/mini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 scale=1 1 1
- link rf2: geometry collision mesh filename=package://mini_pupper_description/meshes/mini_pupper_2/mini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 scale=1 1 1; visual mesh filename=package://mini_pupper_description/meshes/mini_pupper_2/mini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 scale=1 1 1
- link rf3: geometry collision mesh filename=package://mini_pupper_description/meshes/mini_pupper_2/mini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 scale=1 1 1; visual mesh filename=package://mini_pupper_description/meshes/mini_pupper_2/mini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 scale=1 1 1
- link rffoot: geometry collision mesh filename=package://mini_pupper_description/meshes/mini_pupper_2/mini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 scale=1 1 1; visual mesh filename=package://mini_pupper_description/meshes/mini_pupper_2/mini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 scale=1 1 1
- link rpb1: geometry collision mesh filename=package://mini_pupper_description/meshes/mini_pupper_2/mini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 scale=1 1 1; visual mesh filename=package://mini_pupper_description/meshes/mini_pupper_2/mini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 scale=1 1 1
- link rpb2: geometry collision mesh filename=package://mini_pupper_description/meshes/mini_pupper_2/mini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 scale=1 1 1; visual mesh filename=package://mini_pupper_description/meshes/mini_pupper_2/mini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 scale=1 1 1
- link rpf1: geometry collision mesh filename=package://mini_pupper_description/meshes/mini_pupper_2/mini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 scale=1 1 1; visual mesh filename=package://mini_pupper_description/meshes/mini_pupper_2/mini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 scale=1 1 1
- link rpf2: geometry collision mesh filename=package://mini_pupper_description/meshes/mini_pupper_2/mini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 scale=1 1 1; visual mesh filename=package://mini_pupper_description/meshes/mini_pupper_2/mini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 scale=1 1 1

Commit message: fix minor syntax error and rename files in meshes

File: mini_pupper_description/urdf/mini_pupper_2_description.urdf (robot description, URDF)
Before this commit: robot mini_pupper_2, 33 links, 32 joints
Links:
- link Board_PCB: geometry collision mesh filename=package://mini_pupper_description/meshes/mini_pupper_2/Boar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 scale=1 1 1; visual mesh filename=package://mini_pupper_description/meshes/mini_pupper_2/Boar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 scale=1 1 1
- link Board_connectors_1: geometry collision mesh filename=package://mini_pupper_description/meshes/mini_pupper_2/Boar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 scale=1 1 1; visual mesh filename=package://mini_pupper_description/meshes/mini_pupper_2/Boar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 scale=1 1 1
- link Board_connectors_2: geometry collision mesh filename=package://mini_pupper_description/meshes/mini_pupper_2/Boar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 scale=1 1 1; visual mesh filename=package://mini_pupper_description/meshes/mini_pupper_2/Boar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 scale=1 1 1
- link Body_front: geometry collision mesh filename=package://mini_pupper_description/meshes/mini_pupper_2/Body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 scale=1 1 1; visual mesh filename=package://mini_pupper_description/meshes/mini_pupper_2/Body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 scale=1 1 1
- link Shell_Side: geometry collision mesh filename=package://mini_pupper_description/meshes/mini_pupper_2/Shel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 scale=1 1 1; visual mesh filename=package://mini_pupper_description/meshes/mini_pupper_2/Shel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 scale=1 1 1
- link base_link: geometry collision mesh filename=package://mini_pupper_description/meshes/mini_pupper_2/base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 scale=1 1 1; visual mesh filename=package://mini_pupper_description/meshes/mini_pupper_2/base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 scale=1 1 1
- link lb1: geometry collision mesh filename=package://mini_pupper_description/meshes/mini_pupper_2/lb1.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 scale=1 1 1; visual mesh filename=package://mini_pupper_description/meshes/mini_pupper_2/lb1.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 scale=1 1 1
- link lb2: geometry collision mesh filename=package://mini_pupper_description/meshes/mini_pupper_2/lb2.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 scale=1 1 1; visual mesh filename=package://mini_pupper_description/meshes/mini_pupper_2/lb2.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 scale=1 1 1
- link lb3: geometry collision mesh filename=package://mini_pupper_description/meshes/mini_pupper_2/lb3.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 scale=1 1 1; visual mesh filename=package://mini_pupper_description/meshes/mini_pupper_2/lb3.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 scale=1 1 1
- link lbfoot: geometry collision mesh filename=package://mini_pupper_description/meshes/mini_pupper_2/lbfo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 scale=1 1 1; visual mesh filename=package://mini_pupper_description/meshes/mini_pupper_2/lbfo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 scale=1 1 1
- link lf1: geometry collision mesh filename=package://mini_pupper_description/meshes/mini_pupper_2/lf1.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 scale=1 1 1; visual mesh filename=package://mini_pupper_description/meshes/mini_pupper_2/lf1.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 scale=1 1 1
- link lf2: geometry collision mesh filename=package://mini_pupper_description/meshes/mini_pupper_2/lf2.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 scale=1 1 1; visual mesh filename=package://mini_pupper_description/meshes/mini_pupper_2/lf2.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 scale=1 1 1
- link lf3: geometry collision mesh filename=package://mini_pupper_description/meshes/mini_pupper_2/lf3.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 scale=1 1 1; visual mesh filename=package://mini_pupper_description/meshes/mini_pupper_2/lf3.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 scale=1 1 1
- link lffoot: geometry collision mesh filename=package://mini_pupper_description/meshes/mini_pupper_2/lffo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 scale=1 1 1; visual mesh filename=package://mini_pupper_description/meshes/mini_pupper_2/lffo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 scale=1 1 1
- link lidar_link: geometry collision mesh filename=package://mini_pupper_description/meshes/mini_pupper_2/lida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; visual mesh filename=package://mini_pupper_description/meshes/mini_pupper_2/lida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
- link lpb1: geometry collision mesh filename=package://mini_pupper_description/meshes/mini_pupper_2/lpb1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 scale=1 1 1; visual mesh filename=package://mini_pupper_description/meshes/mini_pupper_2/lpb1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 scale=1 1 1
- link lpb2: geometry collision mesh filename=package://mini_pupper_description/meshes/mini_pupper_2/lpb2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 scale=1 1 1; visual mesh filename=package://mini_pupper_description/meshes/mini_pupper_2/lpb2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 scale=1 1 1
- link lpf1: geometry collision mesh filename=package://mini_pupper_description/meshes/mini_pupper_2/lpf1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 scale=1 1 1; visual mesh filename=package://mini_pupper_description/meshes/mini_pupper_2/lpf1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 scale=1 1 1
- link lpf2: geometry collision mesh filename=package://mini_pupper_description/meshes/mini_pupper_2/lpf2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 scale=1 1 1; visual mesh filename=package://mini_pupper_description/meshes/mini_pupper_2/lpf2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 scale=1 1 1
- link rb1: geometry collision mesh filename=package://mini_pupper_description/meshes/mini_pupper_2/rb1.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 scale=1 1 1; visual mesh filename=package://mini_pupper_description/meshes/mini_pupper_2/rb1.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 scale=1 1 1
- link rb2: geometry collision mesh filename=package://mini_pupper_description/meshes/mini_pupper_2/rb2.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 scale=1 1 1; visual mesh filename=package://mini_pupper_description/meshes/mini_pupper_2/rb2.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 scale=1 1 1
- link rb3: geometry collision mesh filename=package://mini_pupper_description/meshes/mini_pupper_2/rb3.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 scale=1 1 1; visual mesh filename=package://mini_pupper_description/meshes/mini_pupper_2/rb3.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 scale=1 1 1
- link rbfoot: geometry collision mesh filename=package://mini_pupper_description/meshes/mini_pupper_2/rbfo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 scale=1 1 1; visual mesh filename=package://mini_pupper_description/meshes/mini_pupper_2/rbfo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 scale=1 1 1
- link rf1: geometry collision mesh filename=package://mini_pupper_description/meshes/mini_pupper_2/rf1.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 scale=1 1 1; visual mesh filename=package://mini_pupper_description/meshes/mini_pupper_2/rf1.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 scale=1 1 1
- link rf2: geometry collision mesh filename=package://mini_pupper_description/meshes/mini_pupper_2/rf2.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 scale=1 1 1; visual mesh filename=package://mini_pupper_description/meshes/mini_pupper_2/rf2.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 scale=1 1 1
- link rf3: geometry collision mesh filename=package://mini_pupper_description/meshes/mini_pupper_2/rf3.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 scale=1 1 1; visual mesh filename=package://mini_pupper_description/meshes/mini_pupper_2/rf3.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 scale=1 1 1
- link rffoot: geometry collision mesh filename=package://mini_pupper_description/meshes/mini_pupper_2/rffo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 scale=1 1 1; visual mesh filename=package://mini_pupper_description/meshes/mini_pupper_2/rffo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 scale=1 1 1
- link rpb1: geometry collision mesh filename=package://mini_pupper_description/meshes/mini_pupper_2/rpb1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 scale=1 1 1; visual mesh filename=package://mini_pupper_description/meshes/mini_pupper_2/rpb1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 scale=1 1 1
- link rpb2: geometry collision mesh filename=package://mini_pupper_description/meshes/mini_pupper_2/rpb2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 scale=1 1 1; visual mesh filename=package://mini_pupper_description/meshes/mini_pupper_2/rpb2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 scale=1 1 1
- link rpf1: geometry collision mesh filename=package://mini_pupper_description/meshes/mini_pupper_2/rpf1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 scale=1 1 1; visual mesh filename=package://mini_pupper_description/meshes/mini_pupper_2/rpf1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 scale=1 1 1
- link rpf2: geometry collision mesh filename=package://mini_pupper_description/meshes/mini_pupper_2/rpf2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 scale=1 1 1; visual mesh filename=package://mini_pupper_description/meshes/mini_pupper_2/rpf2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 scale=1 1 1

File: mini_pupper_description/urdf/mini_pupper_description.urdf (robot description, URDF)
Before this commit: robot mini-pupper, 29 links, 28 joints
Links:
- link base_link: geometry collision mesh filename=package://mini_pupper_description/meshes/mini_pupper/base_l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; visual mesh filename=package://mini_pupper_description/meshes/mini_pupper/base_l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
- link lb1: geometry collision mesh filename=package://mini_pupper_description/meshes/mini_pupper/lb1.STL; visual mesh filename=package://mini_pupper_description/meshes/mini_pupper/lb1.STL
- link lb2: geometry collision mesh filename=package://mini_pupper_description/meshes/mini_pupper/lb2.STL; visual mesh filename=package://mini_pupper_description/meshes/mini_pupper/lb2.STL
- link lb3: geometry collision mesh filename=package://mini_pupper_description/meshes/mini_pupper/lb3.STL; visual mesh filename=package://mini_pupper_description/meshes/mini_pupper/lb3.STL
- link lbfoot: geometry collision mesh filename=package://mini_pupper_description/meshes/mini_pupper/lbfoot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; visual mesh filename=package://mini_pupper_description/meshes/mini_pupper/lbfoot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
- link lf1: geometry collision mesh filename=package://mini_pupper_description/meshes/mini_pupper/lf1.STL; visual mesh filename=package://mini_pupper_description/meshes/mini_pupper/lf1.STL
- link lf2: geometry collision mesh filename=package://mini_pupper_description/meshes/mini_pupper/lf2.STL; visual mesh filename=package://mini_pupper_description/meshes/mini_pupper/lf2.STL
- link lf3: geometry collision mesh filename=package://mini_pupper_description/meshes/mini_pupper/lf3.STL; visual mesh filename=package://mini_pupper_description/meshes/mini_pupper/lf3.STL
- link lffoot: geometry collision mesh filename=package://mini_pupper_description/meshes/mini_pupper/lffoot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; visual mesh filename=package://mini_pupper_description/meshes/mini_pupper/lffoot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
- link lidar_link: geometry collision mesh filename=package://mini_pupper_description/meshes/mini_pupper/lidar.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; visual mesh filename=package://mini_pupper_description/meshes/mini_pupper/lidar.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
- link lpb1: geometry collision mesh filename=package://mini_pupper_description/meshes/mini_pupper/lpb1.S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; visual mesh filename=package://mini_pupper_description/meshes/mini_pupper/lpb1.S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
- link lpb2: geometry collision mesh filename=package://mini_pupper_description/meshes/mini_pupper/lpb2.S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; visual mesh filename=package://mini_pupper_description/meshes/mini_pupper/lpb2.S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
- link lpf1: geometry collision mesh filename=package://mini_pupper_description/meshes/mini_pupper/lpf1.S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; visual mesh filename=package://mini_pupper_description/meshes/mini_pupper/lpf1.S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
- link lpf2: geometry collision mesh filename=package://mini_pupper_description/meshes/mini_pupper/lpf2.S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; visual mesh filename=package://mini_pupper_description/meshes/mini_pupper/lpf2.S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
- link rb1: geometry collision mesh filename=package://mini_pupper_description/meshes/mini_pupper/rb1.STL; visual mesh filename=package://mini_pupper_description/meshes/mini_pupper/rb1.STL
- link rb2: geometry collision mesh filename=package://mini_pupper_description/meshes/mini_pupper/rb2.STL; visual mesh filename=package://mini_pupper_description/meshes/mini_pupper/rb2.STL
- link rb3: geometry collision mesh filename=package://mini_pupper_description/meshes/mini_pupper/rb3.STL; visual mesh filename=package://mini_pupper_description/meshes/mini_pupper/rb3.STL
- link rbfoot: geometry collision mesh filename=package://mini_pupper_description/meshes/mini_pupper/rbfoot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; visual mesh filename=package://mini_pupper_description/meshes/mini_pupper/rbfoot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
- link rf1: geometry collision mesh filename=package://mini_pupper_description/meshes/mini_pupper/rf1.STL; visual mesh filename=package://mini_pupper_description/meshes/mini_pupper/rf1.STL
- link rf2: geometry collision mesh filename=package://mini_pupper_description/meshes/mini_pupper/rf2.STL; visual mesh filename=package://mini_pupper_description/meshes/mini_pupper/rf2.STL
- link rf3: geometry collision mesh filename=package://mini_pupper_description/meshes/mini_pupper/rf3.STL; visual mesh filename=package://mini_pupper_description/meshes/mini_pupper/rf3.STL
- link rffoot: geometry collision mesh filename=package://mini_pupper_description/meshes/mini_pupper/rffoot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; visual mesh filename=package://mini_pupper_description/meshes/mini_pupper/rffoot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
- link rpb1: geometry collision mesh filename=package://mini_pupper_description/meshes/mini_pupper/rpb1.S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; visual mesh filename=package://mini_pupper_description/meshes/mini_pupper/rpb1.S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
- link rpb2: geometry collision mesh filename=package://mini_pupper_description/meshes/mini_pupper/rpb2.S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; visual mesh filename=package://mini_pupper_description/meshes/mini_pupper/rpb2.S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
- link rpf1: geometry collision mesh filename=package://mini_pupper_description/meshes/mini_pupper/rpf1.S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; visual mesh filename=package://mini_pupper_description/meshes/mini_pupper/rpf1.S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
- link rpf2: geometry collision mesh filename=package://mini_pupper_description/meshes/mini_pupper/rpf2.S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; visual mesh filename=package://mini_pupper_description/meshes/mini_pupper/rpf2.S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
- link yellow_plate: geometry collision mesh filename=package://mini_pupper_description/meshes/mini_pupper/yellow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; visual mesh filename=package://mini_pupper_description/meshes/mini_pupper/yellow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
