Commit message: rename to mini-pupper-2-description

File: mini_pupper_2_description/urdf/mini_pupper_2_description.urdf (robot description, URDF)
Before this commit: robot mini_pupper, 32 links, 31 joints
Links:
- link Board_PCB: geometry collision mesh filename=package://mini_pupper_2_description/meshes/Board_PCB.stl scale=1 1 1; visual mesh filename=package://mini_pupper_2_description/meshes/Board_PCB.stl scale=1 1 1
- link Board_connectors_1: geometry collision mesh filename=package://mini_pupper_2_description/meshes/Board_connectors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 scale=1 1 1; visual mesh filename=package://mini_pupper_2_description/meshes/Board_connectors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 scale=1 1 1
- link Board_connectors_2: geometry collision mesh filename=package://mini_pupper_2_description/meshes/Board_connectors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 scale=1 1 1; visual mesh filename=package://mini_pupper_2_description/meshes/Board_connectors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 scale=1 1 1
- link Body_front: geometry collision mesh filename=package://mini_pupper_2_description/meshes/Body_front.stl scale=1 1 1; visual mesh filename=package://mini_pupper_2_description/meshes/Body_front.stl scale=1 1 1
- link Shell_Hip_Left_1: geometry collision mesh filename=package://mini_pupper_2_description/meshes/Shell_Hip_Left_1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 scale=1 1 1; visual mesh filename=package://mini_pupper_2_description/meshes/Shell_Hip_Left_1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 scale=1 1 1
- link Shell_Hip_Left_2: geometry collision mesh filename=package://mini_pupper_2_description/meshes/Shell_Hip_Left_2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 scale=1 1 1; visual mesh filename=package://mini_pupper_2_description/meshes/Shell_Hip_Left_2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 scale=1 1 1
- link Shell_Hip_Right_1: geometry collision mesh filename=package://mini_pupper_2_description/meshes/Shell_Hip_Right_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 scale=1 1 1; visual mesh filename=package://mini_pupper_2_description/meshes/Shell_Hip_Right_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 scale=1 1 1
- link Shell_Hip_Right_2: geometry collision mesh filename=package://mini_pupper_2_description/meshes/Shell_Hip_Right_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 scale=1 1 1; visual mesh filename=package://mini_pupper_2_description/meshes/Shell_Hip_Right_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 scale=1 1 1
- link Shell_Leg_Upper_LeftSide_1: geometry collision mesh filename=package://mini_pupper_2_description/meshes/Shell_Leg_Upper_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 scale=1 1 1; visual mesh filename=package://mini_pupper_2_description/meshes/Shell_Leg_Upper_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 scale=1 1 1
- link Shell_Leg_Upper_LeftSide_2: geometry collision mesh filename=package://mini_pupper_2_description/meshes/Shell_Leg_Upper_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 scale=1 1 1; visual mesh filename=package://mini_pupper_2_description/meshes/Shell_Leg_Upper_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 scale=1 1 1
- link Shell_Leg_Upper_RightSide_1: geometry collision mesh filename=package://mini_pupper_2_description/meshes/Shell_Leg_Upper_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 scale=1 1 1; visual mesh filename=package://mini_pupper_2_description/meshes/Shell_Leg_Upper_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 scale=1 1 1
- link Shell_Leg_Upper_RightSide_2: geometry collision mesh filename=package://mini_pupper_2_description/meshes/Shell_Leg_Upper_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 scale=1 1 1; visual mesh filename=package://mini_pupper_2_description/meshes/Shell_Leg_Upper_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 scale=1 1 1
- link Shell_Side: geometry collision mesh filename=package://mini_pupper_2_description/meshes/Shell_Side.stl scale=1 1 1; visual mesh filename=package://mini_pupper_2_description/meshes/Shell_Side.stl scale=1 1 1
- link base_link: geometry collision mesh filename=package://mini_pupper_2_description/meshes/base_link.stl scale=1 1 1; visual mesh filename=package://mini_pupper_2_description/meshes/base_link.stl scale=1 1 1
- link lb1: geometry collision mesh filename=package://mini_pupper_2_description/meshes/lb1.stl scale=1 1 1; visual mesh filename=package://mini_pupper_2_description/meshes/lb1.stl scale=1 1 1
- link lb2: geometry collision mesh filename=package://mini_pupper_2_description/meshes/lb2.stl scale=1 1 1; visual mesh filename=package://mini_pupper_2_description/meshes/lb2.stl scale=1 1 1
- link lb3: geometry collision mesh filename=package://mini_pupper_2_description/meshes/lb3.stl scale=1 1 1; visual mesh filename=package://mini_pupper_2_description/meshes/lb3.stl scale=1 1 1
- link lbfoot: geometry collision mesh filename=package://mini_pupper_2_description/meshes/lbfoot.stl scale=1 1 1; visual mesh filename=package://mini_pupper_2_description/meshes/lbfoot.stl scale=1 1 1
- link lf1: geometry collision mesh filename=package://mini_pupper_2_description/meshes/lf1.stl scale=1 1 1; visual mesh filename=package://mini_pupper_2_description/meshes/lf1.stl scale=1 1 1
- link lf2: geometry collision mesh filename=package://mini_pupper_2_description/meshes/lf2.stl scale=1 1 1; visual mesh filename=package://mini_pupper_2_description/meshes/lf2.stl scale=1 1 1
- link lf3: geometry collision mesh filename=package://mini_pupper_2_description/meshes/lf3.stl scale=1 1 1; visual mesh filename=package://mini_pupper_2_description/meshes/lf3.stl scale=1 1 1
- link lffoot: geometry collision mesh filename=package://mini_pupper_2_description/meshes/lffoot.stl scale=1 1 1; visual mesh filename=package://mini_pupper_2_description/meshes/lffoot.stl scale=1 1 1
- link rb1: geometry collision mesh filename=package://mini_pupper_2_description/meshes/rb1.stl scale=1 1 1; visual mesh filename=package://mini_pupper_2_description/meshes/rb1.stl scale=1 1 1
- link rb2: geometry collision mesh filename=package://mini_pupper_2_description/meshes/rb2.stl scale=1 1 1; visual mesh filename=package://mini_pupper_2_description/meshes/rb2.stl scale=1 1 1
- link rb3: geometry collision mesh filename=package://mini_pupper_2_description/meshes/rb3.stl scale=1 1 1; visual mesh filename=package://mini_pupper_2_description/meshes/rb3.stl scale=1 1 1
- link rbfoot: geometry collision mesh filename=package://mini_pupper_2_description/meshes/rbfoot.stl scale=1 1 1; visual mesh filename=package://mini_pupper_2_description/meshes/rbfoot.stl scale=1 1 1
- link rf1: geometry collision mesh filename=package://mini_pupper_2_description/meshes/rf1.stl scale=1 1 1; visual mesh filename=package://mini_pupper_2_description/meshes/rf1.stl scale=1 1 1
- link rf2: geometry collision mesh filename=package://mini_pupper_2_description/meshes/rf2.stl scale=1 1 1; visual mesh filename=package://mini_pupper_2_description/meshes/rf2.stl scale=1 1 1
- link rf3: geometry collision mesh filename=package://mini_pupper_2_description/meshes/rf3.stl scale=1 1 1; visual mesh filename=package://mini_pupper_2_description/meshes/rf3.stl scale=1 1 1
- link rffoot: geometry collision mesh filename=package://mini_pupper_2_description/meshes/rffoot.stl scale=1 1 1; visual mesh filename=package://mini_pupper_2_description/meshes/rffoot.stl scale=1 1 1
