Commit message: pick up changes from Peter

File: mini_pupper_2_description/urdf/mini_pupper_description.urdf.xacro (robot description, xacro)
@@ -2,5 +2,5 @@
 <robot name="mini_pupper" xmlns:xacro="http://www.ros.org/wiki/xacro">
   <xacro:include filename="$(find mini_pupper_2_description)/urdf/materials.xacro" />
-  <!-- <xacro:include filename="$(find mini_pupper_2_description)/urdf/mini_pupper_2_description.trans" /> -->
+  <xacro:include filename="$(find mini_pupper_2_description)/urdf/mini_pupper_description.trans" />
   <link name="base_link">
     <visual>
@@ -20,7 +20,7 @@
   <link name="base_inertia">
     <inertial>
-      <origin xyz="-0.008866664732250966 0.0006462612742260995 -0.007154314406453802" rpy="0 0 0"/>
+      <origin xyz="-0.008867 0.000646 -0.007154" rpy="0 0 0"/>
       <mass value="0.09818420433466489"/>
-      <inertia ixx="5.2e-05" iyy="0.000244" izz="0.000252" ixy="1e-06" iyz="1e-06" ixz="-1e-05"/>
+      <inertia ixx="5.2003168e-05" iyy="2.437e-4" izz="2.523e-4" ixy="7.28047e-07" iyz="6.0331e-07" ixz="-9.716561e-06"/>
     </inertial>
   </link>
@@ -29,5 +29,5 @@
       <origin xyz="0.020109281613098752 0.002331771723067172 0.0064994497731911665" rpy="0 0 0"/>
       <mass value="0.020769030109708524"/>
-      <inertia ixx="2e-06" iyy="4e-06" izz="3e-06" ixy="-0.0" iyz="-0.0" ixz="-0.0"/>
+      <inertia ixx="2.494e-06" iyy="3.736e-06" izz="3.223e-06" ixy="-7.659e-9" iyz="0.072e-9" ixz="-33.608e-9"/>
     </inertial>
     <visual>
@@ -47,7 +47,7 @@
   <link name="lf2">
     <inertial>
-      <origin xyz="-2.5728896106275156e-06 0.0009860558893138652 -0.018261345499916863" rpy="0 0 0"/>
+      <origin xyz="-0.0031735030993243693 0.000986055889313886 -0.01798354657247523" rpy="0 0 0"/>
       <mass value="0.0019057729925096327"/>
-      <inertia ixx="0.0" iyy="0.0" izz="0.0" ixy="0.0" iyz="0.0" ixz="-0.0"/>
+      <inertia ixx="0.462154e-6" iyy="0.481174e-6" izz="26.893e-9" ixy="3.117e-9" iyz="17.662e-9" ixz="-79.269e-9"/>
     </inertial>
     <visual>
@@ -67,10 +67,10 @@
   <link name="lf3">
     <inertial>
-      <origin xyz="0.0007046107744873437 0.0034550275861905885 -0.016225601428628958" rpy="0 0 0"/>
+      <origin xyz="0.006210627225594921 0.003455723027058405 -0.015013638057132746" rpy="0 0 0"/>
       <mass value="0.0011438144457690698"/>
-      <inertia ixx="1e-06" iyy="1e-06" izz="0.0" ixy="-0.0" iyz="0.0" ixz="0.0"/>
-    </inertial>
-    <visual>
-      <origin xyz="-0.052159 -0.044445 0.049943" rpy="0 0 0"/>
+      <inertia ixx="0.484118e-6" iyy="0.567346e-06" izz="91.82e-9" ixy="-2.157e-9" iyz="4.945e-9" ixz="0.200546e-6"/>
+    </inertial>
+    <visual>
+      <origin xyz="-0.043476 -0.044445 0.049183" rpy="0 0 0"/>
       <geometry>
         <mesh filename="package://mini_pupper_2_description/meshes/lf3.stl" scale="1 1 1"/>
@@ -79,5 +79,5 @@
     </visual>
     <collision>
-      <origin xyz="-0.052159 -0.044445 0.049943" rpy="0 0 0"/>
+      <origin xyz="-0.043476 -0.044445 0.049183" rpy="0 0 0"/>
       <geometry>
         <mesh filename="package://mini_pupper_2_description/meshes/lf3.stl" scale="1 1 1"/>
@@ -86,8 +86,8 @@
   </link>
   <link name="rf1">
-      <inertial>
+    <inertial>
       <origin xyz="0.020106742599110078 -0.00233237781568562 0.006497900858401761" rpy="0 0 0"/>
       <mass value="0.020769549324466178"/>
-      <inertia ixx="2e-06" iyy="4e-06" izz="3e-06" ixy="0.0" iyz="-0.0" ixz="-0.0"/>
+      <inertia ixx="2.494e-06" iyy="3.736e-06" izz="3.223e-06" ixy="7.618e-9" iyz="0.098e-9" ixz="-37.629e-9"/>
     </inertial>
     <visual>
@@ -107,7 +107,7 @@
   <link name="rf2">
     <inertial>
-      <origin xyz="-4.1025190424676117e-07 -0.0009866275794596438 -0.018261345629717353" rpy="0 0 0"/>
+      <origin xyz="-0.00317137334512671 -0.000986627579459616 -0.01798392230653304" rpy="0 0 0"/>
       <mass value="0.0019057729924780605"/>
-      <inertia ixx="0.0" iyy="0.0" izz="0.0" ixy="-0.0" iyz="-0.0" ixz="-0.0"/>
+      <inertia ixx="0.462172e-6" iyy="0.481174e-6" izz="26.874e-9" ixy="-3.114e-9" iyz="-17.663e-9" ixz="-79.218e-9"/>
     </inertial>
     <visual>
@@ -127,10 +127,10 @@
   <link name="rf3">
     <inertial>
-      <origin xyz="0.0007030898236521158 -0.003457422744677939 -0.016230262912113935" rpy="0 0 0"/>
+      <origin xyz="0.006211719758792998 -0.0034574884973188197 -0.01500899883342268" rpy="0 0 0"/>
       <mass value="0.001143490701517533"/>
-      <inertia ixx="1e-06" iyy="1e-06" izz="0.0" ixy="0.0" iyz="-0.0" ixz="0.0"/>
-    </inertial>
-    <visual>
-      <origin xyz="-0.052165 0.043955 0.049943" rpy="0 0 0"/>
+      <inertia ixx="0.484726e-6" iyy="0.567959e-06" izz="91.882e-9" ixy="2.056e-9" iyz="-4.954e-9" ixz="0.200706e-6"/>
+    </inertial>
+    <visual>
+      <origin xyz="-0.043482 0.043955 0.049184" rpy="0 0 0"/>
       <geometry>
         <mesh filename="package://mini_pupper_2_description/meshes/rf3.stl" scale="1 1 1"/>
@@ -139,5 +139,5 @@
     </visual>
     <collision>
-      <origin xyz="-0.052165 0.043955 0.049943" rpy="0 0 0"/>
+      <origin xyz="-0.043482 0.043955 0.049184" rpy="0 0 0"/>
       <geometry>
         <mesh filename="package://mini_pupper_2_description/meshes/rf3.stl" scale="1 1 1"/>
@@ -149,5 +149,5 @@
       <origin xyz="-0.020107177922528044 -0.0023288309787250286 0.006502376356642127" rpy="0 0 0"/>
       <mass value="0.020769549324363486"/>
-      <inertia ixx="2e-06" iyy="4e-06" izz="3e-06" ixy="-0.0" iyz="-0.0" ixz="-0.0"/>
+      <inertia ixx="2.494e-06" iyy="3.736e-06" izz="3.223e-06" ixy="-7.639e-9" iyz="-0.378e-9" ixz="-37.624e-9"/>
     </inertial>
     <visual>
@@ -167,7 +167,7 @@
   <link name="rb2">
     <inertial>
-      <origin xyz="-2.5070667000748337e-08 -0.000996585764066693 -0.018260149861185754" rpy="0 0 0"/>
+      <origin xyz="-0.0031709881638501275 -0.0009964344348111775 -0.017982726579309202" rpy="0 0 0"/>
       <mass value="0.0019057729926311429"/>
-      <inertia ixx="0.0" iyy="0.0" izz="0.0" ixy="-0.0" iyz="-0.0" ixz="-0.0"/>
+      <inertia ixx="0.462172e-6" iyy="0.481155e-6" izz="26.893e-9" ixy="-3.158e-9" iyz="-17.911e-9" ixz="-79.911e-9"/>
     </inertial>
     <visual>
@@ -187,10 +187,10 @@
   <link name="rb3">
     <inertial>
-      <origin xyz="0.0007031309185970697 -0.0034624258831375196 -0.016220094399306113" rpy="0 0 0"/>
+      <origin xyz="0.006208573190273861 -0.0034623583329196975 -0.015001217060300935" rpy="0 0 0"/>
       <mass value="0.0011440535724654094"/>
-      <inertia ixx="1e-06" iyy="1e-06" izz="0.0" ixy="0.0" iyz="-0.0" ixz="0.0"/>
-    </inertial>
-    <visual>
-      <origin xyz="0.068367 0.043983 0.049932" rpy="0 0 0"/>
+      <inertia ixx="0.484539e-6" iyy="0.567687e-06" izz="91.857e-9" ixy="2.182e-9" iyz="-5.285e-9" ixz="0.200597e-6"/>
+    </inertial>
+    <visual>
+      <origin xyz="0.077049 0.043982 0.049173" rpy="0 0 0"/>
       <geometry>
         <mesh filename="package://mini_pupper_2_description/meshes/rb3.stl" scale="1 1 1"/>
@@ -199,5 +199,5 @@
     </visual>
     <collision>
-      <origin xyz="0.068367 0.043983 0.049932" rpy="0 0 0"/>
+      <origin xyz="0.077049 0.043982 0.049173" rpy="0 0 0"/>
       <geometry>
         <mesh filename="package://mini_pupper_2_description/meshes/rb3.stl" scale="1 1 1"/>
@@ -209,5 +209,5 @@
       <origin xyz="-0.020109716415830967 0.0023317718989125207 0.006499556305653081" rpy="0 0 0"/>
       <mass value="0.020769030189864354"/>
-      <inertia ixx="2e-06" iyy="4e-06" izz="3e-06" ixy="0.0" iyz="0.0" ixz="-0.0"/>
+      <inertia ixx="2.494e-06" iyy="3.736e-06" izz="3.223e-06" ixy="7.659e-9" iyz="-0.072e-9" ixz="-33.608e-9"/>
     </inertial>
     <visual>
@@ -227,7 +227,7 @@
   <link name="lb2">
     <inertial>
-      <origin xyz="-2.486178994620669e-08 0.0009860564153100007 -0.01826134562993383" rpy="0 0 0"/>
+      <origin xyz="-0.0031709879518865836 0.0009860564153100285 -0.01798392227051571" rpy="0 0 0"/>
       <mass value="0.0019057729925095609"/>
-      <inertia ixx="0.0" iyy="0.0" izz="0.0" ixy="0.0" iyz="0.0" ixz="-0.0"/>
+      <inertia ixx="0.462172e-6" iyy="0.481174e-6" izz="26.874e-9" ixy="3.114e-9" iyz="17.663e-9" ixz="-79.218e-9"/>
     </inertial>
     <visual>
@@ -247,10 +247,10 @@
   <link name="lb3">
     <inertial>
-      <origin xyz="0.0007030123702261443 0.0034519487133846394 -0.016218113385159758" rpy="0 0 0"/>
+      <origin xyz="0.006208905683926957 0.0034523757482988054 -0.015005654191541921" rpy="0 0 0"/>
       <mass value="0.001144346207072784"/>
-      <inertia ixx="1e-06" iyy="1e-06" izz="0.0" ixy="-0.0" iyz="0.0" ixz="0.0"/>
-    </inertial>
-    <visual>
-      <origin xyz="0.068367 -0.044445 0.049943" rpy="0 0 0"/>
+      <inertia ixx="0.484492e-6" iyy="0.567176e-06" izz="91.41e-9" ixy="-2.023e-9" iyz="4.977e-9" ixz="0.200063e-6"/>
+    </inertial>
+    <visual>
+      <origin xyz="0.077049 -0.044445 0.049184" rpy="0 0 0"/>
       <geometry>
         <mesh filename="package://mini_pupper_2_description/meshes/lb3.stl" scale="1 1 1"/>
@@ -259,5 +259,5 @@
     </visual>
     <collision>
-      <origin xyz="0.068367 -0.044445 0.049943" rpy="0 0 0"/>
+      <origin xyz="0.077049 -0.044445 0.049184" rpy="0 0 0"/>
       <geometry>
         <mesh filename="package://mini_pupper_2_description/meshes/lb3.stl" scale="1 1 1"/>
@@ -269,5 +269,5 @@
       <origin xyz="-0.005538678480206852 -0.00020424196520824284 0.020222593513387798" rpy="0 0 0"/>
       <mass value="0.00785515871148119"/>
-      <inertia ixx="5e-06" iyy="2e-06" izz="4e-06" ixy="-0.0" iyz="-0.0" ixz="-0.0"/>
+      <inertia ixx="5e-06" iyy="2e-06" izz="4e-06" ixy="0.0" iyz="0.0" ixz="0.0"/>
     </inertial>
     <visual>
@@ -309,5 +309,5 @@
       <origin xyz="-0.07276303117117414 -0.002323344081837563 -0.0010631239213060653" rpy="0 0 0"/>
       <mass value="0.004688613655947816"/>
-      <inertia ixx="0.0" iyy="1.5e-05" izz="1.6e-05" ixy="-1e-06" iyz="0.0" ixz="0.0"/>
+      <inertia ixx="0.203205e-6" iyy="1.5404404e-05" izz="1.5546403e-05" ixy="-0.625328e-06" iyz="42.901e-9" ixz="0.186346e-9"/>
     </inertial>
     <visual>
@@ -329,5 +329,5 @@
       <origin xyz="0.008233541174180986 -0.002138369786547657 -0.00030110978110910874" rpy="0 0 0"/>
       <mass value="0.0019746031301169403"/>
-      <inertia ixx="0.0" iyy="3e-06" izz="4e-06" ixy="-0.0" iyz="0.0" ixz="0.0"/>
+      <inertia ixx="0.458176e-6" iyy="3.284711e-06" izz="3.720353e-06" ixy="-79.81e-9" iyz="4.793e-9" ixz="0.123862e-9"/>
     </inertial>
     <visual>
@@ -347,10 +347,10 @@
   <link name="rffoot">
     <inertial>
-      <origin xyz="-0.0024634044240561814 -2.8557999392359035e-07 0.007801816226636768" rpy="0 0 0"/>
+      <origin xyz="-0.004983173489839052 -2.855799938611403e-07 0.006488367917121082" rpy="0 0 0"/>
       <mass value="0.0014053107976262874"/>
-      <inertia ixx="0.0" iyy="0.0" izz="0.0" ixy="0.0" iyz="-0.0" ixz="-0.0"/>
-    </inertial>
-    <visual>
-      <origin xyz="-0.056689 0.047705 0.109514" rpy="0 0 0"/>
+      <inertia ixx="41.992e-9" iyy="62.399e-9" izz="29.801e-9" ixy="0.0" iyz="0.0" ixz="1.625e-9"/>
+    </inertial>
+    <visual>
+      <origin xyz="-0.068108 0.047705 0.103614" rpy="0 0 0"/>
       <geometry>
         <mesh filename="package://mini_pupper_2_description/meshes/rffoot.stl" scale="1 1 1"/>
@@ -359,5 +359,5 @@
     </visual>
     <collision>
-      <origin xyz="-0.056689 0.047705 0.109514" rpy="0 0 0"/>
+      <origin xyz="-0.068108 0.047705 0.103614" rpy="0 0 0"/>
       <geometry>
         <mesh filename="package://mini_pupper_2_description/meshes/rffoot.stl" scale="1 1 1"/>
@@ -367,10 +367,10 @@
   <link name="rbfoot">
     <inertial>
-      <origin xyz="-0.0024630192318816357 4.2051173794327434e-06 0.0078011683948505245" rpy="0 0 0"/>
+      <origin xyz="-0.004982788301465979 3.706995898918042e-06 0.006488719406103974" rpy="0 0 0"/>
       <mass value="0.0014053107976262874"/>
-      <inertia ixx="0.0" iyy="0.0" izz="0.0" ixy="-0.0" iyz="-0.0" ixz="-0.0"/>
-    </inertial>
-    <visual>
-      <origin xyz="0.063843 0.047765 0.1095" rpy="0 0 0"/>
+      <inertia ixx="41.992e-9" iyy="62.399e-9" izz="29.801e-9" ixy="0.001e-9" iyz="-0.018e-9" ixz="1.625e-9"/>
+    </inertial>
+    <visual>
+      <origin xyz="0.052424 0.047762 0.103601" rpy="0 0 0"/>
       <geometry>
         <mesh filename="package://mini_pupper_2_description/meshes/rbfoot.stl" scale="1 1 1"/>
@@ -379,5 +379,5 @@
     </visual>
     <collision>
-      <origin xyz="0.063843 0.047765 0.1095" rpy="0 0 0"/>
+      <origin xyz="0.052424 0.047762 0.103601" rpy="0 0 0"/>
       <geometry>
         <mesh filename="package://mini_pupper_2_description/meshes/rbfoot.stl" scale="1 1 1"/>
@@ -387,10 +387,10 @@
   <link name="lbfoot">
     <inertial>
-      <origin xyz="-0.0024630193952935586 -2.855826621572799e-07 0.00780181622349041" rpy="0 0 0"/>
+      <origin xyz="-0.004982788451759437 -2.855826620323798e-07 0.0064883680140642025" rpy="0 0 0"/>
       <mass value="0.0014053107976262874"/>
-      <inertia ixx="0.0" iyy="0.0" izz="0.0" ixy="0.0" iyz="-0.0" ixz="-0.0"/>
-    </inertial>
-    <visual>
-      <origin xyz="0.063843 -0.048195 0.109514" rpy="0 0 0"/>
+      <inertia ixx="41.992e-9" iyy="62.399e-9" izz="29.801e-9" ixy="0.0" iyz="0.0" ixz="1.625e-9"/>
+    </inertial>
+    <visual>
+      <origin xyz="0.052424 -0.048195 0.103614" rpy="0 0 0"/>
       <geometry>
         <mesh filename="package://mini_pupper_2_description/meshes/lbfoot.stl" scale="1 1 1"/>
@@ -399,5 +399,5 @@
     </visual>
     <collision>
-      <origin xyz="0.063843 -0.048195 0.109514" rpy="0 0 0"/>
+      <origin xyz="0.052424 -0.048195 0.103614" rpy="0 0 0"/>
       <geometry>
         <mesh filename="package://mini_pupper_2_description/meshes/lbfoot.stl" scale="1 1 1"/>
@@ -407,10 +407,10 @@
   <link name="lffoot">
     <inertial>
-      <origin xyz="-0.002463300234335934 -2.8611328430766525e-07 0.00780127458383767" rpy="0 0 0"/>
+      <origin xyz="-0.004983499344395154 -2.861132842799097e-07 0.006488888240325896" rpy="0 0 0"/>
       <mass value="0.0014053107976262874"/>
-      <inertia ixx="0.0" iyy="0.0" izz="0.0" ixy="0.0" iyz="-0.0" ixz="-0.0"/>
-    </inertial>
-    <visual>
-      <origin xyz="-0.056689 -0.048195 0.109513" rpy="0 0 0"/>
+      <inertia ixx="41.992e-9" iyy="62.399e-9" izz="29.801e-9" ixy="0.0" iyz="0.0" ixz="1.625e-9"/>
+    </inertial>
+    <visual>
+      <origin xyz="-0.068108 -0.048195 0.103611" rpy="0 0 0"/>
       <geometry>
         <mesh filename="package://mini_pupper_2_description/meshes/lffoot.stl" scale="1 1 1"/>
@@ -419,5 +419,5 @@
     </visual>
     <collision>
-      <origin xyz="-0.056689 -0.048195 0.109513" rpy="0 0 0"/>
+      <origin xyz="-0.068108 -0.048195 0.103611" rpy="0 0 0"/>
       <geometry>
         <mesh filename="package://mini_pupper_2_description/meshes/lffoot.stl" scale="1 1 1"/>
@@ -425,14 +425,14 @@
     </collision>
   </link>
-  <link name="Shell_Hip_Left_1">
+  <link name="lpf1">
     <inertial>
       <origin xyz="0.002258882765982295 0.008667473212030541 -0.002747896746317195" rpy="0 0 0"/>
       <mass value="0.002573897544461238"/>
-      <inertia ixx="0.0" iyy="0.0" izz="0.0" ixy="0.0" iyz="0.0" ixz="0.0"/>
+      <inertia ixx="0.390582e-6" iyy="0.412423e-6" izz="0.246322e-6" ixy="24.632e-9" iyz="3.861e-9" ixz="54.103e-9"/>
     </inertial>
     <visual>
       <origin xyz="-0.071565 -0.038245 -0.013057" rpy="0 0 0"/>
       <geometry>
-        <mesh filename="package://mini_pupper_2_description/meshes/Shell_Hip_Left_1.stl" scale="1 1 1"/>
+        <mesh filename="package://mini_pupper_2_description/meshes/lpf1.stl" scale="1 1 1"/>
       </geometry>
       <material name="opaque2552210"/>
@@ -441,18 +441,18 @@
       <origin xyz="-0.071565 -0.038245 -0.013057" rpy="0 0 0"/>
       <geometry>
-        <mesh filename="package://mini_pupper_2_description/meshes/Shell_Hip_Left_1.stl" scale="1 1 1"/>
-      </geometry>
-    </collision>
-  </link>
-  <link name="Shell_Hip_Left_2">
+        <mesh filename="package://mini_pupper_2_description/meshes/lpf1.stl" scale="1 1 1"/>
+      </geometry>
+    </collision>
+  </link>
+  <link name="lpb1">
     <inertial>
       <origin xyz="0.0022592683660053597 0.008667473212031727 -0.0027478967463174797" rpy="0 0 0"/>
       <mass value="0.002573897544461238"/>
-      <inertia ixx="0.0" iyy="0.0" izz="0.0" ixy="0.0" iyz="0.0" ixz="0.0"/>
+      <inertia ixx="0.390582e-6" iyy="0.412423e-6" izz="0.246322e-6" ixy="24.632e-9" iyz="3.861e-9" ixz="54.103e-9"/>
     </inertial>
     <visual>
       <origin xyz="0.048967 -0.038245 -0.013057" rpy="0 0 0"/>
       <geometry>
-        <mesh filename="package://mini_pupper_2_description/meshes/Shell_Hip_Left_2.stl" scale="1 1 1"/>
+        <mesh filename="package://mini_pupper_2_description/meshes/lpb1.stl" scale="1 1 1"/>
       </geometry>
       <material name="opaque2552210"/>
@@ -461,18 +461,18 @@
       <origin xyz="0.048967 -0.038245 -0.013057" rpy="0 0 0"/>
       <geometry>
-        <mesh filename="package://mini_pupper_2_description/meshes/Shell_Hip_Left_2.stl" scale="1 1 1"/>
-      </geometry>
-    </collision>
-  </link>
-  <link name="Shell_Hip_Right_1">
+        <mesh filename="package://mini_pupper_2_description/meshes/lpb1.stl" scale="1 1 1"/>
+      </geometry>
+    </collision>
+  </link>
+  <link name="rpf1">
     <inertial>
       <origin xyz="0.002219644336096324 -0.008605630927951344 -0.002709000699399786" rpy="0 0 0"/>
       <mass value="0.002396251664132183"/>
-      <inertia ixx="0.0" iyy="0.0" izz="0.0" ixy="-0.0" iyz="-0.0" ixz="0.0"/>
+      <inertia ixx="0.364377e-6" iyy="0.38866e-6" izz="0.234177e-6" ixy="-23.674e-9" iyz="-3.338e-9" ixz="52.098e-9"/>
     </inertial>
     <visual>
       <origin xyz="-0.071565 0.037755 -0.013057" rpy="0 0 0"/>
       <geometry>
-        <mesh filename="package://mini_pupper_2_description/meshes/Shell_Hip_Right_1.stl" scale="1 1 1"/>
+        <mesh filename="package://mini_pupper_2_description/meshes/rpf1.stl" scale="1 1 1"/>
       </geometry>
       <material name="opaque2552210"/>
@@ -481,18 +481,18 @@
       <origin xyz="-0.071565 0.037755 -0.013057" rpy="0 0 0"/>
       <geometry>
-        <mesh filename="package://mini_pupper_2_description/meshes/Shell_Hip_Right_1.stl" scale="1 1 1"/>
-      </geometry>
-    </collision>
-  </link>
-  <link name="Shell_Hip_Right_2">
+        <mesh filename="package://mini_pupper_2_description/meshes/rpf1.stl" scale="1 1 1"/>
+      </geometry>
+    </collision>
+  </link>
+  <link name="rpb1">
     <inertial>
       <origin xyz="0.0022200295152449145 -0.008607013686777375 -0.0027033986949916797" rpy="0 0 0"/>
       <mass value="0.002396251664132183"/>
-      <inertia ixx="0.0" iyy="0.0" izz="0.0" ixy="-0.0" iyz="-0.0" ixz="0.0"/>
+      <inertia ixx="0.364377e-6" iyy="0.388657e-6" izz="0.23418e-6" ixy="-23.645e-9" iyz="-3.422e-9" ixz="52.111e-9"/>
     </inertial>
     <visual>
       <origin xyz="0.048967 0.037748 -0.013064" rpy="0 0 0"/>
       <geometry>
-        <mesh filename="package://mini_pupper_2_description/meshes/Shell_Hip_Right_2.stl" scale="1 1 1"/>
+        <mesh filename="package://mini_pupper_2_description/meshes/rpb1.stl" scale="1 1 1"/>
       </geometry>
       <material name="opaque2552210"/>
@@ -501,85 +501,85 @@
       <origin xyz="0.048967 0.037748 -0.013064" rpy="0 0 0"/>
       <geometry>
-        <mesh filename="package://mini_pupper_2_description/meshes/Shell_Hip_Right_2.stl" scale="1 1 1"/>
-      </geometry>
-    </collision>
-  </link>
-  <link name="Shell_Leg_Upper_LeftSide_1">
-    <inertial>
-      <origin xyz="-0.0026521199361419917 0.00790352811362325 0.004979527414372081" rpy="0 0 0"/>
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