Commit message: further fix file path

File: mini_pupper_2_description/urdf/mini_pupper_description.urdf.xacro (robot description, xacro)
@@ -7,5 +7,5 @@
       <origin xyz="0 0 0" rpy="0 0 0"/>
       <geometry>
-        <mesh filename="$(find mini_pupper_2_description)/meshes/base_link.stl" scale="1 1 1"/>
+        <mesh filename="file://$(find mini_pupper_2_description)/meshes/base_link.stl" scale="1 1 1"/>
       </geometry>
       <material name="opaque252525"/>
@@ -14,5 +14,5 @@
       <origin xyz="0 0 0" rpy="0 0 0"/>
       <geometry>
-        <mesh filename="$(find mini_pupper_2_description)/meshes/base_link.stl" scale="1 1 1"/>
+        <mesh filename="file://$(find mini_pupper_2_description)/meshes/base_link.stl" scale="1 1 1"/>
       </geometry>
     </collision>
@@ -34,5 +34,5 @@
       <origin xyz="-0.037299 -0.023745 -5.7e-05" rpy="0 0 0"/>
       <geometry>
-        <mesh filename="$(find mini_pupper_2_description)/meshes/lf1.stl" scale="1 1 1"/>
+        <mesh filename="file://$(find mini_pupper_2_description)/meshes/lf1.stl" scale="1 1 1"/>
       </geometry>
       <material name="opaque666666"/>
@@ -41,5 +41,5 @@
       <origin xyz="-0.037299 -0.023745 -5.7e-05" rpy="0 0 0"/>
       <geometry>
-        <mesh filename="$(find mini_pupper_2_description)/meshes/lf1.stl" scale="1 1 1"/>
+        <mesh filename="file://$(find mini_pupper_2_description)/meshes/lf1.stl" scale="1 1 1"/>
       </geometry>
     </collision>
@@ -54,5 +54,5 @@
       <origin xyz="-0.052165 -0.041445 -5.7e-05" rpy="0 0 0"/>
       <geometry>
-        <mesh filename="$(find mini_pupper_2_description)/meshes/lf2.stl" scale="1 1 1"/>
+        <mesh filename="file://$(find mini_pupper_2_description)/meshes/lf2.stl" scale="1 1 1"/>
       </geometry>
       <material name="opaque636363"/>
@@ -61,5 +61,5 @@
       <origin xyz="-0.052165 -0.041445 -5.7e-05" rpy="0 0 0"/>
       <geometry>
-        <mesh filename="$(find mini_pupper_2_description)/meshes/lf2.stl" scale="1 1 1"/>
+        <mesh filename="file://$(find mini_pupper_2_description)/meshes/lf2.stl" scale="1 1 1"/>
       </geometry>
     </collision>
@@ -74,5 +74,5 @@
       <origin xyz="-0.043476 -0.044445 0.049183" rpy="0 0 0"/>
       <geometry>
-        <mesh filename="$(find mini_pupper_2_description)/meshes/lf3.stl" scale="1 1 1"/>
+        <mesh filename="file://$(find mini_pupper_2_description)/meshes/lf3.stl" scale="1 1 1"/>
       </geometry>
       <material name="opaque252525"/>
@@ -81,5 +81,5 @@
       <origin xyz="-0.043476 -0.044445 0.049183" rpy="0 0 0"/>
       <geometry>
-        <mesh filename="$(find mini_pupper_2_description)/meshes/lf3.stl" scale="1 1 1"/>
+        <mesh filename="file://$(find mini_pupper_2_description)/meshes/lf3.stl" scale="1 1 1"/>
       </geometry>
     </collision>
@@ -94,5 +94,5 @@
       <origin xyz="-0.037299 0.023255 -5.7e-05" rpy="0 0 0"/>
       <geometry>
-        <mesh filename="$(find mini_pupper_2_description)/meshes/rf1.stl" scale="1 1 1"/>
+        <mesh filename="file://$(find mini_pupper_2_description)/meshes/rf1.stl" scale="1 1 1"/>
       </geometry>
       <material name="opaque666666"/>
@@ -101,5 +101,5 @@
       <origin xyz="-0.037299 0.023255 -5.7e-05" rpy="0 0 0"/>
       <geometry>
-        <mesh filename="$(find mini_pupper_2_description)/meshes/rf1.stl" scale="1 1 1"/>
+        <mesh filename="file://$(find mini_pupper_2_description)/meshes/rf1.stl" scale="1 1 1"/>
       </geometry>
     </collision>
@@ -114,5 +114,5 @@
       <origin xyz="-0.052165 0.040955 -5.7e-05" rpy="0 0 0"/>
       <geometry>
-        <mesh filename="$(find mini_pupper_2_description)/meshes/rf2.stl" scale="1 1 1"/>
+        <mesh filename="file://$(find mini_pupper_2_description)/meshes/rf2.stl" scale="1 1 1"/>
       </geometry>
       <material name="opaque636363"/>
@@ -121,5 +121,5 @@
       <origin xyz="-0.052165 0.040955 -5.7e-05" rpy="0 0 0"/>
       <geometry>
-        <mesh filename="$(find mini_pupper_2_description)/meshes/rf2.stl" scale="1 1 1"/>
+        <mesh filename="file://$(find mini_pupper_2_description)/meshes/rf2.stl" scale="1 1 1"/>
       </geometry>
     </collision>
@@ -134,5 +134,5 @@
       <origin xyz="-0.043482 0.043955 0.049184" rpy="0 0 0"/>
       <geometry>
-        <mesh filename="$(find mini_pupper_2_description)/meshes/rf3.stl" scale="1 1 1"/>
+        <mesh filename="file://$(find mini_pupper_2_description)/meshes/rf3.stl" scale="1 1 1"/>
       </geometry>
       <material name="opaque252525"/>
@@ -141,5 +141,5 @@
       <origin xyz="-0.043482 0.043955 0.049184" rpy="0 0 0"/>
       <geometry>
-        <mesh filename="$(find mini_pupper_2_description)/meshes/rf3.stl" scale="1 1 1"/>
+        <mesh filename="file://$(find mini_pupper_2_description)/meshes/rf3.stl" scale="1 1 1"/>
       </geometry>
     </collision>
@@ -154,5 +154,5 @@
       <origin xyz="0.042701 0.023255 -5.7e-05" rpy="0 0 0"/>
       <geometry>
-        <mesh filename="$(find mini_pupper_2_description)/meshes/rb1.stl" scale="1 1 1"/>
+        <mesh filename="file://$(find mini_pupper_2_description)/meshes/rb1.stl" scale="1 1 1"/>
       </geometry>
       <material name="opaque666666"/>
@@ -161,5 +161,5 @@
       <origin xyz="0.042701 0.023255 -5.7e-05" rpy="0 0 0"/>
       <geometry>
-        <mesh filename="$(find mini_pupper_2_description)/meshes/rb1.stl" scale="1 1 1"/>
+        <mesh filename="file://$(find mini_pupper_2_description)/meshes/rb1.stl" scale="1 1 1"/>
       </geometry>
     </collision>
@@ -174,5 +174,5 @@
       <origin xyz="0.068367 0.040955 -6.6e-05" rpy="0 0 0"/>
       <geometry>
-        <mesh filename="$(find mini_pupper_2_description)/meshes/rb2.stl" scale="1 1 1"/>
+        <mesh filename="file://$(find mini_pupper_2_description)/meshes/rb2.stl" scale="1 1 1"/>
       </geometry>
       <material name="opaque636363"/>
@@ -181,5 +181,5 @@
       <origin xyz="0.068367 0.040955 -6.6e-05" rpy="0 0 0"/>
       <geometry>
-        <mesh filename="$(find mini_pupper_2_description)/meshes/rb2.stl" scale="1 1 1"/>
+        <mesh filename="file://$(find mini_pupper_2_description)/meshes/rb2.stl" scale="1 1 1"/>
       </geometry>
     </collision>
@@ -194,5 +194,5 @@
       <origin xyz="0.077049 0.043982 0.049173" rpy="0 0 0"/>
       <geometry>
-        <mesh filename="$(find mini_pupper_2_description)/meshes/rb3.stl" scale="1 1 1"/>
+        <mesh filename="file://$(find mini_pupper_2_description)/meshes/rb3.stl" scale="1 1 1"/>
       </geometry>
       <material name="opaque252525"/>
@@ -201,5 +201,5 @@
       <origin xyz="0.077049 0.043982 0.049173" rpy="0 0 0"/>
       <geometry>
-        <mesh filename="$(find mini_pupper_2_description)/meshes/rb3.stl" scale="1 1 1"/>
+        <mesh filename="file://$(find mini_pupper_2_description)/meshes/rb3.stl" scale="1 1 1"/>
       </geometry>
     </collision>
@@ -214,5 +214,5 @@
       <origin xyz="0.042701 -0.023745 -5.7e-05" rpy="0 0 0"/>
       <geometry>
-        <mesh filename="$(find mini_pupper_2_description)/meshes/lb1.stl" scale="1 1 1"/>
+        <mesh filename="file://$(find mini_pupper_2_description)/meshes/lb1.stl" scale="1 1 1"/>
       </geometry>
       <material name="opaque666666"/>
@@ -221,5 +221,5 @@
       <origin xyz="0.042701 -0.023745 -5.7e-05" rpy="0 0 0"/>
       <geometry>
-        <mesh filename="$(find mini_pupper_2_description)/meshes/lb1.stl" scale="1 1 1"/>
+        <mesh filename="file://$(find mini_pupper_2_description)/meshes/lb1.stl" scale="1 1 1"/>
       </geometry>
     </collision>
@@ -234,5 +234,5 @@
       <origin xyz="0.068367 -0.041445 -5.7e-05" rpy="0 0 0"/>
       <geometry>
-        <mesh filename="$(find mini_pupper_2_description)/meshes/lb2.stl" scale="1 1 1"/>
+        <mesh filename="file://$(find mini_pupper_2_description)/meshes/lb2.stl" scale="1 1 1"/>
       </geometry>
       <material name="opaque636363"/>
@@ -241,5 +241,5 @@
       <origin xyz="0.068367 -0.041445 -5.7e-05" rpy="0 0 0"/>
       <geometry>
-        <mesh filename="$(find mini_pupper_2_description)/meshes/lb2.stl" scale="1 1 1"/>
+        <mesh filename="file://$(find mini_pupper_2_description)/meshes/lb2.stl" scale="1 1 1"/>
       </geometry>
     </collision>
@@ -254,5 +254,5 @@
       <origin xyz="0.077049 -0.044445 0.049184" rpy="0 0 0"/>
       <geometry>
-        <mesh filename="$(find mini_pupper_2_description)/meshes/lb3.stl" scale="1 1 1"/>
+        <mesh filename="file://$(find mini_pupper_2_description)/meshes/lb3.stl" scale="1 1 1"/>
       </geometry>
       <material name="opaque252525"/>
@@ -261,5 +261,5 @@
       <origin xyz="0.077049 -0.044445 0.049184" rpy="0 0 0"/>
       <geometry>
-        <mesh filename="$(find mini_pupper_2_description)/meshes/lb3.stl" scale="1 1 1"/>
+        <mesh filename="file://$(find mini_pupper_2_description)/meshes/lb3.stl" scale="1 1 1"/>
       </geometry>
     </collision>
@@ -274,5 +274,5 @@
       <origin xyz="-0.089299 -0.000245 0.015543" rpy="0 0 0"/>
       <geometry>
-        <mesh filename="$(find mini_pupper_2_description)/meshes/Body_front.stl" scale="1 1 1"/>
+        <mesh filename="file://$(find mini_pupper_2_description)/meshes/Body_front.stl" scale="1 1 1"/>
       </geometry>
       <material name="opaque2552210"/>
@@ -281,5 +281,5 @@
       <origin xyz="-0.089299 -0.000245 0.015543" rpy="0 0 0"/>
       <geometry>
-        <mesh filename="$(find mini_pupper_2_description)/meshes/Body_front.stl" scale="1 1 1"/>
+        <mesh filename="file://$(find mini_pupper_2_description)/meshes/Body_front.stl" scale="1 1 1"/>
       </geometry>
     </collision>
@@ -294,5 +294,5 @@
       <origin xyz="0.087701 0.023255 -0.026457" rpy="0 0 0"/>
       <geometry>
-        <mesh filename="$(find mini_pupper_2_description)/meshes/Board_PCB.stl" scale="1 1 1"/>
+        <mesh filename="file://$(find mini_pupper_2_description)/meshes/Board_PCB.stl" scale="1 1 1"/>
       </geometry>
       <material name="opaque646464"/>
@@ -301,5 +301,5 @@
       <origin xyz="0.087701 0.023255 -0.026457" rpy="0 0 0"/>
       <geometry>
-        <mesh filename="$(find mini_pupper_2_description)/meshes/Board_PCB.stl" scale="1 1 1"/>
+        <mesh filename="file://$(find mini_pupper_2_description)/meshes/Board_PCB.stl" scale="1 1 1"/>
       </geometry>
     </collision>
@@ -314,5 +314,5 @@
       <origin xyz="-0.061334 -0.000217 -0.026457" rpy="0 0 0"/>
       <geometry>
-        <mesh filename="$(find mini_pupper_2_description)/meshes/Board_connectors_1.stl" scale="1 1 1"/>
+        <mesh filename="file://$(find mini_pupper_2_description)/meshes/Board_connectors_1.stl" scale="1 1 1"/>
       </geometry>
       <material name="opaque2491590"/>
@@ -321,5 +321,5 @@
       <origin xyz="-0.061334 -0.000217 -0.026457" rpy="0 0 0"/>
       <geometry>
-        <mesh filename="$(find mini_pupper_2_description)/meshes/Board_connectors_1.stl" scale="1 1 1"/>
+        <mesh filename="file://$(find mini_pupper_2_description)/meshes/Board_connectors_1.stl" scale="1 1 1"/>
       </geometry>
     </collision>
@@ -334,5 +334,5 @@
       <origin xyz="0.045346 -0.000245 -0.026457" rpy="0 0 0"/>
       <geometry>
-        <mesh filename="$(find mini_pupper_2_description)/meshes/Board_connectors_2.stl" scale="1 1 1"/>
+        <mesh filename="file://$(find mini_pupper_2_description)/meshes/Board_connectors_2.stl" scale="1 1 1"/>
       </geometry>
       <material name="opaque255255255"/>
@@ -341,5 +341,5 @@
       <origin xyz="0.045346 -0.000245 -0.026457" rpy="0 0 0"/>
       <geometry>
-        <mesh filename="$(find mini_pupper_2_description)/meshes/Board_connectors_2.stl" scale="1 1 1"/>
+        <mesh filename="file://$(find mini_pupper_2_description)/meshes/Board_connectors_2.stl" scale="1 1 1"/>
       </geometry>
     </collision>
@@ -354,5 +354,5 @@
       <origin xyz="-0.068108 0.047705 0.103614" rpy="0 0 0"/>
       <geometry>
-        <mesh filename="$(find mini_pupper_2_description)/meshes/rffoot.stl" scale="1 1 1"/>
+        <mesh filename="file://$(find mini_pupper_2_description)/meshes/rffoot.stl" scale="1 1 1"/>
       </geometry>
       <material name="opaque666666"/>
@@ -361,5 +361,5 @@
       <origin xyz="-0.068108 0.047705 0.103614" rpy="0 0 0"/>
       <geometry>
-        <mesh filename="$(find mini_pupper_2_description)/meshes/rffoot.stl" scale="1 1 1"/>
+        <mesh filename="file://$(find mini_pupper_2_description)/meshes/rffoot.stl" scale="1 1 1"/>
       </geometry>
     </collision>
@@ -374,5 +374,5 @@
       <origin xyz="0.052424 0.047762 0.103601" rpy="0 0 0"/>
       <geometry>
-        <mesh filename="$(find mini_pupper_2_description)/meshes/rbfoot.stl" scale="1 1 1"/>
+        <mesh filename="file://$(find mini_pupper_2_description)/meshes/rbfoot.stl" scale="1 1 1"/>
       </geometry>
       <material name="opaque666666"/>
@@ -381,5 +381,5 @@
       <origin xyz="0.052424 0.047762 0.103601" rpy="0 0 0"/>
       <geometry>
-        <mesh filename="$(find mini_pupper_2_description)/meshes/rbfoot.stl" scale="1 1 1"/>
+        <mesh filename="file://$(find mini_pupper_2_description)/meshes/rbfoot.stl" scale="1 1 1"/>
       </geometry>
     </collision>
@@ -394,5 +394,5 @@
       <origin xyz="0.052424 -0.048195 0.103614" rpy="0 0 0"/>
       <geometry>
-        <mesh filename="$(find mini_pupper_2_description)/meshes/lbfoot.stl" scale="1 1 1"/>
+        <mesh filename="file://$(find mini_pupper_2_description)/meshes/lbfoot.stl" scale="1 1 1"/>
       </geometry>
       <material name="opaque666666"/>
@@ -401,5 +401,5 @@
       <origin xyz="0.052424 -0.048195 0.103614" rpy="0 0 0"/>
       <geometry>
-        <mesh filename="$(find mini_pupper_2_description)/meshes/lbfoot.stl" scale="1 1 1"/>
+        <mesh filename="file://$(find mini_pupper_2_description)/meshes/lbfoot.stl" scale="1 1 1"/>
       </geometry>
     </collision>
@@ -414,5 +414,5 @@
       <origin xyz="-0.068108 -0.048195 0.103611" rpy="0 0 0"/>
       <geometry>
-        <mesh filename="$(find mini_pupper_2_description)/meshes/lffoot.stl" scale="1 1 1"/>
+        <mesh filename="file://$(find mini_pupper_2_description)/meshes/lffoot.stl" scale="1 1 1"/>
       </geometry>
       <material name="opaque666666"/>
@@ -421,5 +421,5 @@
       <origin xyz="-0.068108 -0.048195 0.103611" rpy="0 0 0"/>
       <geometry>
-        <mesh filename="$(find mini_pupper_2_description)/meshes/lffoot.stl" scale="1 1 1"/>
+        <mesh filename="file://$(find mini_pupper_2_description)/meshes/lffoot.stl" scale="1 1 1"/>
       </geometry>
     </collision>
@@ -434,5 +434,5 @@
       <origin xyz="-0.071565 -0.038245 -0.013057" rpy="0 0 0"/>
       <geometry>
-        <mesh filename="$(find mini_pupper_2_description)/meshes/lpf1.stl" scale="1 1 1"/>
+        <mesh filename="file://$(find mini_pupper_2_description)/meshes/lpf1.stl" scale="1 1 1"/>
       </geometry>
       <material name="opaque2552210"/>
@@ -441,5 +441,5 @@
       <origin xyz="-0.071565 -0.038245 -0.013057" rpy="0 0 0"/>
       <geometry>
-        <mesh filename="$(find mini_pupper_2_description)/meshes/lpf1.stl" scale="1 1 1"/>
+        <mesh filename="file://$(find mini_pupper_2_description)/meshes/lpf1.stl" scale="1 1 1"/>
       </geometry>
     </collision>
@@ -454,5 +454,5 @@
       <origin xyz="0.048967 -0.038245 -0.013057" rpy="0 0 0"/>
       <geometry>
-        <mesh filename="$(find mini_pupper_2_description)/meshes/lpb1.stl" scale="1 1 1"/>
+        <mesh filename="file://$(find mini_pupper_2_description)/meshes/lpb1.stl" scale="1 1 1"/>
       </geometry>
       <material name="opaque2552210"/>
@@ -461,5 +461,5 @@
       <origin xyz="0.048967 -0.038245 -0.013057" rpy="0 0 0"/>
       <geometry>
-        <mesh filename="$(find mini_pupper_2_description)/meshes/lpb1.stl" scale="1 1 1"/>
+        <mesh filename="file://$(find mini_pupper_2_description)/meshes/lpb1.stl" scale="1 1 1"/>
       </geometry>
     </collision>
@@ -474,5 +474,5 @@
       <origin xyz="-0.071565 0.037755 -0.013057" rpy="0 0 0"/>
       <geometry>
-        <mesh filename="$(find mini_pupper_2_description)/meshes/rpf1.stl" scale="1 1 1"/>
+        <mesh filename="file://$(find mini_pupper_2_description)/meshes/rpf1.stl" scale="1 1 1"/>
       </geometry>
       <material name="opaque2552210"/>
@@ -481,5 +481,5 @@
       <origin xyz="-0.071565 0.037755 -0.013057" rpy="0 0 0"/>
       <geometry>
-        <mesh filename="$(find mini_pupper_2_description)/meshes/rpf1.stl" scale="1 1 1"/>
+        <mesh filename="file://$(find mini_pupper_2_description)/meshes/rpf1.stl" scale="1 1 1"/>
       </geometry>
     </collision>
@@ -494,5 +494,5 @@
       <origin xyz="0.048967 0.037748 -0.013064" rpy="0 0 0"/>
       <geometry>
-        <mesh filename="$(find mini_pupper_2_description)/meshes/rpb1.stl" scale="1 1 1"/>
+        <mesh filename="file://$(find mini_pupper_2_description)/meshes/rpb1.stl" scale="1 1 1"/>
       </geometry>
       <material name="opaque2552210"/>
@@ -501,5 +501,5 @@
       <origin xyz="0.048967 0.037748 -0.013064" rpy="0 0 0"/>
       <geometry>
-        <mesh filename="$(find mini_pupper_2_description)/meshes/rpb1.stl" scale="1 1 1"/>
+        <mesh filename="file://$(find mini_pupper_2_description)/meshes/rpb1.stl" scale="1 1 1"/>
       </geometry>
     </collision>
@@ -514,5 +514,5 @@
       <origin xyz="-0.048863 -0.044445 0.018654" rpy="0 0 0"/>
       <geometry>
-        <mesh filename="$(find mini_pupper_2_description)/meshes/lpf2.stl" scale="1 1 1"/>
+        <mesh filename="file://$(find mini_pupper_2_description)/meshes/lpf2.stl" scale="1 1 1"/>
       </geometry>
       <material name="opaque2552210"/>
@@ -521,5 +521,5 @@
       <origin xyz="-0.048863 -0.044445 0.018654" rpy="0 0 0"/>
       <geometry>
-        <mesh filename="$(find mini_pupper_2_description)/meshes/lpf2.stl" scale="1 1 1"/>
+        <mesh filename="file://$(find mini_pupper_2_description)/meshes/lpf2.stl" scale="1 1 1"/>
       </geometry>
     </collision>
@@ -534,5 +534,5 @@
       <origin xyz="0.071666 -0.044445 0.018655" rpy="0 0 0"/>
       <geometry>
-        <mesh filename="$(find mini_pupper_2_description)/meshes/lpb2.stl" scale="1 1 1"/>
+        <mesh filename="file://$(find mini_pupper_2_description)/meshes/lpb2.stl" scale="1 1 1"/>
       </geometry>
       <material name="opaque2552210"/>
@@ -541,5 +541,5 @@
       <origin xyz="0.071666 -0.044445 0.018655" rpy="0 0 0"/>
       <geometry>
-        <mesh filename="$(find mini_pupper_2_description)/meshes/lpb2.stl" scale="1 1 1"/>
+        <mesh filename="file://$(find mini_pupper_2_description)/meshes/lpb2.stl" scale="1 1 1"/>
       </geometry>
     </collision>
@@ -554,5 +554,5 @@
       <origin xyz="-0.048865 0.043955 0.018655" rpy="0 0 0"/>
       <geometry>
-        <mesh filename="$(find mini_pupper_2_description)/meshes/rpf2.stl" scale="1 1 1"/>
+        <mesh filename="file://$(find mini_pupper_2_description)/meshes/rpf2.stl" scale="1 1 1"/>
       </geometry>
       <material name="opaque2552210"/>
@@ -561,5 +561,5 @@
       <origin xyz="-0.048865 0.043955 0.018655" rpy="0 0 0"/>
       <geometry>
-        <mesh filename="$(find mini_pupper_2_description)/meshes/rpf2.stl" scale="1 1 1"/>
+        <mesh filename="file://$(find mini_pupper_2_description)/meshes/rpf2.stl" scale="1 1 1"/>
       </geometry>
     </collision>
@@ -574,5 +574,5 @@
       <origin xyz="0.071666 0.043965 0.018644" rpy="0 0 0"/>
       <geometry>
-        <mesh filename="$(find mini_pupper_2_description)/meshes/rpb2.stl" scale="1 1 1"/>
+        <mesh filename="file://$(find mini_pupper_2_description)/meshes/rpb2.stl" scale="1 1 1"/>
       </geometry>
       <material name="opaque2552210"/>
@@ -581,5 +581,5 @@
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