Commit message: Applied symmetry to all links' center of mass and inertia

File: mini_pupper_description/urdf/mini_pupper_description.urdf (robot description, URDF)
Before this commit: robot mini-pupper, 39 links, 38 joints
Links:
- removed link camera_bottom_screw_frame
- removed link camera_color_frame
- removed link camera_color_optical_frame
- removed link camera_depth_frame
- removed link camera_depth_optical_frame
- removed link camera_infra1_frame
- removed link camera_infra1_optical_frame
- removed link camera_infra2_frame
- removed link camera_infra2_optical_frame
- removed link camera_link
- removed link lidar
- added link lidar_link, mass 0.0001; collision mesh filename=file:///home/peter/ros2_ws/install/mini_pupper_description/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; visual mesh filename=file:///home/peter/ros2_ws/install/mini_pupper_description/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
- link base_inertia: mass 0.2 -> 0.07
- link base_link: geometry collision mesh filename=file:///home/peter/ros2_ws/install/mini_pupper_description/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; visual mesh filename=file:///home/peter/ros2_ws/install/mini_pupper_description/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
- link lb1: mass 0.00025 -> 0.025; geometry collision mesh filename=file:///home/peter/ros2_ws/install/mini_pupper_description/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; visual mesh filename=file:///home/peter/ros2_ws/install/mini_pupper_description/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
- link lb2: mass 0.00125 -> 0.0125; geometry collision mesh filename=file:///home/peter/ros2_ws/install/mini_pupper_description/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; visual mesh filename=file:///home/peter/ros2_ws/install/mini_pupper_description/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
- link lb3: mass 0.000625 -> 0.00625; geometry collision mesh filename=file:///home/peter/ros2_ws/install/mini_pupper_description/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; visual mesh filename=file:///home/peter/ros2_ws/install/mini_pupper_description/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
- link lbfoot: mass 0.000625 -> 0.00625; geometry collision mesh filename=file:///home/peter/ros2_ws/install/mini_pupper_description/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; visual mesh filename=file:///home/peter/ros2_ws/install/mini_pupper_description/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
- link lf1: mass 0.0025 -> 0.025; geometry collision mesh filename=file:///home/peter/ros2_ws/install/mini_pupper_description/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; visual mesh filename=file:///home/peter/ros2_ws/install/mini_pupper_description/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
- link lf2: mass 0.00125 -> 0.0125; geometry collision mesh filename=file:///home/peter/ros2_ws/install/mini_pupper_description/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; visual mesh filename=file:///home/peter/ros2_ws/install/mini_pupper_description/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
- link lf3: mass 0.000625 -> 0.00625; geometry collision mesh filename=file:///home/peter/ros2_ws/install/mini_pupper_description/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; visual mesh filename=file:///home/peter/ros2_ws/install/mini_pupper_description/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
- link lffoot: mass 0.000625 -> 0.00625; geometry collision mesh filename=file:///home/peter/ros2_ws/install/mini_pupper_description/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; visual mesh filename=file:///home/peter/ros2_ws/install/mini_pupper_description/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
- link lpb1: geometry collision mesh filename=file:///home/peter/ros2_ws/install/mini_pupper_description/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; visual mesh filename=file:///home/peter/ros2_ws/install/mini_pupper_description/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
- link lpb2: geometry collision mesh filename=file:///home/peter/ros2_ws/install/mini_pupper_description/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; visual mesh filename=file:///home/peter/ros2_ws/install/mini_pupper_description/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
- link lpf1: geometry collision mesh filename=file:///home/peter/ros2_ws/install/mini_pupper_description/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; visual mesh filename=file:///home/peter/ros2_ws/install/mini_pupper_description/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
- link lpf2: geometry collision mesh filename=file:///home/peter/ros2_ws/install/mini_pupper_description/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; visual mesh filename=file:///home/peter/ros2_ws/install/mini_pupper_description/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
- link rb1: mass 0.0025 -> 0.025; geometry collision mesh filename=file:///home/peter/ros2_ws/install/mini_pupper_description/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; visual mesh filename=file:///home/peter/ros2_ws/install/mini_pupper_description/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
- link rb2: mass 0.00125 -> 0.0125; geometry collision mesh filename=file:///home/peter/ros2_ws/install/mini_pupper_description/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; visual mesh filename=file:///home/peter/ros2_ws/install/mini_pupper_description/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
- link rb3: mass 0.000625 -> 0.00625; geometry collision mesh filename=file:///home/peter/ros2_ws/install/mini_pupper_description/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; visual mesh filename=file:///home/peter/ros2_ws/install/mini_pupper_description/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
- link rbfoot: mass 0.000625 -> 0.00625; geometry collision mesh filename=file:///home/peter/ros2_ws/install/mini_pupper_description/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; visual mesh filename=file:///home/peter/ros2_ws/install/mini_pupper_description/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
- link rf1: mass 0.0025 -> 0.025; geometry collision mesh filename=file:///home/peter/ros2_ws/install/mini_pupper_description/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; visual mesh filename=file:///home/peter/ros2_ws/install/mini_pupper_description/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
- link rf2: mass 0.00125 -> 0.0125; geometry collision mesh filename=file:///home/peter/ros2_ws/install/mini_pupper_description/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; visual mesh filename=file:///home/peter/ros2_ws/install/mini_pupper_description/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
- link rf3: mass 0.000625 -> 0.00625; geometry collision mesh filename=file:///home/peter/ros2_ws/install/mini_pupper_description/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; visual mesh filename=file:///home/peter/ros2_ws/install/mini_pupper_description/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
- link rffoot: mass 0.000625 -> 0.00625; geometry collision mesh filename=file:///home/peter/ros2_ws/install/mini_pupper_description/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; visual mesh filename=file:///home/peter/ros2_ws/install/mini_pupper_description/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
- link rpb1: geometry collision mesh filename=file:///home/peter/ros2_ws/install/mini_pupper_description/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; visual mesh filename=file:///home/peter/ros2_ws/install/mini_pupper_description/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
- link rpb2: geometry collision mesh filename=file:///home/peter/ros2_ws/install/mini_pupper_description/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; visual mesh filename=file:///home/peter/ros2_ws/install/mini_pupper_description/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
- link rpf1: geometry collision mesh filename=file:///home/peter/ros2_ws/install/mini_pupper_description/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; visual mesh filename=file:///home/peter/ros2_ws/install/mini_pupper_description/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
- link rpf2: geometry collision mesh filename=file:///home/peter/ros2_ws/install/mini_pupper_description/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; visual mesh filename=file:///home/peter/ros2_ws/install/mini_pupper_description/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
- link yellow_plate: mass 0.002 -> 0.03; geometry collision mesh filename=file:///home/peter/ros2_ws/install/mini_pupper_description/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; visual mesh filename=file:///home/peter/ros2_ws/install/mini_pupper_description/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
Joints:
- removed joint camera_color_joint
- removed joint camera_color_optical_joint
- removed joint camera_depth_joint
- removed joint camera_depth_optical_joint
- removed joint camera_infra1_joint
- removed joint camera_infra1_optical_joint
- removed joint camera_infra2_joint
- removed joint camera_infra2_optical_joint
- removed joint camera_joint
- removed joint camera_link_joint
- joint base_lb1: limit lower=-3.14 upper=3.14 effort=50 velocity=15 -> lower=-3.14 upper=3.14 effort=5 velocity=1.5
- joint base_lf1: limit lower=-3.14 upper=3.14 effort=50 velocity=15 -> lower=-3.14 upper=3.14 effort=5 velocity=1.5
- joint base_lidar: child lidar -> lidar_link
- joint base_rb1: limit lower=-3.14 upper=3.14 effort=50 velocity=15 -> lower=-3.14 upper=3.14 effort=5 velocity=1.5
- joint base_rf1: limit lower=-3.14 upper=3.14 effort=50 velocity=15 -> lower=-3.14 upper=3.14 effort=5 velocity=1.5
- joint lb1_lb2: limit lower=-3.14 upper=3.14 effort=50 velocity=15 -> lower=-3.14 upper=3.14 effort=5 velocity=1.5
- joint lb2_lb3: limit lower=-3.14 upper=3.14 effort=50 velocity=15 -> lower=-3.14 upper=3.14 effort=5 velocity=1.5
- joint lf1_lf2: limit lower=-3.14 upper=3.14 effort=50 velocity=15 -> lower=-3.14 upper=3.14 effort=5 velocity=1.5
- joint lf2_lf3: limit lower=-3.14 upper=3.14 effort=50 velocity=15 -> lower=-3.14 upper=3.14 effort=5 velocity=1.5
- joint rb1_rb2: limit lower=-3.14 upper=3.14 effort=50 velocity=15 -> lower=-3.14 upper=3.14 effort=5 velocity=1.5
- joint rb2_rb3: limit lower=-3.14 upper=3.14 effort=50 velocity=15 -> lower=-3.14 upper=3.14 effort=5 velocity=1.5
- joint rf1_rf2: limit lower=-3.14 upper=3.14 effort=50 velocity=15 -> lower=-3.14 upper=3.14 effort=5 velocity=1.5
- joint rf2_rf3: limit lower=-3.14 upper=3.14 effort=50 velocity=15 -> lower=-3.14 upper=3.14 effort=5 velocity=1.5
