Commit message: use mp 1 legs

File: mini_pupper_2_description/urdf/mini_pupper_description.urdf.xacro (robot description, xacro)
@@ -49,5 +49,5 @@
     </inertial>
     <visual>
-      <origin xyz="-0.037299 -0.023495 -5.7e-05" rpy="0 0 0"/>
+      <origin xyz="0 0 0" rpy="0 0 0"/>
       <geometry>
         <mesh filename="file://$(find mini_pupper_2_description)/meshes/lf1.stl" scale="1 1 1"/>
@@ -56,5 +56,5 @@
     </visual>
     <collision>
-      <origin xyz="-0.037299 -0.023495 -5.7e-05" rpy="0 0 0"/>
+      <origin xyz="0 0 0" rpy="0 0 0"/>
       <geometry>
         <mesh filename="file://$(find mini_pupper_2_description)/meshes/lf1.stl" scale="1 1 1"/>
@@ -69,5 +69,5 @@
     </inertial>
     <visual>
-      <origin xyz="-0.052165 -0.041195 -5.7e-05" rpy="0 0 0"/>
+      <origin xyz="0 0 0" rpy="0 0 0"/>
       <geometry>
         <mesh filename="file://$(find mini_pupper_2_description)/meshes/lf2.stl" scale="1 1 1"/>
@@ -76,5 +76,5 @@
     </visual>
     <collision>
-      <origin xyz="-0.052165 -0.041195 -5.7e-05" rpy="0 0 0"/>
+      <origin xyz="0 0 0" rpy="0 0 0"/>
       <geometry>
         <mesh filename="file://$(find mini_pupper_2_description)/meshes/lf2.stl" scale="1 1 1"/>
@@ -89,5 +89,5 @@
     </inertial>
     <visual>
-      <origin xyz="-0.043476 -0.044195 0.049184" rpy="0 0 0"/>
+      <origin xyz="0 0 0" rpy="0 0 0"/>
       <geometry>
         <mesh filename="file://$(find mini_pupper_2_description)/meshes/lf3.stl" scale="1 1 1"/>
@@ -96,5 +96,5 @@
     </visual>
     <collision>
-      <origin xyz="-0.043476 -0.044195 0.049184" rpy="0 0 0"/>
+      <origin xyz="0 0 0" rpy="0 0 0"/>
       <geometry>
         <mesh filename="file://$(find mini_pupper_2_description)/meshes/lf3.stl" scale="1 1 1"/>
@@ -109,5 +109,5 @@
     </inertial>
     <visual>
-      <origin xyz="-0.037299 0.023505 -5.7e-05" rpy="0 0 0"/>
+      <origin xyz="0 0 0" rpy="0 0 0"/>
       <geometry>
         <mesh filename="file://$(find mini_pupper_2_description)/meshes/rf1.stl" scale="1 1 1"/>
@@ -116,5 +116,5 @@
     </visual>
     <collision>
-      <origin xyz="-0.037299 0.023505 -5.7e-05" rpy="0 0 0"/>
+      <origin xyz="0 0 0" rpy="0 0 0"/>
       <geometry>
         <mesh filename="file://$(find mini_pupper_2_description)/meshes/rf1.stl" scale="1 1 1"/>
@@ -129,5 +129,5 @@
     </inertial>
     <visual>
-      <origin xyz="-0.052165 0.040955 -5.7e-05" rpy="0 0 0"/>
+      <origin xyz="0 0 0" rpy="0 0 0"/>
       <geometry>
         <mesh filename="file://$(find mini_pupper_2_description)/meshes/rf2.stl" scale="1 1 1"/>
@@ -136,5 +136,5 @@
     </visual>
     <collision>
-      <origin xyz="-0.052165 0.040955 -5.7e-05" rpy="0 0 0"/>
+      <origin xyz="0 0 0" rpy="0 0 0"/>
       <geometry>
         <mesh filename="file://$(find mini_pupper_2_description)/meshes/rf2.stl" scale="1 1 1"/>
@@ -149,5 +149,5 @@
     </inertial>
     <visual>
-      <origin xyz="-0.043482 0.044205 0.049184" rpy="0 0 0"/>
+      <origin xyz="0 0 0" rpy="0 0 0"/>
       <geometry>
         <mesh filename="file://$(find mini_pupper_2_description)/meshes/rf3.stl" scale="1 1 1"/>
@@ -156,5 +156,5 @@
     </visual>
     <collision>
-      <origin xyz="-0.043482 0.044205 0.049184" rpy="0 0 0"/>
+      <origin xyz="0 0 0" rpy="0 0 0"/>
       <geometry>
         <mesh filename="file://$(find mini_pupper_2_description)/meshes/rf3.stl" scale="1 1 1"/>
@@ -169,5 +169,5 @@
     </inertial>
     <visual>
-      <origin xyz="0.042701 0.023505 -5.7e-05" rpy="0 0 0"/>
+      <origin xyz="0 0 0" rpy="0 0 0"/>
       <geometry>
         <mesh filename="file://$(find mini_pupper_2_description)/meshes/rb1.stl" scale="1 1 1"/>
@@ -176,5 +176,5 @@
     </visual>
     <collision>
-      <origin xyz="0.042701 0.023505 -5.7e-05" rpy="0 0 0"/>
+      <origin xyz="0 0 0" rpy="0 0 0"/>
       <geometry>
         <mesh filename="file://$(find mini_pupper_2_description)/meshes/rb1.stl" scale="1 1 1"/>
@@ -189,5 +189,5 @@
     </inertial>
     <visual>
-      <origin xyz="0.068367 0.040955 -5.7e-05" rpy="0 0 0"/>
+      <origin xyz="0 0 0" rpy="0 0 0"/>
       <geometry>
         <mesh filename="file://$(find mini_pupper_2_description)/meshes/rb2.stl" scale="1 1 1"/>
@@ -196,5 +196,5 @@
     </visual>
     <collision>
-      <origin xyz="0.068367 0.040955 -5.7e-05" rpy="0 0 0"/>
+      <origin xyz="0 0 0" rpy="0 0 0"/>
       <geometry>
         <mesh filename="file://$(find mini_pupper_2_description)/meshes/rb2.stl" scale="1 1 1"/>
@@ -209,5 +209,5 @@
     </inertial>
     <visual>
-      <origin xyz="0.077049 0.044205 0.049184" rpy="0 0 0"/>
+      <origin xyz="0 0 0" rpy="0 0 0"/>
       <geometry>
         <mesh filename="file://$(find mini_pupper_2_description)/meshes/rb3.stl" scale="1 1 1"/>
@@ -216,5 +216,5 @@
     </visual>
     <collision>
-      <origin xyz="0.077049 0.044205 0.049184" rpy="0 0 0"/>
+      <origin xyz="0 0 0" rpy="0 0 0"/>
       <geometry>
         <mesh filename="file://$(find mini_pupper_2_description)/meshes/rb3.stl" scale="1 1 1"/>
@@ -229,5 +229,5 @@
     </inertial>
     <visual>
-      <origin xyz="0.042701 -0.023495 -5.7e-05" rpy="0 0 0"/>
+      <origin xyz="0 0 0" rpy="0 0 0"/>
       <geometry>
         <mesh filename="file://$(find mini_pupper_2_description)/meshes/lb1.stl" scale="1 1 1"/>
@@ -236,5 +236,5 @@
     </visual>
     <collision>
-      <origin xyz="0.042701 -0.023495 -5.7e-05" rpy="0 0 0"/>
+      <origin xyz="0 0 0" rpy="0 0 0"/>
       <geometry>
         <mesh filename="file://$(find mini_pupper_2_description)/meshes/lb1.stl" scale="1 1 1"/>
@@ -249,5 +249,5 @@
     </inertial>
     <visual>
-      <origin xyz="0.068367 -0.041195 -5.7e-05" rpy="0 0 0"/>
+      <origin xyz="0 0 0" rpy="0 0 0"/>
       <geometry>
         <mesh filename="file://$(find mini_pupper_2_description)/meshes/lb2.stl" scale="1 1 1"/>
@@ -256,5 +256,5 @@
     </visual>
     <collision>
-      <origin xyz="0.068367 -0.041195 -5.7e-05" rpy="0 0 0"/>
+      <origin xyz="0 0 0" rpy="0 0 0"/>
       <geometry>
         <mesh filename="file://$(find mini_pupper_2_description)/meshes/lb2.stl" scale="1 1 1"/>
@@ -269,5 +269,5 @@
     </inertial>
     <visual>
-      <origin xyz="0.077049 -0.044195 0.049184" rpy="0 0 0"/>
+      <origin xyz="0 0 0" rpy="0 0 0"/>
       <geometry>
         <mesh filename="file://$(find mini_pupper_2_description)/meshes/lb3.stl" scale="1 1 1"/>
@@ -276,5 +276,5 @@
     </visual>
     <collision>
-      <origin xyz="0.077049 -0.044195 0.049184" rpy="0 0 0"/>
+      <origin xyz="0 0 0" rpy="0 0 0"/>
       <geometry>
         <mesh filename="file://$(find mini_pupper_2_description)/meshes/lb3.stl" scale="1 1 1"/>
@@ -369,5 +369,5 @@
     </inertial>
     <visual>
-      <origin xyz="-0.068108 0.047955 0.103614" rpy="0 0 0"/>
+      <origin xyz="0 0 0" rpy="0 0 0"/>
       <geometry>
         <mesh filename="file://$(find mini_pupper_2_description)/meshes/rffoot.stl" scale="1 1 1"/>
@@ -376,5 +376,5 @@
     </visual>
     <collision>
-      <origin xyz="-0.068108 0.047955 0.103614" rpy="0 0 0"/>
+      <origin xyz="0 0 0" rpy="0 0 0"/>
       <geometry>
         <mesh filename="file://$(find mini_pupper_2_description)/meshes/rffoot.stl" scale="1 1 1"/>
@@ -389,5 +389,5 @@
     </inertial>
     <visual>
-      <origin xyz="0.052424 0.047955 0.103614" rpy="0 0 0"/>
+      <origin xyz="0 0 0" rpy="0 0 0"/>
       <geometry>
         <mesh filename="file://$(find mini_pupper_2_description)/meshes/rbfoot.stl" scale="1 1 1"/>
@@ -396,5 +396,5 @@
     </visual>
     <collision>
-      <origin xyz="0.052424 0.047955 0.103614" rpy="0 0 0"/>
+      <origin xyz="0 0 0" rpy="0 0 0"/>
       <geometry>
         <mesh filename="file://$(find mini_pupper_2_description)/meshes/rbfoot.stl" scale="1 1 1"/>
@@ -409,5 +409,5 @@
     </inertial>
     <visual>
-      <origin xyz="0.052424 -0.047945 0.103614" rpy="0 0 0"/>
+      <origin xyz="0 0 0" rpy="0 0 0"/>
       <geometry>
         <mesh filename="file://$(find mini_pupper_2_description)/meshes/lbfoot.stl" scale="1 1 1"/>
@@ -416,5 +416,5 @@
     </visual>
     <collision>
-      <origin xyz="0.052424 -0.047945 0.103614" rpy="0 0 0"/>
+      <origin xyz="0 0 0" rpy="0 0 0"/>
       <geometry>
         <mesh filename="file://$(find mini_pupper_2_description)/meshes/lbfoot.stl" scale="1 1 1"/>
@@ -429,5 +429,5 @@
     </inertial>
     <visual>
-      <origin xyz="-0.068108 -0.047945 0.103614" rpy="0 0 0"/>
+      <origin xyz="0 0 0" rpy="0 0 0"/>
       <geometry>
         <mesh filename="file://$(find mini_pupper_2_description)/meshes/lffoot.stl" scale="1 1 1"/>
@@ -436,5 +436,5 @@
     </visual>
     <collision>
-      <origin xyz="-0.068108 -0.047945 0.103614" rpy="0 0 0"/>
+      <origin xyz="0 0 0" rpy="0 0 0"/>
       <geometry>
         <mesh filename="file://$(find mini_pupper_2_description)/meshes/lffoot.stl" scale="1 1 1"/>
@@ -449,5 +449,5 @@
     </inertial>
     <visual>
-      <origin xyz="-0.071565 -0.037995 -0.013057" rpy="0 0 0"/>
+      <origin xyz="0 0 0" rpy="0 0 0"/>
       <geometry>
         <mesh filename="file://$(find mini_pupper_2_description)/meshes/lpf1.stl" scale="1 1 1"/>
@@ -456,5 +456,5 @@
     </visual>
     <collision>
-      <origin xyz="-0.071565 -0.037995 -0.013057" rpy="0 0 0"/>
+      <origin xyz="0 0 0" rpy="0 0 0"/>
       <geometry>
         <mesh filename="file://$(find mini_pupper_2_description)/meshes/lpf1.stl" scale="1 1 1"/>
@@ -469,5 +469,5 @@
     </inertial>
     <visual>
-      <origin xyz="0.048967 -0.037995 -0.013057" rpy="0 0 0"/>
+      <origin xyz="0 0 0" rpy="0 0 0"/>
       <geometry>
         <mesh filename="file://$(find mini_pupper_2_description)/meshes/lpb1.stl" scale="1 1 1"/>
@@ -476,5 +476,5 @@
     </visual>
     <collision>
-      <origin xyz="0.048967 -0.037995 -0.013057" rpy="0 0 0"/>
+      <origin xyz="0 0 0" rpy="0 0 0"/>
       <geometry>
         <mesh filename="file://$(find mini_pupper_2_description)/meshes/lpb1.stl" scale="1 1 1"/>
@@ -489,5 +489,5 @@
     </inertial>
     <visual>
-      <origin xyz="-0.071565 0.038005 -0.013057" rpy="0 0 0"/>
+      <origin xyz="0 0 0" rpy="0 0 0"/>
       <geometry>
         <mesh filename="file://$(find mini_pupper_2_description)/meshes/rpf1.stl" scale="1 1 1"/>
@@ -496,5 +496,5 @@
     </visual>
     <collision>
-      <origin xyz="-0.071565 0.038005 -0.013057" rpy="0 0 0"/>
+      <origin xyz="0 0 0" rpy="0 0 0"/>
       <geometry>
         <mesh filename="file://$(find mini_pupper_2_description)/meshes/rpf1.stl" scale="1 1 1"/>
@@ -509,5 +509,5 @@
     </inertial>
     <visual>
-      <origin xyz="0.048967 0.037998 -0.013064" rpy="0 0 0"/>
+      <origin xyz="0 0 0" rpy="0 0 0"/>
       <geometry>
         <mesh filename="file://$(find mini_pupper_2_description)/meshes/rpb1.stl" scale="1 1 1"/>
@@ -516,5 +516,5 @@
     </visual>
     <collision>
-      <origin xyz="0.048967 0.037998 -0.013064" rpy="0 0 0"/>
+      <origin xyz="0 0 0" rpy="0 0 0"/>
       <geometry>
         <mesh filename="file://$(find mini_pupper_2_description)/meshes/rpb1.stl" scale="1 1 1"/>
@@ -529,5 +529,5 @@
     </inertial>
     <visual>
-      <origin xyz="-0.048863 -0.044195 0.018654" rpy="0 0 0"/>
+      <origin xyz="0 0 0" rpy="0 0 0"/>
       <geometry>
         <mesh filename="file://$(find mini_pupper_2_description)/meshes/lpf2.stl" scale="1 1 1"/>
@@ -536,5 +536,5 @@
     </visual>
     <collision>
-      <origin xyz="-0.048863 -0.044195 0.018654" rpy="0 0 0"/>
+      <origin xyz="0 0 0" rpy="0 0 0"/>
       <geometry>
         <mesh filename="file://$(find mini_pupper_2_description)/meshes/lpf2.stl" scale="1 1 1"/>
@@ -549,5 +549,5 @@
     </inertial>
     <visual>
-      <origin xyz="0.071666 -0.044195 0.018655" rpy="0 0 0"/>
+      <origin xyz="0 0 0" rpy="0 0 0"/>
       <geometry>
         <mesh filename="file://$(find mini_pupper_2_description)/meshes/lpb2.stl" scale="1 1 1"/>
@@ -556,5 +556,5 @@
     </visual>
     <collision>
-      <origin xyz="0.071666 -0.044195 0.018655" rpy="0 0 0"/>
+      <origin xyz="0 0 0" rpy="0 0 0"/>
       <geometry>
         <mesh filename="file://$(find mini_pupper_2_description)/meshes/lpb2.stl" scale="1 1 1"/>
@@ -569,5 +569,5 @@
     </inertial>
     <visual>
-      <origin xyz="-0.048865 0.044205 0.018655" rpy="0 0 0"/>
+      <origin xyz="0 0 0" rpy="0 0 0"/>
       <geometry>
         <mesh filename="file://$(find mini_pupper_2_description)/meshes/rpf2.stl" scale="1 1 1"/>
@@ -576,5 +576,5 @@
     </visual>
     <collision>
-      <origin xyz="-0.048865 0.044205 0.018655" rpy="0 0 0"/>
+      <origin xyz="0 0 0" rpy="0 0 0"/>
       <geometry>
         <mesh filename="file://$(find mini_pupper_2_description)/meshes/rpf2.stl" scale="1 1 1"/>
@@ -589,5 +589,5 @@
     </inertial>
     <visual>
-      <origin xyz="0.071666 0.044215 0.018644" rpy="0 0 0"/>
+      <origin xyz="0 0 0" rpy="0 0 0"/>
       <geometry>
         <mesh filename="file://$(find mini_pupper_2_description)/meshes/rpb2.stl" scale="1 1 1"/>
@@ -596,5 +596,5 @@
     </visual>
     <collision>
-      <origin xyz="0.071666 0.044215 0.018644" rpy="0 0 0"/>
+      <origin xyz="0 0 0" rpy="0 0 0"/>
       <geometry>
         <mesh filename="file://$(find mini_pupper_2_description)/meshes/rpb2.stl" scale="1 1 1"/>
@@ -629,5 +629,5 @@
   </joint>
   <joint name="base_lf1" type="revolute">
-    <origin xyz="0.037299 0.023495 5.7e-05" rpy="0 0 0"/>
+    <origin xyz="0.05 0.0235 0.0" rpy="0 0 0"/>
     <parent link="base_link"/>
     <child link="lf1"/>
@@ -636,5 +636,5 @@
   </joint>
   <joint name="lf1_lf2" type="revolute">
-    <origin xyz="0.014866 0.0177 0.0" rpy="0 0 0"/>
+    <origin xyz="-4E-05 0.0197 0" rpy="0 0 0"/>
     <parent link="lf1"/>
     <child link="lf2"/>
@@ -643,5 +643,5 @@
   </joint>
   <joint name="lf2_lf3" type="revolute">
-    <origin xyz="-0.008689 0.003 -0.04924" rpy="0 0 0"/>
+    <origin xyz="0 0.00475 -0.05" rpy="0 0 0"/>
     <parent link="lf2"/>
     <child link="lf3"/>
@@ -650,5 +650,5 @@
   </joint>
   <joint name="base_rf1" type="revolute">
-    <origin xyz="0.037299 -0.023505 5.7e-05" rpy="0 0 0"/>
+    <origin xyz="0.05 -0.0235 0.0" rpy="0 0 0"/>
     <parent link="base_link"/>
     <child link="rf1"/>
@@ -657,5 +657,5 @@
   </joint>
   <joint name="rf1_rf2" type="revolute">
-    <origin xyz="0.014866 -0.0177 0.0" rpy="0 0 0"/>
+    <origin xyz="-4E-05 -0.0197 0" rpy="0 0 0"/>
     <parent link="rf1"/>
     <child link="rf2"/>
@@ -664,5 +664,5 @@
   </joint>
   <joint name="rf2_rf3" type="revolute">
-    <origin xyz="-0.008683 -0.003 -0.049241" rpy="0 0 0"/>
+    <origin xyz="0 -0.00475 -0.05" rpy="0 0 0"/>
     <parent link="rf2"/>
     <child link="rf3"/>
@@ -671,5 +671,5 @@
   </joint>
   <joint name="base_rb1" type="revolute">
-    <origin xyz="-0.042701 -0.023505 5.7e-05" rpy="0 0 0"/>
+    <origin xyz="-0.066 -0.0235 0.0" rpy="0 0 0"/>
     <parent link="base_link"/>
     <child link="rb1"/>
@@ -678,5 +678,5 @@
   </joint>
   <joint name="rb1_rb2" type="revolute">
-    <origin xyz="-0.025666 -0.0177 9e-06" rpy="0 0 0"/>
+    <origin xyz="-4E-05 -0.0197 0" rpy="0 0 0"/>
     <parent link="rb1"/>
     <child link="rb2"/>
@@ -685,5 +685,5 @@
   </joint>
   <joint name="rb2_rb3" type="revolute">
-    <origin xyz="-0.008682 -0.003027 -0.049239" rpy="0 0 0"/>
+    <origin xyz="0 -0.00475 -0.05" rpy="0 0 0"/>
     <parent link="rb2"/>
     <child link="rb3"/>
@@ -692,5 +692,5 @@
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
Commit message: Fix colors

File: mini_pupper_2_description/urdf/mini_pupper_description.urdf.xacro (robot description, xacro)
@@ -866,6 +866,18 @@
     <material>Gazebo/FlatBlack</material>
   </gazebo>
+  <gazebo reference="Board_PCB">
+    <material>Gazebo/FlatBlack</material>
+  </gazebo>
+  <gazebo reference="Body_front">
+    <material>Gazebo/Yellow</material>
+  </gazebo>
   <gazebo reference="Shell_Side">
     <material>Gazebo/Yellow</material>
+  </gazebo>
+  <gazebo reference="Board_connectors_1">
+    <material>Gazebo/Orange</material>
+  </gazebo>
+  <gazebo reference="Board_connectors_2">
+    <material>Gazebo/White</material>
   </gazebo>
   <gazebo reference="lf1">

Commit message: Add lidar link
This reverts commit 640768795b3951dca8fa43c07acfa10d20ee931d.

mini_pupper_2_description/urdf/mini_pupper_description.urdf.xacro

File: mini_pupper_2_description/urdf/mini_pupper_description.urdf.xacro (robot description, xacro)
@@ -362,4 +362,37 @@
     </collision>
   </link>
+  <link
+    name="lidar_link">
+    <inertial>
+      <origin
+        xyz="1.56706411611127E-05 -5.16565672073303E-13 -0.0191835739440227"
+        rpy="0 0 -1.57" />
+      <mass value="0.0001" />
+      <inertia
+        ixx="8.74731426973985E-06"
+        ixy="-6.66781590704156E-08"
+        ixz="1.89196685410159E-11"
+        iyy="8.70097486591694E-06"
+        iyz="-1.13397577799603E-17"
+        izz="9.98821295317784E-06" />
+    </inertial>
+    <visual>
+      <origin xyz="0 0 0" rpy="0 0 -1.57"/>
+      <geometry>
+        <mesh
+          filename="file://$(find mini_pupper_2_description)/meshes/lidar.stl" />
+      </geometry>
+      <material name="">
+        <color rgba="0.2 0.2 0.2 1" />
+      </material>
+    </visual>
+    <collision>
+      <origin xyz="0 0 0" rpy="0 0 -1.57" />
+      <geometry>
+        <mesh
+          filename="file://$(find mini_pupper_2_description)/meshes/lidar.stl" />
+      </geometry>
+    </collision>
+  </link>
   <link name="rffoot">
     <inertial>
@@ -731,4 +764,9 @@
     <parent link="Board_PCB"/>
     <child link="Board_connectors_2"/>
+  </joint>
+  <joint name="pcb_lidar" type="fixed">
+    <origin xyz="0.009 0.024 0.042" rpy="0 0 1.57" />
+    <parent link="Board_PCB" />
+    <child link="lidar_link" />
   </joint>
   <joint name="rf3_foot" type="fixed">
@@ -1049,5 +1087,5 @@
     <material>Gazebo/FlatBlack</material>
   </gazebo>
-  <!-- <gazebo reference="lidar_link">
+  <gazebo reference="lidar_link">
     <material>Gazebo/FlatBlack</material>
     <sensor type="ray" name="lidar">
@@ -1081,9 +1119,8 @@
         </ros>
         <output_type>sensor_msgs/LaserScan</output_type>
-        <frame_name>lidar_link</frame_name> -->
-        <!--min_intensity>100.0</min_intensity-->
-      <!-- </plugin>
+        <frame_name>lidar_link</frame_name>
+      </plugin>
     </sensor>
-  </gazebo> -->
+  </gazebo>
   <gazebo>
     <plugin filename="libgazebo_ros_p3d.so" name="p3d_base_controller">
