Commit message: Added new links with correct orientation and adjusted inertia settings accordingly

File: mini_pupper_2_description/urdf/mini_pupper_description.urdf.xacro (robot description, xacro)
@@ -16,8 +16,7 @@
   <!-- Feet - lffoot, rffoot, lbfoot, rbfoot -->
   <xacro:property name="feet_weight" value="0.001405" />
-  <!-- -0.004982788451759437 -2.855826620254409e-07 0.006488368014064216 -->
   <!-- COM-Y: 0.00025 -->
   <xacro:property name="feet_centre_of_mass"
-                  value="-0.014 0.00025 0.002488" />
+                  value="-0.002463 0.0 0.007802" />
   <link name="base_link">
     <visual>
@@ -49,5 +48,5 @@
     </inertial>
     <visual>
-      <origin xyz="0 0 0" rpy="0 0 0"/>
+      <origin xyz="-0.037299 -0.023495 -5.7e-05" rpy="0 0 0"/>
       <geometry>
         <mesh filename="file://$(find mini_pupper_2_description)/meshes/lf1.stl" scale="1 1 1"/>
@@ -56,5 +55,5 @@
     </visual>
     <collision>
-      <origin xyz="0 0 0" rpy="0 0 0"/>
+      <origin xyz="-0.037299 -0.023495 -5.7e-05" rpy="0 0 0"/>
       <geometry>
         <mesh filename="file://$(find mini_pupper_2_description)/meshes/lf1.stl" scale="1 1 1"/>
@@ -64,10 +63,10 @@
   <link name="lf2">
     <inertial>
-      <origin xyz="-0.003174 0.000986 -0.017984" rpy="0 0 0"/>
+      <origin xyz="0.0 0.000986 -0.018260" rpy="0 0 0"/>
       <mass value="${lnkgrp2_weight}"/>
-      <inertia ixx="0.462154e-6" iyy="0.481174e-6" izz="26.893e-9" ixy="3.117e-9" iyz="17.662e-9" ixz="-79.269e-9"/>
-    </inertial>
-    <visual>
-      <origin xyz="0 0 0" rpy="0 0 0"/>
+      <inertia ixx="0.476141e-6" iyy="0.481174e-6" izz="12.925e-9" ixy="0.002e-9" iyz="17.935e-9" ixz="-0.055e-9"/>
+    </inertial>
+    <visual>
+      <origin xyz="-0.052165 -0.041195 -5.7e-05" rpy="0 0 0"/>
       <geometry>
         <mesh filename="file://$(find mini_pupper_2_description)/meshes/lf2.stl" scale="1 1 1"/>
@@ -76,5 +75,5 @@
     </visual>
     <collision>
-      <origin xyz="0 0 0" rpy="0 0 0"/>
+      <origin xyz="-0.052165 -0.041195 -5.7e-05" rpy="0 0 0"/>
       <geometry>
         <mesh filename="file://$(find mini_pupper_2_description)/meshes/lf2.stl" scale="1 1 1"/>
@@ -84,10 +83,10 @@
   <link name="lf3">
     <inertial>
-      <origin xyz="0.006211 0.003456 -0.015014" rpy="0 0 0"/>
+      <origin xyz="0.000705 0.003455 -0.018260" rpy="0 0 0"/>
       <mass value="${lnkgrp3_weight}"/>
-      <inertia ixx="0.484471e-6" iyy="0.567615e-6" izz="91.813e-9" ixy="-2.101e-9" iyz="5.008e-9" ixz="0.20057e-6"/>
-    </inertial>
-    <visual>
-      <origin xyz="0 0 0" rpy="0 0 0"/>
+      <inertia ixx="0.567712e-6" iyy="0.567861e-6" izz="8.805e-9" ixy="-0.236e-9" iyz="5.435e-9" ixz="27.308e-9"/>
+    </inertial>
+    <visual>
+      <origin xyz="-0.052165 -0.044195 0.049943" rpy="0 0 0"/>
       <geometry>
         <mesh filename="file://$(find mini_pupper_2_description)/meshes/lf3.stl" scale="1 1 1"/>
@@ -96,5 +95,5 @@
     </visual>
     <collision>
-      <origin xyz="0 0 0" rpy="0 0 0"/>
+      <origin xyz="-0.052165 -0.044195 0.049943" rpy="0 0 0"/>
       <geometry>
         <mesh filename="file://$(find mini_pupper_2_description)/meshes/lf3.stl" scale="1 1 1"/>
@@ -109,5 +108,5 @@
     </inertial>
     <visual>
-      <origin xyz="0 0 0" rpy="0 0 0"/>
+      <origin xyz="-0.037299 0.023505 -5.7e-05" rpy="0 0 0"/>
       <geometry>
         <mesh filename="file://$(find mini_pupper_2_description)/meshes/rf1.stl" scale="1 1 1"/>
@@ -116,5 +115,5 @@
     </visual>
     <collision>
-      <origin xyz="0 0 0" rpy="0 0 0"/>
+      <origin xyz="-0.037299 0.023505 -5.7e-05" rpy="0 0 0"/>
       <geometry>
         <mesh filename="file://$(find mini_pupper_2_description)/meshes/rf1.stl" scale="1 1 1"/>
@@ -124,10 +123,10 @@
   <link name="rf2">
     <inertial>
-      <origin xyz="-0.003174 -0.000986 -0.017984" rpy="0 0 0"/>
+      <origin xyz="0.0 -0.000986 -0.018260" rpy="0 0 0"/>
       <mass value="${lnkgrp2_weight}"/>
-      <inertia ixx="0.462154e-6" iyy="0.481174e-6" izz="26.893e-9" ixy="-3.117e-9" iyz="-17.662e-9" ixz="-79.269e-9"/>
-    </inertial>
-    <visual>
-      <origin xyz="0 0 0" rpy="0 0 0"/>
+      <inertia ixx="0.476141e-6" iyy="0.481174e-6" izz="12.925e-9" ixy="-0.002e-9" iyz="-17.935e-9" ixz="-0.055e-9"/>
+    </inertial>
+    <visual>
+      <origin xyz="-0.052165 0.040955 -5.7e-05" rpy="0 0 0"/>
       <geometry>
         <mesh filename="file://$(find mini_pupper_2_description)/meshes/rf2.stl" scale="1 1 1"/>
@@ -136,5 +135,5 @@
     </visual>
     <collision>
-      <origin xyz="0 0 0" rpy="0 0 0"/>
+      <origin xyz="-0.052165 0.040955 -5.7e-05" rpy="0 0 0"/>
       <geometry>
         <mesh filename="file://$(find mini_pupper_2_description)/meshes/rf2.stl" scale="1 1 1"/>
@@ -144,10 +143,10 @@
   <link name="rf3">
     <inertial>
-      <origin xyz="0.006211 -0.003456 -0.015014" rpy="0 0 0"/>
+      <origin xyz="0.000705 -0.003455 -0.018260" rpy="0 0 0"/>
       <mass value="${lnkgrp3_weight}"/>
-      <inertia ixx="0.484471e-6" iyy="0.567615e-06" izz="91.813e-9" ixy="2.101e-9" iyz="-5.008e-9" ixz="0.20057e-6"/>
-    </inertial>
-    <visual>
-      <origin xyz="0 0 0" rpy="0 0 0"/>
+      <inertia ixx="0.567712e-6" iyy="0.567861e-6" izz="8.805e-9" ixy="0.236e-9" iyz="-5.435e-9" ixz="27.308e-9"/>
+    </inertial>
+    <visual>
+      <origin xyz="-0.052165 0.044205 0.049943" rpy="0 0 0"/>
       <geometry>
         <mesh filename="file://$(find mini_pupper_2_description)/meshes/rf3.stl" scale="1 1 1"/>
@@ -156,5 +155,5 @@
     </visual>
     <collision>
-      <origin xyz="0 0 0" rpy="0 0 0"/>
+      <origin xyz="-0.052165 0.044205 0.049943" rpy="0 0 0"/>
       <geometry>
         <mesh filename="file://$(find mini_pupper_2_description)/meshes/rf3.stl" scale="1 1 1"/>
@@ -169,5 +168,5 @@
     </inertial>
     <visual>
-      <origin xyz="0 0 0" rpy="0 0 0"/>
+      <origin xyz="0.042701 0.023505 -5.7e-05" rpy="0 0 0"/>
       <geometry>
         <mesh filename="file://$(find mini_pupper_2_description)/meshes/rb1.stl" scale="1 1 1"/>
@@ -176,5 +175,5 @@
     </visual>
     <collision>
-      <origin xyz="0 0 0" rpy="0 0 0"/>
+      <origin xyz="0.042701 0.023505 -5.7e-05" rpy="0 0 0"/>
       <geometry>
         <mesh filename="file://$(find mini_pupper_2_description)/meshes/rb1.stl" scale="1 1 1"/>
@@ -184,10 +183,10 @@
   <link name="rb2">
     <inertial>
-      <origin xyz="-0.003174 -0.000986 -0.017984" rpy="0 0 0"/>
+      <origin xyz="0.0 -0.000986 -0.018260" rpy="0 0 0"/>
       <mass value="${lnkgrp2_weight}"/>
-      <inertia ixx="0.462154e-6" iyy="0.481174e-6" izz="26.893e-9" ixy="-3.117e-9" iyz="-17.662e-9" ixz="-79.269e-9"/>
-    </inertial>
-    <visual>
-      <origin xyz="0 0 0" rpy="0 0 0"/>
+      <inertia ixx="0.476141e-6" iyy="0.481174e-6" izz="12.925e-9" ixy="-0.002e-9" iyz="-17.935e-9" ixz="-0.055e-9"/>
+    </inertial>
+    <visual>
+      <origin xyz="0.068367 0.041205 -5.7e-05" rpy="0 0 0"/>
       <geometry>
         <mesh filename="file://$(find mini_pupper_2_description)/meshes/rb2.stl" scale="1 1 1"/>
@@ -196,5 +195,5 @@
     </visual>
     <collision>
-      <origin xyz="0 0 0" rpy="0 0 0"/>
+      <origin xyz="0.068367 0.041205 -5.7e-05" rpy="0 0 0"/>
       <geometry>
         <mesh filename="file://$(find mini_pupper_2_description)/meshes/rb2.stl" scale="1 1 1"/>
@@ -204,10 +203,10 @@
   <link name="rb3">
     <inertial>
-      <origin xyz="0.006211 -0.003456 -0.015014" rpy="0 0 0"/>
+      <origin xyz="0.000705 -0.003455 -0.018260" rpy="0 0 0"/>
       <mass value="${lnkgrp3_weight}"/>
-      <inertia ixx="0.484816e-6" iyy="0.567883e-06" izz="91.777e-9" ixy="2.212e-9" iyz="-5.34e-9" ixz="0.200564e-6"/>
-    </inertial>
-    <visual>
-      <origin xyz="0 0 0" rpy="0 0 0"/>
+      <inertia ixx="0.567712e-6" iyy="0.567861e-6" izz="8.805e-9" ixy="0.236e-9" iyz="-5.435e-9" ixz="27.308e-9"/>
+    </inertial>
+    <visual>
+      <origin xyz="0.068367 0.044205 0.049943" rpy="0 0 0"/>
       <geometry>
         <mesh filename="file://$(find mini_pupper_2_description)/meshes/rb3.stl" scale="1 1 1"/>
@@ -216,5 +215,5 @@
     </visual>
     <collision>
-      <origin xyz="0 0 0" rpy="0 0 0"/>
+      <origin xyz="0.068367 0.044205 0.049943" rpy="0 0 0"/>
       <geometry>
         <mesh filename="file://$(find mini_pupper_2_description)/meshes/rb3.stl" scale="1 1 1"/>
@@ -229,5 +228,5 @@
     </inertial>
     <visual>
-      <origin xyz="0 0 0" rpy="0 0 0"/>
+      <origin xyz="0.042701 -0.023495 -5.7e-05" rpy="0 0 0"/>
       <geometry>
         <mesh filename="file://$(find mini_pupper_2_description)/meshes/lb1.stl" scale="1 1 1"/>
@@ -236,5 +235,5 @@
     </visual>
     <collision>
-      <origin xyz="0 0 0" rpy="0 0 0"/>
+      <origin xyz="0.042701 -0.023495 -5.7e-05" rpy="0 0 0"/>
       <geometry>
         <mesh filename="file://$(find mini_pupper_2_description)/meshes/lb1.stl" scale="1 1 1"/>
@@ -244,10 +243,10 @@
   <link name="lb2">
     <inertial>
-      <origin xyz="-0.003174 0.000986 -0.017984" rpy="0 0 0"/>
+      <origin xyz="0.0 0.000986 -0.018260" rpy="0 0 0"/>
       <mass value="${lnkgrp2_weight}"/>
-      <inertia ixx="0.462154e-6" iyy="0.481174e-6" izz="26.893e-9" ixy="3.117e-9" iyz="17.662e-9" ixz="-79.269e-9"/>
-    </inertial>
-    <visual>
-      <origin xyz="0 0 0" rpy="0 0 0"/>
+      <inertia ixx="0.476141e-6" iyy="0.481174e-6" izz="12.925e-9" ixy="0.002e-9" iyz="17.935e-9" ixz="-0.055e-9"/>
+    </inertial>
+    <visual>
+      <origin xyz="0.068367 -0.041195 -5.7e-05" rpy="0 0 0"/>
       <geometry>
         <mesh filename="file://$(find mini_pupper_2_description)/meshes/lb2.stl" scale="1 1 1"/>
@@ -256,5 +255,5 @@
     </visual>
     <collision>
-      <origin xyz="0 0 0" rpy="0 0 0"/>
+      <origin xyz="0.068367 -0.041195 -5.7e-05" rpy="0 0 0"/>
       <geometry>
         <mesh filename="file://$(find mini_pupper_2_description)/meshes/lb2.stl" scale="1 1 1"/>
@@ -264,10 +263,10 @@
   <link name="lb3">
     <inertial>
-      <origin xyz="0.006211 0.003456 -0.015014" rpy="0 0 0"/>
+      <origin xyz="0.000705 0.003455 -0.018260" rpy="0 0 0"/>
       <mass value="${lnkgrp3_weight}"/>
-      <inertia ixx="0.484471e-6" iyy="0.567615e-06" izz="91.813e-9" ixy="-2.101e-9" iyz="5.008e-9" ixz="0.20057e-6"/>
-    </inertial>
-    <visual>
-      <origin xyz="0 0 0" rpy="0 0 0"/>
+      <inertia ixx="0.567712e-6" iyy="0.567861e-6" izz="8.805e-9" ixy="-0.236e-9" iyz="5.435e-9" ixz="27.308e-9"/>
+    </inertial>
+    <visual>
+      <origin xyz="0.068367 -0.044195 0.049943" rpy="0 0 0"/>
       <geometry>
         <mesh filename="file://$(find mini_pupper_2_description)/meshes/lb3.stl" scale="1 1 1"/>
@@ -276,5 +275,5 @@
     </visual>
     <collision>
-      <origin xyz="0 0 0" rpy="0 0 0"/>
+      <origin xyz="0.068367 -0.044195 0.049943" rpy="0 0 0"/>
       <geometry>
         <mesh filename="file://$(find mini_pupper_2_description)/meshes/lb3.stl" scale="1 1 1"/>
@@ -369,5 +368,5 @@
     </inertial>
     <visual>
-      <origin xyz="0 0 0" rpy="0 0 0"/>
+      <origin xyz="-0.056689 0.047955 0.109514" rpy="0 0 0"/>
       <geometry>
         <mesh filename="file://$(find mini_pupper_2_description)/meshes/rffoot.stl" scale="1 1 1"/>
@@ -376,5 +375,5 @@
     </visual>
     <collision>
-      <origin xyz="0 0 0" rpy="0 0 0"/>
+      <origin xyz="-0.056689 0.047955 0.109514" rpy="0 0 0"/>
       <geometry>
         <mesh filename="file://$(find mini_pupper_2_description)/meshes/rffoot.stl" scale="1 1 1"/>
@@ -389,5 +388,5 @@
     </inertial>
     <visual>
-      <origin xyz="0 0 0" rpy="0 0 0"/>
+      <origin xyz="0.063843 0.047955 0.109514" rpy="0 0 0"/>
       <geometry>
         <mesh filename="file://$(find mini_pupper_2_description)/meshes/rbfoot.stl" scale="1 1 1"/>
@@ -396,5 +395,5 @@
     </visual>
     <collision>
-      <origin xyz="0 0 0" rpy="0 0 0"/>
+      <origin xyz="0.063843 0.047955 0.109514" rpy="0 0 0"/>
       <geometry>
         <mesh filename="file://$(find mini_pupper_2_description)/meshes/rbfoot.stl" scale="1 1 1"/>
@@ -409,5 +408,5 @@
     </inertial>
     <visual>
-      <origin xyz="0 0 0" rpy="0 0 0"/>
+      <origin xyz="0.063843 -0.047955 0.109514" rpy="0 0 0"/>
       <geometry>
         <mesh filename="file://$(find mini_pupper_2_description)/meshes/lbfoot.stl" scale="1 1 1"/>
@@ -416,5 +415,5 @@
     </visual>
     <collision>
-      <origin xyz="0 0 0" rpy="0 0 0"/>
+      <origin xyz="0.063843 -0.047955 0.109514" rpy="0 0 0"/>
       <geometry>
         <mesh filename="file://$(find mini_pupper_2_description)/meshes/lbfoot.stl" scale="1 1 1"/>
@@ -429,5 +428,5 @@
     </inertial>
     <visual>
-      <origin xyz="0 0 0" rpy="0 0 0"/>
+      <origin xyz="-0.056689 -0.047955 0.109514" rpy="0 0 0"/>
       <geometry>
         <mesh filename="file://$(find mini_pupper_2_description)/meshes/lffoot.stl" scale="1 1 1"/>
@@ -436,5 +435,5 @@
     </visual>
     <collision>
-      <origin xyz="0 0 0" rpy="0 0 0"/>
+      <origin xyz="-0.056689 -0.047955 0.109514" rpy="0 0 0"/>
       <geometry>
         <mesh filename="file://$(find mini_pupper_2_description)/meshes/lffoot.stl" scale="1 1 1"/>
@@ -449,5 +448,5 @@
     </inertial>
     <visual>
-      <origin xyz="0 0 0" rpy="0 0 0"/>
+      <origin xyz="-0.071565 -0.037995 -0.013057" rpy="0 0 0"/>
       <geometry>
         <mesh filename="file://$(find mini_pupper_2_description)/meshes/lpf1.stl" scale="1 1 1"/>
@@ -456,5 +455,5 @@
     </visual>
     <collision>
-      <origin xyz="0 0 0" rpy="0 0 0"/>
+      <origin xyz="-0.071565 -0.037995 -0.013057" rpy="0 0 0"/>
       <geometry>
         <mesh filename="file://$(find mini_pupper_2_description)/meshes/lpf1.stl" scale="1 1 1"/>
@@ -469,5 +468,5 @@
     </inertial>
     <visual>
-      <origin xyz="0 0 0" rpy="0 0 0"/>
+      <origin xyz="0.048967 -0.037995 -0.013057" rpy="0 0 0"/>
       <geometry>
         <mesh filename="file://$(find mini_pupper_2_description)/meshes/lpb1.stl" scale="1 1 1"/>
@@ -476,5 +475,5 @@
     </visual>
     <collision>
-      <origin xyz="0 0 0" rpy="0 0 0"/>
+      <origin xyz="0.048967 -0.037995 -0.013057" rpy="0 0 0"/>
       <geometry>
         <mesh filename="file://$(find mini_pupper_2_description)/meshes/lpb1.stl" scale="1 1 1"/>
@@ -489,5 +488,5 @@
     </inertial>
     <visual>
-      <origin xyz="0 0 0" rpy="0 0 0"/>
+      <origin xyz="-0.071565 0.038005 -0.013057" rpy="0 0 0"/>
       <geometry>
         <mesh filename="file://$(find mini_pupper_2_description)/meshes/rpf1.stl" scale="1 1 1"/>
@@ -496,5 +495,5 @@
     </visual>
     <collision>
-      <origin xyz="0 0 0" rpy="0 0 0"/>
+      <origin xyz="-0.071565 0.038005 -0.013057" rpy="0 0 0"/>
       <geometry>
         <mesh filename="file://$(find mini_pupper_2_description)/meshes/rpf1.stl" scale="1 1 1"/>
@@ -509,5 +508,5 @@
     </inertial>
     <visual>
-      <origin xyz="0 0 0" rpy="0 0 0"/>
+      <origin xyz="0.048967 0.038005 -0.013057" rpy="0 0 0"/>
       <geometry>
         <mesh filename="file://$(find mini_pupper_2_description)/meshes/rpb1.stl" scale="1 1 1"/>
@@ -516,5 +515,5 @@
     </visual>
     <collision>
-      <origin xyz="0 0 0" rpy="0 0 0"/>
+      <origin xyz="0.048967 0.038005 -0.013057" rpy="0 0 0"/>
       <geometry>
         <mesh filename="file://$(find mini_pupper_2_description)/meshes/rpb1.stl" scale="1 1 1"/>
@@ -526,8 +525,8 @@
       <origin xyz="-0.001747 0.007904 0.005365" rpy="0 0 0"/>
       <mass value="${pltgrp2_weight}"/>
-      <inertia ixx="0.862567e-6" iyy="0.991403e-6" izz="0.13904e-6" ixy="1.254e-9" iyz="-13.212e-9" ixz="-0.112894e-6"/>
-    </inertial>
-    <visual>
-      <origin xyz="0 0 0" rpy="0 0 0"/>
+      <inertia ixx="0.862567e-6" iyy="0.991403e-6" izz="0.13904e-6" ixy="1.254e-9" iyz="-13.212e-9" ixz="-0.11152e-6"/>
+    </inertial>
+    <visual>
+      <origin xyz="-0.052162 -0.044195 0.018943" rpy="0 0 0"/>
       <geometry>
         <mesh filename="file://$(find mini_pupper_2_description)/meshes/lpf2.stl" scale="1 1 1"/>
@@ -536,5 +535,5 @@
     </visual>
     <collision>
-      <origin xyz="0 0 0" rpy="0 0 0"/>
+      <origin xyz="-0.052162 -0.044195 0.018943" rpy="0 0 0"/>
       <geometry>
         <mesh filename="file://$(find mini_pupper_2_description)/meshes/lpf2.stl" scale="1 1 1"/>
@@ -546,8 +545,8 @@
       <origin xyz="-0.001747 0.007904 0.005365" rpy="0 0 0"/>
       <mass value="${pltgrp2_weight}"/>
-      <inertia ixx="0.862567e-6" iyy="0.991403e-6" izz="0.13904e-6" ixy="1.254e-9" iyz="-13.212e-9" ixz="-0.112894e-6"/>
-    </inertial>
-    <visual>
-      <origin xyz="0 0 0" rpy="0 0 0"/>
+      <inertia ixx="0.862567e-6" iyy="0.991403e-6" izz="0.13904e-6" ixy="1.254e-9" iyz="-13.212e-9" ixz="-0.11152e-6"/>
+    </inertial>
+    <visual>
+      <origin xyz="0.068367 -0.044195 0.018943" rpy="0 0 0"/>
       <geometry>
         <mesh filename="file://$(find mini_pupper_2_description)/meshes/lpb2.stl" scale="1 1 1"/>
@@ -556,5 +555,5 @@
     </visual>
     <collision>
-      <origin xyz="0 0 0" rpy="0 0 0"/>
+      <origin xyz="0.068367 -0.044195 0.018943" rpy="0 0 0"/>
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
Commit message: create new world for mini pupper

File: mini_pupper_2_description/urdf/mini_pupper_description.urdf.xacro (robot description, xacro)
@@ -368,5 +368,5 @@
         xyz="1.56706411611127E-05 -5.16565672073303E-13 -0.0191835739440227"
         rpy="0 0 -1.57" />
-      <mass value="0.0001" />
+      <mass value="0.108" />
       <inertia
         ixx="8.74731426973985E-06"
@@ -920,5 +920,5 @@
   </gazebo>
   <gazebo reference="lf1">
-    <kp>30000.0</kp>
+    <kp>10000.0</kp>
     <kd>1.0</kd>
     <mu1>0.8</mu1>
@@ -932,5 +932,5 @@
   </gazebo>
   <gazebo reference="lf2">
-    <kp>30000.0</kp>
+    <kp>10000.0</kp>
     <kd>1.0</kd>
     <mu1>0.8</mu1>
@@ -944,5 +944,5 @@
   </gazebo>
   <gazebo reference="lf3">
-    <kp>30000.0</kp>
+    <kp>10000.0</kp>
     <kd>1.0</kd>
     <mu1>0.8</mu1>
@@ -953,5 +953,5 @@
   </gazebo>
   <gazebo reference="lffoot">
-    <kp>30000.0</kp>
+    <kp>10000.0</kp>
     <kd>1.0</kd>
     <mu1>0.8</mu1>
@@ -962,5 +962,5 @@
   </gazebo>
   <gazebo reference="rf1">
-    <kp>30000.0</kp>
+    <kp>10000.0</kp>
     <kd>1.0</kd>
     <mu1>0.8</mu1>
@@ -974,5 +974,5 @@
   </gazebo>
   <gazebo reference="rf2">
-    <kp>30000.0</kp>
+    <kp>10000.0</kp>
     <kd>1.0</kd>
     <mu1>0.8</mu1>
@@ -986,5 +986,5 @@
   </gazebo>
   <gazebo reference="rf3">
-    <kp>30000.0</kp>
+    <kp>10000.0</kp>
     <kd>1.0</kd>
     <mu1>0.8</mu1>
@@ -995,5 +995,5 @@
   </gazebo>
   <gazebo reference="rffoot">
-    <kp>30000.0</kp>
+    <kp>10000.0</kp>
     <kd>1.0</kd>
     <mu1>0.8</mu1>
@@ -1004,5 +1004,5 @@
   </gazebo>
   <gazebo reference="lb1">
-    <kp>30000.0</kp>
+    <kp>10000.0</kp>
     <kd>1.0</kd>
     <mu1>0.8</mu1>
@@ -1016,5 +1016,5 @@
   </gazebo>
   <gazebo reference="lb2">
-    <kp>30000.0</kp>
+    <kp>10000.0</kp>
     <kd>1.0</kd>
     <mu1>0.8</mu1>
@@ -1028,5 +1028,5 @@
   </gazebo>
   <gazebo reference="lb3">
-    <kp>30000.0</kp>
+    <kp>10000.0</kp>
     <kd>1.0</kd>
     <mu1>0.8</mu1>
@@ -1037,5 +1037,5 @@
   </gazebo>
   <gazebo reference="lbfoot">
-    <kp>30000.0</kp>
+    <kp>10000.0</kp>
     <kd>1.0</kd>
     <mu1>0.8</mu1>
@@ -1046,5 +1046,5 @@
   </gazebo>
   <gazebo reference="rb1">
-    <kp>30000.0</kp>
+    <kp>10000.0</kp>
     <kd>1.0</kd>
     <mu1>0.8</mu1>
@@ -1058,5 +1058,5 @@
   </gazebo>
   <gazebo reference="rb2">
-    <kp>30000.0</kp>
+    <kp>10000.0</kp>
     <kd>1.0</kd>
     <mu1>0.8</mu1>
@@ -1070,5 +1070,5 @@
   </gazebo>
   <gazebo reference="rb3">
-    <kp>30000.0</kp>
+    <kp>10000.0</kp>
     <kd>1.0</kd>
     <mu1>0.8</mu1>
@@ -1079,5 +1079,5 @@
   </gazebo>
   <gazebo reference="rbfoot">
-    <kp>30000.0</kp>
+    <kp>10000.0</kp>
     <kd>1.0</kd>
     <mu1>0.8</mu1>
