Commit message: fine tune control parameters

File: mini_pupper_2_description/urdf/mini_pupper_description.urdf.xacro (robot description, xacro)
@@ -666,5 +666,5 @@
     <child link="lf1"/>
     <axis xyz="1.0 0.0 0.0"/>
-    <limit upper="0.425" lower="-0.550" effort="10" velocity="1.5"/>
+    <limit upper="0.425" lower="-0.550" effort="20" velocity="1.5"/>
   </joint>
   <joint name="lf1_lf2" type="revolute">
@@ -673,5 +673,5 @@
     <child link="lf2"/>
     <axis xyz="0.0 1.0 0.0"/>
-    <limit upper="2.40" lower="0.55" effort="10" velocity="1.5"/>
+    <limit upper="2.40" lower="0.55" effort="20" velocity="1.5"/>
   </joint>
   <joint name="lf2_lf3" type="revolute">
@@ -680,5 +680,5 @@
     <child link="lf3"/>
     <axis xyz="0.0 1.0 0.0"/>
-    <limit upper="-0.22" lower="-2.18" effort="10" velocity="1.5"/>
+    <limit upper="-0.22" lower="-2.18" effort="20" velocity="1.5"/>
   </joint>
   <joint name="base_rf1" type="revolute">
@@ -687,5 +687,5 @@
     <child link="rf1"/>
     <axis xyz="1.0 0.0 0.0"/>
-    <limit upper="0.550" lower="-0.425" effort="10" velocity="1.5"/>
+    <limit upper="0.550" lower="-0.425" effort="20" velocity="1.5"/>
   </joint>
   <joint name="rf1_rf2" type="revolute">
@@ -694,5 +694,5 @@
     <child link="rf2"/>
     <axis xyz="0.0 1.0 0.0"/>
-    <limit upper="2.40" lower="0.55" effort="10" velocity="1.5"/>
+    <limit upper="2.40" lower="0.55" effort="20" velocity="1.5"/>
   </joint>
   <joint name="rf2_rf3" type="revolute">
@@ -701,5 +701,5 @@
     <child link="rf3"/>
     <axis xyz="0.0 1.0 0.0"/>
-    <limit upper="-0.22" lower="-2.18" effort="10" velocity="1.5"/>
+    <limit upper="-0.22" lower="-2.18" effort="20" velocity="1.5"/>
   </joint>
   <joint name="base_rb1" type="revolute">
@@ -708,5 +708,5 @@
     <child link="rb1"/>
     <axis xyz="1.0 0.0 0.0"/>
-    <limit upper="0.550" lower="-0.425" effort="10" velocity="1.5"/>
+    <limit upper="0.550" lower="-0.425" effort="20" velocity="1.5"/>
   </joint>
   <joint name="rb1_rb2" type="revolute">
@@ -715,5 +715,5 @@
     <child link="rb2"/>
     <axis xyz="0.0 1.0 0.0"/>
-    <limit upper="2.40" lower="0.55" effort="10" velocity="1.5"/>
+    <limit upper="2.40" lower="0.55" effort="20" velocity="1.5"/>
   </joint>
   <joint name="rb2_rb3" type="revolute">
@@ -722,5 +722,5 @@
     <child link="rb3"/>
     <axis xyz="0.0 1.0 0.0"/>
-    <limit upper="-0.22" lower="-2.18" effort="10" velocity="1.5"/>
+    <limit upper="-0.22" lower="-2.18" effort="20" velocity="1.5"/>
   </joint>
   <joint name="base_lb1" type="revolute">
@@ -729,5 +729,5 @@
     <child link="lb1"/>
     <axis xyz="1.0 0.0 0.0"/>
-    <limit upper="0.425" lower="-0.550" effort="10" velocity="1.5"/>
+    <limit upper="0.425" lower="-0.550" effort="20" velocity="1.5"/>
   </joint>
   <joint name="lb1_lb2" type="revolute">
@@ -736,5 +736,5 @@
     <child link="lb2"/>
     <axis xyz="0.0 1.0 0.0"/>
-    <limit upper="2.40" lower="0.55" effort="10" velocity="1.5"/>
+    <limit upper="2.40" lower="0.55" effort="20" velocity="1.5"/>
   </joint>
   <joint name="lb2_lb3" type="revolute">
@@ -743,5 +743,5 @@
     <child link="lb3"/>
     <axis xyz="0.0 1.0 0.0"/>
-    <limit upper="-0.22" lower="-2.18" effort="10" velocity="1.5"/>
+    <limit upper="-0.22" lower="-2.18" effort="20" velocity="1.5"/>
   </joint>
   <joint name="base_front" type="fixed">
@@ -920,5 +920,5 @@
   </gazebo>
   <gazebo reference="lf1">
-    <kp>10000.0</kp>
+    <kp>100000.0</kp>
     <kd>1.0</kd>
     <mu1>0.8</mu1>
@@ -932,5 +932,5 @@
   </gazebo>
   <gazebo reference="lf2">
-    <kp>10000.0</kp>
+    <kp>100000.0</kp>
     <kd>1.0</kd>
     <mu1>0.8</mu1>
@@ -944,5 +944,5 @@
   </gazebo>
   <gazebo reference="lf3">
-    <kp>10000.0</kp>
+    <kp>100000.0</kp>
     <kd>1.0</kd>
     <mu1>0.8</mu1>
@@ -953,5 +953,5 @@
   </gazebo>
   <gazebo reference="lffoot">
-    <kp>10000.0</kp>
+    <kp>100000.0</kp>
     <kd>1.0</kd>
     <mu1>0.8</mu1>
@@ -962,5 +962,5 @@
   </gazebo>
   <gazebo reference="rf1">
-    <kp>10000.0</kp>
+    <kp>100000.0</kp>
     <kd>1.0</kd>
     <mu1>0.8</mu1>
@@ -974,5 +974,5 @@
   </gazebo>
   <gazebo reference="rf2">
-    <kp>10000.0</kp>
+    <kp>100000.0</kp>
     <kd>1.0</kd>
     <mu1>0.8</mu1>
@@ -986,5 +986,5 @@
   </gazebo>
   <gazebo reference="rf3">
-    <kp>10000.0</kp>
+    <kp>100000.0</kp>
     <kd>1.0</kd>
     <mu1>0.8</mu1>
@@ -995,5 +995,5 @@
   </gazebo>
   <gazebo reference="rffoot">
-    <kp>10000.0</kp>
+    <kp>100000.0</kp>
     <kd>1.0</kd>
     <mu1>0.8</mu1>
@@ -1004,5 +1004,5 @@
   </gazebo>
   <gazebo reference="lb1">
-    <kp>10000.0</kp>
+    <kp>100000.0</kp>
     <kd>1.0</kd>
     <mu1>0.8</mu1>
@@ -1016,5 +1016,5 @@
   </gazebo>
   <gazebo reference="lb2">
-    <kp>10000.0</kp>
+    <kp>100000.0</kp>
     <kd>1.0</kd>
     <mu1>0.8</mu1>
@@ -1028,5 +1028,5 @@
   </gazebo>
   <gazebo reference="lb3">
-    <kp>10000.0</kp>
+    <kp>100000.0</kp>
     <kd>1.0</kd>
     <mu1>0.8</mu1>
@@ -1037,5 +1037,5 @@
   </gazebo>
   <gazebo reference="lbfoot">
-    <kp>10000.0</kp>
+    <kp>100000.0</kp>
     <kd>1.0</kd>
     <mu1>0.8</mu1>
@@ -1046,5 +1046,5 @@
   </gazebo>
   <gazebo reference="rb1">
-    <kp>10000.0</kp>
+    <kp>100000.0</kp>
     <kd>1.0</kd>
     <mu1>0.8</mu1>
@@ -1058,5 +1058,5 @@
   </gazebo>
   <gazebo reference="rb2">
-    <kp>10000.0</kp>
+    <kp>100000.0</kp>
     <kd>1.0</kd>
     <mu1>0.8</mu1>
@@ -1070,5 +1070,5 @@
   </gazebo>
   <gazebo reference="rb3">
-    <kp>10000.0</kp>
+    <kp>100000.0</kp>
     <kd>1.0</kd>
     <mu1>0.8</mu1>
@@ -1079,5 +1079,5 @@
   </gazebo>
   <gazebo reference="rbfoot">
-    <kp>10000.0</kp>
+    <kp>100000.0</kp>
     <kd>1.0</kd>
     <mu1>0.8</mu1>

Commit message: Feature/tidy up slam and nagivation (#90)
* init commit for nagation and slam launch files tidy up

* create new world for mini pupper

* delete useless files

* improve readme and rviz

* fix flake8 errors

* fine tune control parameters

* fix slam parameters and simplify rviz

* enable imu usage

* minor config update for imu

* enable yaw from imu

* Update simulation world and map

File: mini_pupper_2_description/urdf/mini_pupper_description.urdf.xacro (robot description, xacro)
@@ -368,5 +368,5 @@
         xyz="1.56706411611127E-05 -5.16565672073303E-13 -0.0191835739440227"
         rpy="0 0 -1.57" />
-      <mass value="0.0001" />
+      <mass value="0.108" />
       <inertia
         ixx="8.74731426973985E-06"
@@ -666,5 +666,5 @@
     <child link="lf1"/>
     <axis xyz="1.0 0.0 0.0"/>
-    <limit upper="0.425" lower="-0.550" effort="10" velocity="1.5"/>
+    <limit upper="0.425" lower="-0.550" effort="20" velocity="1.5"/>
   </joint>
   <joint name="lf1_lf2" type="revolute">
@@ -673,5 +673,5 @@
     <child link="lf2"/>
     <axis xyz="0.0 1.0 0.0"/>
-    <limit upper="2.40" lower="0.55" effort="10" velocity="1.5"/>
+    <limit upper="2.40" lower="0.55" effort="20" velocity="1.5"/>
   </joint>
   <joint name="lf2_lf3" type="revolute">
@@ -680,5 +680,5 @@
     <child link="lf3"/>
     <axis xyz="0.0 1.0 0.0"/>
-    <limit upper="-0.22" lower="-2.18" effort="10" velocity="1.5"/>
+    <limit upper="-0.22" lower="-2.18" effort="20" velocity="1.5"/>
   </joint>
   <joint name="base_rf1" type="revolute">
@@ -687,5 +687,5 @@
     <child link="rf1"/>
     <axis xyz="1.0 0.0 0.0"/>
-    <limit upper="0.550" lower="-0.425" effort="10" velocity="1.5"/>
+    <limit upper="0.550" lower="-0.425" effort="20" velocity="1.5"/>
   </joint>
   <joint name="rf1_rf2" type="revolute">
@@ -694,5 +694,5 @@
     <child link="rf2"/>
     <axis xyz="0.0 1.0 0.0"/>
-    <limit upper="2.40" lower="0.55" effort="10" velocity="1.5"/>
+    <limit upper="2.40" lower="0.55" effort="20" velocity="1.5"/>
   </joint>
   <joint name="rf2_rf3" type="revolute">
@@ -701,5 +701,5 @@
     <child link="rf3"/>
     <axis xyz="0.0 1.0 0.0"/>
-    <limit upper="-0.22" lower="-2.18" effort="10" velocity="1.5"/>
+    <limit upper="-0.22" lower="-2.18" effort="20" velocity="1.5"/>
   </joint>
   <joint name="base_rb1" type="revolute">
@@ -708,5 +708,5 @@
     <child link="rb1"/>
     <axis xyz="1.0 0.0 0.0"/>
-    <limit upper="0.550" lower="-0.425" effort="10" velocity="1.5"/>
+    <limit upper="0.550" lower="-0.425" effort="20" velocity="1.5"/>
   </joint>
   <joint name="rb1_rb2" type="revolute">
@@ -715,5 +715,5 @@
     <child link="rb2"/>
     <axis xyz="0.0 1.0 0.0"/>
-    <limit upper="2.40" lower="0.55" effort="10" velocity="1.5"/>
+    <limit upper="2.40" lower="0.55" effort="20" velocity="1.5"/>
   </joint>
   <joint name="rb2_rb3" type="revolute">
@@ -722,5 +722,5 @@
     <child link="rb3"/>
     <axis xyz="0.0 1.0 0.0"/>
-    <limit upper="-0.22" lower="-2.18" effort="10" velocity="1.5"/>
+    <limit upper="-0.22" lower="-2.18" effort="20" velocity="1.5"/>
   </joint>
   <joint name="base_lb1" type="revolute">
@@ -729,5 +729,5 @@
     <child link="lb1"/>
     <axis xyz="1.0 0.0 0.0"/>
-    <limit upper="0.425" lower="-0.550" effort="10" velocity="1.5"/>
+    <limit upper="0.425" lower="-0.550" effort="20" velocity="1.5"/>
   </joint>
   <joint name="lb1_lb2" type="revolute">
@@ -736,5 +736,5 @@
     <child link="lb2"/>
     <axis xyz="0.0 1.0 0.0"/>
-    <limit upper="2.40" lower="0.55" effort="10" velocity="1.5"/>
+    <limit upper="2.40" lower="0.55" effort="20" velocity="1.5"/>
   </joint>
   <joint name="lb2_lb3" type="revolute">
@@ -743,5 +743,5 @@
     <child link="lb3"/>
     <axis xyz="0.0 1.0 0.0"/>
-    <limit upper="-0.22" lower="-2.18" effort="10" velocity="1.5"/>
+    <limit upper="-0.22" lower="-2.18" effort="20" velocity="1.5"/>
   </joint>
   <joint name="base_front" type="fixed">
@@ -920,5 +920,5 @@
   </gazebo>
   <gazebo reference="lf1">
-    <kp>5000.0</kp>
+    <kp>100000.0</kp>
     <kd>1.0</kd>
     <mu1>0.8</mu1>
@@ -932,5 +932,5 @@
   </gazebo>
   <gazebo reference="lf2">
-    <kp>5000.0</kp>
+    <kp>100000.0</kp>
     <kd>1.0</kd>
     <mu1>0.8</mu1>
@@ -944,5 +944,5 @@
   </gazebo>
   <gazebo reference="lf3">
-    <kp>5000.0</kp>
+    <kp>100000.0</kp>
     <kd>1.0</kd>
     <mu1>0.8</mu1>
@@ -953,5 +953,5 @@
   </gazebo>
   <gazebo reference="lffoot">
-    <kp>5000.0</kp>
+    <kp>100000.0</kp>
     <kd>1.0</kd>
     <mu1>0.8</mu1>
@@ -962,5 +962,5 @@
   </gazebo>
   <gazebo reference="rf1">
-    <kp>5000.0</kp>
+    <kp>100000.0</kp>
     <kd>1.0</kd>
     <mu1>0.8</mu1>
@@ -974,5 +974,5 @@
   </gazebo>
   <gazebo reference="rf2">
-    <kp>5000.0</kp>
+    <kp>100000.0</kp>
     <kd>1.0</kd>
     <mu1>0.8</mu1>
@@ -986,5 +986,5 @@
   </gazebo>
   <gazebo reference="rf3">
-    <kp>5000.0</kp>
+    <kp>100000.0</kp>
     <kd>1.0</kd>
     <mu1>0.8</mu1>
@@ -995,5 +995,5 @@
   </gazebo>
   <gazebo reference="rffoot">
-    <kp>5000.0</kp>
+    <kp>100000.0</kp>
     <kd>1.0</kd>
     <mu1>0.8</mu1>
@@ -1004,5 +1004,5 @@
   </gazebo>
   <gazebo reference="lb1">
-    <kp>5000.0</kp>
+    <kp>100000.0</kp>
     <kd>1.0</kd>
     <mu1>0.8</mu1>
@@ -1016,5 +1016,5 @@
   </gazebo>
   <gazebo reference="lb2">
-    <kp>5000.0</kp>
+    <kp>100000.0</kp>
     <kd>1.0</kd>
     <mu1>0.8</mu1>
@@ -1028,5 +1028,5 @@
   </gazebo>
   <gazebo reference="lb3">
-    <kp>5000.0</kp>
+    <kp>100000.0</kp>
     <kd>1.0</kd>
     <mu1>0.8</mu1>
@@ -1037,5 +1037,5 @@
   </gazebo>
   <gazebo reference="lbfoot">
-    <kp>5000.0</kp>
+    <kp>100000.0</kp>
     <kd>1.0</kd>
     <mu1>0.8</mu1>
@@ -1046,5 +1046,5 @@
   </gazebo>
   <gazebo reference="rb1">
-    <kp>5000.0</kp>
+    <kp>100000.0</kp>
     <kd>1.0</kd>
     <mu1>0.8</mu1>
@@ -1058,5 +1058,5 @@
   </gazebo>
   <gazebo reference="rb2">
-    <kp>5000.0</kp>
+    <kp>100000.0</kp>
     <kd>1.0</kd>
     <mu1>0.8</mu1>
@@ -1070,5 +1070,5 @@
   </gazebo>
   <gazebo reference="rb3">
-    <kp>5000.0</kp>
+    <kp>100000.0</kp>
     <kd>1.0</kd>
     <mu1>0.8</mu1>
@@ -1079,5 +1079,5 @@
   </gazebo>
   <gazebo reference="rbfoot">
-    <kp>5000.0</kp>
+    <kp>100000.0</kp>
     <kd>1.0</kd>
     <mu1>0.8</mu1>
