Commit message: revert to .xacro description to fix fatal bug

File: mini_pupper_description/urdf/mini_pupper/d435.urdf.xacro (robot description, xacro)
@@ -8,6 +8,6 @@
 <robot name="sensor_d435" xmlns:xacro="http://ros.org/wiki/xacro">
   <!-- Includes -->
-  <xacro:include filename="$(find mini_pupper_description)/urdf/_materials.urdf.xacro" />
-  <xacro:include filename="$(find mini_pupper_description)/urdf/_usb_plug.urdf.xacro" />
+  <xacro:include filename="package://mini_pupper_description/urdf/mini_pupper/materials.urdf.xacro" />
+  <xacro:include filename="package://mini_pupper_description/urdf/mini_pupper/usb_plug.urdf.xacro" />
   <xacro:macro name="sensor_d435" params="parent *origin name:=camera use_nominal_extrinsics:=true add_plug:=false use_mesh:=true">
     <xacro:property name="M_PI" value="3.1415926535897931" />
@@ -53,5 +53,5 @@
           <origin xyz="${d435_zero_depth_to_glass + d435_glass_to_front} ${-d435_cam_depth_py} 0" rpy="${M_PI/2} 0 ${M_PI/2}"/>
           <geometry>
-            <mesh filename="file://$(find mini_pupper_description)/meshes/d435.dae" />
+            <mesh filename="package://mini_pupper_description/meshes/mini_pupper/d435.dae" />
           </geometry>
         </xacro:if>

File: mini_pupper_description/urdf/mini_pupper/usb_plug.urdf.xacro (robot description, xacro)
@@ -20,5 +20,5 @@
         <geometry>
           <!--box size="0.044850 0.008 0.0185" /-->
-          <mesh filename="file://$(find mini_pupper_description)/meshes/plug.stl" />
+          <mesh filename="package://mini_pupper_description/meshes/mini_pupper/plug.stl" />
         </geometry>
         <material name="plastic"/>
@@ -28,5 +28,5 @@
         <geometry>
           <!--box size="0.044850 0.008 0.0185" /-->
-          <mesh filename="file://$(find mini_pupper_description)/meshes/plug_collision.stl" />
+          <mesh filename="package://mini_pupper_description/meshes/mini_pupper/plug_collision.stl" />
         </geometry>
       </collision>

File: mini_pupper_description/urdf/mini_pupper_2/mini_pupper_description.urdf.xacro (robot description, xacro)
@@ -1,158 +1,26 @@
 <?xml version="1.0" ?>
-<!-- =================================================================================== -->
-<!-- |    This document was autogenerated by xacro from mini_pupper_description.urdf.xacro | -->
-<!-- |    EDITING THIS FILE BY HAND IS NOT RECOMMENDED                                 | -->
-<!-- =================================================================================== -->
-<robot name="mini_pupper_2">
-  <material name="silver_default">
-    <color rgba="0.700 0.700 0.700 1.000"/>
-  </material>
-  <material name="opaque666666">
-    <color rgba="0.25882352941176473 0.25882352941176473 0.25882352941176473 1.0"/>
-  </material>
-  <material name="opaque252525">
-    <color rgba="0.09803921568627451 0.09803921568627451 0.09803921568627451 1.0"/>
-  </material>
-  <material name="opaque636363">
-    <color rgba="0.25098039215686274 0.25098039215686274 0.25098039215686274 1.0"/>
-  </material>
-  <material name="opaque2552210">
-    <color rgba="1.0 0.8666666666666667 0.0 1.0"/>
-  </material>
-  <material name="opaque646464">
-    <color rgba="0.25098039215686274 0.25098039215686274 0.25098039215686274 1.0"/>
-  </material>
-  <material name="opaque25524395">
-    <color rgba="1.0 0.9529411764705882 0.37254901960784315 1.0"/>
-  </material>
-  <material name="opaque2491590">
-    <color rgba="0.9764705882352941 0.6235294117647059 0.0 1.0"/>
-  </material>
-  <material name="opaque255255255">
-    <color rgba="1.0 1.0 1.0 1.0"/>
-  </material>
-  <transmission name="base_lf1_tran">
-    <type>transmission_interface/SimpleTransmission</type>
-    <joint name="base_lf1">
-      <hardwareInterface>hardware_interface/EffortJointInterface</hardwareInterface>
-    </joint>
-    <actuator name="base_lf1_actr">
-      <hardwareInterface>hardware_interface/EffortJointInterface</hardwareInterface>
-      <mechanicalReduction>1</mechanicalReduction>
-    </actuator>
-  </transmission>
-  <transmission name="lf1_lf2_tran">
-    <type>transmission_interface/SimpleTransmission</type>
-    <joint name="lf1_lf2">
-      <hardwareInterface>hardware_interface/EffortJointInterface</hardwareInterface>
-    </joint>
-    <actuator name="lf1_lf2_actr">
-      <hardwareInterface>hardware_interface/EffortJointInterface</hardwareInterface>
-      <mechanicalReduction>1</mechanicalReduction>
-    </actuator>
-  </transmission>
-  <transmission name="lf2_lf3_tran">
-    <type>transmission_interface/SimpleTransmission</type>
-    <joint name="lf2_lf3">
-      <hardwareInterface>hardware_interface/EffortJointInterface</hardwareInterface>
-    </joint>
-    <actuator name="lf2_lf3_actr">
-      <hardwareInterface>hardware_interface/EffortJointInterface</hardwareInterface>
-      <mechanicalReduction>1</mechanicalReduction>
-    </actuator>
-  </transmission>
-  <transmission name="base_rf1_tran">
-    <type>transmission_interface/SimpleTransmission</type>
-    <joint name="base_rf1">
-      <hardwareInterface>hardware_interface/EffortJointInterface</hardwareInterface>
-    </joint>
-    <actuator name="base_rf1_actr">
-      <hardwareInterface>hardware_interface/EffortJointInterface</hardwareInterface>
-      <mechanicalReduction>1</mechanicalReduction>
-    </actuator>
-  </transmission>
-  <transmission name="rf1_rf2_tran">
-    <type>transmission_interface/SimpleTransmission</type>
-    <joint name="rf1_rf2">
-      <hardwareInterface>hardware_interface/EffortJointInterface</hardwareInterface>
-    </joint>
-    <actuator name="rf1_rf2_actr">
-      <hardwareInterface>hardware_interface/EffortJointInterface</hardwareInterface>
-      <mechanicalReduction>1</mechanicalReduction>
-    </actuator>
-  </transmission>
-  <transmission name="rf2_rf3_tran">
-    <type>transmission_interface/SimpleTransmission</type>
-    <joint name="rf2_rf3">
-      <hardwareInterface>hardware_interface/EffortJointInterface</hardwareInterface>
-    </joint>
-    <actuator name="rf2_rf3_actr">
-      <hardwareInterface>hardware_interface/EffortJointInterface</hardwareInterface>
-      <mechanicalReduction>1</mechanicalReduction>
-    </actuator>
-  </transmission>
-  <transmission name="base_rb1_tran">
-    <type>transmission_interface/SimpleTransmission</type>
-    <joint name="base_rb1">
-      <hardwareInterface>hardware_interface/EffortJointInterface</hardwareInterface>
-    </joint>
-    <actuator name="base_rb1_actr">
-      <hardwareInterface>hardware_interface/EffortJointInterface</hardwareInterface>
-      <mechanicalReduction>1</mechanicalReduction>
-    </actuator>
-  </transmission>
-  <transmission name="rb1_rb2_tran">
-    <type>transmission_interface/SimpleTransmission</type>
-    <joint name="rb1_rb2">
-      <hardwareInterface>hardware_interface/EffortJointInterface</hardwareInterface>
-    </joint>
-    <actuator name="rb1_rb2_actr">
-      <hardwareInterface>hardware_interface/EffortJointInterface</hardwareInterface>
-      <mechanicalReduction>1</mechanicalReduction>
-    </actuator>
-  </transmission>
-  <transmission name="rb2_rb3_tran">
-    <type>transmission_interface/SimpleTransmission</type>
-    <joint name="rb2_rb3">
-      <hardwareInterface>hardware_interface/EffortJointInterface</hardwareInterface>
-    </joint>
-    <actuator name="rb2_rb3_actr">
-      <hardwareInterface>hardware_interface/EffortJointInterface</hardwareInterface>
-      <mechanicalReduction>1</mechanicalReduction>
-    </actuator>
-  </transmission>
-  <transmission name="base_lb1_tran">
-    <type>transmission_interface/SimpleTransmission</type>
-    <joint name="base_lb1">
-      <hardwareInterface>hardware_interface/EffortJointInterface</hardwareInterface>
-    </joint>
-    <actuator name="base_lb1_actr">
-      <hardwareInterface>hardware_interface/EffortJointInterface</hardwareInterface>
-      <mechanicalReduction>1</mechanicalReduction>
-    </actuator>
-  </transmission>
-  <transmission name="lb1_lb2_tran">
-    <type>transmission_interface/SimpleTransmission</type>
-    <joint name="lb1_lb2">
-      <hardwareInterface>hardware_interface/EffortJointInterface</hardwareInterface>
-    </joint>
-    <actuator name="lb1_lb2_actr">
-      <hardwareInterface>hardware_interface/EffortJointInterface</hardwareInterface>
-      <mechanicalReduction>1</mechanicalReduction>
-    </actuator>
-  </transmission>
-  <transmission name="lb2_lb3_tran">
-    <type>transmission_interface/SimpleTransmission</type>
-    <joint name="lb2_lb3">
-      <hardwareInterface>hardware_interface/EffortJointInterface</hardwareInterface>
-    </joint>
-    <actuator name="lb2_lb3_actr">
-      <hardwareInterface>hardware_interface/EffortJointInterface</hardwareInterface>
-      <mechanicalReduction>1</mechanicalReduction>
-    </actuator>
-  </transmission>
+<robot name="mini_pupper_2" xmlns:xacro="http://www.ros.org/wiki/xacro">
+  <xacro:include filename="package://mini_pupper_description/meshes/mini_pupper_2/materials.xacro" />
+  <xacro:include filename="package://mini_pupper_description/meshes/mini_pupper_2/mini_pupper_description.trans" />
+  <!-- CONSTANTS -->
+  <!-- Link group 1 - lf1, rf1, lb1, rb1 -->
+  <xacro:property name="lnkgrp1_weight" value="0.020769" />
+  <!-- Link group 2 - lf2, rf2, lb2, rb2 -->
+  <xacro:property name="lnkgrp2_weight" value="0.001906" />
+  <!-- Link group 3 - lf3, rf3, lb3, rb3 -->
+  <xacro:property name="lnkgrp3_weight" value="0.001144" />
+  <!-- Plate group 1 - lpf1, rpf1, lpb1, rpb1 -->
+  <xacro:property name="pltgrp1_weight" value="0.002574" />
+  <!-- Plate group 2 - lpf2, rpf2, lpb2, rpb2 -->
+  <xacro:property name="pltgrp2_weight" value="0.002231" />
+  <!-- Feet - lffoot, rffoot, lbfoot, rbfoot -->
+  <xacro:property name="feet_weight" value="0.001405" />
+  <!-- -0.004982788451759437 -2.855826620254409e-07 0.006488368014064216 -->
+  <!-- COM-Y: 0.00025 -->
+  <xacro:property name="feet_centre_of_mass"
+                  value="-0.014 0.00025 0.002488" />
   <link name="base_link">
     <visual>
-      <origin rpy="0 0 0" xyz="0 0 0"/>
+      <origin xyz="0 0 0" rpy="0 0 0"/>
       <geometry>
         <mesh filename="package://mini_pupper_description/meshes/mini_pupper_2/base_link.stl" scale="1 1 1"/>
@@ -161,5 +29,5 @@
     </visual>
     <collision>
-      <origin rpy="0 0 0" xyz="0 0 0"/>
+      <origin xyz="0 0 0" rpy="0 0 0"/>
       <geometry>
         <mesh filename="package://mini_pupper_description/meshes/mini_pupper_2/base_link.stl" scale="1 1 1"/>
@@ -169,17 +37,17 @@
   <link name="base_inertia">
     <inertial>
-      <origin rpy="0 0 0" xyz="-0.008867 0.000396 -0.007154"/>
+      <origin xyz="-0.008867 0.000396 -0.007154" rpy="0 0 0"/>
       <mass value="0.09818420433466489"/>
-      <inertia ixx="5.2003168e-5" ixy="7.28047e-7" ixz="-9.716561e-7" iyy="2.437e-4" iyz="603.31e-11" izz="2.523e-4"/>
+      <inertia ixx="5.2003168e-5" iyy="2.437e-4" izz="2.523e-4" ixy="7.28047e-7" iyz="603.31e-11" ixz="-9.716561e-7"/>
     </inertial>
   </link>
   <link name="lf1">
     <inertial>
-      <origin rpy="0 0 0" xyz="0.020109 0.002332 0.006500"/>
-      <mass value="0.020769"/>
-      <inertia ixx="2.494061e-6" ixy="-7.662e-9" ixz="-33.565e-9" iyy="3.735906e-6" iyz="-0.014e-9" izz="3.222909e-6"/>
-    </inertial>
-    <visual>
-      <origin rpy="0 0 0" xyz="0 0 0"/>
+      <origin xyz="0.020109 0.002332 0.006500" rpy="0 0 0"/>
+      <mass value="${lnkgrp1_weight}"/>
+      <inertia ixx="2.494061e-6" iyy="3.735906e-6" izz="3.222909e-6" ixy="-7.662e-9" iyz="-0.014e-9" ixz="-33.565e-9"/>
+    </inertial>
+    <visual>
+      <origin xyz="0 0 0" rpy="0 0 0"/>
       <geometry>
         <mesh filename="package://mini_pupper_description/meshes/mini_pupper_2/lf1.stl" scale="1 1 1"/>
@@ -188,5 +56,5 @@
     </visual>
     <collision>
-      <origin rpy="0 0 0" xyz="0 0 0"/>
+      <origin xyz="0 0 0" rpy="0 0 0"/>
       <geometry>
         <mesh filename="package://mini_pupper_description/meshes/mini_pupper_2/lf1.stl" scale="1 1 1"/>
@@ -196,10 +64,10 @@
   <link name="lf2">
     <inertial>
-      <origin rpy="0 0 0" xyz="-0.003174 0.000986 -0.017984"/>
-      <mass value="0.001906"/>
-      <inertia ixx="0.462154e-6" ixy="3.117e-9" ixz="-79.269e-9" iyy="0.481174e-6" iyz="17.662e-9" izz="26.893e-9"/>
-    </inertial>
-    <visual>
-      <origin rpy="0 0 0" xyz="0 0 0"/>
+      <origin xyz="-0.003174 0.000986 -0.017984" rpy="0 0 0"/>
+      <mass value="${lnkgrp2_weight}"/>
+      <inertia ixx="0.462154e-6" iyy="0.481174e-6" izz="26.893e-9" ixy="3.117e-9" iyz="17.662e-9" ixz="-79.269e-9"/>
+    </inertial>
+    <visual>
+      <origin xyz="0 0 0" rpy="0 0 0"/>
       <geometry>
         <mesh filename="package://mini_pupper_description/meshes/mini_pupper_2/lf2.stl" scale="1 1 1"/>
@@ -208,5 +76,5 @@
     </visual>
     <collision>
-      <origin rpy="0 0 0" xyz="0 0 0"/>
+      <origin xyz="0 0 0" rpy="0 0 0"/>
       <geometry>
         <mesh filename="package://mini_pupper_description/meshes/mini_pupper_2/lf2.stl" scale="1 1 1"/>
@@ -216,10 +84,10 @@
   <link name="lf3">
     <inertial>
-      <origin rpy="0 0 0" xyz="0.006211 0.003456 -0.015014"/>
-      <mass value="0.001144"/>
-      <inertia ixx="0.484471e-6" ixy="-2.101e-9" ixz="0.20057e-6" iyy="0.567615e-6" iyz="5.008e-9" izz="91.813e-9"/>
-    </inertial>
-    <visual>
-      <origin rpy="0 0 0" xyz="0 0 0"/>
+      <origin xyz="0.006211 0.003456 -0.015014" rpy="0 0 0"/>
+      <mass value="${lnkgrp3_weight}"/>
+      <inertia ixx="0.484471e-6" iyy="0.567615e-6" izz="91.813e-9" ixy="-2.101e-9" iyz="5.008e-9" ixz="0.20057e-6"/>
+    </inertial>
+    <visual>
+      <origin xyz="0 0 0" rpy="0 0 0"/>
       <geometry>
         <mesh filename="package://mini_pupper_description/meshes/mini_pupper_2/lf3.stl" scale="1 1 1"/>
@@ -228,5 +96,5 @@
     </visual>
     <collision>
-      <origin rpy="0 0 0" xyz="0 0 0"/>
+      <origin xyz="0 0 0" rpy="0 0 0"/>
       <geometry>
         <mesh filename="package://mini_pupper_description/meshes/mini_pupper_2/lf3.stl" scale="1 1 1"/>
@@ -236,10 +104,10 @@
   <link name="rf1">
     <inertial>
-      <origin rpy="0 0 0" xyz="0.020109 -0.002332 0.006500"/>
-      <mass value="0.020769"/>
-      <inertia ixx="2.494061e-06" ixy="7.662e-9" ixz="-33.565e-9" iyy="3.735906e-06" iyz="-0.014e-9" izz="3.222909e-06"/>
-    </inertial>
-    <visual>
-      <origin rpy="0 0 0" xyz="0 0 0"/>
+      <origin xyz="0.020109 -0.002332 0.006500" rpy="0 0 0"/>
+      <mass value="${lnkgrp1_weight}"/>
+      <inertia ixx="2.494061e-06" iyy="3.735906e-06" izz="3.222909e-06" ixy="7.662e-9" iyz="-0.014e-9" ixz="-33.565e-9"/>
+    </inertial>
+    <visual>
+      <origin xyz="0 0 0" rpy="0 0 0"/>
       <geometry>
         <mesh filename="package://mini_pupper_description/meshes/mini_pupper_2/rf1.stl" scale="1 1 1"/>
@@ -248,5 +116,5 @@
     </visual>
     <collision>
-      <origin rpy="0 0 0" xyz="0 0 0"/>
+      <origin xyz="0 0 0" rpy="0 0 0"/>
       <geometry>
         <mesh filename="package://mini_pupper_description/meshes/mini_pupper_2/rf1.stl" scale="1 1 1"/>
@@ -256,10 +124,10 @@
   <link name="rf2">
     <inertial>
-      <origin rpy="0 0 0" xyz="-0.003174 -0.000986 -0.017984"/>
-      <mass value="0.001906"/>
-      <inertia ixx="0.462154e-6" ixy="-3.117e-9" ixz="-79.269e-9" iyy="0.481174e-6" iyz="-17.662e-9" izz="26.893e-9"/>
-    </inertial>
-    <visual>
-      <origin rpy="0 0 0" xyz="0 0 0"/>
+      <origin xyz="-0.003174 -0.000986 -0.017984" rpy="0 0 0"/>
+      <mass value="${lnkgrp2_weight}"/>
+      <inertia ixx="0.462154e-6" iyy="0.481174e-6" izz="26.893e-9" ixy="-3.117e-9" iyz="-17.662e-9" ixz="-79.269e-9"/>
+    </inertial>
+    <visual>
+      <origin xyz="0 0 0" rpy="0 0 0"/>
       <geometry>
         <mesh filename="package://mini_pupper_description/meshes/mini_pupper_2/rf2.stl" scale="1 1 1"/>
@@ -268,5 +136,5 @@
     </visual>
     <collision>
-      <origin rpy="0 0 0" xyz="0 0 0"/>
+      <origin xyz="0 0 0" rpy="0 0 0"/>
       <geometry>
         <mesh filename="package://mini_pupper_description/meshes/mini_pupper_2/rf2.stl" scale="1 1 1"/>
@@ -276,10 +144,10 @@
   <link name="rf3">
     <inertial>
-      <origin rpy="0 0 0" xyz="0.006211 -0.003456 -0.015014"/>
-      <mass value="0.001144"/>
-      <inertia ixx="0.484471e-6" ixy="2.101e-9" ixz="0.20057e-6" iyy="0.567615e-06" iyz="-5.008e-9" izz="91.813e-9"/>
-    </inertial>
-    <visual>
-      <origin rpy="0 0 0" xyz="0 0 0"/>
+      <origin xyz="0.006211 -0.003456 -0.015014" rpy="0 0 0"/>
+      <mass value="${lnkgrp3_weight}"/>
+      <inertia ixx="0.484471e-6" iyy="0.567615e-06" izz="91.813e-9" ixy="2.101e-9" iyz="-5.008e-9" ixz="0.20057e-6"/>
+    </inertial>
+    <visual>
+      <origin xyz="0 0 0" rpy="0 0 0"/>
       <geometry>
         <mesh filename="package://mini_pupper_description/meshes/mini_pupper_2/rf3.stl" scale="1 1 1"/>
@@ -288,5 +156,5 @@
     </visual>
     <collision>
-      <origin rpy="0 0 0" xyz="0 0 0"/>
+      <origin xyz="0 0 0" rpy="0 0 0"/>
       <geometry>
         <mesh filename="package://mini_pupper_description/meshes/mini_pupper_2/rf3.stl" scale="1 1 1"/>
@@ -296,10 +164,10 @@
   <link name="rb1">
     <inertial>
-      <origin rpy="0 0 0" xyz="-0.020109 -0.002332 0.006500"/>
-      <mass value="0.020769"/>
-      <inertia ixx="2.494061e-06" ixy="-7.662e-9" ixz="-33.565e-9" iyy="3.735906e-06" iyz="-0.014e-9" izz="3.222909e-06"/>
-    </inertial>
-    <visual>
-      <origin rpy="0 0 0" xyz="0 0 0"/>
+      <origin xyz="-0.020109 -0.002332 0.006500" rpy="0 0 0"/>
+      <mass value="${lnkgrp1_weight}"/>
+      <inertia ixx="2.494061e-06" iyy="3.735906e-06" izz="3.222909e-06" ixy="-7.662e-9" iyz="-0.014e-9" ixz="-33.565e-9"/>
+    </inertial>
+    <visual>
+      <origin xyz="0 0 0" rpy="0 0 0"/>
       <geometry>
         <mesh filename="package://mini_pupper_description/meshes/mini_pupper_2/rb1.stl" scale="1 1 1"/>
@@ -308,5 +176,5 @@
     </visual>
     <collision>
-      <origin rpy="0 0 0" xyz="0 0 0"/>
+      <origin xyz="0 0 0" rpy="0 0 0"/>
       <geometry>
         <mesh filename="package://mini_pupper_description/meshes/mini_pupper_2/rb1.stl" scale="1 1 1"/>
@@ -316,10 +184,10 @@
   <link name="rb2">
     <inertial>
-      <origin rpy="0 0 0" xyz="-0.003174 -0.000986 -0.017984"/>
-      <mass value="0.001906"/>
-      <inertia ixx="0.462154e-6" ixy="-3.117e-9" ixz="-79.269e-9" iyy="0.481174e-6" iyz="-17.662e-9" izz="26.893e-9"/>
-    </inertial>
-    <visual>
-      <origin rpy="0 0 0" xyz="0 0 0"/>
+      <origin xyz="-0.003174 -0.000986 -0.017984" rpy="0 0 0"/>
+      <mass value="${lnkgrp2_weight}"/>
+      <inertia ixx="0.462154e-6" iyy="0.481174e-6" izz="26.893e-9" ixy="-3.117e-9" iyz="-17.662e-9" ixz="-79.269e-9"/>
+    </inertial>
+    <visual>
+      <origin xyz="0 0 0" rpy="0 0 0"/>
       <geometry>
         <mesh filename="package://mini_pupper_description/meshes/mini_pupper_2/rb2.stl" scale="1 1 1"/>
@@ -328,5 +196,5 @@
     </visual>
     <collision>
-      <origin rpy="0 0 0" xyz="0 0 0"/>
+      <origin xyz="0 0 0" rpy="0 0 0"/>
       <geometry>
         <mesh filename="package://mini_pupper_description/meshes/mini_pupper_2/rb2.stl" scale="1 1 1"/>
@@ -336,10 +204,10 @@
   <link name="rb3">
     <inertial>
-      <origin rpy="0 0 0" xyz="0.006211 -0.003456 -0.015014"/>
-      <mass value="0.001144"/>
-      <inertia ixx="0.484816e-6" ixy="2.212e-9" ixz="0.200564e-6" iyy="0.567883e-06" iyz="-5.34e-9" izz="91.777e-9"/>
-    </inertial>
-    <visual>
-      <origin rpy="0 0 0" xyz="0 0 0"/>
+      <origin xyz="0.006211 -0.003456 -0.015014" rpy="0 0 0"/>
+      <mass value="${lnkgrp3_weight}"/>
+      <inertia ixx="0.484816e-6" iyy="0.567883e-06" izz="91.777e-9" ixy="2.212e-9" iyz="-5.34e-9" ixz="0.200564e-6"/>
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