Commit message: fix mesh file path

File: mini_pupper_description/urdf/mini_pupper/mini_pupper_description.urdf.xacro (robot description, xacro)
@@ -9,5 +9,5 @@
       <geometry>
         <mesh
-          filename="$(find mini_pupper_description)/meshes/mini_pupper/base_link.STL" />
+          filename="file://$(find mini_pupper_description)/meshes/mini_pupper/base_link.STL" />
       </geometry>
       <material
@@ -23,5 +23,5 @@
       <geometry>
         <mesh
-          filename="$(find mini_pupper_description)/meshes/mini_pupper/base_link.STL" />
+          filename="file://$(find mini_pupper_description)/meshes/mini_pupper/base_link.STL" />
       </geometry>
     </collision>
@@ -70,5 +70,5 @@
       <geometry>
         <mesh
-          filename="$(find mini_pupper_description)/meshes/mini_pupper/yellow_plate.STL" />
+          filename="file://$(find mini_pupper_description)/meshes/mini_pupper/yellow_plate.STL" />
       </geometry>
       <material
@@ -84,5 +84,5 @@
       <geometry>
         <mesh
-          filename="$(find mini_pupper_description)/meshes/mini_pupper/yellow_plate.STL" />
+          filename="file://$(find mini_pupper_description)/meshes/mini_pupper/yellow_plate.STL" />
       </geometry>
     </collision>
@@ -123,5 +123,5 @@
       <geometry>
         <mesh
-          filename="$(find mini_pupper_description)/meshes/mini_pupper/lidar.STL" />
+          filename="file://$(find mini_pupper_description)/meshes/mini_pupper/lidar.STL" />
       </geometry>
       <material
@@ -137,5 +137,5 @@
       <geometry>
         <mesh
-          filename="$(find mini_pupper_description)/meshes/mini_pupper/lidar.STL" />
+          filename="file://$(find mini_pupper_description)/meshes/mini_pupper/lidar.STL" />
       </geometry>
     </collision>
@@ -176,5 +176,5 @@
       <geometry>
         <mesh
-          filename="$(find mini_pupper_description)/meshes/mini_pupper/lf1.STL" />
+          filename="file://$(find mini_pupper_description)/meshes/mini_pupper/lf1.STL" />
       </geometry>
       <material
@@ -190,5 +190,5 @@
       <geometry>
         <mesh
-          filename="$(find mini_pupper_description)/meshes/mini_pupper/lf1.STL" />
+          filename="file://$(find mini_pupper_description)/meshes/mini_pupper/lf1.STL" />
       </geometry>
     </collision>
@@ -234,5 +234,5 @@
       <geometry>
         <mesh
-          filename="$(find mini_pupper_description)/meshes/mini_pupper/lpf1.STL" />
+          filename="file://$(find mini_pupper_description)/meshes/mini_pupper/lpf1.STL" />
       </geometry>
       <material
@@ -248,5 +248,5 @@
       <geometry>
         <mesh
-          filename="$(find mini_pupper_description)/meshes/mini_pupper/lpf1.STL" />
+          filename="file://$(find mini_pupper_description)/meshes/mini_pupper/lpf1.STL" />
       </geometry>
     </collision>
@@ -287,5 +287,5 @@
       <geometry>
         <mesh
-          filename="$(find mini_pupper_description)/meshes/mini_pupper/lf2.STL" />
+          filename="file://$(find mini_pupper_description)/meshes/mini_pupper/lf2.STL" />
       </geometry>
       <material
@@ -301,5 +301,5 @@
       <geometry>
         <mesh
-          filename="$(find mini_pupper_description)/meshes/mini_pupper/lf2.STL" />
+          filename="file://$(find mini_pupper_description)/meshes/mini_pupper/lf2.STL" />
       </geometry>
     </collision>
@@ -345,5 +345,5 @@
       <geometry>
         <mesh
-          filename="$(find mini_pupper_description)/meshes/mini_pupper/lpf2.STL" />
+          filename="file://$(find mini_pupper_description)/meshes/mini_pupper/lpf2.STL" />
       </geometry>
       <material
@@ -359,5 +359,5 @@
       <geometry>
         <mesh
-          filename="$(find mini_pupper_description)/meshes/mini_pupper/lpf2.STL" />
+          filename="file://$(find mini_pupper_description)/meshes/mini_pupper/lpf2.STL" />
       </geometry>
     </collision>
@@ -398,5 +398,5 @@
       <geometry>
         <mesh
-          filename="$(find mini_pupper_description)/meshes/mini_pupper/lf3.STL" />
+          filename="file://$(find mini_pupper_description)/meshes/mini_pupper/lf3.STL" />
       </geometry>
       <material
@@ -412,5 +412,5 @@
       <geometry>
         <mesh
-          filename="$(find mini_pupper_description)/meshes/mini_pupper/lf3.STL" />
+          filename="file://$(find mini_pupper_description)/meshes/mini_pupper/lf3.STL" />
       </geometry>
     </collision>
@@ -456,5 +456,5 @@
       <geometry>
         <mesh
-          filename="$(find mini_pupper_description)/meshes/mini_pupper/lffoot.STL" />
+          filename="file://$(find mini_pupper_description)/meshes/mini_pupper/lffoot.STL" />
       </geometry>
       <material
@@ -470,5 +470,5 @@
       <geometry>
         <mesh
-          filename="$(find mini_pupper_description)/meshes/mini_pupper/lffoot.STL" />
+          filename="file://$(find mini_pupper_description)/meshes/mini_pupper/lffoot.STL" />
       </geometry>
     </collision>
@@ -509,5 +509,5 @@
       <geometry>
         <mesh
-          filename="$(find mini_pupper_description)/meshes/mini_pupper/rf1.STL" />
+          filename="file://$(find mini_pupper_description)/meshes/mini_pupper/rf1.STL" />
       </geometry>
       <material
@@ -523,5 +523,5 @@
       <geometry>
         <mesh
-          filename="$(find mini_pupper_description)/meshes/mini_pupper/rf1.STL" />
+          filename="file://$(find mini_pupper_description)/meshes/mini_pupper/rf1.STL" />
       </geometry>
     </collision>
@@ -567,5 +567,5 @@
       <geometry>
         <mesh
-          filename="$(find mini_pupper_description)/meshes/mini_pupper/rpf1.STL" />
+          filename="file://$(find mini_pupper_description)/meshes/mini_pupper/rpf1.STL" />
       </geometry>
       <material
@@ -581,5 +581,5 @@
       <geometry>
         <mesh
-          filename="$(find mini_pupper_description)/meshes/mini_pupper/rpf1.STL" />
+          filename="file://$(find mini_pupper_description)/meshes/mini_pupper/rpf1.STL" />
       </geometry>
     </collision>
@@ -620,5 +620,5 @@
       <geometry>
         <mesh
-          filename="$(find mini_pupper_description)/meshes/mini_pupper/rf2.STL" />
+          filename="file://$(find mini_pupper_description)/meshes/mini_pupper/rf2.STL" />
       </geometry>
       <material
@@ -634,5 +634,5 @@
       <geometry>
         <mesh
-          filename="$(find mini_pupper_description)/meshes/mini_pupper/rf2.STL" />
+          filename="file://$(find mini_pupper_description)/meshes/mini_pupper/rf2.STL" />
       </geometry>
     </collision>
@@ -678,5 +678,5 @@
       <geometry>
         <mesh
-          filename="$(find mini_pupper_description)/meshes/mini_pupper/rpf2.STL" />
+          filename="file://$(find mini_pupper_description)/meshes/mini_pupper/rpf2.STL" />
       </geometry>
       <material
@@ -692,5 +692,5 @@
       <geometry>
         <mesh
-          filename="$(find mini_pupper_description)/meshes/mini_pupper/rpf2.STL" />
+          filename="file://$(find mini_pupper_description)/meshes/mini_pupper/rpf2.STL" />
       </geometry>
     </collision>
@@ -731,5 +731,5 @@
       <geometry>
         <mesh
-          filename="$(find mini_pupper_description)/meshes/mini_pupper/rf3.STL" />
+          filename="file://$(find mini_pupper_description)/meshes/mini_pupper/rf3.STL" />
       </geometry>
       <material
@@ -745,5 +745,5 @@
       <geometry>
         <mesh
-          filename="$(find mini_pupper_description)/meshes/mini_pupper/rf3.STL" />
+          filename="file://$(find mini_pupper_description)/meshes/mini_pupper/rf3.STL" />
       </geometry>
     </collision>
@@ -789,5 +789,5 @@
       <geometry>
         <mesh
-          filename="$(find mini_pupper_description)/meshes/mini_pupper/rffoot.STL" />
+          filename="file://$(find mini_pupper_description)/meshes/mini_pupper/rffoot.STL" />
       </geometry>
       <material
@@ -803,5 +803,5 @@
       <geometry>
         <mesh
-          filename="$(find mini_pupper_description)/meshes/mini_pupper/rffoot.STL" />
+          filename="file://$(find mini_pupper_description)/meshes/mini_pupper/rffoot.STL" />
       </geometry>
     </collision>
@@ -842,5 +842,5 @@
       <geometry>
         <mesh
-          filename="$(find mini_pupper_description)/meshes/mini_pupper/lb1.STL" />
+          filename="file://$(find mini_pupper_description)/meshes/mini_pupper/lb1.STL" />
       </geometry>
       <material
@@ -856,5 +856,5 @@
       <geometry>
         <mesh
-          filename="$(find mini_pupper_description)/meshes/mini_pupper/lb1.STL" />
+          filename="file://$(find mini_pupper_description)/meshes/mini_pupper/lb1.STL" />
       </geometry>
     </collision>
@@ -900,5 +900,5 @@
       <geometry>
         <mesh
-          filename="$(find mini_pupper_description)/meshes/mini_pupper/lpb1.STL" />
+          filename="file://$(find mini_pupper_description)/meshes/mini_pupper/lpb1.STL" />
       </geometry>
       <material
@@ -914,5 +914,5 @@
       <geometry>
         <mesh
-          filename="$(find mini_pupper_description)/meshes/mini_pupper/lpb1.STL" />
+          filename="file://$(find mini_pupper_description)/meshes/mini_pupper/lpb1.STL" />
       </geometry>
     </collision>
@@ -953,5 +953,5 @@
       <geometry>
         <mesh
-          filename="$(find mini_pupper_description)/meshes/mini_pupper/lb2.STL" />
+          filename="file://$(find mini_pupper_description)/meshes/mini_pupper/lb2.STL" />
       </geometry>
       <material
@@ -967,5 +967,5 @@
       <geometry>
         <mesh
-          filename="$(find mini_pupper_description)/meshes/mini_pupper/lb2.STL" />
+          filename="file://$(find mini_pupper_description)/meshes/mini_pupper/lb2.STL" />
       </geometry>
     </collision>
@@ -1011,5 +1011,5 @@
       <geometry>
         <mesh
-          filename="$(find mini_pupper_description)/meshes/mini_pupper/lpb2.STL" />
+          filename="file://$(find mini_pupper_description)/meshes/mini_pupper/lpb2.STL" />
       </geometry>
       <material
@@ -1025,5 +1025,5 @@
       <geometry>
         <mesh
-          filename="$(find mini_pupper_description)/meshes/mini_pupper/lpb2.STL" />
+          filename="file://$(find mini_pupper_description)/meshes/mini_pupper/lpb2.STL" />
       </geometry>
     </collision>
@@ -1064,5 +1064,5 @@
       <geometry>
         <mesh
-          filename="$(find mini_pupper_description)/meshes/mini_pupper/lb3.STL" />
+          filename="file://$(find mini_pupper_description)/meshes/mini_pupper/lb3.STL" />
       </geometry>
       <material
@@ -1078,5 +1078,5 @@
       <geometry>
         <mesh
-          filename="$(find mini_pupper_description)/meshes/mini_pupper/lb3.STL" />
+          filename="file://$(find mini_pupper_description)/meshes/mini_pupper/lb3.STL" />
       </geometry>
     </collision>
@@ -1122,5 +1122,5 @@
       <geometry>
         <mesh
-          filename="$(find mini_pupper_description)/meshes/mini_pupper/lbfoot.STL" />
+          filename="file://$(find mini_pupper_description)/meshes/mini_pupper/lbfoot.STL" />
       </geometry>
       <material
@@ -1136,5 +1136,5 @@
       <geometry>
         <mesh
-          filename="$(find mini_pupper_description)/meshes/mini_pupper/lbfoot.STL" />
+          filename="file://$(find mini_pupper_description)/meshes/mini_pupper/lbfoot.STL" />
       </geometry>
     </collision>
@@ -1175,5 +1175,5 @@
       <geometry>
         <mesh
-          filename="$(find mini_pupper_description)/meshes/mini_pupper/rb1.STL" />
+          filename="file://$(find mini_pupper_description)/meshes/mini_pupper/rb1.STL" />
       </geometry>
       <material
@@ -1189,5 +1189,5 @@
       <geometry>
         <mesh
-          filename="$(find mini_pupper_description)/meshes/mini_pupper/rb1.STL" />
+          filename="file://$(find mini_pupper_description)/meshes/mini_pupper/rb1.STL" />
       </geometry>
     </collision>
@@ -1233,5 +1233,5 @@
       <geometry>
         <mesh
-          filename="$(find mini_pupper_description)/meshes/mini_pupper/rpb1.STL" />
+          filename="file://$(find mini_pupper_description)/meshes/mini_pupper/rpb1.STL" />
       </geometry>
       <material
@@ -1247,5 +1247,5 @@
       <geometry>
         <mesh
-          filename="$(find mini_pupper_description)/meshes/mini_pupper/rpb1.STL" />
+          filename="file://$(find mini_pupper_description)/meshes/mini_pupper/rpb1.STL" />
       </geometry>
     </collision>
@@ -1286,5 +1286,5 @@
       <geometry>
         <mesh
-          filename="$(find mini_pupper_description)/meshes/mini_pupper/rb2.STL" />
+          filename="file://$(find mini_pupper_description)/meshes/mini_pupper/rb2.STL" />
       </geometry>
       <material
@@ -1300,5 +1300,5 @@
       <geometry>
         <mesh
-          filename="$(find mini_pupper_description)/meshes/mini_pupper/rb2.STL" />
+          filename="file://$(find mini_pupper_description)/meshes/mini_pupper/rb2.STL" />
       </geometry>
     </collision>
@@ -1344,5 +1344,5 @@
       <geometry>
         <mesh
-          filename="$(find mini_pupper_description)/meshes/mini_pupper/rpb2.STL" />
+          filename="file://$(find mini_pupper_description)/meshes/mini_pupper/rpb2.STL" />
       </geometry>
       <material
@@ -1358,5 +1358,5 @@
       <geometry>
         <mesh
-          filename="$(find mini_pupper_description)/meshes/mini_pupper/rpb2.STL" />
+          filename="file://$(find mini_pupper_description)/meshes/mini_pupper/rpb2.STL" />
       </geometry>
     </collision>
@@ -1397,5 +1397,5 @@
       <geometry>
         <mesh
-          filename="$(find mini_pupper_description)/meshes/mini_pupper/rb3.STL" />
+          filename="file://$(find mini_pupper_description)/meshes/mini_pupper/rb3.STL" />
       </geometry>
       <material
@@ -1411,5 +1411,5 @@
       <geometry>
         <mesh
-          filename="$(find mini_pupper_description)/meshes/mini_pupper/rb3.STL" />
+          filename="file://$(find mini_pupper_description)/meshes/mini_pupper/rb3.STL" />
       </geometry>
     </collision>
@@ -1455,5 +1455,5 @@
       <geometry>
         <mesh
-          filename="$(find mini_pupper_description)/meshes/mini_pupper/rbfoot.STL" />
+          filename="file://$(find mini_pupper_description)/meshes/mini_pupper/rbfoot.STL" />
       </geometry>
       <material
@@ -1469,5 +1469,5 @@
       <geometry>
         <mesh
-          filename="$(find mini_pupper_description)/meshes/mini_pupper/rbfoot.STL" />
+          filename="file://$(find mini_pupper_description)/meshes/mini_pupper/rbfoot.STL" />
       </geometry>
     </collision>
