Commit message: feat: ROS 2 Jazzy migration (Gazebo Harmonic, Nav2, real robot)
Gazebo Classic → Harmonic:
- URDF sensors use native <topic> + <gz_frame_id> (no bridge needed)
- gz_ros2_control/GazeboSimSystem replaces gazebo_ros2_control
- gz-sim-odometry-publisher-system replaces libgazebo_ros_p3d.so
- d435 depth camera migrated to Harmonic
- World file updated with Gz Harmonic system plugins

Nav2 Jazzy:
- Remove plugin_lib_names (auto-loaded in Jazzy, duplicates crash)
- navfn plugin separator / → :: (required in Jazzy)
- Add collision_monitor + docking_server config (hardcoded in lifecycle)
- Add real_table.yaml Nav2 Jazzy configs

Real robot:
- LiDAR driver: ldlidar_stl_ros2 → ldlidar_node
- Update .minipupper.repos for new ldlidar driver

Docs & infra:
- All Humble/Ubuntu 22.04 references → Jazzy/Ubuntu 24.04
- CI updated for Jazzy
- Install scripts updated for Jazzy

Co-Authored-By: Claude Opus 4.6 (1M context) <noreply@anthropic.com>

File: mini_pupper_description/urdf/mini_pupper/mini_pupper_description.urdf.xacro (robot description, xacro)
@@ -1488,5 +1488,5 @@
   <ros2_control name="GazeboSystem" type="system">
     <hardware>
-      <plugin>gazebo_ros2_control/GazeboSystem</plugin>
+      <plugin>gz_ros2_control/GazeboSimSystem</plugin>
     </hardware>
     <joint name="base_lf1">
@@ -1728,10 +1728,10 @@
   <gazebo reference="lidar_link">
     <material>Gazebo/FlatBlack</material>
-    <sensor type="ray" name="lidar">
+    <sensor type="gpu_lidar" name="lidar">
       <always_on>true</always_on>
       <update_rate>30</update_rate>
       <pose>0 0 0 0 0 0</pose>
       <visualize>false</visualize>
-      <ray>
+      <lidar>
         <scan>
           <horizontal>
@@ -1752,30 +1752,19 @@
           <stddev>0.004</stddev>
         </noise>
-      </ray>
-      <plugin name="gazebo_ros_lidar_controller" filename="libgazebo_ros_ray_sensor.so">
-        <ros>
-          <remapping>~/out:=/scan</remapping>
-        </ros>
-        <output_type>sensor_msgs/LaserScan</output_type>
-        <frame_name>lidar_link</frame_name>
-        <!--min_intensity>100.0</min_intensity-->
-      </plugin>
+      </lidar>
+      <topic>/scan</topic>
+      <gz_frame_id>lidar_link</gz_frame_id>
     </sensor>
   </gazebo>
   <gazebo>
-    <plugin filename="libgazebo_ros_p3d.so" name="p3d_base_controller">
-      <ros>
-          <remapping>odom:=odom/ground_truth</remapping>
-      </ros>
-      <body_name>base_link</body_name>
-      <frame_name>world</frame_name>
-      <update_rate>10.0</update_rate>
-      <xyz_offset>0 0 0</xyz_offset>
-      <rpy_offset>0 0 0</rpy_offset>
-      <gaussian_noise>0.01</gaussian_noise>
+    <plugin filename="gz-sim-odometry-publisher-system" name="gz::sim::systems::OdometryPublisher">
+      <odom_frame>world</odom_frame>
+      <robot_base_frame>base_link</robot_base_frame>
+      <odom_publish_frequency>10.0</odom_publish_frequency>
+      <odom_topic>odom/ground_truth</odom_topic>
     </plugin>
   </gazebo>
   <gazebo>
-    <plugin filename="libgazebo_ros2_control.so" name="gazebo_ros2_control">
+    <plugin filename="gz_ros2_control-system" name="gz_ros2_control::GazeboSimROS2ControlPlugin">
       <parameters>$(find mini_pupper_description)/config/ros_control/mini_pupper_controller.yaml</parameters>
     </plugin>
@@ -1796,10 +1785,6 @@
       <always_on>true</always_on>
       <update_rate>50</update_rate>
-      <plugin name="gazebo_ros_imu_sensor" filename="libgazebo_ros_imu_sensor.so">
-          <ros>
-              <namespace>/imu</namespace>
-              <remapping>~/out:=data</remapping>
-          </ros>
-      </plugin>
+      <topic>/imu/data</topic>
+      <gz_frame_id>imu_link</gz_frame_id>
     </sensor>
   </gazebo>

File: mini_pupper_description/urdf/mini_pupper_2/mini_pupper_description.urdf.xacro (robot description, xacro)
@@ -837,5 +837,5 @@
   <ros2_control name="GazeboSystem" type="system">
     <hardware>
-      <plugin>gazebo_ros2_control/GazeboSystem</plugin>
+      <plugin>gz_ros2_control/GazeboSimSystem</plugin>
     </hardware>
     <joint name="base_lf1">
@@ -1089,10 +1089,10 @@
   <gazebo reference="lidar_link">
     <material>Gazebo/FlatBlack</material>
-    <sensor type="ray" name="lidar">
+    <sensor type="gpu_lidar" name="lidar">
       <always_on>true</always_on>
       <update_rate>30</update_rate>
       <pose>0 0 0 0 0 0</pose>
       <visualize>false</visualize>
-      <ray>
+      <lidar>
         <scan>
           <horizontal>
@@ -1113,29 +1113,19 @@
           <stddev>0.004</stddev>
         </noise>
-      </ray>
-      <plugin name="gazebo_ros_lidar_controller" filename="libgazebo_ros_ray_sensor.so">
-        <ros>
-          <remapping>~/out:=/scan</remapping>
-        </ros>
-        <output_type>sensor_msgs/LaserScan</output_type>
-        <frame_name>lidar_link</frame_name>
-      </plugin>
+      </lidar>
+      <topic>/scan</topic>
+      <gz_frame_id>lidar_link</gz_frame_id>
     </sensor>
   </gazebo>
   <gazebo>
-    <plugin filename="libgazebo_ros_p3d.so" name="p3d_base_controller">
-      <ros>
-        <remapping>odom:=odom/ground_truth</remapping>
-      </ros>
-      <body_name>base_link</body_name>
-      <frame_name>world</frame_name>
-      <update_rate>10.0</update_rate>
-      <xyz_offset>0 0 0</xyz_offset>
-      <rpy_offset>0 0 0</rpy_offset>
-      <gaussian_noise>0.01</gaussian_noise>
+    <plugin filename="gz-sim-odometry-publisher-system" name="gz::sim::systems::OdometryPublisher">
+      <odom_frame>world</odom_frame>
+      <robot_base_frame>base_link</robot_base_frame>
+      <odom_publish_frequency>10.0</odom_publish_frequency>
+      <odom_topic>odom/ground_truth</odom_topic>
     </plugin>
   </gazebo>
   <gazebo>
-    <plugin filename="libgazebo_ros2_control.so" name="gazebo_ros2_control">
+    <plugin filename="gz_ros2_control-system" name="gz_ros2_control::GazeboSimROS2ControlPlugin">
       <parameters>$(find mini_pupper_description)/config/ros_control/mini_pupper_2_controller.yaml</parameters>
     </plugin>
@@ -1156,10 +1146,6 @@
       <always_on>true</always_on>
       <update_rate>50</update_rate>
-      <plugin name="gazebo_ros_imu_sensor" filename="libgazebo_ros_imu_sensor.so">
-          <ros>
-              <namespace>/imu</namespace>
-              <remapping>~/out:=data</remapping>
-          </ros>
-      </plugin>
+      <topic>/imu/data</topic>
+      <gz_frame_id>imu_link</gz_frame_id>
     </sensor>
   </gazebo>
@@ -1168,9 +1154,7 @@
     <visual>
       <geometry>
-        <box>
-          <size>0.02 0.02 0.02</size>
-        </box>
-      </geometry>
-      <material>
+        <box size="0.02 0.02 0.02"/>
+      </geometry>
+      <material name="blue">
         <ambient>0 0 1 1</ambient>
         <diffuse>0 0 1 1</diffuse>
@@ -1200,12 +1184,6 @@
         </clip>
       </camera>
-      <!-- Gazebo ROS plugin to publish /image_raw -->
-      <plugin name="camera_controller" filename="libgazebo_ros_camera.so">
-        <always_on>true</always_on>
-        <update_rate>30.0</update_rate>
-        <frame_name>camera_link</frame_name>
-        <image_topic_name>/image_raw</image_topic_name>
-        <!-- camera_info omitted to disable /camera_info -->
-      </plugin>
+      <topic>/image_raw</topic>
+      <gz_frame_id>camera_link</gz_frame_id>
     </sensor>
   </gazebo>
