Commit message: add mini_pupper_hardware package and wire up for real robot

File: mini_pupper_description/urdf/ros2_control/mini_pupper.ros2_control.xacro (robot description, xacro)
@@ -1,5 +1,5 @@
 <?xml version="1.0"?>
 <robot xmlns:xacro="http://www.ros.org/wiki/xacro">
-  <xacro:macro name="mini_pupper_ros2_control" params="use_mock_hardware:=^|true">
+  <xacro:macro name="mini_pupper_ros2_control" params="use_gazebo_hardware:=^|true">
     <gazebo>
       <plugin name="gazebo_ros2_control" filename="libgazebo_ros2_control.so">
@@ -8,8 +8,16 @@
     </gazebo>
     <ros2_control name="MiniPupper" type="system">
-      <hardware>
-        <plugin>gazebo_ros2_control/GazeboSystem</plugin>
-        <param name="hold_joints">true</param>
-      </hardware>
+      <xacro:if value="${use_gazebo_hardware}">
+        <hardware>
+          <plugin>gazebo_ros2_control/GazeboSystem</plugin>
+          <param name="hold_joints">true</param>
+        </hardware>
+      </xacro:if>
+      <xacro:unless value="${use_gazebo_hardware}">
+        <hardware>
+          <plugin>mini_pupper_hardware/MiniPupperHardware</plugin>
+          <param name="hardware_interface_type">esp32_proxy</param>
+        </hardware>
+      </xacro:unless>
       <joint name="base_lf1">
         <command_interface name="position"/>

Commit message: refactor

File: mini_pupper_description/urdf/ros2_control/mini_pupper.ros2_control.xacro (robot description, xacro)
@@ -21,16 +21,13 @@
     </joint>
   </xacro:macro>
-  <xacro:macro name="mini_pupper_ros2_control" params="use_gazebo_hardware:=^|true">
-    <gazebo>
-      <plugin name="gazebo_ros2_control" filename="libgazebo_ros2_control.so">
-        <xacro:if value="${use_gazebo_hardware}">
-          <parameters>$(find mini_pupper_controllers)/config/mini_pupper_2_controllers_sim.yaml</parameters>
+  <xacro:macro name="mini_pupper_ros2_control" params="use_gazebo_hardware">
+    <xacro:if value="${use_gazebo_hardware}">
+      <gazebo>
+        <plugin name="gazebo_ros2_control" filename="libgazebo_ros2_control.so">
+          <parameters>$(find mini_pupper_simulation)/config/ros2_control/mini_pupper_2_controllers_sim.yaml</parameters>
           <hold_joints>false</hold_joints>
-        </xacro:if>
-        <xacro:unless value="${use_gazebo_hardware}">
-          <parameters>$(find mini_pupper_controllers)/config/mini_pupper_2_controllers.yaml</parameters>
-        </xacro:unless>
-      </plugin>
-    </gazebo>
+        </plugin>
+      </gazebo>
+    </xacro:if>
     <ros2_control name="MiniPupper" type="system">
       <hardware>
