Commit message: feat: added camera to URDF of robot, enabling camera usage in Gazebo

File: mini_pupper_description/urdf/mini_pupper_2/mini_pupper_description.urdf.xacro (robot description, xacro)
@@ -1164,3 +1164,49 @@
     </sensor>
   </gazebo>
+  <!-- Simulated camera mounted to the front body -->
+  <link name="camera_link">
+    <visual>
+      <geometry>
+        <box>
+          <size>0.02 0.02 0.02</size>
+        </box>
+      </geometry>
+      <material>
+        <ambient>0 0 1 1</ambient>
+        <diffuse>0 0 1 1</diffuse>
+      </material>
+    </visual>
+  </link>
+  <joint name="bodyfront_camera_joint" type="fixed">
+    <parent link="Body_front"/>
+    <child link="camera_link"/>
+    <origin xyz="0.02 0 0.02" rpy="0 0 0"/>
+  </joint>
+  <gazebo reference="camera_link">
+    <sensor type="camera" name="sim_camera">
+      <always_on>true</always_on>
+      <update_rate>30.0</update_rate>
+      <visualize>true</visualize>
+      <camera name="camera">
+        <horizontal_fov>1.3962634</horizontal_fov>
+        <image>
+          <width>640</width>
+          <height>480</height>
+          <format>R8G8B8</format>
+        </image>
+        <clip>
+          <near>0.02</near>
+          <far>50</far>
+        </clip>
+      </camera>
+      <!-- Gazebo ROS plugin to publish /image_raw -->
+      <plugin name="camera_controller" filename="libgazebo_ros_camera.so">
+        <always_on>true</always_on>
+        <update_rate>30.0</update_rate>
+        <frame_name>camera_link</frame_name>
+        <image_topic_name>/image_raw</image_topic_name>
+        <!-- camera_info omitted to disable /camera_info -->
+      </plugin>
+    </sensor>
+  </gazebo>
 </robot>

Commit message: make mini-pupper be able to move on a stand

File: mini_pupper_description/urdf/mini_pupper_2/mini_pupper_description.urdf.xacro (robot description, xacro)
@@ -2,5 +2,9 @@
 <robot name="mini_pupper_2" xmlns:xacro="http://www.ros.org/wiki/xacro">
   <xacro:include filename="$(find mini_pupper_description)/urdf/mini_pupper_2/materials.xacro" />
-  <xacro:include filename="$(find mini_pupper_description)/urdf/mini_pupper_2/mini_pupper_description.trans" />
+  <!-- Import Mini Pupper ros2_control description -->
+  <xacro:include filename="$(find mini_pupper_description)/urdf/ros2_control/mini_pupper.ros2_control.xacro" />
+  <!-- Arguments -->
+  <xacro:arg name="use_mock_hardware" default="true"/>
+  <xacro:arg name="use_debug_stand" default="false"/>
   <!-- CONSTANTS -->
   <!-- Link group 1 - lf1, rf1, lb1, rb1 -->
@@ -835,69 +839,4 @@
     <child link="Shell_Side"/>
   </joint>
-  <ros2_control name="GazeboSystem" type="system">
-    <hardware>
-      <plugin>gazebo_ros2_control/GazeboSystem</plugin>
-    </hardware>
-    <joint name="base_lf1">
-      <command_interface name="effort"/>
-      <state_interface name="position"/>
-      <state_interface name="velocity"/>
-    </joint>
-    <joint name="lf1_lf2">
-      <command_interface name="effort"/>
-      <state_interface name="position"/>
-      <state_interface name="velocity"/>
-    </joint>
-    <joint name="lf2_lf3">
-      <command_interface name="effort"/>
-      <state_interface name="position"/>
-      <state_interface name="velocity"/>
-    </joint>
-    <joint name="base_rf1">
-      <command_interface name="effort"/>
-      <state_interface name="position"/>
-      <state_interface name="velocity"/>
-    </joint>
-    <joint name="rf1_rf2">
-      <command_interface name="effort"/>
-      <state_interface name="position"/>
-      <state_interface name="velocity"/>
-    </joint>
-    <joint name="rf2_rf3">
-      <command_interface name="effort"/>
-      <state_interface name="position"/>
-      <state_interface name="velocity"/>
-    </joint>
-    <joint name="base_lb1">
-      <command_interface name="effort"/>
-      <state_interface name="position"/>
-      <state_interface name="velocity"/>
-    </joint>
-    <joint name="lb1_lb2">
-      <command_interface name="effort"/>
-      <state_interface name="position"/>
-      <state_interface name="velocity"/>
-    </joint>
-    <joint name="lb2_lb3">
-      <command_interface name="effort"/>
-      <state_interface name="position"/>
-      <state_interface name="velocity"/>
-    </joint>
-    <joint name="base_rb1">
-      <command_interface name="effort"/>
-      <state_interface name="position"/>
-      <state_interface name="velocity"/>
-    </joint>
-    <joint name="rb1_rb2">
-      <command_interface name="effort"/>
-      <state_interface name="position"/>
-      <state_interface name="velocity"/>
-    </joint>
-    <joint name="rb2_rb3">
-      <command_interface name="effort"/>
-      <state_interface name="position"/>
-      <state_interface name="velocity"/>
-    </joint>
-  </ros2_control>
   <!-- coloring Gazebo model -->
   <gazebo reference="base_link">
@@ -1136,9 +1075,4 @@
     </plugin>
   </gazebo>
-  <gazebo>
-    <plugin filename="libgazebo_ros2_control.so" name="gazebo_ros2_control">
-      <parameters>$(find mini_pupper_description)/config/ros_control/mini_pupper_2_controller.yaml</parameters>
-    </plugin>
-  </gazebo>
   <link name="imu_link">
     <inertial>
@@ -1164,3 +1098,9 @@
     </sensor>
   </gazebo>
+  <xacro:mini_pupper_ros2_control use_mock_hardware="$(arg use_mock_hardware)" />
+  <!-- Conditional debug support stand -->
+  <xacro:if value="$(arg use_debug_stand)">
+    <xacro:include filename="$(find mini_pupper_description)/urdf/ros2_control/support_stand.debug.xacro" />
+    <xacro:support_stand_debug robot_base_link="base_link"/>
+  </xacro:if>
 </robot>

Commit message: rebot can stand in gazebo

File: mini_pupper_description/urdf/mini_pupper_2/mini_pupper_description.urdf.xacro (robot description, xacro)
@@ -8,4 +8,15 @@
   <xacro:arg name="use_debug_stand" default="false"/>
   <!-- CONSTANTS -->
+  <xacro:property name="startup_abduction" value="0.0" />
+  <xacro:property name="startup_hip" value="0.977" />
+  <xacro:property name="startup_knee" value="-0.794" />
+  <xacro:property name="foot_mu1" value="50.0" />
+  <xacro:property name="foot_mu2" value="50.0" />
+  <xacro:property name="foot_kp" value="1000000.0" />
+  <xacro:property name="foot_kd" value="100.0" />
+  <xacro:property name="foot_max_contacts" value="40" />
+  <xacro:property name="foot_slip" value="0.0" />
+  <xacro:property name="servo_damping" value="5.0" />
+  <xacro:property name="servo_friction" value="1.0" />
   <!-- Link group 1 - lf1, rf1, lb1, rb1 -->
   <xacro:property name="lnkgrp1_weight" value="0.020769" />
@@ -25,4 +36,9 @@
                   value="-0.014 0.00025 0.002488" />
   <link name="base_link">
+    <inertial>
+      <origin xyz="-0.008867 0.000396 -0.007154" rpy="0 0 0"/>
+      <mass value="0.174884"/>
+      <inertia ixx="0.00090939" iyy="0.00426716" izz="0.00440707" ixy="1.27324e-7" iyz="1.05509e-9" ixz="-1.69927e-7"/>
+    </inertial>
     <visual>
       <origin xyz="0 0 0" rpy="0 0 0"/>
@@ -42,6 +58,6 @@
     <inertial>
       <origin xyz="-0.008867 0.000396 -0.007154" rpy="0 0 0"/>
-      <mass value="0.09818420433466489"/>
-      <inertia ixx="5.2003168e-5" iyy="2.437e-4" izz="2.523e-4" ixy="7.28047e-7" iyz="603.31e-11" ixz="-9.716561e-7"/>
+      <mass value="0.174884"/>
+      <inertia ixx="0.00090939" iyy="0.00426716" izz="0.00440707" ixy="1.27324e-7" iyz="1.05509e-9" ixz="-1.69927e-7"/>
     </inertial>
   </link>
@@ -419,4 +435,16 @@
     </collision>
   </link>
+  <gazebo reference="rffoot">
+    <mu1>${foot_mu1}</mu1>
+    <mu2>${foot_mu2}</mu2>
+    <kp>${foot_kp}</kp>
+    <kd>${foot_kd}</kd>
+    <max_contacts>${foot_max_contacts}</max_contacts>
+    <slip1>${foot_slip}</slip1>
+    <slip2>${foot_slip}</slip2>
+    <maxVel>0.0</maxVel>
+    <minDepth>0.001</minDepth>
+    <material>Gazebo/FlatBlack</material>
+  </gazebo>
   <link name="rbfoot">
     <inertial>
@@ -439,4 +467,16 @@
     </collision>
   </link>
+  <gazebo reference="rbfoot">
+    <mu1>${foot_mu1}</mu1>
+    <mu2>${foot_mu2}</mu2>
+    <kp>${foot_kp}</kp>
+    <kd>${foot_kd}</kd>
+    <max_contacts>${foot_max_contacts}</max_contacts>
+    <slip1>${foot_slip}</slip1>
+    <slip2>${foot_slip}</slip2>
+    <maxVel>0.0</maxVel>
+    <minDepth>0.001</minDepth>
+    <material>Gazebo/FlatBlack</material>
+  </gazebo>
   <link name="lbfoot">
     <inertial>
@@ -459,4 +499,16 @@
     </collision>
   </link>
+  <gazebo reference="lbfoot">
+    <mu1>${foot_mu1}</mu1>
+    <mu2>${foot_mu2}</mu2>
+    <kp>${foot_kp}</kp>
+    <kd>${foot_kd}</kd>
+    <max_contacts>${foot_max_contacts}</max_contacts>
+    <slip1>${foot_slip}</slip1>
+    <slip2>${foot_slip}</slip2>
+    <maxVel>0.0</maxVel>
+    <minDepth>0.001</minDepth>
+    <material>Gazebo/FlatBlack</material>
+  </gazebo>
   <link name="lffoot">
     <inertial>
@@ -479,4 +531,16 @@
     </collision>
   </link>
+  <gazebo reference="lffoot">
+    <mu1>${foot_mu1}</mu1>
+    <mu2>${foot_mu2}</mu2>
+    <kp>${foot_kp}</kp>
+    <kd>${foot_kd}</kd>
+    <max_contacts>${foot_max_contacts}</max_contacts>
+    <slip1>${foot_slip}</slip1>
+    <slip2>${foot_slip}</slip2>
+    <maxVel>0.0</maxVel>
+    <minDepth>0.001</minDepth>
+    <material>Gazebo/FlatBlack</material>
+  </gazebo>
   <link name="lpf1">
     <inertial>
@@ -670,5 +734,6 @@
     <child link="lf1"/>
     <axis xyz="1.0 0.0 0.0"/>
-    <limit upper="0.425" lower="-0.550" effort="20" velocity="1.5"/>
+    <dynamics damping="${servo_damping}" friction="${servo_friction}"/>
+    <limit upper="0.425" lower="-0.550" effort="10.0" velocity="10.47"/>
   </joint>
   <joint name="lf1_lf2" type="revolute">
@@ -677,5 +742,6 @@
     <child link="lf2"/>
     <axis xyz="0.0 1.0 0.0"/>
-    <limit upper="2.40" lower="0.55" effort="20" velocity="1.5"/>
+    <dynamics damping="${servo_damping}" friction="${servo_friction}"/>
+    <limit upper="2.40" lower="0.55" effort="10.0" velocity="10.47"/>
   </joint>
   <joint name="lf2_lf3" type="revolute">
@@ -684,5 +750,6 @@
     <child link="lf3"/>
     <axis xyz="0.0 1.0 0.0"/>
-    <limit upper="-0.22" lower="-2.18" effort="20" velocity="1.5"/>
+    <dynamics damping="${servo_damping}" friction="${servo_friction}"/>
+    <limit upper="-0.22" lower="-3.0" effort="10.0" velocity="10.47"/>
   </joint>
   <joint name="base_rf1" type="revolute">
@@ -691,5 +758,6 @@
     <child link="rf1"/>
     <axis xyz="1.0 0.0 0.0"/>
-    <limit upper="0.550" lower="-0.425" effort="20" velocity="1.5"/>
+    <dynamics damping="${servo_damping}" friction="${servo_friction}"/>
+    <limit upper="0.550" lower="-0.425" effort="10.0" velocity="10.47"/>
   </joint>
   <joint name="rf1_rf2" type="revolute">
@@ -698,5 +766,6 @@
     <child link="rf2"/>
     <axis xyz="0.0 1.0 0.0"/>
-    <limit upper="2.40" lower="0.55" effort="20" velocity="1.5"/>
+    <dynamics damping="${servo_damping}" friction="${servo_friction}"/>
+    <limit upper="2.40" lower="0.55" effort="10.0" velocity="10.47"/>
   </joint>
   <joint name="rf2_rf3" type="revolute">
@@ -705,5 +774,6 @@
     <child link="rf3"/>
     <axis xyz="0.0 1.0 0.0"/>
-    <limit upper="-0.22" lower="-2.18" effort="20" velocity="1.5"/>
+    <dynamics damping="${servo_damping}" friction="${servo_friction}"/>
+    <limit upper="-0.22" lower="-3.0" effort="10.0" velocity="10.47"/>
   </joint>
   <joint name="base_rb1" type="revolute">
@@ -712,5 +782,6 @@
     <child link="rb1"/>
     <axis xyz="1.0 0.0 0.0"/>
-    <limit upper="0.550" lower="-0.425" effort="20" velocity="1.5"/>
+    <dynamics damping="${servo_damping}" friction="${servo_friction}"/>
+    <limit upper="0.550" lower="-0.425" effort="10.0" velocity="10.47"/>
   </joint>
   <joint name="rb1_rb2" type="revolute">
@@ -719,5 +790,6 @@
     <child link="rb2"/>
     <axis xyz="0.0 1.0 0.0"/>
-    <limit upper="2.40" lower="0.55" effort="20" velocity="1.5"/>
+    <dynamics damping="${servo_damping}" friction="${servo_friction}"/>
+    <limit upper="2.40" lower="0.55" effort="10.0" velocity="10.47"/>
   </joint>
   <joint name="rb2_rb3" type="revolute">
@@ -726,5 +798,6 @@
     <child link="rb3"/>
     <axis xyz="0.0 1.0 0.0"/>
-    <limit upper="-0.22" lower="-2.18" effort="20" velocity="1.5"/>
+    <dynamics damping="${servo_damping}" friction="${servo_friction}"/>
+    <limit upper="-0.22" lower="-3.0" effort="10.0" velocity="10.47"/>
   </joint>
   <joint name="base_lb1" type="revolute">
@@ -733,5 +806,6 @@
     <child link="lb1"/>
     <axis xyz="1.0 0.0 0.0"/>
-    <limit upper="0.425" lower="-0.550" effort="20" velocity="1.5"/>
+    <dynamics damping="${servo_damping}" friction="${servo_friction}"/>
+    <limit upper="0.425" lower="-0.550" effort="10.0" velocity="10.47"/>
   </joint>
   <joint name="lb1_lb2" type="revolute">
@@ -740,5 +814,6 @@
     <child link="lb2"/>
     <axis xyz="0.0 1.0 0.0"/>
-    <limit upper="2.40" lower="0.55" effort="20" velocity="1.5"/>
+    <dynamics damping="${servo_damping}" friction="${servo_friction}"/>
+    <limit upper="2.40" lower="0.55" effort="10.0" velocity="10.47"/>
   </joint>
   <joint name="lb2_lb3" type="revolute">
@@ -747,5 +822,6 @@
     <child link="lb3"/>
     <axis xyz="0.0 1.0 0.0"/>
-    <limit upper="-0.22" lower="-2.18" effort="20" velocity="1.5"/>
+    <dynamics damping="${servo_damping}" friction="${servo_friction}"/>
+    <limit upper="-0.22" lower="-3.0" effort="10.0" velocity="10.47"/>
   </joint>
   <joint name="base_front" type="fixed">
@@ -891,13 +967,4 @@
     <material>Gazebo/FlatBlack</material>
   </gazebo>
-  <gazebo reference="lffoot">
-    <kp>100000.0</kp>
-    <kd>1.0</kd>
-    <mu1>0.8</mu1>
-    <mu2>0.8</mu2>
-    <maxVel>0.0</maxVel>
-    <minDepth>0.001</minDepth>
-    <material>Gazebo/FlatBlack</material>
-  </gazebo>
   <gazebo reference="rf1">
     <kp>100000.0</kp>
@@ -933,13 +1000,4 @@
     <material>Gazebo/FlatBlack</material>
   </gazebo>
-  <gazebo reference="rffoot">
-    <kp>100000.0</kp>
-    <kd>1.0</kd>
-    <mu1>0.8</mu1>
-    <mu2>0.8</mu2>
-    <maxVel>0.0</maxVel>
-    <minDepth>0.001</minDepth>
-    <material>Gazebo/FlatBlack</material>
-  </gazebo>
   <gazebo reference="lb1">
     <kp>100000.0</kp>
@@ -975,13 +1033,4 @@
     <material>Gazebo/FlatBlack</material>
   </gazebo>
-  <gazebo reference="lbfoot">
-    <kp>100000.0</kp>
-    <kd>1.0</kd>
-    <mu1>0.8</mu1>
-    <mu2>0.8</mu2>
-    <maxVel>0.0</maxVel>
-    <minDepth>0.001</minDepth>
-    <material>Gazebo/FlatBlack</material>
-  </gazebo>
   <gazebo reference="rb1">
     <kp>100000.0</kp>
@@ -1009,13 +1058,4 @@
   </gazebo>
   <gazebo reference="rb3">
-    <kp>100000.0</kp>
-    <kd>1.0</kd>
-    <mu1>0.8</mu1>
-    <mu2>0.8</mu2>
-    <maxVel>0.0</maxVel>
-    <minDepth>0.001</minDepth>
-    <material>Gazebo/FlatBlack</material>
-  </gazebo>
-  <gazebo reference="rbfoot">
     <kp>100000.0</kp>
     <kd>1.0</kd>

File: mini_pupper_description/urdf/ros2_control/mini_pupper.ros2_control.xacro (robot description, xacro)
@@ -13,49 +13,73 @@
       <joint name="base_lf1">
         <command_interface name="position"/>
-        <state_interface name="position"/>
+        <state_interface name="position">
+          <param name="initial_value">${startup_abduction}</param>
+        </state_interface>
       </joint>
       <joint name="lf1_lf2">
         <command_interface name="position"/>
-        <state_interface name="position"/>
+        <state_interface name="position">
+          <param name="initial_value">${startup_hip}</param>
+        </state_interface>
       </joint>
       <joint name="lf2_lf3">
         <command_interface name="position"/>
-        <state_interface name="position"/>
+        <state_interface name="position">
+          <param name="initial_value">${startup_knee}</param>
+        </state_interface>
       </joint>
       <joint name="base_rf1">
         <command_interface name="position"/>
-        <state_interface name="position"/>
+        <state_interface name="position">
+          <param name="initial_value">${startup_abduction}</param>
+        </state_interface>
       </joint>
       <joint name="rf1_rf2">
         <command_interface name="position"/>
-        <state_interface name="position"/>
+        <state_interface name="position">
+          <param name="initial_value">${startup_hip}</param>
+        </state_interface>
       </joint>
       <joint name="rf2_rf3">
         <command_interface name="position"/>
-        <state_interface name="position"/>
+        <state_interface name="position">
+          <param name="initial_value">${startup_knee}</param>
+        </state_interface>
       </joint>
       <joint name="base_lb1">
         <command_interface name="position"/>
-        <state_interface name="position"/>
+        <state_interface name="position">
+          <param name="initial_value">${startup_abduction}</param>
+        </state_interface>
       </joint>
       <joint name="lb1_lb2">
         <command_interface name="position"/>
-        <state_interface name="position"/>
+        <state_interface name="position">
+          <param name="initial_value">${startup_hip}</param>
+        </state_interface>
       </joint>
       <joint name="lb2_lb3">
         <command_interface name="position"/>
-        <state_interface name="position"/>
+        <state_interface name="position">
+          <param name="initial_value">${startup_knee}</param>
+        </state_interface>
       </joint>
       <joint name="base_rb1">
         <command_interface name="position"/>
-        <state_interface name="position"/>
+        <state_interface name="position">
+          <param name="initial_value">${startup_abduction}</param>
+        </state_interface>
       </joint>
       <joint name="rb1_rb2">
         <command_interface name="position"/>
-        <state_interface name="position"/>
+        <state_interface name="position">
+          <param name="initial_value">${startup_hip}</param>
+        </state_interface>
       </joint>
       <joint name="rb2_rb3">
         <command_interface name="position"/>
-        <state_interface name="position"/>
+        <state_interface name="position">
+          <param name="initial_value">${startup_knee}</param>
+        </state_interface>
       </joint>
     </ros2_control>

Commit message: set correct initial values

File: mini_pupper_description/urdf/mini_pupper_2/mini_pupper_description.urdf.xacro (robot description, xacro)
@@ -9,6 +9,6 @@
   <!-- CONSTANTS -->
   <xacro:property name="startup_abduction" value="0.0" />
-  <xacro:property name="startup_hip" value="0.977" />
-  <xacro:property name="startup_knee" value="-0.794" />
+  <xacro:property name="startup_hip" value="0.994" />
+  <xacro:property name="startup_knee" value="-1.767" />
   <xacro:property name="foot_mu1" value="50.0" />
   <xacro:property name="foot_mu2" value="50.0" />

Commit message: increase limit of all the joints

File: mini_pupper_description/urdf/mini_pupper_2/mini_pupper_description.urdf.xacro (robot description, xacro)
@@ -735,5 +735,5 @@
     <axis xyz="1.0 0.0 0.0"/>
     <dynamics damping="${servo_damping}" friction="${servo_friction}"/>
-    <limit upper="0.425" lower="-0.550" effort="10.0" velocity="10.47"/>
+    <limit upper="3.14" lower="-3.14" effort="10.0" velocity="10.47"/>
   </joint>
   <joint name="lf1_lf2" type="revolute">
@@ -743,5 +743,5 @@
     <axis xyz="0.0 1.0 0.0"/>
     <dynamics damping="${servo_damping}" friction="${servo_friction}"/>
-    <limit upper="2.40" lower="0.55" effort="10.0" velocity="10.47"/>
+    <limit upper="3.14" lower="-3.14" effort="10.0" velocity="10.47"/>
   </joint>
   <joint name="lf2_lf3" type="revolute">
@@ -751,5 +751,5 @@
     <axis xyz="0.0 1.0 0.0"/>
     <dynamics damping="${servo_damping}" friction="${servo_friction}"/>
-    <limit upper="-0.22" lower="-3.0" effort="10.0" velocity="10.47"/>
+    <limit upper="3.14" lower="-3.14" effort="10.0" velocity="10.47"/>
   </joint>
   <joint name="base_rf1" type="revolute">
@@ -759,5 +759,5 @@
     <axis xyz="1.0 0.0 0.0"/>
     <dynamics damping="${servo_damping}" friction="${servo_friction}"/>
-    <limit upper="0.550" lower="-0.425" effort="10.0" velocity="10.47"/>
+    <limit upper="3.14" lower="-3.14" effort="10.0" velocity="10.47"/>
   </joint>
   <joint name="rf1_rf2" type="revolute">
@@ -767,5 +767,5 @@
     <axis xyz="0.0 1.0 0.0"/>
     <dynamics damping="${servo_damping}" friction="${servo_friction}"/>
-    <limit upper="2.40" lower="0.55" effort="10.0" velocity="10.47"/>
+    <limit upper="3.14" lower="-3.14" effort="10.0" velocity="10.47"/>
   </joint>
   <joint name="rf2_rf3" type="revolute">
@@ -775,5 +775,5 @@
     <axis xyz="0.0 1.0 0.0"/>
     <dynamics damping="${servo_damping}" friction="${servo_friction}"/>
-    <limit upper="-0.22" lower="-3.0" effort="10.0" velocity="10.47"/>
+    <limit upper="3.14" lower="-3.14" effort="10.0" velocity="10.47"/>
   </joint>
   <joint name="base_rb1" type="revolute">
@@ -783,5 +783,5 @@
     <axis xyz="1.0 0.0 0.0"/>
     <dynamics damping="${servo_damping}" friction="${servo_friction}"/>
-    <limit upper="0.550" lower="-0.425" effort="10.0" velocity="10.47"/>
+    <limit upper="3.14" lower="-3.14" effort="10.0" velocity="10.47"/>
   </joint>
   <joint name="rb1_rb2" type="revolute">
@@ -791,5 +791,5 @@
     <axis xyz="0.0 1.0 0.0"/>
     <dynamics damping="${servo_damping}" friction="${servo_friction}"/>
-    <limit upper="2.40" lower="0.55" effort="10.0" velocity="10.47"/>
+    <limit upper="3.14" lower="-3.14" effort="10.0" velocity="10.47"/>
   </joint>
   <joint name="rb2_rb3" type="revolute">
@@ -799,5 +799,5 @@
     <axis xyz="0.0 1.0 0.0"/>
     <dynamics damping="${servo_damping}" friction="${servo_friction}"/>
-    <limit upper="-0.22" lower="-3.0" effort="10.0" velocity="10.47"/>
+    <limit upper="3.14" lower="-3.14" effort="10.0" velocity="10.47"/>
   </joint>
   <joint name="base_lb1" type="revolute">
@@ -807,5 +807,5 @@
     <axis xyz="1.0 0.0 0.0"/>
     <dynamics damping="${servo_damping}" friction="${servo_friction}"/>
-    <limit upper="0.425" lower="-0.550" effort="10.0" velocity="10.47"/>
+    <limit upper="3.14" lower="-3.14" effort="10.0" velocity="10.47"/>
   </joint>
   <joint name="lb1_lb2" type="revolute">
@@ -815,5 +815,5 @@
     <axis xyz="0.0 1.0 0.0"/>
     <dynamics damping="${servo_damping}" friction="${servo_friction}"/>
-    <limit upper="2.40" lower="0.55" effort="10.0" velocity="10.47"/>
+    <limit upper="3.14" lower="-3.14" effort="10.0" velocity="10.47"/>
   </joint>
   <joint name="lb2_lb3" type="revolute">
@@ -823,5 +823,5 @@
     <axis xyz="0.0 1.0 0.0"/>
     <dynamics damping="${servo_damping}" friction="${servo_friction}"/>
-    <limit upper="-0.22" lower="-3.0" effort="10.0" velocity="10.47"/>
+    <limit upper="3.14" lower="-3.14" effort="10.0" velocity="10.47"/>
   </joint>
   <joint name="base_front" type="fixed">
