Commit message: Feature/integrate ros2 control (#147)
* make mini-pupper be able to move on a stand

* rebot can stand in gazebo

* set correct initial values

* update ros2_control gazebo parameters to a separate file

* tidy up logic

* add mini_pupper_hardware package and wire up for real robot

* disable legacy hardware interface

* fix wrong xacro parameter

* fix hardware xml

* fix cmake

* fix joint names

* feed right robot description

* fix the description

* fix joint matrix issue

* fix hardware mappings

* fix controllers launch files

* fix esp interface connection dead issue

* update timeout for esp32

* tune frequency

* fix typo

* move ros2 controller to a separate package

* fix sim_time seting

* fix hardware mapping

* fix the joints mapping again

* add logs

* add even more logs

* fix hardware mapping

* fix joints mapping again

* add more logs for troubleshooting

* add config for broadcast

* update more debug log

* add more logs

* add more logs

* add more logs

* increase limit of all the joints

* update mappings

* Revert "update mappings"

This reverts commit a0cc1d951db3048d4a94ed83b7ac8b5beb3cbc6b.

* add more logs

* fix typo

* fix the logs

* fix another typo for the lanuch file

* change default positions

* reorder to match command protocol

* fix joints orders

* fix the states order

* fix the joints again

* fix the wrong yaml file

* fix the multipler numbers

* test: add standalone hardware test (no ROS2 required)

* fix: move servo_labels to function scope in standalone test

* fix: change torque from 1 to 500 to match Python DEFAULT_TORQUE

The ESP32 interprets torque_enable as a 0-1023 torque LIMIT, not a
binary on/off flag. Python uses DEFAULT_TORQUE=[500,...] giving ~49%
torque - enough to hold position against gravity. C++ was using 1
(~0.1% torque), causing servos to go limp and fall to physical stops
(observed: ch0=218, ch4=32, etc. instead of commanded positions).

This is why Python bringup worked but C++ ros2_control did not.

* fix: correct wrong angle signs in RB/LB abduction math test cases

* test: add Python standalone hardware test

* fix: use BB12B12H packet format (torque as uint8, 38 bytes total)

The installed esp32-proxy on Mini Pupper 2 uses BB12B12H format:
  BB   = 2 bytes header (size=38, cmd=1)
  12B  = 12 x uint8 torque (binary enable, 1=on)
  12H  = 12 x uint16 positions (little-endian)
  Total = 38 bytes

Our code was using BB12H12H (50 bytes, torque as uint16). The robot's
SOCK_SEQPACKET server buffer is 38 bytes, so our 50-byte packets were
truncated - positions for channels 6-11 were cut off, and channels 0-5
received torque data as position values instead of actual positions.

This explains all observed symptoms:
- Channels 6-11 received RF/LF position data (bytes 26-37)
- RB/LB position data (bytes 38-49) was always truncated
- Front leg positions (channels 0-5) received value=1 (torque bytes)
  and tried to move to position=1 (near mechanical stop)

* test: fix stale comments and misleading labels in standalone tests

- cpp: fix send_positions() comment BB12H12H → BB12B12H
- py: remove dead torque_1 variable (duplicate of torque_on)
- py: fix [2a] compare label '2a torque=500' → '2a torque=1'
- py: fix [2b] label 'broken' removed (torque=1 is correct)
- py: fix docstring 'torque=500 (correct)' → 'torque=1 (correct)'
All servo values commanded are identical between cpp and py tests.

* test: simplify Python live test to match C++ structure

* refactor: remove knee angle subtract+add roundtrip

Stanford controller joint_angles[2,x] is already knee_abs (from IK).
convert_to_JTP_positions was subtracting hip to get relative knee,
then mini_pupper_hardware.cpp was adding hip back to get knee_abs again.

Now knee_abs flows directly end-to-end:
- Utilities.py: pass joint_angles[2,x] unchanged (no - hip)
- send_commands_to_hardware: extract as lf/rf/lb/rb_knee_abs directly
- read_state_from_hardware: store knee_abs in hw_positions_ (no - hip)

hw_positions_[] now stores absolute knee angles, consistent with
hw_position_commands_[], so on_activate initialisation is also correct.

* refactor: remove knee angle subtract+add roundtrip, fix YAML default_positions

* cleanup: remove debug logging, keep only essential lifecycle and error logs

* tidy up codes

* refine for polishing the pr

* fine tune angles

* fine tune angles1

* further fine tune to align between different components

* further fine tune angles

* tidy up read me file

* update read me

* fix syntax

* rearrange folder locations

* make basic simulation works

* make simulation works, basic slam + navigation

* make simulation stable

* make twist converter default to be launched

* add ekf nodes

* simplify ekf nodes

* improve odometry

* restore part of the startup to keep champ in place, to be removed later

* fix launch errors

* fix imu data not used issue

* minor tune for the speed

* fix flake 8 errors

* fix syntax

* clean up pr

* fix cpp lint

* fine tune the pr

* revert the unnecessary change

* refactor

* fix code review issues

* fix code smell

* fix review comments from github

* fix build error

* fix syntax

* fix new line issues

* update documentation

* minor tune for the navigation parameters

* fine tune documenation

File: mini_pupper_description/urdf/mini_pupper_2/mini_pupper_description.urdf.xacro (robot description, xacro)
@@ -2,6 +2,45 @@
 <robot name="mini_pupper_2" xmlns:xacro="http://www.ros.org/wiki/xacro">
   <xacro:include filename="$(find mini_pupper_description)/urdf/mini_pupper_2/materials.xacro" />
-  <xacro:include filename="$(find mini_pupper_description)/urdf/mini_pupper_2/mini_pupper_description.trans" />
+  <!-- Import Mini Pupper ros2_control description -->
+  <xacro:include filename="$(find mini_pupper_description)/urdf/ros2_control/mini_pupper.ros2_control.xacro" />
+  <!-- Arguments -->
+  <xacro:arg name="use_gazebo_hardware" default="true"/>
+  <xacro:arg name="use_debug_stand" default="false"/>
   <!-- CONSTANTS -->
+  <xacro:if value="$(arg use_gazebo_hardware)">
+    <!-- Measured passive settled pose in Gazebo with no stand controller loaded. -->
+    <xacro:property name="startup_abduction_left" value="-0.33" />
+    <xacro:property name="startup_abduction_right" value="0.33" />
+    <xacro:property name="startup_hip" value="1.326" />
+    <xacro:property name="startup_knee" value="-2.927" />
+  </xacro:if>
+  <xacro:unless value="$(arg use_gazebo_hardware)">
+    <xacro:property name="startup_abduction_left" value="0.0" />
+    <xacro:property name="startup_abduction_right" value="0.0" />
+    <xacro:property name="startup_hip" value="0.994" />
+    <xacro:property name="startup_knee" value="-1.767" />
+  </xacro:unless>
+  <xacro:property name="foot_mu1" value="1.5" />
+  <xacro:property name="foot_mu2" value="1.5" />
+  <xacro:property name="foot_kp" value="50000.0" />
+  <xacro:property name="foot_kd" value="5.0" />
+  <xacro:property name="foot_max_contacts" value="10" />
+  <xacro:property name="foot_slip" value="0.0" />
+  <!-- Joint dynamics: ODE implicit damping must be small relative to link inertia
+       (~2.5e-6 kg·m²). Values above ~0.005 cause ODE to lock joints at origin. -->
+  <xacro:if value="$(arg use_gazebo_hardware)">
+    <xacro:property name="servo_damping" value="0.001" />
+    <xacro:property name="servo_friction" value="0.0" />
+    <!-- Keep limb inertia high enough for stable joint PID, but keep the trunk
+         lighter so pitch/roll corrections still move the body during gait. -->
+    <xacro:property name="sim_inertia_scale" value="100" />
+    <xacro:property name="sim_body_inertia_scale" value="100" />
+  </xacro:if>
+  <xacro:unless value="$(arg use_gazebo_hardware)">
+    <xacro:property name="servo_damping" value="5.0" />
+    <xacro:property name="servo_friction" value="1.0" />
+    <xacro:property name="sim_inertia_scale" value="1" />
+    <xacro:property name="sim_body_inertia_scale" value="1" />
+  </xacro:unless>
   <!-- Link group 1 - lf1, rf1, lb1, rb1 -->
   <xacro:property name="lnkgrp1_weight" value="0.020769" />
@@ -21,4 +60,9 @@
                   value="-0.014 0.00025 0.002488" />
   <link name="base_link">
+    <inertial>
+      <origin xyz="-0.008867 0.000396 -0.007154" rpy="0 0 0"/>
+      <mass value="0.174884"/>
+      <inertia ixx="${0.00090939 * sim_body_inertia_scale}" iyy="${0.00426716 * sim_body_inertia_scale}" izz="${0.00440707 * sim_body_inertia_scale}" ixy="${1.27324e-7 * sim_body_inertia_scale}" iyz="${1.05509e-9 * sim_body_inertia_scale}" ixz="${-1.69927e-7 * sim_body_inertia_scale}"/>
+    </inertial>
     <visual>
       <origin xyz="0 0 0" rpy="0 0 0"/>
@@ -38,6 +82,6 @@
     <inertial>
       <origin xyz="-0.008867 0.000396 -0.007154" rpy="0 0 0"/>
-      <mass value="0.09818420433466489"/>
-      <inertia ixx="5.2003168e-5" iyy="2.437e-4" izz="2.523e-4" ixy="7.28047e-7" iyz="603.31e-11" ixz="-9.716561e-7"/>
+      <mass value="0.174884"/>
+      <inertia ixx="${0.00090939 * sim_body_inertia_scale}" iyy="${0.00426716 * sim_body_inertia_scale}" izz="${0.00440707 * sim_body_inertia_scale}" ixy="${1.27324e-7 * sim_body_inertia_scale}" iyz="${1.05509e-9 * sim_body_inertia_scale}" ixz="${-1.69927e-7 * sim_body_inertia_scale}"/>
     </inertial>
   </link>
@@ -46,5 +90,5 @@
       <origin xyz="0.020109 0.002332 0.006500" rpy="0 0 0"/>
       <mass value="${lnkgrp1_weight}"/>
-      <inertia ixx="2.494061e-6" iyy="3.735906e-6" izz="3.222909e-6" ixy="-7.662e-9" iyz="-0.014e-9" ixz="-33.565e-9"/>
+      <inertia ixx="${2.494061e-6 * sim_inertia_scale}" iyy="${3.735906e-6 * sim_inertia_scale}" izz="${3.222909e-6 * sim_inertia_scale}" ixy="${-7.662e-9 * sim_inertia_scale}" iyz="${-0.014e-9 * sim_inertia_scale}" ixz="${-33.565e-9 * sim_inertia_scale}"/>
     </inertial>
     <visual>
@@ -66,5 +110,5 @@
       <origin xyz="-0.003174 0.000986 -0.017984" rpy="0 0 0"/>
       <mass value="${lnkgrp2_weight}"/>
-      <inertia ixx="0.462154e-6" iyy="0.481174e-6" izz="26.893e-9" ixy="3.117e-9" iyz="17.662e-9" ixz="-79.269e-9"/>
+      <inertia ixx="${0.462154e-6 * sim_inertia_scale}" iyy="${0.481174e-6 * sim_inertia_scale}" izz="${26.893e-9 * sim_inertia_scale}" ixy="${3.117e-9 * sim_inertia_scale}" iyz="${17.662e-9 * sim_inertia_scale}" ixz="${-79.269e-9 * sim_inertia_scale}"/>
     </inertial>
     <visual>
@@ -86,5 +130,5 @@
       <origin xyz="0.006211 0.003456 -0.015014" rpy="0 0 0"/>
       <mass value="${lnkgrp3_weight}"/>
-      <inertia ixx="0.484471e-6" iyy="0.567615e-6" izz="91.813e-9" ixy="-2.101e-9" iyz="5.008e-9" ixz="0.20057e-6"/>
+      <inertia ixx="${0.484471e-6 * sim_inertia_scale}" iyy="${0.567615e-6 * sim_inertia_scale}" izz="${91.813e-9 * sim_inertia_scale}" ixy="${-2.101e-9 * sim_inertia_scale}" iyz="${5.008e-9 * sim_inertia_scale}" ixz="${0.20057e-6 * sim_inertia_scale}"/>
     </inertial>
     <visual>
@@ -106,5 +150,5 @@
       <origin xyz="0.020109 -0.002332 0.006500" rpy="0 0 0"/>
       <mass value="${lnkgrp1_weight}"/>
-      <inertia ixx="2.494061e-06" iyy="3.735906e-06" izz="3.222909e-06" ixy="7.662e-9" iyz="-0.014e-9" ixz="-33.565e-9"/>
+      <inertia ixx="${2.494061e-06 * sim_inertia_scale}" iyy="${3.735906e-06 * sim_inertia_scale}" izz="${3.222909e-06 * sim_inertia_scale}" ixy="${7.662e-9 * sim_inertia_scale}" iyz="${-0.014e-9 * sim_inertia_scale}" ixz="${-33.565e-9 * sim_inertia_scale}"/>
     </inertial>
     <visual>
@@ -126,5 +170,5 @@
       <origin xyz="-0.003174 -0.000986 -0.017984" rpy="0 0 0"/>
       <mass value="${lnkgrp2_weight}"/>
-      <inertia ixx="0.462154e-6" iyy="0.481174e-6" izz="26.893e-9" ixy="-3.117e-9" iyz="-17.662e-9" ixz="-79.269e-9"/>
+      <inertia ixx="${0.462154e-6 * sim_inertia_scale}" iyy="${0.481174e-6 * sim_inertia_scale}" izz="${26.893e-9 * sim_inertia_scale}" ixy="${-3.117e-9 * sim_inertia_scale}" iyz="${-17.662e-9 * sim_inertia_scale}" ixz="${-79.269e-9 * sim_inertia_scale}"/>
     </inertial>
     <visual>
@@ -146,5 +190,5 @@
       <origin xyz="0.006211 -0.003456 -0.015014" rpy="0 0 0"/>
       <mass value="${lnkgrp3_weight}"/>
-      <inertia ixx="0.484471e-6" iyy="0.567615e-06" izz="91.813e-9" ixy="2.101e-9" iyz="-5.008e-9" ixz="0.20057e-6"/>
+      <inertia ixx="${0.484471e-6 * sim_inertia_scale}" iyy="${0.567615e-06 * sim_inertia_scale}" izz="${91.813e-9 * sim_inertia_scale}" ixy="${2.101e-9 * sim_inertia_scale}" iyz="${-5.008e-9 * sim_inertia_scale}" ixz="${0.20057e-6 * sim_inertia_scale}"/>
     </inertial>
     <visual>
@@ -166,5 +210,5 @@
       <origin xyz="-0.020109 -0.002332 0.006500" rpy="0 0 0"/>
       <mass value="${lnkgrp1_weight}"/>
-      <inertia ixx="2.494061e-06" iyy="3.735906e-06" izz="3.222909e-06" ixy="-7.662e-9" iyz="-0.014e-9" ixz="-33.565e-9"/>
+      <inertia ixx="${2.494061e-06 * sim_inertia_scale}" iyy="${3.735906e-06 * sim_inertia_scale}" izz="${3.222909e-06 * sim_inertia_scale}" ixy="${-7.662e-9 * sim_inertia_scale}" iyz="${-0.014e-9 * sim_inertia_scale}" ixz="${-33.565e-9 * sim_inertia_scale}"/>
     </inertial>
     <visual>
@@ -186,5 +230,5 @@
       <origin xyz="-0.003174 -0.000986 -0.017984" rpy="0 0 0"/>
       <mass value="${lnkgrp2_weight}"/>
-      <inertia ixx="0.462154e-6" iyy="0.481174e-6" izz="26.893e-9" ixy="-3.117e-9" iyz="-17.662e-9" ixz="-79.269e-9"/>
+      <inertia ixx="${0.462154e-6 * sim_inertia_scale}" iyy="${0.481174e-6 * sim_inertia_scale}" izz="${26.893e-9 * sim_inertia_scale}" ixy="${-3.117e-9 * sim_inertia_scale}" iyz="${-17.662e-9 * sim_inertia_scale}" ixz="${-79.269e-9 * sim_inertia_scale}"/>
     </inertial>
     <visual>
@@ -206,5 +250,5 @@
       <origin xyz="0.006211 -0.003456 -0.015014" rpy="0 0 0"/>
       <mass value="${lnkgrp3_weight}"/>
-      <inertia ixx="0.484816e-6" iyy="0.567883e-06" izz="91.777e-9" ixy="2.212e-9" iyz="-5.34e-9" ixz="0.200564e-6"/>
+      <inertia ixx="${0.484816e-6 * sim_inertia_scale}" iyy="${0.567883e-06 * sim_inertia_scale}" izz="${91.777e-9 * sim_inertia_scale}" ixy="${2.212e-9 * sim_inertia_scale}" iyz="${-5.34e-9 * sim_inertia_scale}" ixz="${0.200564e-6 * sim_inertia_scale}"/>
     </inertial>
     <visual>
@@ -226,5 +270,5 @@
       <origin xyz="-0.020109 0.002332 0.006500" rpy="0 0 0"/>
       <mass value="${lnkgrp1_weight}"/>
-      <inertia ixx="2.494061e-06" iyy="3.735906e-06" izz="3.222909e-06" ixy="7.662e-9" iyz="-0.014e-9" ixz="-33.565e-9"/>
+      <inertia ixx="${2.494061e-06 * sim_inertia_scale}" iyy="${3.735906e-06 * sim_inertia_scale}" izz="${3.222909e-06 * sim_inertia_scale}" ixy="${7.662e-9 * sim_inertia_scale}" iyz="${-0.014e-9 * sim_inertia_scale}" ixz="${-33.565e-9 * sim_inertia_scale}"/>
     </inertial>
     <visual>
@@ -246,5 +290,5 @@
       <origin xyz="-0.003174 0.000986 -0.017984" rpy="0 0 0"/>
       <mass value="${lnkgrp2_weight}"/>
-      <inertia ixx="0.462154e-6" iyy="0.481174e-6" izz="26.893e-9" ixy="3.117e-9" iyz="17.662e-9" ixz="-79.269e-9"/>
+      <inertia ixx="${0.462154e-6 * sim_inertia_scale}" iyy="${0.481174e-6 * sim_inertia_scale}" izz="${26.893e-9 * sim_inertia_scale}" ixy="${3.117e-9 * sim_inertia_scale}" iyz="${17.662e-9 * sim_inertia_scale}" ixz="${-79.269e-9 * sim_inertia_scale}"/>
     </inertial>
     <visual>
@@ -266,5 +310,5 @@
       <origin xyz="0.006211 0.003456 -0.015014" rpy="0 0 0"/>
       <mass value="${lnkgrp3_weight}"/>
-      <inertia ixx="0.484471e-6" iyy="0.567615e-06" izz="91.813e-9" ixy="-2.101e-9" iyz="5.008e-9" ixz="0.20057e-6"/>
+      <inertia ixx="${0.484471e-6 * sim_inertia_scale}" iyy="${0.567615e-06 * sim_inertia_scale}" izz="${91.813e-9 * sim_inertia_scale}" ixy="${-2.101e-9 * sim_inertia_scale}" iyz="${5.008e-9 * sim_inertia_scale}" ixz="${0.20057e-6 * sim_inertia_scale}"/>
     </inertial>
     <visual>
@@ -286,5 +330,5 @@
       <origin xyz="-0.005539 -0.000204 0.020223" rpy="0 0 0"/>
       <mass value="0.00785515871148119"/>
-      <inertia ixx="5.306048e-6" iyy="1.837621e-6" izz="3.61974e-6" ixy="-22.863e-9" iyz="-4.925e-9" ixz="-9.195e-9"/>
+      <inertia ixx="${5.306048e-6 * sim_body_inertia_scale}" iyy="${1.837621e-6 * sim_body_inertia_scale}" izz="${3.61974e-6 * sim_body_inertia_scale}" ixy="${-22.863e-9 * sim_body_inertia_scale}" iyz="${-4.925e-9 * sim_body_inertia_scale}" ixz="${-9.195e-9 * sim_body_inertia_scale}"/>
     </inertial>
     <visual>
@@ -306,5 +350,5 @@
       <origin xyz="0.089461 0.023505 0.0" rpy="0 0 0"/>
       <mass value="0.014261552601793053"/>
-      <inertia ixx="4.425965e-6" iyy="3.4560775e-5" izz="3.8954441e-5" ixy="0.104871e-6" iyz="75.406e-9" ixz="0.113313e-6"/>
+      <inertia ixx="${4.425965e-6 * sim_body_inertia_scale}" iyy="${3.4560775e-5 * sim_body_inertia_scale}" izz="${3.8954441e-5 * sim_body_inertia_scale}" ixy="${0.104871e-6 * sim_body_inertia_scale}" iyz="${75.406e-9 * sim_body_inertia_scale}" ixz="${0.113313e-6 * sim_body_inertia_scale}"/>
     </inertial>
     <visual>
@@ -370,10 +414,10 @@
       <mass value="0.108" />
       <inertia
-        ixx="8.74731426973985E-06"
-        ixy="-6.66781590704156E-08"
-        ixz="1.89196685410159E-11"
-        iyy="8.70097486591694E-06"
-        iyz="-1.13397577799603E-17"
-        izz="9.98821295317784E-06" />
+        ixx="${8.74731426973985E-06 * sim_body_inertia_scale}"
+        ixy="${-6.66781590704156E-08 * sim_body_inertia_scale}"
+        ixz="${1.89196685410159E-11 * sim_body_inertia_scale}"
+        iyy="${8.70097486591694E-06 * sim_body_inertia_scale}"
+        iyz="${-1.13397577799603E-17 * sim_body_inertia_scale}"
+        izz="${9.98821295317784E-06 * sim_body_inertia_scale}" />
     </inertial>
     <visual>
@@ -399,5 +443,5 @@
       <origin xyz="${feet_centre_of_mass}" rpy="0 0 0"/>
       <mass value="${feet_weight}"/>
-      <inertia ixx="41.995e-9" iyy="62.40e-9" izz="29.798e-9" ixy="0.0e-9" iyz="0.0e-9" ixz="1.616e-9"/>
+      <inertia ixx="${41.995e-9 * sim_inertia_scale}" iyy="${62.40e-9 * sim_inertia_scale}" izz="${29.798e-9 * sim_inertia_scale}" ixy="${0.0e-9 * sim_inertia_scale}" iyz="${0.0e-9 * sim_inertia_scale}" ixz="${1.616e-9 * sim_inertia_scale}"/>
     </inertial>
     <visual>
@@ -415,9 +459,21 @@
     </collision>
   </link>
+  <gazebo reference="rffoot">
+    <mu1>${foot_mu1}</mu1>
+    <mu2>${foot_mu2}</mu2>
+    <kp>${foot_kp}</kp>
+    <kd>${foot_kd}</kd>
+    <max_contacts>${foot_max_contacts}</max_contacts>
+    <slip1>${foot_slip}</slip1>
+    <slip2>${foot_slip}</slip2>
+    <maxVel>0.0</maxVel>
+    <minDepth>0.001</minDepth>
+    <material>Gazebo/FlatBlack</material>
+  </gazebo>
   <link name="rbfoot">
     <inertial>
       <origin xyz="${feet_centre_of_mass}" rpy="0 0 0"/>
       <mass value="${feet_weight}"/>
-      <inertia ixx="41.995e-9" iyy="62.40e-9" izz="29.798e-9" ixy="0.0e-9" iyz="0.0e-9" ixz="1.616e-9"/>
+      <inertia ixx="${41.995e-9 * sim_inertia_scale}" iyy="${62.40e-9 * sim_inertia_scale}" izz="${29.798e-9 * sim_inertia_scale}" ixy="${0.0e-9 * sim_inertia_scale}" iyz="${0.0e-9 * sim_inertia_scale}" ixz="${1.616e-9 * sim_inertia_scale}"/>
     </inertial>
     <visual>
@@ -435,9 +491,21 @@
     </collision>
   </link>
+  <gazebo reference="rbfoot">
+    <mu1>${foot_mu1}</mu1>
+    <mu2>${foot_mu2}</mu2>
+    <kp>${foot_kp}</kp>
+    <kd>${foot_kd}</kd>
+    <max_contacts>${foot_max_contacts}</max_contacts>
+    <slip1>${foot_slip}</slip1>
+    <slip2>${foot_slip}</slip2>
+    <maxVel>0.0</maxVel>
+    <minDepth>0.001</minDepth>
+    <material>Gazebo/FlatBlack</material>
+  </gazebo>
   <link name="lbfoot">
     <inertial>
       <origin xyz="${feet_centre_of_mass}" rpy="0 0 0"/>
       <mass value="${feet_weight}"/>
-      <inertia ixx="41.995e-9" iyy="62.40e-9" izz="29.798e-9" ixy="0.0e-9" iyz="0.0e-9" ixz="1.616e-9"/>
+      <inertia ixx="${41.995e-9 * sim_inertia_scale}" iyy="${62.40e-9 * sim_inertia_scale}" izz="${29.798e-9 * sim_inertia_scale}" ixy="${0.0e-9 * sim_inertia_scale}" iyz="${0.0e-9 * sim_inertia_scale}" ixz="${1.616e-9 * sim_inertia_scale}"/>
     </inertial>
     <visual>
@@ -455,9 +523,21 @@
     </collision>
   </link>
+  <gazebo reference="lbfoot">
+    <mu1>${foot_mu1}</mu1>
+    <mu2>${foot_mu2}</mu2>
+    <kp>${foot_kp}</kp>
+    <kd>${foot_kd}</kd>
+    <max_contacts>${foot_max_contacts}</max_contacts>
+    <slip1>${foot_slip}</slip1>
+    <slip2>${foot_slip}</slip2>
+    <maxVel>0.0</maxVel>
+    <minDepth>0.001</minDepth>
+    <material>Gazebo/FlatBlack</material>
+  </gazebo>
   <link name="lffoot">
     <inertial>
       <origin xyz="${feet_centre_of_mass}" rpy="0 0 0"/>
       <mass value="${feet_weight}"/>
-      <inertia ixx="41.995e-9" iyy="62.40e-9" izz="29.798e-9" ixy="0.0e-9" iyz="0.0e-9" ixz="1.616e-9"/>
+      <inertia ixx="${41.995e-9 * sim_inertia_scale}" iyy="${62.40e-9 * sim_inertia_scale}" izz="${29.798e-9 * sim_inertia_scale}" ixy="${0.0e-9 * sim_inertia_scale}" iyz="${0.0e-9 * sim_inertia_scale}" ixz="${1.616e-9 * sim_inertia_scale}"/>
     </inertial>
     <visual>
@@ -475,9 +555,21 @@
     </collision>
   </link>
+  <gazebo reference="lffoot">
+    <mu1>${foot_mu1}</mu1>
+    <mu2>${foot_mu2}</mu2>
+    <kp>${foot_kp}</kp>
+    <kd>${foot_kd}</kd>
+    <max_contacts>${foot_max_contacts}</max_contacts>
+    <slip1>${foot_slip}</slip1>
+    <slip2>${foot_slip}</slip2>
+    <maxVel>0.0</maxVel>
+    <minDepth>0.001</minDepth>
+    <material>Gazebo/FlatBlack</material>
+  </gazebo>
   <link name="lpf1">
     <inertial>
       <origin xyz="0.002259 0.008667 -0.002748" rpy="0 0 0"/>
       <mass value="${pltgrp1_weight}"/>
-      <inertia ixx="0.39059e-6" iyy="0.412444e-6" izz="0.246337e-6" ixy="24.631e-9" iyz="3.861e-9" ixz="54.116e-9"/>
+      <inertia ixx="${0.39059e-6 * sim_inertia_scale}" iyy="${0.412444e-6 * sim_inertia_scale}" izz="${0.246337e-6 * sim_inertia_scale}" ixy="${24.631e-9 * sim_inertia_scale}" iyz="${3.861e-9 * sim_inertia_scale}" ixz="${54.116e-9 * sim_inertia_scale}"/>
     </inertial>
     <visual>
@@ -499,5 +591,5 @@
       <origin xyz="0.002259 0.008667 -0.002748" rpy="0 0 0"/>
       <mass value="${pltgrp1_weight}"/>
-      <inertia ixx="0.39059e-6" iyy="0.412444e-6" izz="0.246337e-6" ixy="24.631e-9" iyz="3.861e-9" ixz="54.116e-9"/>
+      <inertia ixx="${0.39059e-6 * sim_inertia_scale}" iyy="${0.412444e-6 * sim_inertia_scale}" izz="${0.246337e-6 * sim_inertia_scale}" ixy="${24.631e-9 * sim_inertia_scale}" iyz="${3.861e-9 * sim_inertia_scale}" ixz="${54.116e-9 * sim_inertia_scale}"/>
     </inertial>
     <visual>
@@ -519,5 +611,5 @@
       <origin xyz="0.002259 -0.008667 -0.002748" rpy="0 0 0"/>
       <mass value="${pltgrp1_weight}"/>
-      <inertia ixx="0.39059e-6" iyy="0.412444e-6" izz="0.246337e-6" ixy="-24.631e-9" iyz="-3.861e-9" ixz="54.116e-9"/>
+      <inertia ixx="${0.39059e-6 * sim_inertia_scale}" iyy="${0.412444e-6 * sim_inertia_scale}" izz="${0.246337e-6 * sim_inertia_scale}" ixy="${-24.631e-9 * sim_inertia_scale}" iyz="${-3.861e-9 * sim_inertia_scale}" ixz="${54.116e-9 * sim_inertia_scale}"/>
     </inertial>
     <visual>
@@ -539,5 +631,5 @@
       <origin xyz="0.002259 -0.008667 -0.002748" rpy="0 0 0"/>
       <mass value="${pltgrp1_weight}"/>
-      <inertia ixx="0.39059e-6" iyy="0.412444e-6" izz="0.246337e-6" ixy="-24.631e-9" iyz="-3.861e-9" ixz="54.116e-9"/>
+      <inertia ixx="${0.39059e-6 * sim_inertia_scale}" iyy="${0.412444e-6 * sim_inertia_scale}" izz="${0.246337e-6 * sim_inertia_scale}" ixy="${-24.631e-9 * sim_inertia_scale}" iyz="${-3.861e-9 * sim_inertia_scale}" ixz="${54.116e-9 * sim_inertia_scale}"/>
     </inertial>
     <visual>
@@ -559,5 +651,5 @@
       <origin xyz="-0.001747 0.007904 0.005365" rpy="0 0 0"/>
       <mass value="${pltgrp2_weight}"/>
-      <inertia ixx="0.862567e-6" iyy="0.991403e-6" izz="0.13904e-6" ixy="1.254e-9" iyz="-13.212e-9" ixz="-0.112894e-6"/>
+      <inertia ixx="${0.862567e-6 * sim_inertia_scale}" iyy="${0.991403e-6 * sim_inertia_scale}" izz="${0.13904e-6 * sim_inertia_scale}" ixy="${1.254e-9 * sim_inertia_scale}" iyz="${-13.212e-9 * sim_inertia_scale}" ixz="${-0.112894e-6 * sim_inertia_scale}"/>
     </inertial>
     <visual>
@@ -579,5 +671,5 @@
       <origin xyz="-0.001747 0.007904 0.005365" rpy="0 0 0"/>
       <mass value="${pltgrp2_weight}"/>
-      <inertia ixx="0.862567e-6" iyy="0.991403e-6" izz="0.13904e-6" ixy="1.254e-9" iyz="-13.212e-9" ixz="-0.112894e-6"/>
+      <inertia ixx="${0.862567e-6 * sim_inertia_scale}" iyy="${0.991403e-6 * sim_inertia_scale}" izz="${0.13904e-6 * sim_inertia_scale}" ixy="${1.254e-9 * sim_inertia_scale}" iyz="${-13.212e-9 * sim_inertia_scale}" ixz="${-0.112894e-6 * sim_inertia_scale}"/>
     </inertial>
     <visual>
@@ -599,5 +691,5 @@
       <origin xyz="-0.001747 -0.007904 0.005365" rpy="0 0 0"/>
       <mass value="${pltgrp2_weight}"/>
-      <inertia ixx="0.862567e-6" iyy="0.991403e-6" izz="0.13904e-6" ixy="-1.254e-9" iyz="13.212e-9" ixz="-0.11152e-6"/>
+      <inertia ixx="${0.862567e-6 * sim_inertia_scale}" iyy="${0.991403e-6 * sim_inertia_scale}" izz="${0.13904e-6 * sim_inertia_scale}" ixy="${-1.254e-9 * sim_inertia_scale}" iyz="${13.212e-9 * sim_inertia_scale}" ixz="${-0.11152e-6 * sim_inertia_scale}"/>
     </inertial>
     <visual>
@@ -619,5 +711,5 @@
       <origin xyz="-0.001747 -0.007904 0.005365" rpy="0 0 0"/>
       <mass value="${pltgrp2_weight}"/>
-      <inertia ixx="0.862567e-6" iyy="0.991403e-6" izz="0.13904e-6" ixy="-1.254e-9" iyz="13.212e-9" ixz="-0.11152e-6"/>
+      <inertia ixx="${0.862567e-6 * sim_inertia_scale}" iyy="${0.991403e-6 * sim_inertia_scale}" izz="${0.13904e-6 * sim_inertia_scale}" ixy="${-1.254e-9 * sim_inertia_scale}" iyz="${13.212e-9 * sim_inertia_scale}" ixz="${-0.11152e-6 * sim_inertia_scale}"/>
     </inertial>
     <visual>
@@ -640,5 +732,5 @@
       <origin xyz="-0.00003 0.030005 0.022371" rpy="0 0 0"/>
       <mass value="0.0051928835390001775"/>
-      <inertia ixx="5.834352e-6" iyy="3.214872e-6" izz="6.996514e-6" ixy="0.0e-9" iyz="0.0e-9" ixz="15.218e-9"/>
+      <inertia ixx="${5.834352e-6 * sim_body_inertia_scale}" iyy="${3.214872e-6 * sim_body_inertia_scale}" izz="${6.996514e-6 * sim_body_inertia_scale}" ixy="${0.0e-9 * sim_body_inertia_scale}" iyz="${0.0e-9 * sim_body_inertia_scale}" ixz="${15.218e-9 * sim_body_inertia_scale}"/>
     </inertial>
     <visual>
@@ -666,5 +758,6 @@
     <child link="lf1"/>
     <axis xyz="1.0 0.0 0.0"/>
-    <limit upper="0.425" lower="-0.550" effort="20" velocity="1.5"/>
+    <dynamics damping="${servo_damping}" friction="${servo_friction}"/>
+    <limit upper="3.14" lower="-3.14" effort="10.0" velocity="10.47"/>
   </joint>
   <joint name="lf1_lf2" type="revolute">
@@ -673,5 +766,6 @@
     <child link="lf2"/>
     <axis xyz="0.0 1.0 0.0"/>
-    <limit upper="2.40" lower="0.55" effort="20" velocity="1.5"/>
+    <dynamics damping="${servo_damping}" friction="${servo_friction}"/>
+    <limit upper="3.14" lower="-3.14" effort="10.0" velocity="10.47"/>
   </joint>
   <joint name="lf2_lf3" type="revolute">
@@ -680,5 +774,6 @@
     <child link="lf3"/>
     <axis xyz="0.0 1.0 0.0"/>
-    <limit upper="-0.22" lower="-2.18" effort="20" velocity="1.5"/>
+    <dynamics damping="${servo_damping}" friction="${servo_friction}"/>
+    <limit upper="3.14" lower="-3.14" effort="10.0" velocity="10.47"/>
   </joint>
   <joint name="base_rf1" type="revolute">
@@ -687,5 +782,6 @@
     <child link="rf1"/>
     <axis xyz="1.0 0.0 0.0"/>
-    <limit upper="0.550" lower="-0.425" effort="20" velocity="1.5"/>
+    <dynamics damping="${servo_damping}" friction="${servo_friction}"/>
+    <limit upper="3.14" lower="-3.14" effort="10.0" velocity="10.47"/>
   </joint>
   <joint name="rf1_rf2" type="revolute">
@@ -694,5 +790,6 @@
     <child link="rf2"/>
     <axis xyz="0.0 1.0 0.0"/>
-    <limit upper="2.40" lower="0.55" effort="20" velocity="1.5"/>
+    <dynamics damping="${servo_damping}" friction="${servo_friction}"/>
+    <limit upper="3.14" lower="-3.14" effort="10.0" velocity="10.47"/>
   </joint>
   <joint name="rf2_rf3" type="revolute">
@@ -701,5 +798,6 @@
     <child link="rf3"/>
     <axis xyz="0.0 1.0 0.0"/>
-    <limit upper="-0.22" lower="-2.18" effort="20" velocity="1.5"/>
+    <dynamics damping="${servo_damping}" friction="${servo_friction}"/>
+    <limit upper="3.14" lower="-3.14" effort="10.0" velocity="10.47"/>
   </joint>
   <joint name="base_rb1" type="revolute">
@@ -708,5 +806,6 @@
     <child link="rb1"/>
     <axis xyz="1.0 0.0 0.0"/>
-    <limit upper="0.550" lower="-0.425" effort="20" velocity="1.5"/>
+    <dynamics damping="${servo_damping}" friction="${servo_friction}"/>
+    <limit upper="3.14" lower="-3.14" effort="10.0" velocity="10.47"/>
   </joint>
   <joint name="rb1_rb2" type="revolute">
@@ -715,5 +814,6 @@
     <child link="rb2"/>
     <axis xyz="0.0 1.0 0.0"/>
-    <limit upper="2.40" lower="0.55" effort="20" velocity="1.5"/>
+    <dynamics damping="${servo_damping}" friction="${servo_friction}"/>
+    <limit upper="3.14" lower="-3.14" effort="10.0" velocity="10.47"/>
   </joint>
   <joint name="rb2_rb3" type="revolute">
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