Commit message: Fix camera link xarco geometry

File: mini_pupper_description/urdf/mini_pupper_2/mini_pupper_description.urdf.xacro (robot description, xacro)
@@ -1163,11 +1163,8 @@
     <visual>
       <geometry>
-        <box>
-          <size>0.02 0.02 0.02</size>
-        </box>
-      </geometry>
-      <material>
-        <ambient>0 0 1 1</ambient>
-        <diffuse>0 0 1 1</diffuse>
+          <box size="0.02 0.02 0.02" />
+      </geometry>
+      <material name="Cyan">
+        <color rgba="0 1.0 1.0 1.0"/>
       </material>
     </visual>

Commit message: Ros2 Jazzy migration

File: mini_pupper_description/urdf/mini_pupper_2/mini_pupper_description.urdf.xacro (robot description, xacro)
@@ -36,4 +36,17 @@
     <xacro:property name="sim_inertia_scale" value="100" />
     <xacro:property name="sim_body_inertia_scale" value="100" />
+    <xacro:property name="sim_mass_scale" value="30.0" />
+    <xacro:property name="base_link_mass" value="${0.174884 * sim_mass_scale}" />
+    <xacro:property name="lnkgrp1_mass" value="${0.020769 * sim_mass_scale}" />
+    <xacro:property name="lnkgrp2_mass" value="${0.001906 * sim_mass_scale}" />
+    <xacro:property name="lnkgrp3_mass" value="${0.001144 * sim_mass_scale}" />
+    <xacro:property name="pltgrp1_mass" value="${0.002574 * sim_mass_scale}" />
+    <xacro:property name="pltgrp2_mass" value="${0.002231 * sim_mass_scale}" />
+    <xacro:property name="feet_mass" value="${0.001405 * sim_mass_scale}" />
+    <xacro:property name="body_front_mass" value="${0.00785515871148119 * sim_mass_scale}" />
+    <xacro:property name="board_pcb_mass" value="${0.014261552601793053 * sim_mass_scale}" />
+    <xacro:property name="lidar_mass" value="${0.108 * sim_mass_scale}" />
+    <xacro:property name="shell_side_mass" value="${0.0051928835390001775 * sim_mass_scale}" />
+    <xacro:property name="imu_mass" value="${0.0001 * sim_mass_scale}" />
   </xacro:if>
   <xacro:unless value="$(arg use_gazebo_hardware)">
@@ -42,4 +55,16 @@
     <xacro:property name="sim_inertia_scale" value="1" />
     <xacro:property name="sim_body_inertia_scale" value="1" />
+    <xacro:property name="base_link_mass" value="0.174884" />
+    <xacro:property name="lnkgrp1_mass" value="0.020769" />
+    <xacro:property name="lnkgrp2_mass" value="0.001906" />
+    <xacro:property name="lnkgrp3_mass" value="0.001144" />
+    <xacro:property name="pltgrp1_mass" value="0.002574" />
+    <xacro:property name="pltgrp2_mass" value="0.002231" />
+    <xacro:property name="feet_mass" value="0.001405" />
+    <xacro:property name="body_front_mass" value="0.00785515871148119" />
+    <xacro:property name="board_pcb_mass" value="0.014261552601793053" />
+    <xacro:property name="lidar_mass" value="0.108" />
+    <xacro:property name="shell_side_mass" value="0.0051928835390001775" />
+    <xacro:property name="imu_mass" value="0.0001" />
   </xacro:unless>
   <!-- Link group 1 - lf1, rf1, lb1, rb1 -->
@@ -62,5 +87,5 @@
     <inertial>
       <origin xyz="-0.008867 0.000396 -0.007154" rpy="0 0 0"/>
-      <mass value="0.174884"/>
+      <mass value="${base_link_mass}"/>
       <inertia ixx="${0.00090939 * sim_body_inertia_scale}" iyy="${0.00426716 * sim_body_inertia_scale}" izz="${0.00440707 * sim_body_inertia_scale}" ixy="${1.27324e-7 * sim_body_inertia_scale}" iyz="${1.05509e-9 * sim_body_inertia_scale}" ixz="${-1.69927e-7 * sim_body_inertia_scale}"/>
     </inertial>
@@ -68,5 +93,5 @@
       <origin xyz="0 0 0" rpy="0 0 0"/>
       <geometry>
-        <mesh filename="file://$(find mini_pupper_description)/meshes/mini_pupper_2/base_link.stl" scale="1 1 1"/>
+        <mesh filename="package://mini_pupper_description/meshes/mini_pupper_2/base_link.stl" scale="1 1 1"/>
       </geometry>
       <material name="opaque252525"/>
@@ -75,5 +100,5 @@
       <origin xyz="0 0 0" rpy="0 0 0"/>
       <geometry>
-        <mesh filename="file://$(find mini_pupper_description)/meshes/mini_pupper_2/base_link.stl" scale="1 1 1"/>
+        <mesh filename="package://mini_pupper_description/meshes/mini_pupper_2/base_link.stl" scale="1 1 1"/>
       </geometry>
     </collision>
@@ -82,5 +107,5 @@
     <inertial>
       <origin xyz="-0.008867 0.000396 -0.007154" rpy="0 0 0"/>
-      <mass value="0.174884"/>
+      <mass value="${base_link_mass}"/>
       <inertia ixx="${0.00090939 * sim_body_inertia_scale}" iyy="${0.00426716 * sim_body_inertia_scale}" izz="${0.00440707 * sim_body_inertia_scale}" ixy="${1.27324e-7 * sim_body_inertia_scale}" iyz="${1.05509e-9 * sim_body_inertia_scale}" ixz="${-1.69927e-7 * sim_body_inertia_scale}"/>
     </inertial>
@@ -89,5 +114,5 @@
     <inertial>
       <origin xyz="0.020109 0.002332 0.006500" rpy="0 0 0"/>
-      <mass value="${lnkgrp1_weight}"/>
+      <mass value="${lnkgrp1_mass}"/>
       <inertia ixx="${2.494061e-6 * sim_inertia_scale}" iyy="${3.735906e-6 * sim_inertia_scale}" izz="${3.222909e-6 * sim_inertia_scale}" ixy="${-7.662e-9 * sim_inertia_scale}" iyz="${-0.014e-9 * sim_inertia_scale}" ixz="${-33.565e-9 * sim_inertia_scale}"/>
     </inertial>
@@ -95,5 +120,5 @@
       <origin xyz="0 0 0" rpy="0 0 0"/>
       <geometry>
-        <mesh filename="file://$(find mini_pupper_description)/meshes/mini_pupper_2/lf1.stl" scale="1 1 1"/>
+        <mesh filename="package://mini_pupper_description/meshes/mini_pupper_2/lf1.stl" scale="1 1 1"/>
       </geometry>
       <material name="opaque666666"/>
@@ -102,5 +127,5 @@
       <origin xyz="0 0 0" rpy="0 0 0"/>
       <geometry>
-        <mesh filename="file://$(find mini_pupper_description)/meshes/mini_pupper_2/lf1.stl" scale="1 1 1"/>
+        <mesh filename="package://mini_pupper_description/meshes/mini_pupper_2/lf1.stl" scale="1 1 1"/>
       </geometry>
     </collision>
@@ -109,5 +134,5 @@
     <inertial>
       <origin xyz="-0.003174 0.000986 -0.017984" rpy="0 0 0"/>
-      <mass value="${lnkgrp2_weight}"/>
+      <mass value="${lnkgrp2_mass}"/>
       <inertia ixx="${0.462154e-6 * sim_inertia_scale}" iyy="${0.481174e-6 * sim_inertia_scale}" izz="${26.893e-9 * sim_inertia_scale}" ixy="${3.117e-9 * sim_inertia_scale}" iyz="${17.662e-9 * sim_inertia_scale}" ixz="${-79.269e-9 * sim_inertia_scale}"/>
     </inertial>
@@ -115,5 +140,5 @@
       <origin xyz="0 0 0" rpy="0 0 0"/>
       <geometry>
-        <mesh filename="file://$(find mini_pupper_description)/meshes/mini_pupper_2/lf2.stl" scale="1 1 1"/>
+        <mesh filename="package://mini_pupper_description/meshes/mini_pupper_2/lf2.stl" scale="1 1 1"/>
       </geometry>
       <material name="opaque636363"/>
@@ -122,5 +147,5 @@
       <origin xyz="0 0 0" rpy="0 0 0"/>
       <geometry>
-        <mesh filename="file://$(find mini_pupper_description)/meshes/mini_pupper_2/lf2.stl" scale="1 1 1"/>
+        <mesh filename="package://mini_pupper_description/meshes/mini_pupper_2/lf2.stl" scale="1 1 1"/>
       </geometry>
     </collision>
@@ -129,5 +154,5 @@
     <inertial>
       <origin xyz="0.006211 0.003456 -0.015014" rpy="0 0 0"/>
-      <mass value="${lnkgrp3_weight}"/>
+      <mass value="${lnkgrp3_mass}"/>
       <inertia ixx="${0.484471e-6 * sim_inertia_scale}" iyy="${0.567615e-6 * sim_inertia_scale}" izz="${91.813e-9 * sim_inertia_scale}" ixy="${-2.101e-9 * sim_inertia_scale}" iyz="${5.008e-9 * sim_inertia_scale}" ixz="${0.20057e-6 * sim_inertia_scale}"/>
     </inertial>
@@ -135,5 +160,5 @@
       <origin xyz="0 0 0" rpy="0 0 0"/>
       <geometry>
-        <mesh filename="file://$(find mini_pupper_description)/meshes/mini_pupper_2/lf3.stl" scale="1 1 1"/>
+        <mesh filename="package://mini_pupper_description/meshes/mini_pupper_2/lf3.stl" scale="1 1 1"/>
       </geometry>
       <material name="opaque252525"/>
@@ -142,5 +167,5 @@
       <origin xyz="0 0 0" rpy="0 0 0"/>
       <geometry>
-        <mesh filename="file://$(find mini_pupper_description)/meshes/mini_pupper_2/lf3.stl" scale="1 1 1"/>
+        <mesh filename="package://mini_pupper_description/meshes/mini_pupper_2/lf3.stl" scale="1 1 1"/>
       </geometry>
     </collision>
@@ -149,5 +174,5 @@
     <inertial>
       <origin xyz="0.020109 -0.002332 0.006500" rpy="0 0 0"/>
-      <mass value="${lnkgrp1_weight}"/>
+      <mass value="${lnkgrp1_mass}"/>
       <inertia ixx="${2.494061e-06 * sim_inertia_scale}" iyy="${3.735906e-06 * sim_inertia_scale}" izz="${3.222909e-06 * sim_inertia_scale}" ixy="${7.662e-9 * sim_inertia_scale}" iyz="${-0.014e-9 * sim_inertia_scale}" ixz="${-33.565e-9 * sim_inertia_scale}"/>
     </inertial>
@@ -155,5 +180,5 @@
       <origin xyz="0 0 0" rpy="0 0 0"/>
       <geometry>
-        <mesh filename="file://$(find mini_pupper_description)/meshes/mini_pupper_2/rf1.stl" scale="1 1 1"/>
+        <mesh filename="package://mini_pupper_description/meshes/mini_pupper_2/rf1.stl" scale="1 1 1"/>
       </geometry>
       <material name="opaque666666"/>
@@ -162,5 +187,5 @@
       <origin xyz="0 0 0" rpy="0 0 0"/>
       <geometry>
-        <mesh filename="file://$(find mini_pupper_description)/meshes/mini_pupper_2/rf1.stl" scale="1 1 1"/>
+        <mesh filename="package://mini_pupper_description/meshes/mini_pupper_2/rf1.stl" scale="1 1 1"/>
       </geometry>
     </collision>
@@ -169,5 +194,5 @@
     <inertial>
       <origin xyz="-0.003174 -0.000986 -0.017984" rpy="0 0 0"/>
-      <mass value="${lnkgrp2_weight}"/>
+      <mass value="${lnkgrp2_mass}"/>
       <inertia ixx="${0.462154e-6 * sim_inertia_scale}" iyy="${0.481174e-6 * sim_inertia_scale}" izz="${26.893e-9 * sim_inertia_scale}" ixy="${-3.117e-9 * sim_inertia_scale}" iyz="${-17.662e-9 * sim_inertia_scale}" ixz="${-79.269e-9 * sim_inertia_scale}"/>
     </inertial>
@@ -175,5 +200,5 @@
       <origin xyz="0 0 0" rpy="0 0 0"/>
       <geometry>
-        <mesh filename="file://$(find mini_pupper_description)/meshes/mini_pupper_2/rf2.stl" scale="1 1 1"/>
+        <mesh filename="package://mini_pupper_description/meshes/mini_pupper_2/rf2.stl" scale="1 1 1"/>
       </geometry>
       <material name="opaque636363"/>
@@ -182,5 +207,5 @@
       <origin xyz="0 0 0" rpy="0 0 0"/>
       <geometry>
-        <mesh filename="file://$(find mini_pupper_description)/meshes/mini_pupper_2/rf2.stl" scale="1 1 1"/>
+        <mesh filename="package://mini_pupper_description/meshes/mini_pupper_2/rf2.stl" scale="1 1 1"/>
       </geometry>
     </collision>
@@ -189,5 +214,5 @@
     <inertial>
       <origin xyz="0.006211 -0.003456 -0.015014" rpy="0 0 0"/>
-      <mass value="${lnkgrp3_weight}"/>
+      <mass value="${lnkgrp3_mass}"/>
       <inertia ixx="${0.484471e-6 * sim_inertia_scale}" iyy="${0.567615e-06 * sim_inertia_scale}" izz="${91.813e-9 * sim_inertia_scale}" ixy="${2.101e-9 * sim_inertia_scale}" iyz="${-5.008e-9 * sim_inertia_scale}" ixz="${0.20057e-6 * sim_inertia_scale}"/>
     </inertial>
@@ -195,5 +220,5 @@
       <origin xyz="0 0 0" rpy="0 0 0"/>
       <geometry>
-        <mesh filename="file://$(find mini_pupper_description)/meshes/mini_pupper_2/rf3.stl" scale="1 1 1"/>
+        <mesh filename="package://mini_pupper_description/meshes/mini_pupper_2/rf3.stl" scale="1 1 1"/>
       </geometry>
       <material name="opaque252525"/>
@@ -202,5 +227,5 @@
       <origin xyz="0 0 0" rpy="0 0 0"/>
       <geometry>
-        <mesh filename="file://$(find mini_pupper_description)/meshes/mini_pupper_2/rf3.stl" scale="1 1 1"/>
+        <mesh filename="package://mini_pupper_description/meshes/mini_pupper_2/rf3.stl" scale="1 1 1"/>
       </geometry>
     </collision>
@@ -209,5 +234,5 @@
     <inertial>
       <origin xyz="-0.020109 -0.002332 0.006500" rpy="0 0 0"/>
-      <mass value="${lnkgrp1_weight}"/>
+      <mass value="${lnkgrp1_mass}"/>
       <inertia ixx="${2.494061e-06 * sim_inertia_scale}" iyy="${3.735906e-06 * sim_inertia_scale}" izz="${3.222909e-06 * sim_inertia_scale}" ixy="${-7.662e-9 * sim_inertia_scale}" iyz="${-0.014e-9 * sim_inertia_scale}" ixz="${-33.565e-9 * sim_inertia_scale}"/>
     </inertial>
@@ -215,5 +240,5 @@
       <origin xyz="0 0 0" rpy="0 0 0"/>
       <geometry>
-        <mesh filename="file://$(find mini_pupper_description)/meshes/mini_pupper_2/rb1.stl" scale="1 1 1"/>
+        <mesh filename="package://mini_pupper_description/meshes/mini_pupper_2/rb1.stl" scale="1 1 1"/>
       </geometry>
       <material name="opaque666666"/>
@@ -222,5 +247,5 @@
       <origin xyz="0 0 0" rpy="0 0 0"/>
       <geometry>
-        <mesh filename="file://$(find mini_pupper_description)/meshes/mini_pupper_2/rb1.stl" scale="1 1 1"/>
+        <mesh filename="package://mini_pupper_description/meshes/mini_pupper_2/rb1.stl" scale="1 1 1"/>
       </geometry>
     </collision>
@@ -229,5 +254,5 @@
     <inertial>
       <origin xyz="-0.003174 -0.000986 -0.017984" rpy="0 0 0"/>
-      <mass value="${lnkgrp2_weight}"/>
+      <mass value="${lnkgrp2_mass}"/>
       <inertia ixx="${0.462154e-6 * sim_inertia_scale}" iyy="${0.481174e-6 * sim_inertia_scale}" izz="${26.893e-9 * sim_inertia_scale}" ixy="${-3.117e-9 * sim_inertia_scale}" iyz="${-17.662e-9 * sim_inertia_scale}" ixz="${-79.269e-9 * sim_inertia_scale}"/>
     </inertial>
@@ -235,5 +260,5 @@
       <origin xyz="0 0 0" rpy="0 0 0"/>
       <geometry>
-        <mesh filename="file://$(find mini_pupper_description)/meshes/mini_pupper_2/rb2.stl" scale="1 1 1"/>
+        <mesh filename="package://mini_pupper_description/meshes/mini_pupper_2/rb2.stl" scale="1 1 1"/>
       </geometry>
       <material name="opaque636363"/>
@@ -242,5 +267,5 @@
       <origin xyz="0 0 0" rpy="0 0 0"/>
       <geometry>
-        <mesh filename="file://$(find mini_pupper_description)/meshes/mini_pupper_2/rb2.stl" scale="1 1 1"/>
+        <mesh filename="package://mini_pupper_description/meshes/mini_pupper_2/rb2.stl" scale="1 1 1"/>
       </geometry>
     </collision>
@@ -249,5 +274,5 @@
     <inertial>
       <origin xyz="0.006211 -0.003456 -0.015014" rpy="0 0 0"/>
-      <mass value="${lnkgrp3_weight}"/>
+      <mass value="${lnkgrp3_mass}"/>
       <inertia ixx="${0.484816e-6 * sim_inertia_scale}" iyy="${0.567883e-06 * sim_inertia_scale}" izz="${91.777e-9 * sim_inertia_scale}" ixy="${2.212e-9 * sim_inertia_scale}" iyz="${-5.34e-9 * sim_inertia_scale}" ixz="${0.200564e-6 * sim_inertia_scale}"/>
     </inertial>
@@ -255,5 +280,5 @@
       <origin xyz="0 0 0" rpy="0 0 0"/>
       <geometry>
-        <mesh filename="file://$(find mini_pupper_description)/meshes/mini_pupper_2/rb3.stl" scale="1 1 1"/>
+        <mesh filename="package://mini_pupper_description/meshes/mini_pupper_2/rb3.stl" scale="1 1 1"/>
       </geometry>
       <material name="opaque252525"/>
@@ -262,5 +287,5 @@
       <origin xyz="0 0 0" rpy="0 0 0"/>
       <geometry>
-        <mesh filename="file://$(find mini_pupper_description)/meshes/mini_pupper_2/rb3.stl" scale="1 1 1"/>
+        <mesh filename="package://mini_pupper_description/meshes/mini_pupper_2/rb3.stl" scale="1 1 1"/>
       </geometry>
     </collision>
@@ -269,5 +294,5 @@
     <inertial>
       <origin xyz="-0.020109 0.002332 0.006500" rpy="0 0 0"/>
-      <mass value="${lnkgrp1_weight}"/>
+      <mass value="${lnkgrp1_mass}"/>
       <inertia ixx="${2.494061e-06 * sim_inertia_scale}" iyy="${3.735906e-06 * sim_inertia_scale}" izz="${3.222909e-06 * sim_inertia_scale}" ixy="${7.662e-9 * sim_inertia_scale}" iyz="${-0.014e-9 * sim_inertia_scale}" ixz="${-33.565e-9 * sim_inertia_scale}"/>
     </inertial>
@@ -275,5 +300,5 @@
       <origin xyz="0 0 0" rpy="0 0 0"/>
       <geometry>
-        <mesh filename="file://$(find mini_pupper_description)/meshes/mini_pupper_2/lb1.stl" scale="1 1 1"/>
+        <mesh filename="package://mini_pupper_description/meshes/mini_pupper_2/lb1.stl" scale="1 1 1"/>
       </geometry>
       <material name="opaque666666"/>
@@ -282,5 +307,5 @@
       <origin xyz="0 0 0" rpy="0 0 0"/>
       <geometry>
-        <mesh filename="file://$(find mini_pupper_description)/meshes/mini_pupper_2/lb1.stl" scale="1 1 1"/>
+        <mesh filename="package://mini_pupper_description/meshes/mini_pupper_2/lb1.stl" scale="1 1 1"/>
       </geometry>
     </collision>
@@ -289,5 +314,5 @@
     <inertial>
       <origin xyz="-0.003174 0.000986 -0.017984" rpy="0 0 0"/>
-      <mass value="${lnkgrp2_weight}"/>
+      <mass value="${lnkgrp2_mass}"/>
       <inertia ixx="${0.462154e-6 * sim_inertia_scale}" iyy="${0.481174e-6 * sim_inertia_scale}" izz="${26.893e-9 * sim_inertia_scale}" ixy="${3.117e-9 * sim_inertia_scale}" iyz="${17.662e-9 * sim_inertia_scale}" ixz="${-79.269e-9 * sim_inertia_scale}"/>
     </inertial>
@@ -295,5 +320,5 @@
       <origin xyz="0 0 0" rpy="0 0 0"/>
       <geometry>
-        <mesh filename="file://$(find mini_pupper_description)/meshes/mini_pupper_2/lb2.stl" scale="1 1 1"/>
+        <mesh filename="package://mini_pupper_description/meshes/mini_pupper_2/lb2.stl" scale="1 1 1"/>
       </geometry>
       <material name="opaque636363"/>
@@ -302,5 +327,5 @@
       <origin xyz="0 0 0" rpy="0 0 0"/>
       <geometry>
-        <mesh filename="file://$(find mini_pupper_description)/meshes/mini_pupper_2/lb2.stl" scale="1 1 1"/>
+        <mesh filename="package://mini_pupper_description/meshes/mini_pupper_2/lb2.stl" scale="1 1 1"/>
       </geometry>
     </collision>
@@ -309,5 +334,5 @@
     <inertial>
       <origin xyz="0.006211 0.003456 -0.015014" rpy="0 0 0"/>
-      <mass value="${lnkgrp3_weight}"/>
+      <mass value="${lnkgrp3_mass}"/>
       <inertia ixx="${0.484471e-6 * sim_inertia_scale}" iyy="${0.567615e-06 * sim_inertia_scale}" izz="${91.813e-9 * sim_inertia_scale}" ixy="${-2.101e-9 * sim_inertia_scale}" iyz="${5.008e-9 * sim_inertia_scale}" ixz="${0.20057e-6 * sim_inertia_scale}"/>
     </inertial>
@@ -315,5 +340,5 @@
       <origin xyz="0 0 0" rpy="0 0 0"/>
       <geometry>
-        <mesh filename="file://$(find mini_pupper_description)/meshes/mini_pupper_2/lb3.stl" scale="1 1 1"/>
+        <mesh filename="package://mini_pupper_description/meshes/mini_pupper_2/lb3.stl" scale="1 1 1"/>
       </geometry>
       <material name="opaque252525"/>
@@ -322,5 +347,5 @@
       <origin xyz="0 0 0" rpy="0 0 0"/>
       <geometry>
-        <mesh filename="file://$(find mini_pupper_description)/meshes/mini_pupper_2/lb3.stl" scale="1 1 1"/>
+        <mesh filename="package://mini_pupper_description/meshes/mini_pupper_2/lb3.stl" scale="1 1 1"/>
       </geometry>
     </collision>
@@ -329,5 +354,5 @@
     <inertial>
       <origin xyz="-0.005539 -0.000204 0.020223" rpy="0 0 0"/>
-      <mass value="0.00785515871148119"/>
+      <mass value="${body_front_mass}"/>
       <inertia ixx="${5.306048e-6 * sim_body_inertia_scale}" iyy="${1.837621e-6 * sim_body_inertia_scale}" izz="${3.61974e-6 * sim_body_inertia_scale}" ixy="${-22.863e-9 * sim_body_inertia_scale}" iyz="${-4.925e-9 * sim_body_inertia_scale}" ixz="${-9.195e-9 * sim_body_inertia_scale}"/>
     </inertial>
@@ -335,5 +360,5 @@
       <origin xyz="-0.089299 0 0.015543" rpy="0 0 0"/>
       <geometry>
-        <mesh filename="file://$(find mini_pupper_description)/meshes/mini_pupper_2/Body_front.stl" scale="1 1 1"/>
+        <mesh filename="package://mini_pupper_description/meshes/mini_pupper_2/Body_front.stl" scale="1 1 1"/>
       </geometry>
       <material name="opaque2552210"/>
@@ -342,5 +367,5 @@
       <origin xyz="-0.089299 0 0.015543" rpy="0 0 0"/>
       <geometry>
-        <mesh filename="file://$(find mini_pupper_description)/meshes/mini_pupper_2/Body_front.stl" scale="1 1 1"/>
+        <mesh filename="package://mini_pupper_description/meshes/mini_pupper_2/Body_front.stl" scale="1 1 1"/>
       </geometry>
     </collision>
@@ -349,5 +374,5 @@
     <inertial>
       <origin xyz="0.089461 0.023505 0.0" rpy="0 0 0"/>
-      <mass value="0.014261552601793053"/>
+      <mass value="${board_pcb_mass}"/>
       <inertia ixx="${4.425965e-6 * sim_body_inertia_scale}" iyy="${3.4560775e-5 * sim_body_inertia_scale}" izz="${3.8954441e-5 * sim_body_inertia_scale}" ixy="${0.104871e-6 * sim_body_inertia_scale}" iyz="${75.406e-9 * sim_body_inertia_scale}" ixz="${0.113313e-6 * sim_body_inertia_scale}"/>
     </inertial>
@@ -355,5 +380,5 @@
       <origin xyz="0.087701 0.023505 -0.026457" rpy="0 0 0"/>
       <geometry>
-        <mesh filename="file://$(find mini_pupper_description)/meshes/mini_pupper_2/Board_PCB.stl" scale="1 1 1"/>
+        <mesh filename="package://mini_pupper_description/meshes/mini_pupper_2/Board_PCB.stl" scale="1 1 1"/>
       </geometry>
       <material name="opaque646464"/>
@@ -362,18 +387,13 @@
       <origin xyz="0.087701 0.023505 -0.026457" rpy="0 0 0"/>
       <geometry>
-        <mesh filename="file://$(find mini_pupper_description)/meshes/mini_pupper_2/Board_PCB.stl" scale="1 1 1"/>
+        <mesh filename="package://mini_pupper_description/meshes/mini_pupper_2/Board_PCB.stl" scale="1 1 1"/>
       </geometry>
     </collision>
   </link>
   <link name="Board_connectors_1">
-    <!-- <inertial>
-      <origin xyz="-0.07276303117117414 -0.002323344081837562 -0.0010631239213060653" rpy="0 0 0"/>
-      <mass value="0.004688613655947816"/>
-      <inertia ixx="0.203205e-6" iyy="1.5404404e-5" izz="1.5546403e-5" ixy="-0.625328e-6" iyz="42.901e-9" ixz="0.186346e-9"/>
-    </inertial> -->
     <visual>
       <origin xyz="-0.061334 3.3e-05 -0.026457" rpy="0 0 0"/>
       <geometry>
-        <mesh filename="file://$(find mini_pupper_description)/meshes/mini_pupper_2/Board_connectors_1.stl" scale="1 1 1"/>
+        <mesh filename="package://mini_pupper_description/meshes/mini_pupper_2/Board_connectors_1.stl" scale="1 1 1"/>
       </geometry>
       <material name="opaque2491590"/>
@@ -382,18 +402,13 @@
       <origin xyz="-0.061334 3.3e-05 -0.026457" rpy="0 0 0"/>
       <geometry>
-        <mesh filename="file://$(find mini_pupper_description)/meshes/mini_pupper_2/Board_connectors_1.stl" scale="1 1 1"/>
+        <mesh filename="package://mini_pupper_description/meshes/mini_pupper_2/Board_connectors_1.stl" scale="1 1 1"/>
       </geometry>
     </collision>
   </link>
   <link name="Board_connectors_2">
-    <!-- <inertial>
-      <origin xyz="0.008233541174180986 -0.0021383697865476553 -0.00030110978110910874" rpy="0 0 0"/>
-      <mass value="0.0019746031301169403"/>
-      <inertia ixx="0.458183e-6" iyy="3.284548e-6" izz="3.720196e-6" ixy="-79.741e-9" iyz="4.796e-9" ixz="0.123868e-9"/>
-    </inertial> -->
     <visual>
       <origin xyz="0.045346 5e-06 -0.026457" rpy="0 0 0"/>
       <geometry>
-        <mesh filename="file://$(find mini_pupper_description)/meshes/mini_pupper_2/Board_connectors_2.stl" scale="1 1 1"/>
+        <mesh filename="package://mini_pupper_description/meshes/mini_pupper_2/Board_connectors_2.stl" scale="1 1 1"/>
       </geometry>
       <material name="opaque255255255"/>
@@ -402,5 +417,5 @@
       <origin xyz="0.045346 5e-06 -0.026457" rpy="0 0 0"/>
       <geometry>
-        <mesh filename="file://$(find mini_pupper_description)/meshes/mini_pupper_2/Board_connectors_2.stl" scale="1 1 1"/>
+        <mesh filename="package://mini_pupper_description/meshes/mini_pupper_2/Board_connectors_2.stl" scale="1 1 1"/>
       </geometry>
     </collision>
@@ -412,5 +427,5 @@
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