Commit message: Ros2 Jazzy migration

File: mini_pupper_description/urdf/ros2_control/mini_pupper.ros2_control.xacro (robot description, xacro)
@@ -3,12 +3,5 @@
   <xacro:macro name="pupper_joint" params="joint_name initial_value use_gazebo_hardware">
     <joint name="${joint_name}">
-      <xacro:if value="${use_gazebo_hardware}">
-        <command_interface name="position_pid"/>
-        <param name="pos_kp">5.0</param>
-        <param name="pos_kd">0.05</param>
-      </xacro:if>
-      <xacro:unless value="${use_gazebo_hardware}">
-        <command_interface name="position"/>
-      </xacro:unless>
+      <command_interface name="position"/>
       <state_interface name="position">
         <param name="initial_value">${initial_value}</param>
@@ -20,5 +13,5 @@
     <xacro:if value="${use_gazebo_hardware}">
       <gazebo>
-        <plugin name="gazebo_ros2_control" filename="libgazebo_ros2_control.so">
+          <plugin filename="gz_ros2_control-system" name="gz_ros2_control::GazeboSimROS2ControlPlugin">
           <parameters>$(find mini_pupper_simulation)/config/ros2_control/mini_pupper_2_controllers_sim.yaml</parameters>
           <hold_joints>false</hold_joints>
@@ -29,6 +22,5 @@
       <hardware>
         <xacro:if value="${use_gazebo_hardware}">
-          <plugin>gazebo_ros2_control/GazeboSystem</plugin>
-          <param name="hold_joints">true</param>
+            <plugin>gz_ros2_control/GazeboSimSystem</plugin>
         </xacro:if>
         <xacro:unless value="${use_gazebo_hardware}">
